Commit message: [clearpath_platform_description] Fixed incorrect path.

File: clearpath_platform_description/urdf/a200/a200_macro.urdf.xacro (robot description, xacro)
@@ -37,5 +37,5 @@
         <origin xyz="0 0 0" rpy="0 0 0" />
         <geometry>
-          <mesh filename="package://a200_description/meshes/base_link.dae" />
+          <mesh filename="package://clearpath_platform_description/meshes/a200/base_link.dae" />
         </geometry>
       </visual>
