Commit message: Move clearpath_description to clearpath_platform_description and switched robot names to robot model number.

File: clearpath_platform_description/urdf/a200/a200.urdf.xacro (robot description, xacro)
@@ -1,11 +1,11 @@
 <?xml version="1.0"?>
-<robot xmlns:xacro="http://ros.org/wiki/xacro" name="husky">
+<robot xmlns:xacro="http://ros.org/wiki/xacro" name="a200">
   <!-- robot name parameter -->
   <!-- <xacro:arg name="name" default="" /> -->
   <xacro:arg name="prefix" default="" />
   <xacro:arg name="gazebo_controllers" default="$(find clearpath_control)/config/control.yaml" />
-  <xacro:include filename="$(find clearpath_description)/urdf/husky/husky_macro.urdf.xacro" />
-  <!-- Load husky description -->
-  <xacro:husky prefix="$(arg prefix)" />
+  <xacro:include filename="$(find clearpath_platform_description)/urdf/a200/a200_macro.urdf.xacro" />
+  <!-- Load a200 description -->
+  <xacro:a200 prefix="$(arg prefix)" />
   <xacro:if value="$(arg is_sim)">
     <gazebo>

File: clearpath_platform_description/urdf/a200/a200_macro.urdf.xacro (robot description, xacro)
@@ -8,17 +8,17 @@
   <xacro:arg name="realsense_rpy" default="$(optenv CPR_REALSENSE_RPY 0 0 0)" />
   <xacro:arg name="realsense_mount" default="$(optenv CPR_REALSENSE_MOUNT_FRAME sensor_arch_mount_link)" />
-  <xacro:property name="husky_front_bumper_extend" value="$(optenv HUSKY_FRONT_BUMPER_EXTEND 0)" />
-  <xacro:property name="husky_rear_bumper_extend" value="$(optenv HUSKY_REAR_BUMPER_EXTEND 0)" />
+  <xacro:property name="a200_front_bumper_extend" value="$(optenv A200_FRONT_BUMPER_EXTEND 0)" />
+  <xacro:property name="a200_rear_bumper_extend" value="$(optenv A200_REAR_BUMPER_EXTEND 0)" />
   <xacro:arg name="robot_namespace" default="/" />
   <xacro:arg name="is_sim" default="false" />
   <xacro:arg name="urdf_extras" default="$(optenv CPR_URDF_EXTRAS empty.urdf)" />
   <!-- Included URDF/XACRO Files -->
-  <xacro:include filename="$(find clearpath_description)/urdf/husky/decorations.urdf.xacro" />
-  <xacro:include filename="$(find clearpath_description)/urdf/husky/wheel.urdf.xacro" />
-  <xacro:include filename="$(find clearpath_description)/urdf/husky/accessories/intel_realsense.urdf.xacro"/>
-  <!-- <xacro:include filename="$(find clearpath_description)/urdf/husky/accessories/sick_lms1xx_mount.urdf.xacro"/> -->
-  <xacro:include filename="$(find clearpath_description)/urdf/husky/accessories/sensor_arch.urdf.xacro"/>
+  <xacro:include filename="$(find clearpath_platform_description)/urdf/a200/decorations.urdf.xacro" />
+  <xacro:include filename="$(find clearpath_platform_description)/urdf/a200/wheel.urdf.xacro" />
+  <xacro:include filename="$(find clearpath_platform_description)/urdf/a200/accessories/intel_realsense.urdf.xacro"/>
+  <!-- <xacro:include filename="$(find clearpath_platform_description)/urdf/a200/accessories/sick_lms1xx_mount.urdf.xacro"/> -->
+  <xacro:include filename="$(find clearpath_platform_description)/urdf/a200/accessories/sensor_arch.urdf.xacro"/>
   <xacro:property name="M_PI" value="3.14159"/>
-  <xacro:macro name="husky" params="prefix">
+  <xacro:macro name="a200" params="prefix">
     <!-- Base Size -->
     <xacro:property name="base_x_size" value="0.98740000" />
@@ -37,11 +37,11 @@
         <origin xyz="0 0 0" rpy="0 0 0" />
         <geometry>
-          <mesh filename="package://husky_description/meshes/base_link.dae" />
+          <mesh filename="package://a200_description/meshes/base_link.dae" />
         </geometry>
       </visual>
       <collision>
-        <origin xyz="${( husky_front_bumper_extend - husky_rear_bumper_extend ) / 2.0} 0 ${base_z_size/4}" rpy="0 0 0" />
+        <origin xyz="${( a200_front_bumper_extend - a200_rear_bumper_extend ) / 2.0} 0 ${base_z_size/4}" rpy="0 0 0" />
         <geometry>
-          <box size="${ base_x_size + husky_front_bumper_extend + husky_rear_bumper_extend } ${base_y_size} ${base_z_size/2}"/>
+          <box size="${ base_x_size + a200_front_bumper_extend + a200_rear_bumper_extend } ${base_y_size} ${base_z_size/2}"/>
         </geometry>
       </collision>
@@ -89,18 +89,18 @@
       <child link="${prefix}gps_link" />
     </joint>
-    <!-- Husky wheel macros -->
-    <xacro:husky_wheel wheel_prefix="${prefix}front_left">
+    <!-- A200 wheel macros -->
+    <xacro:a200_wheel wheel_prefix="${prefix}front_left">
       <origin xyz="${wheelbase/2} ${track/2} ${wheel_vertical_offset}" rpy="0 0 0" />
-    </xacro:husky_wheel>
-    <xacro:husky_wheel wheel_prefix="${prefix}front_right">
+    </xacro:a200_wheel>
+    <xacro:a200_wheel wheel_prefix="${prefix}front_right">
       <origin xyz="${wheelbase/2} ${-track/2} ${wheel_vertical_offset}" rpy="0 0 0" />
-    </xacro:husky_wheel>
-    <xacro:husky_wheel wheel_prefix="${prefix}rear_left">
+    </xacro:a200_wheel>
+    <xacro:a200_wheel wheel_prefix="${prefix}rear_left">
       <origin xyz="${-wheelbase/2} ${track/2} ${wheel_vertical_offset}" rpy="0 0 0" />
-    </xacro:husky_wheel>
-    <xacro:husky_wheel wheel_prefix="${prefix}rear_right">
+    </xacro:a200_wheel>
+    <xacro:a200_wheel wheel_prefix="${prefix}rear_right">
       <origin xyz="${-wheelbase/2} ${-track/2} ${wheel_vertical_offset}" rpy="0 0 0" />
-    </xacro:husky_wheel>
-    <xacro:husky_decorate />
+    </xacro:a200_wheel>
+    <xacro:a200_decorate />
     <!-- <xacro:if value="$(arg laser_enabled)">
       <xacro:sick_lms1xx_mount prefix="base"/>
@@ -133,5 +133,5 @@
       <xacro:intel_realsense_mount prefix="camera" topic="realsense" parent_link="realsense_mountpoint"/>
     </xacro:if>
-    <ros2_control name="${prefix}husky_hardware" type="system">
+    <ros2_control name="${prefix}a200_hardware" type="system">
       <hardware>
         <xacro:if value="$(arg is_sim)">
@@ -139,5 +139,5 @@
         </xacro:if>
         <xacro:unless value="$(arg is_sim)">
-          <plugin>husky_base/HuskyHardware</plugin>
+          <plugin>a200_base/A200Hardware</plugin>
           <plugin>fake_components/GenericSystem</plugin>
           <param name="hw_start_duration_sec">2.0</param>

File: clearpath_platform_description/urdf/a200/accessories/sensor_arch.urdf.xacro (robot description, xacro)
@@ -7,5 +7,5 @@
              <visual>
                  <geometry>
-                     <mesh filename="package://clearpath_description/meshes/husky/accessories/${size}_mm_sensor_arch.dae" />
+                     <mesh filename="package://clearpath_platform_description/meshes/a200/accessories/${size}_mm_sensor_arch.dae" />
                  </geometry>
              </visual>
@@ -13,5 +13,5 @@
                  <origin xyz="0 0 0" rpy="0 0 0"/>
                  <geometry>
-                     <mesh filename="package://clearpath_description/meshes/husky/accessories/${size}_mm_sensor_arch.dae" />
+                     <mesh filename="package://clearpath_platform_description/meshes/a200/accessories/${size}_mm_sensor_arch.dae" />
                  </geometry>
              </collision>

File: clearpath_platform_description/urdf/a200/accessories/sick_lms1xx_mount.urdf.xacro (robot description, xacro)
@@ -25,32 +25,28 @@
 SOFTWARE, EVEN IF ADVISED OF THE POSSIBILITY OF SUCH DAMAGE.
 -->
-<robot xmlns:xacro="http://www.ros.org/wiki/xacro">
+<robot xmlns:xacro="http://ros.org/wiki/xacro">
   <xacro:include filename="$(find lms1xx)/urdf/sick_lms1xx.urdf.xacro" />
-  <xacro:macro name="sick_lms1xx_mount" params="prefix topic parent_link *origin">
-    <xacro:sick_lms1xx frame="${prefix}_laser" topic="${topic}" />
-    <joint name="${prefix}_laser_mount_joint" type="fixed">
-      <xacro:insert_block name="origin" />
-      <parent link="${parent_link}" />
-      <child link="${prefix}_laser_mount" />
-    </joint>
+  <xacro:macro name="sick_lms1xx_mount" params="prefix">
     <link name="${prefix}_laser_mount">
       <visual>
-        <origin xyz="0 0 0" rpy="0 0 0" />
+        <origin xyz="0 0 0" rpy="0 0 ${-M_PI/2}" />
         <geometry>
           <!-- Origin of this mesh is the base of the bracket. -->
-          <mesh filename="package://clearpath_description/meshes/jackal/sick-lms1xx-bracket.stl" />
+          <mesh filename="package://clearpath_platform_description/meshes/a200/accessories/lms1xx_mount.dae" />
         </geometry>
-        <material name="dark_grey" />
       </visual>
+      <collision>
+        <origin xyz="0 0 .0585" rpy="0 0 0" />
+        <geometry>
+          <box size=".1 .108 .117" />
+        </geometry>
+      </collision>
     </link>
     <joint name="${prefix}_laser_joint" type="fixed">
       <!-- This offset is from the base of the bracket to the LIDAR's focal point. -->
-      <origin xyz="0 0 0.149" rpy="0 0 0" />
+      <origin xyz="0.0352 0 0.0566" rpy="${M_PI} 0 0" />
       <parent link="${prefix}_laser_mount" />
       <child link="${prefix}_laser" />
     </joint>
-    <gazebo reference="${prefix}_laser_mount">
-      <material>Gazebo/DarkGrey</material>
-    </gazebo>
   </xacro:macro>
 </robot>

File: clearpath_platform_description/urdf/a200/decorations.urdf.xacro (robot description, xacro)
@@ -1,4 +1,4 @@
 <?xml version="1.0"?>
-<robot name="husky_decorations" xmlns:xacro="http://ros.org/wiki/xacro">
+<robot name="a200_decorations" xmlns:xacro="http://ros.org/wiki/xacro">
   <material name="dark_grey"><color rgba="0.2 0.2 0.2 1.0" /></material>
   <material name="medium_grey"><color rgba="0.6 0.6 0.6 1.0" /></material>
@@ -8,13 +8,13 @@
   <material name="white"><color rgba="1.0 1.0 1.0 1.0" /></material>
   <material name="red"><color rgba="1.0 0.0 0.0 1.0" /></material>
-  <xacro:macro name="husky_decorate">
-    <xacro:property name="husky_front_bumper_extend" value="$(optenv HUSKY_FRONT_BUMPER_EXTEND 0)" />
-    <xacro:property name="husky_rear_bumper_extend" value="$(optenv HUSKY_REAR_BUMPER_EXTEND 0)" />
-    <!-- Spawn Husky chassis -->
+  <xacro:macro name="a200_decorate">
+    <xacro:property name="a200_front_bumper_extend" value="$(optenv A200_FRONT_BUMPER_EXTEND 0)" />
+    <xacro:property name="a200_rear_bumper_extend" value="$(optenv A200_REAR_BUMPER_EXTEND 0)" />
+    <!-- Spawn A200 chassis -->
     <link name="top_chassis_link">
       <visual>
         <origin xyz="0 0 0" rpy="0 0 0" />
         <geometry>
-          <mesh filename="package://clearpath_description/meshes/husky/top_chassis.dae" />
+          <mesh filename="package://clearpath_platform_description/meshes/a200/top_chassis.dae" />
         </geometry>
       </visual>
@@ -25,10 +25,10 @@
       <child link="top_chassis_link" />
     </joint>
-    <xacro:if value="$(optenv HUSKY_USER_RAIL_ENABLED true)">
+    <xacro:if value="$(optenv A200_USER_RAIL_ENABLED true)">
       <!-- Spawn user rails -->
       <link name="user_rail_link">
         <visual>
           <geometry>
-            <mesh filename="package://clearpath_description/meshes/husky/user_rail.dae" />
+            <mesh filename="package://clearpath_platform_description/meshes/a200/user_rail.dae" />
           </geometry>
         </visual>
@@ -45,5 +45,5 @@
       <visual>
         <geometry>
-          <mesh filename="package://clearpath_description/meshes/husky/bumper.dae" />
+          <mesh filename="package://clearpath_platform_description/meshes/a200/bumper.dae" />
         </geometry>
       </visual>
@@ -51,18 +51,18 @@
     <!-- Attach front bumper -->
     <joint name="front_bumper" type="fixed">
-      <origin xyz="${0.48 + husky_front_bumper_extend} 0 0.091" rpy="0 0 0" />
+      <origin xyz="${0.48 + a200_front_bumper_extend} 0 0.091" rpy="0 0 0" />
       <parent link="base_link" />
       <child link="front_bumper_link" />
     </joint>
-    <xacro:if value="${husky_front_bumper_extend}">
+    <xacro:if value="${a200_front_bumper_extend}">
       <link name="front_bumper_extension_link">
           <visual>
               <geometry>
-                  <mesh filename="package://clearpath_description/meshes/husky/bumper_extension.dae" />
+                  <mesh filename="package://clearpath_platform_description/meshes/a200/bumper_extension.dae" />
               </geometry>
           </visual>
       </link>
       <joint name="front_bumper_extension" type="fixed">
-        <origin xyz="${0.48 + husky_front_bumper_extend} 0 0.091" rpy="0 0 0" />
+        <origin xyz="${0.48 + a200_front_bumper_extend} 0 0.091" rpy="0 0 0" />
         <parent link="base_link" />
         <child link="front_bumper_extension_link" />
@@ -73,5 +73,5 @@
       <visual>
         <geometry>
-          <mesh filename="package://clearpath_description/meshes/husky/bumper.dae" />
+          <mesh filename="package://clearpath_platform_description/meshes/a200/bumper.dae" />
         </geometry>
       </visual>
@@ -79,30 +79,30 @@
     <!-- Attach rear bumper -->
     <joint name="rear_bumper" type="fixed">
-      <origin xyz="${-0.48 - husky_rear_bumper_extend} 0 0.091" rpy="0 0 ${M_PI}" />
+      <origin xyz="${-0.48 - a200_rear_bumper_extend} 0 0.091" rpy="0 0 ${M_PI}" />
       <parent link="base_link" />
       <child link="rear_bumper_link" />
     </joint>
-    <xacro:if value="${husky_rear_bumper_extend}">
+    <xacro:if value="${a200_rear_bumper_extend}">
       <link name="rear_bumper_extension_link">
           <visual>
               <geometry>
-                  <mesh filename="package://clearpath_description/meshes/husky/bumper_extension.dae" />
+                  <mesh filename="package://clearpath_platform_description/meshes/a200/bumper_extension.dae" />
               </geometry>
           </visual>
       </link>
       <joint name="rear_bumper_extension" type="fixed">
-        <origin xyz="${-0.48 - husky_rear_bumper_extend} 0 0.091" rpy="0 0 ${M_PI}" />
+        <origin xyz="${-0.48 - a200_rear_bumper_extend} 0 0.091" rpy="0 0 ${M_PI}" />
         <parent link="base_link" />
         <child link="rear_bumper_extension_link" />
       </joint>
     </xacro:if>
-    <xacro:if value="$(optenv HUSKY_TOP_PLATE_ENABLED true)">
+    <xacro:if value="$(optenv A200_TOP_PLATE_ENABLED true)">
       <!-- Spawn the top plate -->
-      <xacro:if value="$(optenv HUSKY_LARGE_TOP_PLATE false)">
+      <xacro:if value="$(optenv A200_LARGE_TOP_PLATE false)">
         <link name="top_plate_link">
           <visual>
             <origin xyz="0 0 0" rpy="0 0 0" />
             <geometry>
-              <mesh filename="package://clearpath_description/meshes/husky/large_top_plate.dae" />
+              <mesh filename="package://clearpath_platform_description/meshes/a200/large_top_plate.dae" />
             </geometry>
           </visual>
@@ -110,5 +110,5 @@
             <origin xyz="0 0 0" rpy="0 0 0"/>
             <geometry>
-              <mesh filename="package://clearpath_description/meshes/husky/large_top_plate_collision.stl" />
+              <mesh filename="package://clearpath_platform_description/meshes/a200/large_top_plate_collision.stl" />
             </geometry>
           </collision>
@@ -133,10 +133,10 @@
         </joint>
       </xacro:if>
-      <xacro:unless value="$(optenv HUSKY_LARGE_TOP_PLATE false)">
+      <xacro:unless value="$(optenv A200_LARGE_TOP_PLATE false)">
         <link name="top_plate_link">
           <visual>
             <origin xyz="0 0 0" rpy="0 0 0" />
             <geometry>
-              <mesh filename="package://clearpath_description/meshes/husky/top_plate.dae" />
+              <mesh filename="package://clearpath_platform_description/meshes/a200/top_plate.dae" />
             </geometry>
           </visual>
@@ -144,5 +144,5 @@
             <origin xyz="0 0 0" rpy="0 0 0"/>
             <geometry>
-              <mesh filename="package://clearpath_description/meshes/husky/top_plate.stl" />
+              <mesh filename="package://clearpath_platform_description/meshes/a200/top_plate.stl" />
             </geometry>
           </collision>

File: clearpath_platform_description/urdf/a200/wheel.urdf.xacro (robot description, xacro)
@@ -1,5 +1,5 @@
 <?xml version="1.0"?>
-<robot xmlns:xacro="http://ros.org/wiki/xacro" name="husky_wheel">
-  <xacro:macro name="husky_wheel" params="wheel_prefix *joint_pose">
+<robot xmlns:xacro="http://ros.org/wiki/xacro" name="a200_wheel">
+  <xacro:macro name="a200_wheel" params="wheel_prefix *joint_pose">
     <link name="${wheel_prefix}_wheel">
       <inertial>
@@ -11,5 +11,5 @@
         <origin xyz="0 0 0" rpy="0 0 0" />
         <geometry>
-          <mesh filename="package://clearpath_description/meshes/husky/wheel.dae" />
+          <mesh filename="package://clearpath_platform_description/meshes/a200/wheel.dae" />
         </geometry>
       </visual>

File: clearpath_platform_description/urdf/j100/accessories.urdf.xacro (robot description, xacro)
@@ -10,13 +10,13 @@
   -->
   <!-- Macros to generate standoffs for offset payload mounting. -->
-  <xacro:include filename="$(find clearpath_description)/urdf/jackal/accessories/standoffs.urdf.xacro" />
+  <xacro:include filename="$(find clearpath_platform_description)/urdf/j100/accessories/standoffs.urdf.xacro" />
   <!-- This optional plate mounts both the upgraded GPS and the Velodyne 3D LIDAR. -->
-  <xacro:include filename="$(find clearpath_description)/urdf/jackal/accessories/bridge_plate.urdf.xacro" />
+  <xacro:include filename="$(find clearpath_platform_description)/urdf/j100/accessories/bridge_plate.urdf.xacro" />
   <!-- 2D Lidars -->
   <!-- <xacro:include filename="$(find lms1xx)/urdf/sick_lms1xx.urdf.xacro" />
-  <xacro:include filename="$(find clearpath_description)/urdf/jackal/accessories/sick_lms1xx_mount.urdf.xacro" />-->
-  <xacro:include filename="$(find clearpath_description)/urdf/jackal/accessories/hokuyo_ust10.urdf.xacro" />
-  <xacro:include filename="$(find clearpath_description)/urdf/jackal/accessories/vlp16_mount.urdf.xacro" />
-  <xacro:include filename="$(find clearpath_description)/urdf/jackal/accessories/hdl32_mount.urdf.xacro" />
+  <xacro:include filename="$(find clearpath_platform_description)/urdf/j100/accessories/sick_lms1xx_mount.urdf.xacro" />-->
+  <xacro:include filename="$(find clearpath_platform_description)/urdf/j100/accessories/hokuyo_ust10.urdf.xacro" />
+  <xacro:include filename="$(find clearpath_platform_description)/urdf/j100/accessories/vlp16_mount.urdf.xacro" />
+  <xacro:include filename="$(find clearpath_platform_description)/urdf/j100/accessories/hdl32_mount.urdf.xacro" />
   <!--
     Add primary/secondary 2D lidar sensors.  By default these are SICK LMS1xx but can be changed with the
@@ -135,6 +135,6 @@
     - smart7              :: Novatel Smart7
   -->
-  <xacro:include filename="$(find clearpath_description)/urdf/jackal/accessories/novatel_smart6.urdf.xacro" />
-  <xacro:include filename="$(find clearpath_description)/urdf/jackal/accessories/novatel_smart7.urdf.xacro" />
+  <xacro:include filename="$(find clearpath_platform_description)/urdf/j100/accessories/novatel_smart6.urdf.xacro" />
+  <xacro:include filename="$(find clearpath_platform_description)/urdf/j100/accessories/novatel_smart7.urdf.xacro" />
   <xacro:if value="$(optenv CPR_NAVSAT 0)">
     <xacro:property name="mount" value="$(optenv CPR_NAVSAT_MOUNT rear)" />
@@ -197,5 +197,5 @@
   -->
   <!-- Common camera mounts and accessory URDFs. -->
-  <xacro:include filename="$(find clearpath_description)/urdf/jackal/accessories/camera_mount.urdf.xacro" />
+  <xacro:include filename="$(find clearpath_platform_description)/urdf/j100/accessories/camera_mount.urdf.xacro" />
   <!--xacro:include filename="$(find pointgrey_camera_description)/urdf/pointgrey_flea3.urdf.xacro" /-->
   <!-- If enabled, generate the flea3 camera payload with a tilt of 30 degrees. -->
@@ -242,5 +242,5 @@
     </xacro:unless>
   </xacro:if>
-  <xacro:include filename="$(find clearpath_description)/urdf/jackal/accessories/stereo_camera_mount.urdf.xacro" />
+  <xacro:include filename="$(find clearpath_platform_description)/urdf/j100/accessories/stereo_camera_mount.urdf.xacro" />
   <!-- If enabled, generates a pair of flea3 cameras for stereo vision with a tilt of 30 degrees. -->
   <!-- Disabled temporarily due to metapackage issue. -->
@@ -322,5 +322,5 @@
   <!-- Fender Accessories -->
   <xacro:if value="$(optenv CPR_FRONT_ACCESSORY_FENDER 0)">
-    <xacro:include filename="$(find clearpath_description)/urdf/jackal/accessories/hokuyo_ust10.urdf.xacro" />
+    <xacro:include filename="$(find clearpath_platform_description)/urdf/j100/accessories/hokuyo_ust10.urdf.xacro" />
     <xacro:if value="$(optenv CPR_FRONT_FENDER_UST10 0)">
       <xacro:hokuyo_ust10_mount
@@ -351,5 +351,5 @@
         <origin xyz="0 0 0" rpy="0 0 0"/>
         <geometry>
-          <mesh filename="package://clearpath_description/meshes/jackal/ark_enclosure.stl"/>
+          <mesh filename="package://clearpath_platform_description/meshes/j100/ark_enclosure.stl"/>
         </geometry>
         <material name="dark_grey" />

File: clearpath_platform_description/urdf/j100/accessories/bridge_plate.urdf.xacro (robot description, xacro)
@@ -17,5 +17,5 @@
         <origin xyz="0 0 0" rpy="1.5707 0.0 1.5707" />
         <geometry>
-          <mesh filename="package://clearpath_description/meshes/jackal/bridge-plate.stl"/>
+          <mesh filename="package://clearpath_platform_description/meshes/j100/bridge-plate.stl"/>
         </geometry>
         <material name="dark_grey" />

File: clearpath_platform_description/urdf/j100/accessories/camera_mount.urdf.xacro (robot description, xacro)
@@ -5,5 +5,5 @@
         <origin xyz="0 0 0" rpy="1.5707 0 1.5707" />
         <geometry>
-          <mesh filename="package://clearpath_description/meshes/jackal/camera-bracket.stl" scale="0.001 0.001 0.001" />
+          <mesh filename="package://clearpath_platform_description/meshes/j100/camera-bracket.stl" scale="0.001 0.001 0.001" />
         </geometry>
         <material name="dark_grey" />
@@ -14,5 +14,5 @@
         <origin xyz="0 0 0" rpy="0 0 1.5707" />
         <geometry>
-          <mesh filename="package://clearpath_description/meshes/jackal/camera-beam.stl" scale="0.001 0.001 0.001" />
+          <mesh filename="package://clearpath_platform_description/meshes/j100/camera-beam.stl" scale="0.001 0.001 0.001" />
         </geometry>
         <material name="dark_grey" />

File: clearpath_platform_description/urdf/j100/accessories/hdl32_mount.urdf.xacro (robot description, xacro)
@@ -6,5 +6,5 @@
         <visual>
           <geometry>
-            <mesh filename="package://clearpath_description/meshes/jackal/velodyne_tower.stl"/>
+            <mesh filename="package://clearpath_platform_description/meshes/j100/velodyne_tower.stl"/>
           </geometry>
           <origin xyz="0 0 0" rpy="0 0 0" />
@@ -13,5 +13,5 @@
         <collision>
           <geometry>
-            <mesh filename="package://clearpath_description/meshes/jackal/velodyne_tower.stl"/>
+            <mesh filename="package://clearpath_platform_description/meshes/j100/velodyne_tower.stl"/>
           </geometry>
           <origin xyz="0 0 0" rpy="0 0 0" />
