Commit message: Move clearpath_description to clearpath_platform_description and switched robot names to robot model number.

File: clearpath_platform_description/urdf/j100/accessories/hokuyo_ust10.urdf.xacro (robot description, xacro)
@@ -61,5 +61,5 @@
         <geometry>
           <!-- Origin of this mesh is the base of the bracket. -->
-          <mesh filename="package://clearpath_description/meshes/jackal/hokuyo_ust10.stl" />
+          <mesh filename="package://clearpath_platform_description/meshes/j100/hokuyo_ust10.stl" />
         </geometry>
         <material name="dark_grey" />

File: clearpath_platform_description/urdf/j100/accessories/novatel_smart6.urdf.xacro (robot description, xacro)
@@ -6,5 +6,5 @@
       <origin xyz="0 0 0" rpy="0 0 0" />
       <geometry>
-        <mesh filename="package://clearpath_description/meshes/jackal/novatel-smart6.stl"/>
+        <mesh filename="package://clearpath_platform_description/meshes/j100/novatel-smart6.stl"/>
       </geometry>
       <material name="novatel_white">

File: clearpath_platform_description/urdf/j100/accessories/novatel_smart7.urdf.xacro (robot description, xacro)
@@ -6,5 +6,5 @@
         <origin xyz="-0.095 0 0" rpy="${pi/2} 0 -${pi/2}" />
         <geometry>
-          <mesh filename="package://clearpath_description/meshes/jackal/novatel-smart7.stl"/>
+          <mesh filename="package://clearpath_platform_description/meshes/j100/novatel-smart7.stl"/>
         </geometry>
         <material name="novatel_white">
@@ -15,5 +15,5 @@
         <origin xyz="-0.095 0 0" rpy="${pi/2} 0 -${pi/2}" />
         <geometry>
-          <mesh filename="package://clearpath_description/meshes/jackal/novatel-smart7.stl"/>
+          <mesh filename="package://clearpath_platform_description/meshes/j100/novatel-smart7.stl"/>
         </geometry>
       </collision>

File: clearpath_platform_description/urdf/j100/accessories/sick_lms1xx_mount.urdf.xacro (robot description, xacro)
@@ -25,28 +25,32 @@
 SOFTWARE, EVEN IF ADVISED OF THE POSSIBILITY OF SUCH DAMAGE.
 -->
-<robot xmlns:xacro="http://ros.org/wiki/xacro">
+<robot xmlns:xacro="http://www.ros.org/wiki/xacro">
   <xacro:include filename="$(find lms1xx)/urdf/sick_lms1xx.urdf.xacro" />
-  <xacro:macro name="sick_lms1xx_mount" params="prefix">
+  <xacro:macro name="sick_lms1xx_mount" params="prefix topic parent_link *origin">
+    <xacro:sick_lms1xx frame="${prefix}_laser" topic="${topic}" />
+    <joint name="${prefix}_laser_mount_joint" type="fixed">
+      <xacro:insert_block name="origin" />
+      <parent link="${parent_link}" />
+      <child link="${prefix}_laser_mount" />
+    </joint>
     <link name="${prefix}_laser_mount">
       <visual>
-        <origin xyz="0 0 0" rpy="0 0 ${-M_PI/2}" />
+        <origin xyz="0 0 0" rpy="0 0 0" />
         <geometry>
           <!-- Origin of this mesh is the base of the bracket. -->
-          <mesh filename="package://clearpath_description/meshes/husky/accessories/lms1xx_mount.dae" />
+          <mesh filename="package://clearpath_platform_description/meshes/j100/sick-lms1xx-bracket.stl" />
         </geometry>
+        <material name="dark_grey" />
       </visual>
-      <collision>
-        <origin xyz="0 0 .0585" rpy="0 0 0" />
-        <geometry>
-          <box size=".1 .108 .117" />
-        </geometry>
-      </collision>
     </link>
     <joint name="${prefix}_laser_joint" type="fixed">
       <!-- This offset is from the base of the bracket to the LIDAR's focal point. -->
-      <origin xyz="0.0352 0 0.0566" rpy="${M_PI} 0 0" />
+      <origin xyz="0 0 0.149" rpy="0 0 0" />
       <parent link="${prefix}_laser_mount" />
       <child link="${prefix}_laser" />
     </joint>
+    <gazebo reference="${prefix}_laser_mount">
+      <material>Gazebo/DarkGrey</material>
+    </gazebo>
   </xacro:macro>
 </robot>

File: clearpath_platform_description/urdf/j100/accessories/stereo_camera_mount.urdf.xacro (robot description, xacro)
@@ -6,5 +6,5 @@
         <origin xyz="0 0 0" rpy="0 0 0" />
         <geometry>
-          <mesh filename="package://clearpath_description/meshes/jackal/stereo-camera-bracket.stl" />
+          <mesh filename="package://clearpath_platform_description/meshes/j100/stereo-camera-bracket.stl" />
         </geometry>
         <material name="dark_grey" />
@@ -15,5 +15,5 @@
         <origin xyz="0 0 0" rpy="0 0 0" />
         <geometry>
-          <mesh filename="package://clearpath_description/meshes/jackal/stereo-camera-beam.stl" />
+          <mesh filename="package://clearpath_platform_description/meshes/j100/stereo-camera-beam.stl" />
         </geometry>
         <material name="dark_grey" />

File: clearpath_platform_description/urdf/j100/j100.urdf.xacro (robot description, xacro)
@@ -1,4 +1,4 @@
 <?xml version="1.0"?>
-<robot name="jackal" xmlns:xacro="http://www.ros.org/wiki/xacro">
+<robot name="j100" xmlns:xacro="http://www.ros.org/wiki/xacro">
   <xacro:arg name="is_sim" default="false" />
   <xacro:arg name="prefix" default="" />
@@ -25,5 +25,5 @@
         <origin xyz="0 0 0" rpy="${PI/2} 0 0"/>
         <geometry>
-          <mesh filename="package://clearpath_description/meshes/jackal/jackal-wheel.stl"/>
+          <mesh filename="package://clearpath_platform_description/meshes/j100/j100-wheel.stl"/>
         </geometry>
         <material name="black" />
@@ -59,5 +59,5 @@
       <axis xyz="0 1 0" />
     </joint>
-    <!-- In reality, Jackal has only two motors, one per side. However, it's more
+    <!-- In reality, J100 has only two motors, one per side. However, it's more
          straightforward for Gazebo to simulate as if there's an actuator per wheel. -->
     <transmission name="${prefix}_wheel_trans">
@@ -93,5 +93,5 @@
       <origin xyz="0 0 ${footprint_vertical_offset}" rpy="${PI/2} 0 ${PI/2}"/>
       <geometry>
-        <mesh filename="package://clearpath_description/meshes/jackal/jackal-base.stl"/>
+        <mesh filename="package://clearpath_platform_description/meshes/j100/j100-base.stl"/>
       </geometry>
       <material name="dark_grey" />
@@ -114,9 +114,9 @@
       </inertial>
   </link>
-  <xacro:unless value="$(optenv JACKAL_FRONT_ACCESSORY_FENDER 0)">
+  <xacro:unless value="$(optenv J100_FRONT_ACCESSORY_FENDER 0)">
     <link name="front_fender_link">
       <visual>
         <geometry>
-          <mesh filename="package://clearpath_description/meshes/jackal/jackal-fender.stl"/>
+          <mesh filename="package://clearpath_platform_description/meshes/j100/j100-fender.stl"/>
         </geometry>
         <material name="yellow" />
@@ -124,9 +124,9 @@
     </link>
   </xacro:unless>
-  <xacro:if value="$(optenv JACKAL_FRONT_ACCESSORY_FENDER 0)">
+  <xacro:if value="$(optenv J100_FRONT_ACCESSORY_FENDER 0)">
     <link name="front_fender_link">
       <visual>
         <geometry>
-          <mesh filename="package://clearpath_description/meshes/jackal/accessory_fender.stl"/>
+          <mesh filename="package://clearpath_platform_description/meshes/j100/accessory_fender.stl"/>
         </geometry>
         <material name="yellow" />
@@ -145,9 +145,9 @@
     <child link="front_fender_link" />
   </joint>
-  <xacro:unless value="$(optenv JACKAL_REAR_ACCESSORY_FENDER 0)">
+  <xacro:unless value="$(optenv J100_REAR_ACCESSORY_FENDER 0)">
     <link name="rear_fender_link">
       <visual>
         <geometry>
-          <mesh filename="package://clearpath_description/meshes/jackal/jackal-fender.stl"/>
+          <mesh filename="package://clearpath_platform_description/meshes/j100/j100-fender.stl"/>
         </geometry>
         <material name="yellow" />
@@ -155,9 +155,9 @@
     </link>
   </xacro:unless>
-  <xacro:if value="$(optenv JACKAL_REAR_ACCESSORY_FENDER 0)">
+  <xacro:if value="$(optenv J100_REAR_ACCESSORY_FENDER 0)">
     <link name="rear_fender_link">
       <visual>
         <geometry>
-          <mesh filename="package://clearpath_description/meshes/jackal/accessory_fender.stl"/>
+          <mesh filename="package://clearpath_platform_description/meshes/j100/accessory_fender.stl"/>
         </geometry>
         <material name="yellow" />
@@ -225,5 +225,5 @@
   </joint>
   <!-- ROS2 controls -->
-  <ros2_control name="jackal_hardware" type="system">
+  <ros2_control name="j100_hardware" type="system">
     <hardware>
       <xacro:if value="$(arg is_sim)">
@@ -231,5 +231,5 @@
       </xacro:if>
       <xacro:unless value="$(arg is_sim)">
-        <plugin>jackal_hardware/JackalHardware</plugin>
+        <plugin>j100_hardware/J100Hardware</plugin>
         <plugin>fake_components/GenericSystem</plugin>
       </xacro:unless>
@@ -258,10 +258,10 @@
   <!-- Bring in simulation data for Gazebo. -->
   <xacro:if value="$(arg is_sim)">
-    <xacro:include filename="$(find clearpath_description)/urdf/jackal/jackal.gazebo" />
+    <xacro:include filename="$(find clearpath_platform_description)/urdf/j100/j100.gazebo" />
   </xacro:if>
   <!-- Optional standard accessories, including their simulation data. The rendering
        of these into the final description is controlled by optenv variables, which
        default each one to off.-->
-  <xacro:include filename="$(find clearpath_description)/urdf/jackal/accessories.urdf.xacro" />
+  <xacro:include filename="$(find clearpath_platform_description)/urdf/j100/accessories.urdf.xacro" />
   <!-- Optional custom includes. -->
   <xacro:include filename="$(optenv CPR_URDF_EXTRAS empty.urdf)" />

Commit message: Sim fixes

File: clearpath_platform_description/urdf/a200/a200.urdf.xacro (robot description, xacro)
@@ -101,8 +101,40 @@
       <child link="rear_bumper_mount" />
     </joint>
+    <xacro:if value="$(arg is_sim)">
+      <gazebo>
+        <plugin filename="libign_ros2_control-system.so" name="ign_ros2_control::IgnitionROS2ControlPlugin">
+          <parameters>$(find clearpath_control)/config/a200/control.yaml</parameters>
+          <ros>
+            <remapping>~/odom:=platform/odom</remapping>
+            <remapping>~/cmd_vel_unstamped:=platform/cmd_vel_unstamped</remapping>
+            <remapping>/tf:=tf</remapping>
+            <remapping>/tf_static:=tf_static</remapping>
+            <remapping>/diagnostics:=diagnostics</remapping>
+            <remapping>joint_states:=platform/joint_states</remapping>
+            <!-- <namespace>$(arg namespace)</namespace> -->
+          </ros>
+        </plugin>
+      </gazebo>
+      <gazebo>
+        <plugin filename="libignition-gazebo-pose-publisher-system.so" name="ignition::gazebo::systems::PosePublisher">
+          <publish_link_pose>true</publish_link_pose>
+          <publish_nested_model_pose>true</publish_nested_model_pose>
+          <use_pose_vector_msg>true</use_pose_vector_msg>
+          <update_frequency>62</update_frequency>
+        </plugin>
+      </gazebo>
+      <gazebo>
+        <plugin filename="libignition-gazebo-contact-system.so" name="ignition::gazebo::systems::Contact"></plugin>
+      </gazebo>
+      <gazebo>
+        <plugin filename="libignition-gazebo-sensors-system.so" name="ignition::gazebo::systems::Sensors">
+          <render_engine>ogre</render_engine>
+        </plugin>
+      </gazebo>
+    </xacro:if>
     <ros2_control name="a200_hardware" type="system">
       <hardware>
         <xacro:if value="$(arg is_sim)">
-          <plugin>gazebo_ros2_control/GazeboSystem</plugin>
+          <plugin>ign_ros2_control/IgnitionSystem</plugin>
         </xacro:if>
         <xacro:unless value="$(arg is_sim)">

File: clearpath_platform_description/urdf/a200/decorations/structure.urdf.xacro (robot description, xacro)
@@ -12,5 +12,5 @@
         </visual>
         <collision>
-          <origin xyz="0 0 0" rpy="0 0 0"/>
+          <origin xyz="0 0 0.51" rpy="0 0 0"/>
           <geometry>
             <mesh filename="package://clearpath_platform_description/meshes/a200/decorations/510_mm_sensor_arch.dae" />
@@ -41,5 +41,5 @@
         </visual>
         <collision>
-          <origin xyz="0 0 0" rpy="0 0 0"/>
+          <origin xyz="0 0 0.3" rpy="0 0 0"/>
           <geometry>
             <mesh filename="package://clearpath_platform_description/meshes/a200/decorations/300_mm_sensor_arch.dae" />

File: clearpath_platform_description/urdf/a200/wheel.urdf.xacro (robot description, xacro)
@@ -6,5 +6,5 @@
         <mass value="2.637" />
         <origin xyz="0 0 0" />
-        <inertia  ixx="0.02467" ixy="0" ixz="0" iyy="0.04411" iyz="0" izz="0.02467" />
+        <inertia ixx="0.02467" ixy="0" ixz="0" iyy="0.04411" iyz="0" izz="0.02467" />
       </inertial>
       <visual>

File: clearpath_sensors_description/urdf/sick_lms1xx.urdf.xacro (robot description, xacro)
@@ -7,7 +7,4 @@
           <mesh filename="package://clearpath_sensors_description/meshes/sick_lms1xx_small.dae" />
         </geometry>
-        <material name="blue" >
-          <color rgba="0 0 1 1" />
-        </material>
       </visual>
       <collision>

Commit message: use_sim_time support Added lidar gazebo plugins

File: clearpath_platform_description/urdf/a200/a200.urdf.xacro (robot description, xacro)
@@ -121,5 +121,5 @@
           <publish_nested_model_pose>true</publish_nested_model_pose>
           <use_pose_vector_msg>true</use_pose_vector_msg>
-          <update_frequency>62</update_frequency>
+          <update_frequency>50</update_frequency>
         </plugin>
       </gazebo>

File: clearpath_sensors_description/urdf/hokuyo_ust10.urdf.xacro (robot description, xacro)
@@ -1,5 +1,7 @@
 <?xml version="1.0"?>
 <robot xmlns:xacro="http://ros.org/wiki/xacro">
-  <xacro:macro name="hokuyo_ust10" params="name parent_link *origin">
+  <xacro:macro name="hokuyo_ust10" params="name parent_link *origin
+                                          ang_res:=0.25 min_ang:=-2.35619 max_ang:=2.35619
+                                          update_rate:=40 min_range:=0.06 max_range:=30.0">
     <link name="${name}_link">
       <visual>
@@ -32,4 +34,33 @@
       <child link="${name}_laser" />
     </joint>
+    <xacro:property name="samples" value="${round((max_ang - min_ang) * 180 / (ang_res * pi))}"/>
+    <gazebo reference="${name}_laser">
+      <sensor name="${name}" type="gpu_lidar">
+        <update_rate>${update_rate}</update_rate>
+        <visualize>true</visualize>
+        <always_on>true</always_on>
+        <lidar>
+          <scan>
+            <horizontal>
+              <samples>${samples}</samples>
+              <resolution>1</resolution>
+              <min_angle>${min_ang}</min_angle>
+              <max_angle>${max_ang}</max_angle>
+            </horizontal>
+            <vertical>
+              <samples>1</samples>
+              <resolution>1</resolution>
+              <min_angle>0</min_angle>
+              <max_angle>0</max_angle>
+            </vertical>
+          </scan>
+          <range>
+            <min>${min_range}</min>
+            <max>${max_range}</max>
+            <resolution>0.01</resolution>
+          </range>
+        </lidar>
+      </sensor>
+    </gazebo>
   </xacro:macro>
 </robot>

File: clearpath_sensors_description/urdf/intel_realsense.urdf.xacro (robot description, xacro)
@@ -133,4 +133,23 @@
       <xacro:insert_block name="origin" />
     </xacro:sensor_d435>
+    <gazebo reference="${name}_color_frame">
+      <sensor name="rgbd_camera" type="rgbd_camera">
+        <camera>
+          <horizontal_fov>1.25</horizontal_fov>
+          <image>
+            <width>640</width>
+            <height>480</height>
+          </image>
+          <clip>
+            <near>0.3</near>
+            <far>100</far>
+          </clip>
+          <optical_frame_id>${name}_color_optical_frame</optical_frame_id>
+        </camera>
+        <always_on>1</always_on>
+        <update_rate>30</update_rate>
+        <visualize>true</visualize>
+      </sensor>
+    </gazebo>
   </xacro:macro>
 </robot>

File: clearpath_sensors_description/urdf/sick_lms1xx.urdf.xacro (robot description, xacro)
@@ -1,5 +1,7 @@
 <?xml version="1.0"?>
 <robot xmlns:xacro="http://www.ros.org/wiki/xacro">
-  <xacro:macro name="sick_lms1xx" params="name parent_link *origin">
+  <xacro:macro name="sick_lms1xx" params="name parent_link *origin
+                                          ang_res:=0.5 min_ang:=-2.35619 max_ang:=2.35619
+                                          update_rate:=50 min_range:=0.05 max_range:=25.0">
     <link name="${name}_link">
       <visual>
@@ -25,4 +27,33 @@
       <origin rpy="0 0 0" xyz="0.0549 0 0.0367"/>
     </joint>
+    <xacro:property name="samples" value="${round((max_ang - min_ang) * 180 / (ang_res * pi))}"/>
+    <gazebo reference="${name}_laser">
+      <sensor name="${name}" type="gpu_lidar">
+        <update_rate>${update_rate}</update_rate>
+        <visualize>true</visualize>
+        <always_on>true</always_on>
+        <lidar>
+          <scan>
+            <horizontal>
+              <samples>${samples}</samples>
+              <resolution>1</resolution>
+              <min_angle>${min_ang}</min_angle>
+              <max_angle>${max_ang}</max_angle>
+            </horizontal>
+            <vertical>
+              <samples>1</samples>
+              <resolution>1</resolution>
+              <min_angle>0</min_angle>
+              <max_angle>0</max_angle>
+            </vertical>
+          </scan>
+          <range>
+            <min>${min_range}</min>
+            <max>${max_range}</max>
+            <resolution>0.01</resolution>
+          </range>
+        </lidar>
+      </sensor>
+    </gazebo>
   </xacro:macro>
 </robot>

File: clearpath_sensors_description/urdf/velodyne_lidar.urdf.xacro (robot description, xacro)
@@ -2,5 +2,8 @@
 <robot xmlns:xacro="http://www.ros.org/wiki/xacro">
   <xacro:include filename="$(find velodyne_description)/urdf/VLP-16.urdf.xacro" />
-  <xacro:macro name="velodyne_lidar" params="name parent_link *origin">
+  <xacro:macro name="velodyne_lidar" params="name parent_link *origin
+                                             ang_res_h:=0.4 min_ang_h:=-3.141592 max_ang_h:=3.141592
+                                             ang_res_v:=2.0 min_ang_v:=-0.261799 max_ang_v:=0.261799
+                                             update_rate:=20 min_range:=0.9 max_range:=130.0">
     <link name="${name}_link">
       <inertial>
@@ -54,4 +57,34 @@
       <child link="${name}_laser"/>
     </joint>
+    <xacro:property name="samples_h" value="${round((max_ang_h - min_ang_h) * 180 / (ang_res_h * pi))}"/>
+    <xacro:property name="samples_v" value="${round((max_ang_v - min_ang_v) * 180 / (ang_res_v * pi))}"/>
+    <gazebo reference="${name}_laser">
+      <sensor name="${name}" type="gpu_lidar">
+        <update_rate>${update_rate}</update_rate>
+        <visualize>true</visualize>
+        <always_on>true</always_on>
+        <lidar>
+          <scan>
+            <horizontal>
+              <samples>${samples_h}</samples>
+              <resolution>1</resolution>
+              <min_angle>${min_ang_h}</min_angle>
+              <max_angle>${max_ang_h}</max_angle>
+            </horizontal>
+            <vertical>
+              <samples>${samples_v}</samples>
+              <resolution>1</resolution>
+              <min_angle>${min_ang_v}</min_angle>
+              <max_angle>${max_ang_v}</max_angle>
+            </vertical>
+          </scan>
+          <range>
+            <min>${min_range}</min>
+            <max>${max_range}</max>
+            <resolution>0.01</resolution>
+          </range>
+        </lidar>
+      </sensor>
+    </gazebo>
   </xacro:macro>
 </robot>

Commit message: Added gazebo IMU plugin

File: clearpath_platform_description/urdf/a200/a200.urdf.xacro (robot description, xacro)
@@ -132,4 +132,7 @@
         </plugin>
       </gazebo>
+      <gazebo>
+        <plugin filename="libignition-gazebo-imu-system.so" name="ignition::gazebo::systems::Imu"></plugin>
+      </gazebo>
     </xacro:if>
     <ros2_control name="a200_hardware" type="system">

File: clearpath_sensors_description/urdf/microstrain_imu.urdf.xacro (robot description, xacro)
@@ -1,5 +1,5 @@
 <?xml version="1.0"?>
 <robot xmlns:xacro="http://ros.org/wiki/xacro">
-  <xacro:macro name="microstrain_imu" params="name parent_link *origin">
+  <xacro:macro name="microstrain_imu" params="name parent_link update_rate:=100 *origin">
     <link name="${name}_base_link"/>
     <link name="${name}_link">
@@ -21,4 +21,11 @@
       <child link="${name}_link" />
     </joint>
+    <gazebo reference="${name}_link">
+      <sensor type="imu" name="${name}">
+        <always_on>true</always_on>
+        <update_rate>${update_rate}</update_rate>
+        <visualize>true</visualize>
+      </sensor>
+    </gazebo>
   </xacro:macro>
 </robot>
