Commit message: Added GPS Added realsense gazebo parameters

File: clearpath_platform_description/urdf/a200/a200.urdf.xacro (robot description, xacro)
@@ -135,4 +135,7 @@
         <plugin filename="libignition-gazebo-imu-system.so" name="ignition::gazebo::systems::Imu"></plugin>
       </gazebo>
+      <gazebo>
+        <plugin filename="libignition-gazebo-navsat-system.so" name="ignition::gazebo::systems::NavSat"></plugin>
+      </gazebo>
     </xacro:if>
     <ros2_control name="a200_hardware" type="system">

File: clearpath_sensors_description/urdf/intel_realsense.urdf.xacro (robot description, xacro)
@@ -1,6 +1,9 @@
 <?xml version="1.0"?>
 <robot xmlns:xacro="http://ros.org/wiki/xacro">
-  <xacro:macro name="intel_realsense" params="name parent_link *origin">
-    <xacro:macro name="sensor_d435" params="parent *origin name:=camera use_nominal_extrinsics:=false add_plug:=false use_mesh:=true">
+  <xacro:macro name="intel_realsense" params="name parent_link *origin
+                                              update_rate:=30.0 image_height:=480 image_width:=640">
+    <xacro:macro name="sensor_d435"
+                 params="parent *origin name:=camera
+                         use_nominal_extrinsics:=false add_plug:=false use_mesh:=true">
       <xacro:property name="M_PI" value="3.1415926535897931" />
       <!-- The following values are approximate, and the camera node
@@ -133,11 +136,11 @@
       <xacro:insert_block name="origin" />
     </xacro:sensor_d435>
-    <gazebo reference="${name}_color_frame">
-      <sensor name="rgbd_camera" type="rgbd_camera">
+    <gazebo reference="${name}_link">
+      <sensor name="${name}" type="rgbd_camera">
         <camera>
           <horizontal_fov>1.25</horizontal_fov>
           <image>
-            <width>640</width>
-            <height>480</height>
+            <width>${image_width}</width>
+            <height>${image_height}</height>
           </image>
           <clip>
@@ -148,5 +151,5 @@
         </camera>
         <always_on>1</always_on>
-        <update_rate>30</update_rate>
+        <update_rate>${update_rate}</update_rate>
         <visualize>true</visualize>
       </sensor>

File: clearpath_sensors_description/urdf/swiftnav_duro.urdf.xacro (robot description, xacro)
@@ -22,4 +22,10 @@
       <xacro:insert_block name="origin"/>
     </joint>
+    <gazebo reference="${name}_link">
+      <sensor name="${name}" type="navsat">
+        <always_on>1</always_on>
+        <update_rate>1</update_rate>
+      </sensor>
+    </gazebo>
   </xacro:macro>
 </robot>

Commit message: Jackal sim support

File: clearpath_platform_description/urdf/a200/a200.urdf.xacro (robot description, xacro)
@@ -124,18 +124,4 @@
         </plugin>
       </gazebo>
-      <gazebo>
-        <plugin filename="libignition-gazebo-contact-system.so" name="ignition::gazebo::systems::Contact"></plugin>
-      </gazebo>
-      <gazebo>
-        <plugin filename="libignition-gazebo-sensors-system.so" name="ignition::gazebo::systems::Sensors">
-          <render_engine>ogre</render_engine>
-        </plugin>
-      </gazebo>
-      <gazebo>
-        <plugin filename="libignition-gazebo-imu-system.so" name="ignition::gazebo::systems::Imu"></plugin>
-      </gazebo>
-      <gazebo>
-        <plugin filename="libignition-gazebo-navsat-system.so" name="ignition::gazebo::systems::NavSat"></plugin>
-      </gazebo>
     </xacro:if>
     <ros2_control name="a200_hardware" type="system">

File: clearpath_platform_description/urdf/j100/decorations/bumper.urdf.xacro (robot description, xacro)
@@ -1,5 +1,5 @@
 <?xml version="1.0"?>
 <robot xmlns:xacro="http://ros.org/wiki/xacro">
-  <xacro:macro name="bumper" params="name extension:=0">
+  <xacro:macro name="bumper" params="name extension:=0 *origin">
     <xacro:property name="yaw" value="0" />
     <xacro:if value="${'rear' in name}">

File: clearpath_platform_description/urdf/j100/j100.urdf.xacro (robot description, xacro)
@@ -74,4 +74,11 @@
       <child link="imu_link" />
     </joint>
+    <gazebo reference="imu_link">
+      <sensor type="imu" name="imu_link">
+        <always_on>true</always_on>
+        <update_rate>50</update_rate>
+        <visualize>true</visualize>
+      </sensor>
+    </gazebo>
     <!-- TODO: Same note as applies to imu_link -->
     <link name="navsat_link">
@@ -89,4 +96,10 @@
       <origin xyz="-0.180 0.126 0.1815" />
     </joint>
+    <gazebo reference="navsat_link">
+      <sensor name="navsat_link" type="navsat">
+        <always_on>1</always_on>
+        <update_rate>1</update_rate>
+      </sensor>
+    </gazebo>
     <link name="mid_mount"></link>
     <joint name="mid_mount_joint" type="fixed">
@@ -107,9 +120,33 @@
       <origin xyz="${mount_spacing} 0 0" />
     </joint>
+    <xacro:if value="$(arg is_sim)">
+      <gazebo>
+        <plugin filename="libign_ros2_control-system.so" name="ign_ros2_control::IgnitionROS2ControlPlugin">
+          <parameters>$(find clearpath_control)/config/j100/control.yaml</parameters>
+          <ros>
+            <remapping>~/odom:=platform/odom</remapping>
+            <remapping>~/cmd_vel_unstamped:=platform/cmd_vel_unstamped</remapping>
+            <remapping>/tf:=tf</remapping>
+            <remapping>/tf_static:=tf_static</remapping>
+            <remapping>/diagnostics:=diagnostics</remapping>
+            <remapping>joint_states:=platform/joint_states</remapping>
+            <!-- <namespace>$(arg namespace)</namespace> -->
+          </ros>
+        </plugin>
+      </gazebo>
+      <gazebo>
+        <plugin filename="libignition-gazebo-pose-publisher-system.so" name="ignition::gazebo::systems::PosePublisher">
+          <publish_link_pose>true</publish_link_pose>
+          <publish_nested_model_pose>true</publish_nested_model_pose>
+          <use_pose_vector_msg>true</use_pose_vector_msg>
+          <update_frequency>50</update_frequency>
+        </plugin>
+      </gazebo>
+    </xacro:if>
     <!-- ROS2 controls -->
     <ros2_control name="j100_hardware" type="system">
       <hardware>
         <xacro:if value="$(arg is_sim)">
-          <plugin>gazebo_ros2_control/GazeboSystem</plugin>
+          <plugin>ign_ros2_control/IgnitionSystem</plugin>
         </xacro:if>
         <xacro:unless value="$(arg is_sim)">

Commit message: Updated husky track value

File: clearpath_platform_description/urdf/a200/a200.urdf.xacro (robot description, xacro)
@@ -15,5 +15,5 @@
     <!-- Wheel Mounting Positions -->
     <xacro:property name="wheelbase" value="0.5120" />
-    <xacro:property name="track" value="0.5708" />
+    <xacro:property name="track" value="0.555" />
     <xacro:property name="wheel_vertical_offset" value="0.03282" />
     <!-- Wheel Properties -->

Commit message: Updated gazebo simulation

File: clearpath_platform_description/urdf/a200/a200.urdf.xacro (robot description, xacro)
@@ -4,4 +4,5 @@
   <xacro:arg name="is_sim" default="false" />
   <xacro:arg name="serial_port" default="/dev/clearpath/prolific" />
+  <xacro:arg name="gazebo_controllers" default="$(find clearpath_control)/config/a200/control.yaml"/>
   <!-- Included URDF/XACRO Files -->
   <xacro:include filename="$(find clearpath_platform_description)/urdf/a200/wheel.urdf.xacro" />
@@ -136,4 +137,7 @@
       <origin xyz="0.0 0.0 0.224"/>
     </joint>
+    <!-- Gazebo Controller -->
+    <xacro:include filename="$(find clearpath_platform_description)/urdf/generic/gazebo.urdf.xacro"/>
+    <!-- ROS2 controls -->
     <ros2_control name="a200_hardware" type="system">
       <hardware>

File: clearpath_platform_description/urdf/w200/w200.urdf.xacro (robot description, xacro)
@@ -4,4 +4,5 @@
   <xacro:arg name="namespace" default="" />
   <xacro:arg name="is_sim" default="false" />
+  <xacro:arg name="gazebo_controllers" default="$(find clearpath_control)/config/w200/control.yaml"/>
   <xacro:property name="PI" value="3.1415926535897931"/>
   <xacro:property name="wheel_radius" value="0.3" />
@@ -86,6 +87,6 @@
       <mu1>0.5</mu1>
       <mu2>0.5</mu2>
-      <kp value="10000000.0" />
-      <kd value="1.0" />
+      <!-- <kp value="10000000.0" /> -->
+      <!-- <kd value="1.0" /> -->
       <fdir1 value="1 0 0" />
       <material>Gazebo/DarkGrey</material>
@@ -209,5 +210,5 @@
       </visual>
     </link>
-    <joint name="${prefix}_diff_unit_joint" type="revolute">
+    <joint name="${prefix}_diff_unit_joint" type="fixed">
       <limit upper="0.4" lower="-0.4" effort="100" velocity="1"/>
       <parent link="chassis_link"/>
@@ -349,34 +350,26 @@
       <origin xyz="-0.5826 0 0.24979" rpy="0 0 0" />
     </joint>
-    <link name="imu_link" />
-    <joint name="imu_link_joint" type="fixed">
-      <origin xyz="$(optenv WARTHOG_IMU_XYZ 0 0 0)" rpy="$(optenv WARTHOG_IMU_RPY 0 0 0)" />
-      <parent link="chassis_link"/>
-      <child link="imu_link" />
-    </joint>
-     <xacro:if value="$(arg is_sim)">
-      <gazebo>
-        <plugin filename="libign_ros2_control-system.so" name="ign_ros2_control::IgnitionROS2ControlPlugin">
-          <parameters>$(arg gazebo_controllers)</parameters>
-          <ros>
-            <remapping>~/odom:=platform/odom</remapping>
-            <remapping>~/cmd_vel_unstamped:=platform/cmd_vel_unstamped</remapping>
-            <remapping>/tf:=tf</remapping>
-            <remapping>/tf_static:=tf_static</remapping>
-            <remapping>/diagnostics:=diagnostics</remapping>
-            <remapping>joint_states:=platform/joint_states</remapping>
-            <namespace>$(arg namespace)</namespace>
-          </ros>
-        </plugin>
-      </gazebo>
-      <gazebo>
-        <plugin filename="libignition-gazebo-pose-publisher-system.so" name="ignition::gazebo::systems::PosePublisher">
-          <publish_link_pose>true</publish_link_pose>
-          <publish_nested_model_pose>true</publish_nested_model_pose>
-          <use_pose_vector_msg>true</use_pose_vector_msg>
-          <update_frequency>50</update_frequency>
-        </plugin>
-      </gazebo>
-    </xacro:if>
+    <link name="imu_0_link">
+      <inertial>
+        <mass value="0.001"/>
+        <origin xyz="0 0 0" rpy="0 0 0"/>
+        <inertia ixx="${dummy_inertia}" ixy="0.0" ixz="0.0" iyy="${dummy_inertia}" iyz="0.0" izz="${dummy_inertia}"/>
+      </inertial>
+    </link>
+    <joint name="imu_joint" type="fixed">
+      <parent link="chassis_link" />
+      <child link="imu_0_link" />
+    </joint>
+    <gazebo reference="imu_0_link">
+      <sensor type="imu" name="imu_0">
+        <always_on>true</always_on>
+        <update_rate>50</update_rate>
+        <visualize>true</visualize>
+        <ignition_frame_id>imu_0_link</ignition_frame_id>
+      </sensor>
+    </gazebo>
+    <!-- Gazebo Controller -->
+    <xacro:include filename="$(find clearpath_platform_description)/urdf/generic/gazebo.urdf.xacro"/>
+    <!-- ROS2 controls -->
     <ros2_control name="w200_hardware" type="system">
       <hardware>
@@ -428,4 +421,34 @@
       </joint>
     </ros2_control>
+    <xacro:if value="$(arg is_sim)">
+      <gazebo>
+        <plugin filename="libignition-gazebo-wheel-slip-system.so" name="ignition::gazebo::systems::WheelSlip">
+          <wheel link_name="front_left_wheel_link">
+            <slip_compliance_lateral>1.0</slip_compliance_lateral>
+            <slip_compliance_longitudinal>1.0</slip_compliance_longitudinal>
+            <wheel_normal_force>686</wheel_normal_force>
+            <wheel_radius>${wheel_radius}</wheel_radius>
+          </wheel>
+          <wheel link_name="front_right_wheel_link">
+            <slip_compliance_lateral>1.0</slip_compliance_lateral>
+            <slip_compliance_longitudinal>1.0</slip_compliance_longitudinal>
+            <wheel_normal_force>686</wheel_normal_force>
+            <wheel_radius>${wheel_radius}</wheel_radius>
+          </wheel>
+          <wheel link_name="rear_left_wheel_link">
+            <slip_compliance_lateral>1.0</slip_compliance_lateral>
+            <slip_compliance_longitudinal>1.0</slip_compliance_longitudinal>
+            <wheel_normal_force>686</wheel_normal_force>
+            <wheel_radius>${wheel_radius}</wheel_radius>
+          </wheel>
+          <wheel link_name="rear_right_wheel_link">
+            <slip_compliance_lateral>1.0</slip_compliance_lateral>
+            <slip_compliance_longitudinal>1.0</slip_compliance_longitudinal>
+            <wheel_normal_force>686</wheel_normal_force>
+            <wheel_radius>${wheel_radius}</wheel_radius>
+          </wheel>
+        </plugin>
+      </gazebo>
+    </xacro:if>
   </xacro:macro>
 </robot>

Commit message: Added wheel parameters to all robot

File: clearpath_platform_description/urdf/a200/a200.urdf.xacro (robot description, xacro)
@@ -6,7 +6,7 @@
   <xacro:arg name="gazebo_controllers" default="$(find clearpath_control)/config/a200/control.yaml"/>
   <!-- Included URDF/XACRO Files -->
-  <xacro:include filename="$(find clearpath_platform_description)/urdf/a200/wheel.urdf.xacro" />
+  <xacro:include filename="$(find clearpath_platform_description)/urdf/a200/wheels/wheel.urdf.xacro" />
   <xacro:property name="M_PI" value="3.14159"/>
-  <xacro:macro name="a200">
+  <xacro:macro name="a200" params="wheel:='default'">
     <!-- Base Size -->
     <xacro:property name="base_x_size" value="0.98740000" />

File: clearpath_platform_description/urdf/dd100/dd100.urdf.xacro (robot description, xacro)
@@ -5,8 +5,8 @@
   <xacro:arg name="gazebo_controllers" default="$(find clearpath_control)/config/dd100/control.yaml"/>
   <!-- Included URDF/XACRO Files -->
-  <xacro:include filename="$(find clearpath_platform_description)/urdf/dd100/wheel.urdf.xacro"/>
+  <xacro:include filename="$(find clearpath_platform_description)/urdf/dd100/wheels/wheel.urdf.xacro"/>
   <xacro:property name="PI" value="3.1415926535897931" />
   <!-- DD100 Platform Macro -->
-  <xacro:macro name="dd100">
+  <xacro:macro name="dd100" params="wheel:='default'">
     <!-- Variables -->
     <xacro:property name="wheel_radius" value="0.049" />

File: clearpath_platform_description/urdf/dd150/dd150.urdf.xacro (robot description, xacro)
@@ -5,8 +5,8 @@
   <xacro:arg name="gazebo_controllers" default="$(find clearpath_control)/config/dd150/control.yaml"/>
   <!-- Included URDF/XACRO Files -->
-  <xacro:include filename="$(find clearpath_platform_description)/urdf/dd150/wheel.urdf.xacro"/>
+  <xacro:include filename="$(find clearpath_platform_description)/urdf/dd150/wheels/wheel.urdf.xacro"/>
   <xacro:property name="PI" value="3.1415926535897931" />
   <!-- DD150 Platform Macro -->
-  <xacro:macro name="dd150">
+  <xacro:macro name="dd150" params="wheel:='default'">
     <!-- Variables -->
     <xacro:property name="wheel_radius" value="0.049" />

File: clearpath_platform_description/urdf/j100/j100.urdf.xacro (robot description, xacro)
@@ -2,5 +2,5 @@
 <robot name="j100"
   xmlns:xacro="http://www.ros.org/wiki/xacro">
-  <xacro:include filename="$(find clearpath_platform_description)/urdf/j100/wheel.urdf.xacro"/>
+  <xacro:include filename="$(find clearpath_platform_description)/urdf/j100/wheels/wheel.urdf.xacro"/>
   <xacro:arg name="is_sim" default="false" />
   <xacro:arg name="prefix" default="" />
@@ -19,5 +19,5 @@
   <xacro:property name="dummy_inertia" value="1e-09"/>
   <xacro:property name="mount_spacing" value="0.120" />
-  <xacro:macro name="j100">
+  <xacro:macro name="j100" params="wheel:='default'">
     <xacro:j100_wheel prefix="front_left">
       <origin xyz="${wheelbase/2} ${track/2} ${wheel_vertical_offset}" rpy="0 0 0" />
