Commit message: [clearpath_platform_description] Renamed all dashes to underscores.

File: clearpath_platform_description/urdf/j100/accessories/bridge_plate.urdf.xacro (robot description, xacro)
@@ -17,5 +17,5 @@
         <origin xyz="0 0 0" rpy="1.5707 0.0 1.5707" />
         <geometry>
-          <mesh filename="package://clearpath_platform_description/meshes/j100/bridge-plate.stl"/>
+          <mesh filename="package://clearpath_platform_description/meshes/j100/bridge_plate.stl"/>
         </geometry>
         <material name="dark_grey" />

File: clearpath_platform_description/urdf/j100/accessories/camera_mount.urdf.xacro (robot description, xacro)
@@ -5,5 +5,5 @@
         <origin xyz="0 0 0" rpy="1.5707 0 1.5707" />
         <geometry>
-          <mesh filename="package://clearpath_platform_description/meshes/j100/camera-bracket.stl" scale="0.001 0.001 0.001" />
+          <mesh filename="package://clearpath_platform_description/meshes/j100/camera_bracket.stl" scale="0.001 0.001 0.001" />
         </geometry>
         <material name="dark_grey" />
@@ -14,5 +14,5 @@
         <origin xyz="0 0 0" rpy="0 0 1.5707" />
         <geometry>
-          <mesh filename="package://clearpath_platform_description/meshes/j100/camera-beam.stl" scale="0.001 0.001 0.001" />
+          <mesh filename="package://clearpath_platform_description/meshes/j100/camera_beam.stl" scale="0.001 0.001 0.001" />
         </geometry>
         <material name="dark_grey" />

File: clearpath_platform_description/urdf/j100/accessories/novatel_smart6.urdf.xacro (robot description, xacro)
@@ -6,5 +6,5 @@
       <origin xyz="0 0 0" rpy="0 0 0" />
       <geometry>
-        <mesh filename="package://clearpath_platform_description/meshes/j100/novatel-smart6.stl"/>
+        <mesh filename="package://clearpath_platform_description/meshes/j100/novatel_smart6.stl"/>
       </geometry>
       <material name="novatel_white">

File: clearpath_platform_description/urdf/j100/accessories/novatel_smart7.urdf.xacro (robot description, xacro)
@@ -6,5 +6,5 @@
         <origin xyz="-0.095 0 0" rpy="${pi/2} 0 -${pi/2}" />
         <geometry>
-          <mesh filename="package://clearpath_platform_description/meshes/j100/novatel-smart7.stl"/>
+          <mesh filename="package://clearpath_platform_description/meshes/j100/novatel_smart7.stl"/>
         </geometry>
         <material name="novatel_white">

File: clearpath_platform_description/urdf/j100/accessories/sick_lms1xx_mount.urdf.xacro (robot description, xacro)
@@ -39,5 +39,5 @@
         <geometry>
           <!-- Origin of this mesh is the base of the bracket. -->
-          <mesh filename="package://clearpath_platform_description/meshes/j100/sick-lms1xx-bracket.stl" />
+          <mesh filename="package://clearpath_platform_description/meshes/j100/sick_lms1xx_bracket.stl" />
         </geometry>
         <material name="dark_grey" />

File: clearpath_platform_description/urdf/j100/accessories/stereo_camera_mount.urdf.xacro (robot description, xacro)
@@ -6,5 +6,5 @@
         <origin xyz="0 0 0" rpy="0 0 0" />
         <geometry>
-          <mesh filename="package://clearpath_platform_description/meshes/j100/stereo-camera-bracket.stl" />
+          <mesh filename="package://clearpath_platform_description/meshes/j100/stereo_camera_bracket.stl" />
         </geometry>
         <material name="dark_grey" />
@@ -15,5 +15,5 @@
         <origin xyz="0 0 0" rpy="0 0 0" />
         <geometry>
-          <mesh filename="package://clearpath_platform_description/meshes/j100/stereo-camera-beam.stl" />
+          <mesh filename="package://clearpath_platform_description/meshes/j100/stereo_camera_beam.stl" />
         </geometry>
         <material name="dark_grey" />
