Commit message: [clearpath_sensors_description] Moved Novatel and Hokuyo into sensors from J100.

File: clearpath_platform_description/urdf/j100/accessories.urdf.xacro (robot description, xacro)
@@ -16,5 +16,5 @@
   <!-- <xacro:include filename="$(find lms1xx)/urdf/sick_lms1xx.urdf.xacro" />
   <xacro:include filename="$(find clearpath_platform_description)/urdf/j100/accessories/sick_lms1xx_mount.urdf.xacro" />-->
-  <xacro:include filename="$(find clearpath_platform_description)/urdf/j100/accessories/hokuyo_ust10.urdf.xacro" />
+  <xacro:include filename="$(find clearpath_sensors_description)/urdf/hokuyo_ust10.urdf.xacro" />
   <xacro:include filename="$(find clearpath_platform_description)/urdf/j100/accessories/vlp16_mount.urdf.xacro" />
   <xacro:include filename="$(find clearpath_platform_description)/urdf/j100/accessories/hdl32_mount.urdf.xacro" />
@@ -135,6 +135,6 @@
     - smart7              :: Novatel Smart7
   -->
-  <xacro:include filename="$(find clearpath_platform_description)/urdf/j100/accessories/novatel_smart6.urdf.xacro" />
-  <xacro:include filename="$(find clearpath_platform_description)/urdf/j100/accessories/novatel_smart7.urdf.xacro" />
+  <xacro:include filename="$(find clearpath_sensors_description)/urdf/novatel_smart6.urdf.xacro" />
+  <xacro:include filename="$(find clearpath_sensors_description)/urdf/novatel_smart7.urdf.xacro" />
   <xacro:if value="$(optenv CPR_NAVSAT 0)">
     <xacro:property name="mount" value="$(optenv CPR_NAVSAT_MOUNT rear)" />
@@ -198,5 +198,4 @@
   <!-- Common camera mounts and accessory URDFs. -->
   <xacro:include filename="$(find clearpath_platform_description)/urdf/j100/accessories/camera_mount.urdf.xacro" />
-  <!--xacro:include filename="$(find pointgrey_camera_description)/urdf/pointgrey_flea3.urdf.xacro" /-->
   <!-- If enabled, generate the flea3 camera payload with a tilt of 30 degrees. -->
   <xacro:if value="$(optenv CPR_FLEA3 0)">
@@ -322,5 +321,4 @@
   <!-- Fender Accessories -->
   <xacro:if value="$(optenv CPR_FRONT_ACCESSORY_FENDER 0)">
-    <xacro:include filename="$(find clearpath_platform_description)/urdf/j100/accessories/hokuyo_ust10.urdf.xacro" />
     <xacro:if value="$(optenv CPR_FRONT_FENDER_UST10 0)">
       <xacro:hokuyo_ust10_mount

File: clearpath_sensors_description/urdf/hokuyo_ust10.urdf.xacro (robot description, xacro)
@@ -61,5 +61,5 @@
         <geometry>
           <!-- Origin of this mesh is the base of the bracket. -->
-          <mesh filename="package://clearpath_platform_description/meshes/j100/hokuyo_ust10.stl" />
+          <mesh filename="package://clearpath_sensors_description/meshes/hokuyo_ust10.stl" />
         </geometry>
         <material name="dark_grey" />

File: clearpath_sensors_description/urdf/novatel_smart6.urdf.xacro (robot description, xacro)
@@ -6,5 +6,5 @@
       <origin xyz="0 0 0" rpy="0 0 0" />
       <geometry>
-        <mesh filename="package://clearpath_platform_description/meshes/j100/novatel_smart6.stl"/>
+        <mesh filename="package://clearpath_sensors_description/meshes/novatel_smart6.stl"/>
       </geometry>
       <material name="novatel_white">

File: clearpath_sensors_description/urdf/novatel_smart7.urdf.xacro (robot description, xacro)
@@ -6,5 +6,5 @@
         <origin xyz="-0.095 0 0" rpy="${pi/2} 0 -${pi/2}" />
         <geometry>
-          <mesh filename="package://clearpath_platform_description/meshes/j100/novatel_smart7.stl"/>
+          <mesh filename="package://clearpath_sensors_description/meshes/novatel_smart7.stl"/>
         </geometry>
         <material name="novatel_white">
@@ -15,5 +15,5 @@
         <origin xyz="-0.095 0 0" rpy="${pi/2} 0 -${pi/2}" />
         <geometry>
-          <mesh filename="package://clearpath_platform_description/meshes/j100/novatel-smart7.stl"/>
+          <mesh filename="package://clearpath_sensors_description/meshes/novatel-smart7.stl"/>
         </geometry>
       </collision>
