Commit message: Description classes

File: clearpath_mounts_description/urdf/pacs/bracket.urdf.xacro (robot description, xacro)
@@ -22,4 +22,5 @@
 -->
 <robot xmlns:xacro="http://ros.org/wiki/xacro">
+  <!-- <xacro:include filename="$(find clearpath_platform_description)/urdf/common.urdf.xacro" /> -->
   <!--
       Brackets: add user defined bracket per mount name (i.e. A01)

File: clearpath_mounts_description/urdf/pacs/quad_post.urdf.xacro (robot description, xacro)
@@ -22,4 +22,5 @@
 -->
 <robot xmlns:xacro="http://ros.org/wiki/xacro">
+	<!-- <xacro:include filename="$(find clearpath_platform_description)/urdf/common.urdf.xacro" /> -->
 	<!-- Post Quad: adds four posts in a rectangular configuration -->
 	<xacro:macro name="quad_post" params="name parent_link length:=0.08 width:=0.08 height radius:=0.006 *origin">

File: clearpath_mounts_description/urdf/pacs/riser.urdf.xacro (robot description, xacro)
@@ -22,5 +22,5 @@
 -->
 <robot xmlns:xacro="http://ros.org/wiki/xacro">
-    <xacro:include filename="$(find clearpath_mounts_description)/urdf/common.urdf.xacro" />
+    <!-- <xacro:include filename="$(find clearpath_platform_description)/urdf/common.urdf.xacro" /> -->
     <!--
         Full Riser: add plate sized riser

File: clearpath_mounts_description/urdf/pacs/riser_leg.urdf.xacro (robot description, xacro)
@@ -22,4 +22,5 @@
 -->
 <robot xmlns:xacro="http://ros.org/wiki/xacro">
+	<!-- <xacro:include filename="$(find clearpath_platform_description)/urdf/common.urdf.xacro" /> -->
 	<!--
 	Riser Leg: standard leg for partial and full risers

File: clearpath_platform_description/urdf/a200/a200.urdf.xacro (robot description, xacro)
@@ -86,4 +86,18 @@
       <origin xyz="${-wheelbase/2} ${-track/2} ${wheel_vertical_offset}" rpy="0 0 0" />
     </xacro:a200_wheel>
+    <!-- Front bumper mount -->
+    <link name="front_bumper_mount"/>
+    <joint name="front_bumper_mount_joint" type="fixed">
+      <origin xyz="0.406 0 0.091" rpy="0 0 0" />
+      <parent link="base_link" />
+      <child link="front_bumper_mount" />
+    </joint>
+    <!-- Rear bumper mount -->
+    <link name="rear_bumper_mount"/>
+    <joint name="rear_bumper_mount_joint" type="fixed">
+      <origin xyz="-0.406 0 0.091" rpy="0 0 ${M_PI}" />
+      <parent link="base_link" />
+      <child link="rear_bumper_mount" />
+    </joint>
     <ros2_control name="a200_hardware" type="system">
       <hardware>

File: clearpath_platform_description/urdf/a200/decorations/top_plate.urdf.xacro (robot description, xacro)
@@ -1,5 +1,5 @@
 <?xml version="1.0"?>
 <robot xmlns:xacro="http://ros.org/wiki/xacro">
-    <xacro:include filename="$(find clearpath_mounts_description)/urdf/common.urdf.xacro" />
+    <!-- <xacro:include filename="$(find clearpath_platform_description)/urdf/common.urdf.xacro" /> -->
     <xacro:macro name="top_plate" params="model:=default">
         <!-- Spawn the top plate -->
@@ -93,5 +93,5 @@
         <link name="top_plate_link">
           <visual>
-            <material name="dark_grey"><color rgba="0.2 0.2 0.2 1.0" /></material>
+            <material name="dark_grey" />
             <geometry>
               <mesh filename="package://clearpath_platform_description/meshes/a200/decorations/pacs_top_plate.stl" />
@@ -99,5 +99,5 @@
           </visual>
           <collision>
-            <material name="dark_grey"><color rgba="0.2 0.2 0.2 1.0" /></material>
+            <material name="dark_grey" />
             <origin xyz="0 0 0.00317500531673" rpy="0 0 0"/>
             <geometry>

File: clearpath_platform_description/urdf/common.urdf.xacro (robot description, xacro)
@@ -2,7 +2,8 @@
 <!--
 Software License Agreement (BSD)
-\file      mounts.urdf.xacro
+\file      common.urdf.xacro
 \authors   Luis Camero <lcamero@clearpathrobotics.com>
-\copyright Copyright (c) 2022, Clearpath Robotics, Inc., All rights reserved.
+           Roni Kreinin <rkreinin@clearpathrobotics.com>
+\copyright Copyright (c) 2023, Clearpath Robotics, Inc., All rights reserved.
 Redistribution and use in source and binary forms, with or without modification, are permitted provided that
 the following conditions are met:
@@ -22,4 +23,11 @@
 -->
 <robot xmlns:xacro="http://ros.org/wiki/xacro">
+    <material name="dark_grey"><color rgba="0.2 0.2 0.2 1.0" /></material>
+    <material name="medium_grey"><color rgba="0.6 0.6 0.6 1.0" /></material>
+    <material name="light_grey"><color rgba="0.8 0.8 0.8 1.0" /></material>
+    <material name="yellow"><color rgba="0.8 0.8 0.0 1.0" /></material>
+    <material name="black"><color rgba="0.15 0.15 0.15 1.0" /></material>
+    <material name="white"><color rgba="1.0 1.0 1.0 1.0" /></material>
+    <material name="red"><color rgba="1.0 0.0 0.0 1.0" /></material>
     <!--
         Standard Mount: adds link (w/o geometry) at given position

File: clearpath_sensors_description/urdf/hokuyo_ust10.urdf.xacro (robot description, xacro)
@@ -1,4 +1,5 @@
 <?xml version="1.0"?>
 <robot xmlns:xacro="http://ros.org/wiki/xacro">
+  <xacro:include filename="$(find clearpath_platform_description)/urdf/common.urdf.xacro" />
   <xacro:macro name="hokuyo_ust10" params="name parent_link *origin">
     <link name="${name}_link">
