Commit message: Standard urdf and yaml file name and path Fixed spacing in urdfs

File: clearpath_mounts_description/urdf/pacs/quad_post.urdf.xacro (robot description, xacro)
@@ -22,81 +22,80 @@
 -->
 <robot xmlns:xacro="http://ros.org/wiki/xacro">
-	<!-- <xacro:include filename="$(find clearpath_platform_description)/urdf/common.urdf.xacro" /> -->
-	<!-- Post Quad: adds four posts in a rectangular configuration -->
-	<xacro:macro name="quad_post" params="name parent_link length:=0.08 width:=0.08 height radius:=0.006 *origin">
-		<link name="${name}_link">
-			<!-- Top Left -->
-			<visual>
-				<material name="light_grey" />
-				<origin xyz="${length/2} ${width/2} ${height/2}" />
-				<geometry>
-					<cylinder radius="${radius}" length="${height}" />
-				</geometry>
-			</visual>
-			<collision>
-				<material name="light_grey" />
-				<origin xyz="${length/2} ${width/2} ${height/2}" />
-				<geometry>
-					<cylinder radius="${radius}" length="${height}" />
-				</geometry>
-			</collision>
-			<!-- Top Right -->
-			<visual>
-				<material name="light_grey" />
-				<origin xyz="${length/2} ${-width/2} ${height/2}" />
-				<geometry>
-					<cylinder radius="${radius}" length="${height}" />
-				</geometry>
-			</visual>
-			<collision>
-				<material name="light_grey" />
-				<origin xyz="${length/2} ${-width/2} ${height/2}" />
-				<geometry>
-					<cylinder radius="${radius}" length="${height}" />
-				</geometry>
-			</collision>
-			<!-- Bottom Left -->
-			<visual>
-				<material name="light_grey" />
-				<origin xyz="${-length/2} ${width/2} ${height/2}" />
-				<geometry>
-					<cylinder radius="${radius}" length="${height}" />
-				</geometry>
-			</visual>
-			<collision>
-				<material name="light_grey" />
-				<origin xyz="${-length/2} ${width/2} ${height/2}" />
-				<geometry>
-					<cylinder radius="${radius}" length="${height}" />
-				</geometry>
-			</collision>
-			<!-- Bottom Right -->
-			<visual>
-				<material name="light_grey" />
-				<origin xyz="${-length/2} ${-width/2} ${height/2}" />
-				<geometry>
-					<cylinder radius="${radius}" length="${height}" />
-				</geometry>
-			</visual>
-			<collision>
-				<material name="light_grey" />
-				<origin xyz="${-length/2} ${-width/2} ${height/2}" />
-				<geometry>
-					<cylinder radius="${radius}" length="${height}" />
-				</geometry>
-			</collision>
-		</link>
-		<link name="${name}_mount"/>
-		<joint name="${name}_joint" type="fixed">
-			<child link="${name}_link" />
-			<parent link="${parent_link}" />
-			<insert_block name="origin" />
-		</joint>
-		<joint name="${name}_mount_joint" type="fixed">
-			<child link="${name}_mount" />
-			<parent link="${name}_link" />
-			<origin xyz="0 0 ${height}">
-			</origin>
-		</joint>
-	</xacro:macro>
+  <!-- Post Quad: adds four posts in a rectangular configuration -->
+  <xacro:macro name="quad_post" params="name parent_link length:=0.08 width:=0.08 height radius:=0.006 *origin">
+    <link name="${name}_link">
+      <!-- Top Left -->
+      <visual>
+        <material name="light_grey" />
+        <origin xyz="${length/2} ${width/2} ${height/2}" />
+        <geometry>
+          <cylinder radius="${radius}" length="${height}" />
+        </geometry>
+      </visual>
+      <collision>
+        <material name="light_grey" />
+        <origin xyz="${length/2} ${width/2} ${height/2}" />
+        <geometry>
+          <cylinder radius="${radius}" length="${height}" />
+        </geometry>
+      </collision>
+      <!-- Top Right -->
+      <visual>
+        <material name="light_grey" />
+        <origin xyz="${length/2} ${-width/2} ${height/2}" />
+        <geometry>
+          <cylinder radius="${radius}" length="${height}" />
+        </geometry>
+      </visual>
+      <collision>
+        <material name="light_grey" />
+        <origin xyz="${length/2} ${-width/2} ${height/2}" />
+        <geometry>
+          <cylinder radius="${radius}" length="${height}" />
+        </geometry>
+      </collision>
+      <!-- Bottom Left -->
+      <visual>
+        <material name="light_grey" />
+        <origin xyz="${-length/2} ${width/2} ${height/2}" />
+        <geometry>
+          <cylinder radius="${radius}" length="${height}" />
+        </geometry>
+      </visual>
+      <collision>
+        <material name="light_grey" />
+        <origin xyz="${-length/2} ${width/2} ${height/2}" />
+        <geometry>
+          <cylinder radius="${radius}" length="${height}" />
+        </geometry>
+      </collision>
+      <!-- Bottom Right -->
+      <visual>
+        <material name="light_grey" />
+        <origin xyz="${-length/2} ${-width/2} ${height/2}" />
+        <geometry>
+          <cylinder radius="${radius}" length="${height}" />
+        </geometry>
+      </visual>
+      <collision>
+        <material name="light_grey" />
+        <origin xyz="${-length/2} ${-width/2} ${height/2}" />
+        <geometry>
+          <cylinder radius="${radius}" length="${height}" />
+        </geometry>
+      </collision>
+    </link>
+    <link name="${name}_mount"/>
+    <joint name="${name}_joint" type="fixed">
+      <child link="${name}_link" />
+      <parent link="${parent_link}" />
+      <insert_block name="origin" />
+    </joint>
+    <joint name="${name}_mount_joint" type="fixed">
+      <child link="${name}_mount" />
+      <parent link="${name}_link" />
+      <origin xyz="0 0 ${height}">
+      </origin>
+    </joint>
+  </xacro:macro>
 </robot>

File: clearpath_mounts_description/urdf/pacs/riser.urdf.xacro (robot description, xacro)
@@ -22,58 +22,50 @@
 -->
 <robot xmlns:xacro="http://ros.org/wiki/xacro">
-    <!-- <xacro:include filename="$(find clearpath_platform_description)/urdf/common.urdf.xacro" /> -->
-    <!--
+  <!--
         Full Riser: add plate sized riser
         - within PACS grid framework, only input required is 'level' (height)
         - adds legs and mounts
     -->
-    <xacro:macro name="riser" params="name parent_link thickness:=0.00635 rows:=8 columns:=7 *origin">
-      <xacro:property name="spacing" value="0.08" />
-      <xacro:property name="parent_coordinate" value="${parent_link[-2:]}"/>
-      <xacro:property name="standard_size" value="False"/>
-      <!-- Partial Riser Plate Link -->
-      <link name="${name}_link">
-        <visual>
-          <geometry>
-            <xacro:if value="${rows == 8 and columns == 7}">
-                <xacro:property name="standard_size" value="True"/>
-                <xacro:property name="thickness" value="0.00635"/>
-                <mesh filename="package://clearpath_mounts_description/meshes/pacs/riser_8x7.stl" />
-            </xacro:if>
-            <xacro:if value="${rows == 1 and columns == 7}">
-                <xacro:property name="standard_size" value="True"/>
-                <xacro:property name="thickness" value="0.00635"/>
-                <mesh filename="package://clearpath_mounts_description/meshes/pacs/riser_1x7.stl" />
-            </xacro:if>
-            <xacro:unless value="${standard_size}">
-                <box size="${rows * spacing} ${columns * spacing} ${thickness}"/>
-            </xacro:unless>
-          </geometry>
-          <material name="dark_grey" />
-          <origin xyz="${-(rows / 2) * spacing + spacing / 2} ${-(columns / 2) * spacing + spacing / 2} ${thickness / 2}" rpy="0 0 0" />
-        </visual>
-        <collision>
-          <origin xyz="0 0 ${thickness/2}" rpy="0 0 0" />
-          <geometry>
-            <box size="0.11 0.59 ${thickness}" />
-          </geometry>
-          <material name="dark_grey" />
-        </collision>
-      </link>
-      <!-- Row Riser Plate Joint -->
-      <joint name="${name}_joint" type="fixed">
-        <child link="${name}_link" />
-        <parent link="${parent_link}" />
-        <xacro:insert_block name="origin" />
-      </joint>
-      <!-- Row Riser Mounts -->
-      <xacro:full_mounts
-        name="${name}"
-        parent_link="${name}_link"
-        column="${parent_coordinate[0]}"
-		    row="${parent_coordinate[1]}"
-        columns="${columns}"
-        rows="${rows}"
-        z="${thickness}" />
-    </xacro:macro>
+  <xacro:macro name="riser" params="name parent_link thickness:=0.00635 rows:=8 columns:=7 *origin">
+    <xacro:property name="spacing" value="0.08" />
+    <xacro:property name="parent_coordinate" value="${parent_link[-2:]}"/>
+    <xacro:property name="standard_size" value="False"/>
+    <!-- Partial Riser Plate Link -->
+    <link name="${name}_link">
+      <visual>
+        <geometry>
+          <xacro:if value="${rows == 8 and columns == 7}">
+            <xacro:property name="standard_size" value="True"/>
+            <xacro:property name="thickness" value="0.00635"/>
+            <mesh filename="package://clearpath_mounts_description/meshes/pacs/riser_8x7.stl" />
+          </xacro:if>
+          <xacro:if value="${rows == 1 and columns == 7}">
+            <xacro:property name="standard_size" value="True"/>
+            <xacro:property name="thickness" value="0.00635"/>
+            <mesh filename="package://clearpath_mounts_description/meshes/pacs/riser_1x7.stl" />
+          </xacro:if>
+          <xacro:unless value="${standard_size}">
+            <box size="${rows * spacing} ${columns * spacing} ${thickness}"/>
+          </xacro:unless>
+        </geometry>
+        <material name="dark_grey" />
+        <origin xyz="${-(rows / 2) * spacing + spacing / 2} ${-(columns / 2) * spacing + spacing / 2} ${thickness / 2}" rpy="0 0 0" />
+      </visual>
+      <collision>
+        <origin xyz="0 0 ${thickness/2}" rpy="0 0 0" />
+        <geometry>
+          <box size="0.11 0.59 ${thickness}" />
+        </geometry>
+        <material name="dark_grey" />
+      </collision>
+    </link>
+    <!-- Row Riser Plate Joint -->
+    <joint name="${name}_joint" type="fixed">
+      <child link="${name}_link" />
+      <parent link="${parent_link}" />
+      <xacro:insert_block name="origin" />
+    </joint>
+    <!-- Row Riser Mounts -->
+    <xacro:full_mounts name="${name}" parent_link="${name}_link" column="${parent_coordinate[0]}" row="${parent_coordinate[1]}" columns="${columns}" rows="${rows}" z="${thickness}" />
+  </xacro:macro>
 </robot>

File: clearpath_mounts_description/urdf/pacs/riser_leg.urdf.xacro (robot description, xacro)
@@ -22,37 +22,36 @@
 -->
 <robot xmlns:xacro="http://ros.org/wiki/xacro">
-	<!-- <xacro:include filename="$(find clearpath_platform_description)/urdf/common.urdf.xacro" /> -->
-	<!--
+  <!--
 	Riser Leg: standard leg for partial and full risers
 	- 'height' is from parent to the bottom of riser (should substract thickness of riser)
 	-->
-	<xacro:macro name="riser_leg" params="name parent_link height *origin">
-		<link name="${name}_link">
-			<visual>
-				<origin xyz="0 0 ${height/2}" rpy="0 0 0" />
-				<geometry>
-					<box size="0.04 0.02 ${height}" />
-				</geometry>
-				<material name="dark_grey" />
-			</visual>
-			<collision>
-				<origin xyz="0 0 ${height/2}" rpy="0 0 0" />
-				<geometry>
-					<box size="0.04 0.02 ${height}" />
-				</geometry>
-				<material name="dark_grey" />
-			</collision>
-		</link>
-		<link name="${name}_mount"/>
-		<joint name="${name}_joint" type="fixed">
-			<child link="${name}_link" />
-			<parent link="${parent_link}" />
-            <insert_block name="origin" />
-		</joint>
-        <joint name="${name}_mount_joint" type="fixed">
-			<child link="${name}_mount" />
-			<parent link="${name}_link" />
-            <origin xyz="0 0 ${height}"/>
-		</joint>
-	</xacro:macro>
+  <xacro:macro name="riser_leg" params="name parent_link height *origin">
+    <link name="${name}_link">
+      <visual>
+        <origin xyz="0 0 ${height/2}" rpy="0 0 0" />
+        <geometry>
+          <box size="0.04 0.02 ${height}" />
+        </geometry>
+        <material name="dark_grey" />
+      </visual>
+      <collision>
+        <origin xyz="0 0 ${height/2}" rpy="0 0 0" />
+        <geometry>
+          <box size="0.04 0.02 ${height}" />
+        </geometry>
+        <material name="dark_grey" />
+      </collision>
+    </link>
+    <link name="${name}_mount"/>
+    <joint name="${name}_joint" type="fixed">
+      <child link="${name}_link" />
+      <parent link="${parent_link}" />
+      <insert_block name="origin" />
+    </joint>
+    <joint name="${name}_mount_joint" type="fixed">
+      <child link="${name}_mount" />
+      <parent link="${name}_link" />
+      <origin xyz="0 0 ${height}"/>
+    </joint>
+  </xacro:macro>
 </robot>

File: clearpath_sensors_description/urdf/hokuyo_ust10.urdf.xacro (robot description, xacro)
@@ -18,6 +18,6 @@
         <origin xyz="0 0 0" />
         <inertia ixx="${0.0833333 * 1.1 * (0.102*0.102 + 0.152*0.152)}" ixy="0.0" ixz="0.0"
-                  iyy="${0.0833333 * 1.1 * (0.105*0.105 + 0.152*0.152)}" iyz="0.0"
-                  izz="${0.0833333 * 1.1 * (0.105*0.105 + 0.102*0.102)}" />
+                 iyy="${0.0833333 * 1.1 * (0.105*0.105 + 0.152*0.152)}" iyz="0.0"
+                 izz="${0.0833333 * 1.1 * (0.105*0.105 + 0.102*0.102)}" />
       </inertial>
     </link>

File: clearpath_sensors_description/urdf/novatel_smart6.urdf.xacro (robot description, xacro)
@@ -2,15 +2,15 @@
 <robot xmlns:xacro="http://www.ros.org/wiki/xacro">
   <xacro:macro name="novatel_smart6" params="name">
-  <link name="${name}_link">
-    <visual>
-      <origin xyz="0 0 0" rpy="0 0 0" />
-      <geometry>
-        <mesh filename="package://clearpath_sensors_description/meshes/novatel_smart6.stl"/>
-      </geometry>
-      <material name="novatel_white">
-        <color rgba="0.8 0.8 0.8 1.0" />
-      </material>
-    </visual>
-  </link>
+    <link name="${name}_link">
+      <visual>
+        <origin xyz="0 0 0" rpy="0 0 0" />
+        <geometry>
+          <mesh filename="package://clearpath_sensors_description/meshes/novatel_smart6.stl"/>
+        </geometry>
+        <material name="novatel_white">
+          <color rgba="0.8 0.8 0.8 1.0" />
+        </material>
+      </visual>
+    </link>
   </xacro:macro>
 </robot>
