Commit message: Sensor descriptions

File: clearpath_sensors_description/urdf/ust10.urdf.xacro (robot description, xacro)
@@ -1,6 +1,5 @@
 <?xml version="1.0"?>
 <robot xmlns:xacro="http://ros.org/wiki/xacro">
-  <xacro:include filename="$(find clearpath_platform_description)/urdf/common.urdf.xacro" />
-  <xacro:macro name="hokuyo_ust10" params="name parent_link *origin">
+  <xacro:macro name="ust10" params="name parent_link *origin">
     <link name="${name}_link">
       <visual>
