Commit message: Updated sensor naming

File: clearpath_sensors_description/urdf/hokuyo_ust10.urdf.xacro (robot description, xacro)
@@ -1,5 +1,5 @@
 <?xml version="1.0"?>
 <robot xmlns:xacro="http://ros.org/wiki/xacro">
-  <xacro:macro name="ust10" params="name parent_link *origin">
+  <xacro:macro name="hokuyo_ust10" params="name parent_link *origin">
     <link name="${name}_link">
       <visual>
