Commit message: Correct optical frame naming and fix gazebo section

File: clearpath_sensors_description/urdf/flir_blackfly.urdf.xacro (robot description, xacro)
@@ -1,72 +1,73 @@
 <?xml version="1.0"?>
 <robot xmlns:xacro="http://www.ros.org/wiki/xacro" name="flir_blackfly">
-<!--
-    camera_{x,y,z,mass} are physical properties of camera collision model
-    lens_{r, h, mass} are physical properties of the camera lens
-    hfov, fps, width, height, format, near, and far are simulation
--->
-<xacro:macro name="flir_blackfly"
-    params="name parent_link *origin update_rate:=30.0 width:=720 height:=540 format:=R8G8B8 near:=0.5 far:=300">
-    <link name="${name}_link">
-    <!-- The following are not reliable values, and should not be used for modeling -->
-        <inertial>
-            <mass value= "0.03" />
-            <inertia ixx="1e-6" ixy="0" ixz="0" iyy="1e-6" iyz="0" izz="1e-6" />
-        </inertial>
-        <visual>
-            <origin xyz="0 0 0.01425" rpy="0 0 0" />
-            <geometry>
-                <mesh filename="package://clearpath_sensors_description/meshes/flir_blackfly.stl"/>
-            </geometry>
-            <material name="dark_grey" />
-        </visual>
-        <collision>
-            <origin xyz="0.003 0 0.0145" rpy="0 0 0" />
-            <geometry>
-            <box size="0.047758 0.029 0.029" />
-            </geometry>
-        </collision>
-    </link>
-    <joint name="${name}_joint" type="fixed">
-        <xacro:insert_block name="origin"/>
-        <parent link="${parent_link}"/>
-        <child link="${name}_link"/>
-    </joint>
-    <link name="${name}_lens">
-        <intertial>
-            <mass values="0.05" />
-            <inertia ixx="1e-6" ixy="0" ixz="0" iyy="1e-6" iyz="0" izz="1e-6" />
-        </intertial>
-        <visual>
-            <origin xyz="0.02 0 0" rpy="0 1.5707 0" />
-            <geometry>
-            <cylinder radius="0.016" length="0.04"/>
-            </geometry>
-            <material name="dark_grey" />
-        </visual>
-        <collision>
-            <origin xyz="0.02 0 0" rpy="0 1.5707 0" />
-            <geometry>
-            <cylinder radius="0.016" length="0.04"/>
-            </geometry>
-        </collision>
-    </link>
-    <link name="${name}_optical" />
-    <joint name="${name}_lens_joint" type="fixed">
-    <origin xyz="0.02685 0 0.01425" rpy="0 0 0" />
-    <parent link="${name}_link" />
-    <child link="${name}_lens" />
-    </joint>
-    <joint name="${name}_optical_joint" type="fixed">
-    <origin xyz="0.04 0 0" rpy="-1.570796 0 -1.570796" />
-    <parent link="${name}_lens" />
-    <child link="${name}_optical" />
-    </joint>
-    <!-- Gazebo -->
-    <gazebo reference="${name}_optical">
-        <sensor type="rgbd_camera" name="${name}">
-            <camera>
+    <!--
+        camera_{x,y,z,mass} are physical properties of camera collision model
+        lens_{r, h, mass} are physical properties of the camera lens
+        hfov, fps, width, height, format, near, and far are simulation
+    -->
+    <xacro:macro name="flir_blackfly"
+        params="name parent_link *origin hfov:=1.0471975512 update_rate:=30.0 width:=720
+                height:=540 format:=R8G8B8 near:=0.5 far:=300">
+        <link name="${name}_link">
+        <!-- The following are not reliable values, and should not be used for modeling -->
+            <inertial>
+                <mass value= "0.03" />
+                <inertia ixx="1e-6" ixy="0" ixz="0" iyy="1e-6" iyz="0" izz="1e-6" />
+            </inertial>
+            <visual>
+                <origin xyz="0 0 0.01425" rpy="0 0 0" />
+                <geometry>
+                    <mesh filename="package://clearpath_sensors_description/meshes/flir_blackfly.stl"/>
+                </geometry>
+                <material name="dark_grey" />
+            </visual>
+            <collision>
+                <origin xyz="0.003 0 0.0145" rpy="0 0 0" />
+                <geometry>
+                <box size="0.047758 0.029 0.029" />
+                </geometry>
+            </collision>
+        </link>
+        <joint name="${name}_joint" type="fixed">
+            <xacro:insert_block name="origin"/>
+            <parent link="${parent_link}"/>
+            <child link="${name}_link"/>
+        </joint>
+        <link name="${name}_lens">
+            <intertial>
+                <mass values="0.05" />
+                <inertia ixx="1e-6" ixy="0" ixz="0" iyy="1e-6" iyz="0" izz="1e-6" />
+            </intertial>
+            <visual>
+                <origin xyz="0.02 0 0" rpy="0 1.5707 0" />
+                <geometry>
+                <cylinder radius="0.016" length="0.04"/>
+                </geometry>
+                <material name="dark_grey" />
+            </visual>
+            <collision>
+                <origin xyz="0.02 0 0" rpy="0 1.5707 0" />
+                <geometry>
+                <cylinder radius="0.016" length="0.04"/>
+                </geometry>
+            </collision>
+        </link>
+        <link name="${name}_color_optical_frame" />
+        <joint name="${name}_lens_joint" type="fixed">
+            <origin xyz="0.02685 0 0.01425" rpy="0 0 0" />
+            <parent link="${name}_link" />
+            <child link="${name}_lens" />
+        </joint>
+        <joint name="${name}_optical_joint" type="fixed">
+            <origin xyz="0.04 0 0" rpy="0 0 0" />
+            <parent link="${name}_lens" />
+            <child link="${name}_color_optical_frame" />
+        </joint>
+        <!-- Gazebo -->
+        <gazebo reference="${name}_color_optical_frame">
+            <sensor type="camera" name="${name}">
+                <camera name="${name}">
                 <pose>0 0 0 0 -1.5707 1.5707</pose>
-                <horizontal_fov>1.0471975512</horizontal_fov>
+                <horizontal_fov>${hfov}</horizontal_fov>
                 <image>
                     <width>${width}</width>
@@ -83,21 +84,20 @@
                     <stddev>0.007</stddev>
                 </noise>
-                <optical_frame_id>${name}_color_optical_frame</optical_frame_id>
-            </camera>
-            <plugin name="camera_controller" filename="libgazebo_ros_camera.so">
-            <alwaysOn>true</alwaysOn>
-            <update_rate>${update_rate}</update_rate>
-            <cameraName>${name}</cameraName>
-            <imageTopicName>image_raw</imageTopicName>
-            <cameraInfoTopicName>camera_info</cameraInfoTopicName>
-            <hackBaseline>0.07</hackBaseline>
-            <distortionK1>0.0</distortionK1>
-            <distortionK2>0.0</distortionK2>
-            <distortionK3>0.0</distortionK3>
-            <distortionT1>0.0</distortionT1>
-            <distortionT2>0.0</distortionT2>
-            </plugin>
-        </sensor>
-    </gazebo>
-</xacro:macro>
+                </camera>
+                <plugin name="camera_controller" filename="libgazebo_ros_camera.so">
+                <alwaysOn>true</alwaysOn>
+                <updateRate>${update_rate}</updateRate>
+                <cameraName>${name}</cameraName>
+                <imageTopicName>image_raw</imageTopicName>
+                <cameraInfoTopicName>camera_info</cameraInfoTopicName>
+                <hackBaseline>0.07</hackBaseline>
+                <distortionK1>0.0</distortionK1>
+                <distortionK2>0.0</distortionK2>
+                <distortionK3>0.0</distortionK3>
+                <distortionT1>0.0</distortionT1>
+                <distortionT2>0.0</distortionT2>
+                </plugin>
+            </sensor>
+        </gazebo>
+    </xacro:macro>
 </robot>
