Commit message: Fix the path for the meshes

File: clearpath_sensors_description/urdf/axis_dome_fixed.urdf.xacro (robot description, xacro)
@@ -13,5 +13,5 @@
       <visual>
         <geometry>
-          <mesh filename="package://axis_description/meshes/axis_dome.stl" scale="1 1 1" />
+          <mesh filename="package://clearpth_sensors_description/meshes/axis_dome.stl" scale="1 1 1" />
         </geometry>
         <material name="axis_white">

File: clearpath_sensors_description/urdf/axis_dome_ptz.urdf.xacro (robot description, xacro)
@@ -13,5 +13,5 @@
       <visual>
         <geometry>
-          <mesh filename="package://axis_description/meshes/axis_dome.stl" scale="1 1 1" />
+          <mesh filename="package://clearpth_sensors_description/meshes/axis_dome.stl" scale="1 1 1" />
         </geometry>
         <material name="axis_white">
