Commit message: Keep sensor origin directly above base_link

File: clearpath_sensors_description/urdf/seyond_lidar.urdf.xacro (robot description, xacro)
@@ -45,5 +45,5 @@
             <parent link="${name}_base_link" />
             <child link="${name}_laser" />
-            <origin xyz="0.04 0 0.042" rpy="0 0 0" />
+            <origin xyz="0 0 0.042" rpy="0 0 0" />
         </joint>
         <xacro:property name="samples_h" value="${round((max_ang_h - min_ang_h) * 180 / (ang_res_h * pi))}"/>

Commit message: Make the shade of grey darker

File: clearpath_sensors_description/urdf/seyond_lidar.urdf.xacro (robot description, xacro)
@@ -19,6 +19,6 @@
                     <mesh filename="package://clearpath_sensors_description/meshes/seyond_robin_w.stl"/>
                 </geometry>
-                <material name="silver">
-                    <color rgba="0.7 0.7 0.7 1.0" />
+                <material name="seyond_dark_grey">
+                    <color rgba="0.3 0.3 0.3 1.0" />
                 </material>
             </visual>
