Commit message: Fix collision bodies for patch, helical antennas

File: clearpath_sensors_description/urdf/gnss_antenna.urdf.xacro (robot description, xacro)
@@ -38,4 +38,10 @@
                     <origin xyz="0 0 0" rpy="0 0 0" />
                 </visual>
+                <collision>
+                    <geometry>
+                        <cylinder radius="0.015" length="0.055"/>
+                    </geometry>
+                    <origin xyz="0 0 0.0275" rpy="0 0 0" />
+                </collision>
                 <!--
                     TODO: cylinder collision
@@ -55,11 +61,10 @@
                         <mesh filename="package://clearpath_sensors_description/meshes/gnss_patch.stl" />
                     </geometry>
-                    <origin xyz="0 0 0.005" />
                 </visual>
                 <collision>
                     <geometry>
-                        <box size="0.025 0.025 0.01" />
+                        <box size="0.06 0.06 0.02" />
                     </geometry>
-                    <origin xyz="0 0 0.005" rpy="0 0 0" />
+                    <origin xyz="0 0 0.01" rpy="0 0 0" />
                 </collision>
             </link>

Commit message: Use the new gnss_antenna for the Swiftnav Duro URDF

File: clearpath_sensors_description/urdf/gnss_antenna.urdf.xacro (robot description, xacro)
@@ -1,4 +1,13 @@
 <?xml version="1.0" encoding="UTF-8"?>
 <robot xmlns:xacro="http://wiki.ros.org/xacro">
+    <!--
+        Macro for adding GNSS (aka: GPS) antennas to robots
+        3 types are supported:
+            - "spherical" - dome-shaped antennas commonly used with SwiftNav Duro receivers
+            - "helical" - cylindrical antennas included by default with Fixposition systems
+            - "patch" - small, square antennas used with low-cost units like Ublox
+        The antenna has 1 link (the physical mounting point) called ${prefix}_link and 1
+        fixed joint called ${prefix}_joint connecting parent_link to ${prefix}_link.
+    -->
     <xacro:macro name="gnss_antenna" params="
         prefix

File: clearpath_sensors_description/urdf/swiftnav_duro.urdf.xacro (robot description, xacro)
@@ -2,24 +2,8 @@
 <robot xmlns:xacro="http://www.ros.org/wiki/xacro">
   <xacro:macro name="swiftnav_duro" params="name parent_link *origin">
-    <link name="${name}_link">
-      <visual>
-        <material name="clearpath_white"/>
-        <geometry>
-          <mesh filename="package://clearpath_sensors_description/meshes/gnss_spherical.stl"/>
-        </geometry>
-      </visual>
-      <collision>
-        <material name="clearpath_white"/>
-        <origin xyz="0.0000 -0.0000 0.0324"/>
-        <geometry>
-          <sphere radius="0.1122" />
-        </geometry>
-      </collision>
-    </link>
-    <joint name="${name}_joint" type="fixed">
-      <child link="${name}_link"/>
-      <parent link="${parent_link}"/>
+    <xacro:include filename="$(find clearpath_sensors_description)/urdf/gnss_antenna.urdf.xacro" />
+    <xacro:gnss_antenna prefix="${name}" parent_link="${parent_link}" type="spherical">
       <xacro:insert_block name="origin"/>
-    </joint>
+    </xacro:gnss_antenna>
     <gazebo reference="${name}_link">
       <sensor name="${name}" type="navsat">

Commit message: Rename the antenna joint to just _joint, not _base_joint

File: clearpath_sensors_description/urdf/gnss_antenna.urdf.xacro (robot description, xacro)
@@ -32,5 +32,5 @@
                 </collision>
             </link>
-            <joint name="${prefix}_base_joint" type="fixed">
+            <joint name="${prefix}_joint" type="fixed">
                 <parent link="${parent_link}" />
                 <child link="${prefix}_link" />
@@ -54,5 +54,5 @@
                 </collision>
             </link>
-            <joint name="${prefix}_base_joint" type="fixed">
+            <joint name="${prefix}_joint" type="fixed">
                 <parent link="${parent_link}" />
                 <child link="${prefix}_link" />
@@ -75,5 +75,5 @@
                 </collision>
             </link>
-            <joint name="${prefix}_base_joint" type="fixed">
+            <joint name="${prefix}_joint" type="fixed">
                 <parent link="${parent_link}" />
                 <child link="${prefix}_link" />
