Commit message: Rename swift_antenna -> gnss_spherical, add gnss_helical, start filling in the fixposition URDF. Waiting for the STL from Rhys

File: clearpath_sensors_description/urdf/fixposition.urdf.xacro (robot description, xacro)
@@ -1,3 +1,7 @@
 <?xml version="1.0" encoding="UTF-8"?>
+<!--
+    Fixposition mesh originally sourced from
+    https://docs.fixposition.com/fd/step-model-and-camera-fov-data#STEPmodelandcameraFOVdata-LinktotheSTEPfile
+-->
 <robot xmlns:xacro="http://wiki.ros.org/xacro">
     <xacro:macro name="fixposition" params="
@@ -7,6 +11,119 @@
         model:=xvn
         topic:=platform/odom/filtered
-        update_rate:=100
+        update_rate:=200
+        num_gps:=2
+        gps_0_type:=spherical
+        gps_0_xyz:=0 0 0
+        gps_0_rpy:=0 0 0
+        gps_0_parent:=base_link
+        gps_1_type:=spherical
+        gps_1_xyz:=0 0 0
+        gps_1_rpy:=0 0 0
+        gps_1_parent:=base_link
     ">
+        <xacro:macro name="gnss_antenna" params="
+            prefix
+            parent_link
+            *origin
+            type:=spherical
+        ">
+            <xacro:if value="${type == 'spherical'}">
+                <link name="${prefix}_base_link">
+                    <visual>
+                        <material name="clearpath_white"/>
+                        <geometry>
+                            <mesh filename="package://clearpath_sensors_description/meshes/gnss_spherical.stl"/>
+                        </geometry>
+                    </visual>
+                    <collision>
+                        <material name="clearpath_white"/>
+                        <origin xyz="0.0000 -0.0000 0.0324"/>
+                        <geometry>
+                            <sphere radius="0.1122" />
+                        </geometry>
+                    </collision>
+                </link>
+                <joint name="${prefix}_base_joint" type="fixed">
+                    <parent link="${parent_link}" />
+                    <child link="${prefix}_base_link" />
+                    <xacro:insert_block name="origin" />
+                </joint>
+            </xacro:if>
+            <xacro:if value="${type == 'helical'}">
+                <link name="${prefix}_base_link">
+                    <visual>
+                        <material name="clearpath_white"/>
+                        <geometry>
+                            <mesh filename="package://clearpath_sensors_description/meshes/gnss_helical.stl"/>
+                        </geometry>
+                    </visual>
+                    <!--
+                        TODO: cylinder collision
+                    -->
+                </link>
+                <joint name="${prefix}_base_joint" type="fixed">
+                    <parent link="${parent_link}" />
+                    <child link="${prefix}_base_link" />
+                    <xacro:insert_block name="origin" />
+                </joint>
+            </xacro:if>
+            <xacro:if value="${type == 'patch'}">
+                <link name="${prefix}_base_link">
+                    <!--
+                        TODO: assuming 25mm square for now, but this may be incorrect
+                    -->
+                    <visual>
+                        <material name="clearpath_black" />
+                        <geometry>
+                            <box size="0.025 0.025 0.01" />
+                        </geometry>
+                        <origin xyz="0 0 0.005" />
+                    </visual>
+                    <collision>
+                        <geometry>
+                            <box size="0.025 0.025 0.01" />
+                        </geometry>
+                        <origin xyz="0 0 0.005" rpy="0 0 0" />
+                    </collision>
+                </link>
+                <joint name="${prefix}_base_joint" type="fixed">
+                    <parent link="${parent_link}" />
+                    <child link="${prefix}_base_link" />
+                    <xacro:insert_block name="origin" />
+                </joint>
+            </xacro:if>
+        </xacro:macro>
+        <link name="${name}_base_link">
+            <visual>
+            </visual>
+            <collision>
+                <geometry>
+                    <box size="0.1291 0.1136 0.03" />
+                </geometry>
+                <origin xyz="0 0 0.015" rpy="0 0 0" />
+            </collision>
+        </link>
+        <joint name="${name}_base_joint" type="fixed">
+            <parent link="${parent_link}" />
+            <child link="${name}_base_link" />
+            <xacro:insert_block name="origin" />
+        </joint>
+        <!--
+            1 antenna is mandatory, second is optional
+        -->
+        <xacro:gnss_antenna
+            prefix="${name}_gps0"
+            parent_link="${gps_0_parent"
+            type="${gps_0_type">
+            <origin xyz="${gps_0_xyz}" rpy="{gps0_rpy}" />
+        </xacro:gnss_antenna>
+        <xacro:if value="${num_gps > 1}">
+            <xacro:gnss_antenna
+                prefix="${name}_gps1"
+                parent_link="${gps_1_parent"
+                type="${gps_1_type">
+                <origin xyz="${gps_1_xyz}" rpy="{gps_1_rpy}" />
+            </xacro:gnss_antenna>
+        </xacro:if>
     </xacro:macro>
 </robot>

File: clearpath_sensors_description/urdf/swiftnav_duro.urdf.xacro (robot description, xacro)
@@ -6,5 +6,5 @@
         <material name="clearpath_white"/>
         <geometry>
-          <mesh filename="package://clearpath_sensors_description/meshes/swift_antenna.stl"/>
+          <mesh filename="package://clearpath_sensors_description/meshes/gnss_spherical.stl"/>
         </geometry>
       </visual>

Commit message: Add patch antenna STL, move gnss_antenna macro to its own file, fix parameters in the fixposition macro

File: clearpath_sensors_description/urdf/fixposition.urdf.xacro (robot description, xacro)
@@ -14,89 +14,35 @@
         num_gps:=2
         gps_0_type:=spherical
-        gps_0_xyz:=0 0 0
-        gps_0_rpy:=0 0 0
+        gps_0_xyz_x:=0
+        gps_0_xyz_y:=0
+        gps_0_xyz_z:=0
+        gps_0_rpy_r:=0
+        gps_0_rpy_p:=0
+        gps_0_rpy_y:=0
         gps_0_parent:=base_link
         gps_1_type:=spherical
-        gps_1_xyz:=0 0 0
-        gps_1_rpy:=0 0 0
+        gps_1_xyz_x:=0
+        gps_1_xyz_y:=0
+        gps_1_xyz_z:=0
+        gps_1_rpy_r:=0
+        gps_1_rpy_p:=0
+        gps_1_rpy_y:=0
         gps_1_parent:=base_link
     ">
-        <xacro:macro name="gnss_antenna" params="
-            prefix
-            parent_link
-            *origin
-            type:=spherical
-        ">
-            <xacro:if value="${type == 'spherical'}">
-                <link name="${prefix}_base_link">
-                    <visual>
-                        <material name="clearpath_white"/>
-                        <geometry>
-                            <mesh filename="package://clearpath_sensors_description/meshes/gnss_spherical.stl"/>
-                        </geometry>
-                    </visual>
-                    <collision>
-                        <material name="clearpath_white"/>
-                        <origin xyz="0.0000 -0.0000 0.0324"/>
-                        <geometry>
-                            <sphere radius="0.1122" />
-                        </geometry>
-                    </collision>
-                </link>
-                <joint name="${prefix}_base_joint" type="fixed">
-                    <parent link="${parent_link}" />
-                    <child link="${prefix}_base_link" />
-                    <xacro:insert_block name="origin" />
-                </joint>
-            </xacro:if>
-            <xacro:if value="${type == 'helical'}">
-                <link name="${prefix}_base_link">
-                    <visual>
-                        <material name="clearpath_white"/>
-                        <geometry>
-                            <mesh filename="package://clearpath_sensors_description/meshes/gnss_helical.stl"/>
-                        </geometry>
-                    </visual>
-                    <!--
-                        TODO: cylinder collision
-                    -->
-                </link>
-                <joint name="${prefix}_base_joint" type="fixed">
-                    <parent link="${parent_link}" />
-                    <child link="${prefix}_base_link" />
-                    <xacro:insert_block name="origin" />
-                </joint>
-            </xacro:if>
-            <xacro:if value="${type == 'patch'}">
-                <link name="${prefix}_base_link">
-                    <!--
-                        TODO: assuming 25mm square for now, but this may be incorrect
-                    -->
-                    <visual>
-                        <material name="clearpath_black" />
-                        <geometry>
-                            <box size="0.025 0.025 0.01" />
-                        </geometry>
-                        <origin xyz="0 0 0.005" />
-                    </visual>
-                    <collision>
-                        <geometry>
-                            <box size="0.025 0.025 0.01" />
-                        </geometry>
-                        <origin xyz="0 0 0.005" rpy="0 0 0" />
-                    </collision>
-                </link>
-                <joint name="${prefix}_base_joint" type="fixed">
-                    <parent link="${parent_link}" />
-                    <child link="${prefix}_base_link" />
-                    <xacro:insert_block name="origin" />
-                </joint>
-            </xacro:if>
-        </xacro:macro>
+        <xacro:include filename="$(find clearpath_sensors_description)/urdf/gnss_antenna.urdf.xacro" />
         <link name="${name}_base_link">
             <visual>
+                <material name="clearpath_white"/>
+                <geometry>
+                    <mesh filename="package://clearpath_sensors_description/meshes/fixposition.stl" />
+                </geometry>
+                <origin xyz="0 0 0" rpy="0 0 0" />
             </visual>
             <collision>
                 <geometry>
+                    <!--
+                        Bounding box dimensions from
+                        https://docs.fixposition.com/__attachments/73072655/VRTK2_integration_manual_v2.3.3.pdf
+                    -->
                     <box size="0.1291 0.1136 0.03" />
                 </geometry>
@@ -114,14 +60,20 @@
         <xacro:gnss_antenna
             prefix="${name}_gps0"
-            parent_link="${gps_0_parent"
-            type="${gps_0_type">
-            <origin xyz="${gps_0_xyz}" rpy="{gps0_rpy}" />
+            parent_link="${gps_0_parent}"
+            type="${gps_0_type}">
+            <origin
+                xyz="${gps_0_xyz_x} ${gps_0_xyz_y} ${gps_0_xyz_z}"
+                rpy="${gps_0_rpy_r} ${gps_0_rpy_p} ${gps_0_rpy_y}"
+            />
         </xacro:gnss_antenna>
         <xacro:if value="${num_gps > 1}">
             <xacro:gnss_antenna
                 prefix="${name}_gps1"
-                parent_link="${gps_1_parent"
-                type="${gps_1_type">
-                <origin xyz="${gps_1_xyz}" rpy="{gps_1_rpy}" />
+                parent_link="${gps_1_parent}"
+                type="${gps_1_type}">
+                <origin
+                    xyz="${gps_1_xyz_x} ${gps_1_xyz_y} ${gps_1_xyz_z}"
+                    rpy="${gps_1_rpy_r} ${gps_1_rpy_p} ${gps_1_rpy_y}"
+                />
             </xacro:gnss_antenna>
         </xacro:if>

Commit message: Rename antenna frames, set scale of XVN mesh, add a sensor frame to the top of the XVN

File: clearpath_sensors_description/urdf/fixposition.urdf.xacro (robot description, xacro)
@@ -33,5 +33,5 @@
                 <material name="clearpath_white"/>
                 <geometry>
-                    <mesh filename="package://clearpath_sensors_description/meshes/fixposition.stl" />
+                    <mesh filename="package://clearpath_sensors_description/meshes/fixposition.stl" scale="0.001 0.001 0.001" />
                 </geometry>
                 <origin xyz="0 0 0" rpy="0 0 0" />
@@ -54,8 +54,17 @@
         </joint>
         <!--
+            Sensor origin is on the top of the unit, but base_link is on the bottom
+        -->
+        <link name="${name}_sensor"/>
+        <joint name="${name}_sensor_joint" type="fixed">
+            <parent link="${name}_base_link" />
+            <child link="${name}_sensor" />
+            <origin xyz="0 0 0.03" rpy="0 0 0" />
+        </joint>
+        <!--
             1 antenna is mandatory, second is optional
         -->
         <xacro:gnss_antenna
-            prefix="${name}_gps0"
+            prefix="${name}_gps_0"
             parent_link="${gps_0_parent}"
             type="${gps_0_type}">
@@ -67,5 +76,5 @@
         <xacro:if value="${num_antennas > 1}">
             <xacro:gnss_antenna
-                prefix="${name}_gps1"
+                prefix="${name}_gps_1"
                 parent_link="${gps_1_parent}"
                 type="${gps_1_type}">

File: clearpath_sensors_description/urdf/gnss_antenna.urdf.xacro (robot description, xacro)
@@ -8,5 +8,5 @@
     ">
         <xacro:if value="${type == 'spherical'}">
-            <link name="${prefix}_base_link">
+            <link name="${prefix}_link">
                 <visual>
                     <material name="clearpath_white"/>
@@ -25,10 +25,10 @@
             <joint name="${prefix}_base_joint" type="fixed">
                 <parent link="${parent_link}" />
-                <child link="${prefix}_base_link" />
+                <child link="${prefix}_link" />
                 <xacro:insert_block name="origin" />
             </joint>
         </xacro:if>
         <xacro:if value="${type == 'helical'}">
-            <link name="${prefix}_base_link">
+            <link name="${prefix}_link">
                 <visual>
                     <material name="clearpath_white"/>
@@ -44,10 +44,10 @@
             <joint name="${prefix}_base_joint" type="fixed">
                 <parent link="${parent_link}" />
-                <child link="${prefix}_base_link" />
+                <child link="${prefix}_link" />
                 <xacro:insert_block name="origin" />
             </joint>
         </xacro:if>
         <xacro:if value="${type == 'patch'}">
-            <link name="${prefix}_base_link">
+            <link name="${prefix}_link">
                 <visual>
                     <material name="clearpath_black" />
@@ -66,5 +66,5 @@
             <joint name="${prefix}_base_joint" type="fixed">
                 <parent link="${parent_link}" />
-                <child link="${prefix}_base_link" />
+                <child link="${prefix}_link" />
                 <xacro:insert_block name="origin" />
             </joint>

Commit message: Add the 3.5cm front offset between the XVN physical mounting point & the sensor origin

File: clearpath_sensors_description/urdf/fixposition.urdf.xacro (robot description, xacro)
@@ -54,5 +54,5 @@
         </joint>
         <!--
-            Sensor origin is on the top of the unit, but base_link is on the bottom
+            Sensor origin is on the top of the unit, slightly in front of the mounting point
         -->
         <link name="${name}_sensor"/>
@@ -60,5 +60,5 @@
             <parent link="${name}_base_link" />
             <child link="${name}_sensor" />
-            <origin xyz="0 0 0.03" rpy="0 0 0" />
+            <origin xyz="0.035 0 0.03" rpy="0 0 0" />
         </joint>
         <!--
