Commit message: Resize Wiferion

File: clearpath_sensors_description/urdf/wiferion.urdf.xacro (robot description, xacro)
@@ -2,4 +2,6 @@
 <robot xmlns:xacro="http://www.ros.org/wiki/xacro">
   <xacro:macro name="wiferion" params="name parent_link *origin">
+    <xacro:property name="thickness" value="0.03"/>
+    <xacro:property name="length" value="0.16"/>
     <link name="${name}_link">
       <visual>
@@ -7,6 +9,7 @@
           <color rgba="0.06 0.32 0.73 1.0" />
         </material>
+        <origin xyz="${thickness/2} 0 0"/>
         <geometry>
-          <box size="0.015 0.25 0.25"/>
+          <box size="${thickness} ${length} ${length}"/>
         </geometry>
       </visual>
@@ -15,6 +18,7 @@
           <color rgba="0.06 0.32 0.73 1.0" />
         </material>
+        <origin xyz="${thickness/2} 0 0"/>
         <geometry>
-          <box size="0.015 0.25 0.25"/>
+          <box size="${thickness} ${length} ${length}"/>
         </geometry>
       </collision>
