Commit message: 0. -> 0.0

File: clearpath_sensors_description/urdf/ouster_os1.urdf.xacro (robot description, xacro)
@@ -30,12 +30,12 @@
     <xacro:property name="lidar_diameter" value="0.087"/>
     <xacro:if value="${base == 'base'}">
-      <xacro:property name="base_mass" value="0."/>
+      <xacro:property name="base_mass" value="0.0"/>
       <xacro:property name="base_height" value="0.0225"/>
       <xacro:property name="base_length" value="0.110"/>
     </xacro:if>
     <xacro:unless value="${base == 'base'}">
-      <xacro:property name="base_mass" value="0."/>
-      <xacro:property name="base_height" value="0."/>
-      <xacro:property name="base_length" value="0."/>
+      <xacro:property name="base_mass" value="0.0"/>
+      <xacro:property name="base_height" value="0.0"/>
+      <xacro:property name="base_length" value="0.0"/>
     </xacro:unless>
     <xacro:property name="fins_mass" value="0.079"/>
