Commit message: Add corrected D435 mesh with fixed normals

File: clearpath_sensors_description/urdf/intel_realsense.urdf.xacro (robot description, xacro)
@@ -48,5 +48,5 @@
             <origin xyz="${d435_zero_depth_to_glass + d435_glass_to_front} ${-d435_cam_depth_py} 0" rpy="${M_PI/2} 0 ${M_PI/2}"/>
             <geometry>
-              <mesh filename="package://realsense2_description/meshes/d435.dae" />
+              <mesh filename="package://clearpath_sensors_description/meshes/d435.dae" />
             </geometry>
           </xacro:if>
