Commit message: control launch fixes Added ark enclosure for j100 top_plate

File: clearpath_platform_description/urdf/j100/decorations/top_plate.urdf.xacro (robot description, xacro)
@@ -1,156 +1,19 @@
 <?xml version="1.0"?>
 <robot xmlns:xacro="http://ros.org/wiki/xacro">
-    <!-- <xacro:include filename="$(find clearpath_platform_description)/urdf/common.urdf.xacro" /> -->
     <xacro:macro name="top_plate" params="model:=default">
-        <!-- Spawn the top plate -->
-      <xacro:if value="${model == 'default'}">
-        <link name="top_plate_link">
+      <xacro:if value="${model == 'ark_enclosure'}">
+         <link name="ark_enclosure_link">
           <visual>
-            <origin xyz="0 0 0" rpy="0 0 0" />
-            <geometry>
-              <mesh filename="package://clearpath_platform_description/meshes/a200/decorations/large_top_plate.dae" />
-            </geometry>
-          </visual>
-          <collision>
             <origin xyz="0 0 0" rpy="0 0 0"/>
             <geometry>
-              <mesh filename="package://clearpath_platform_description/meshes/a200/decorations/large_top_plate_collision.stl" />
+              <mesh filename="package://clearpath_platform_description/meshes/j100/decorations/ark_enclosure.stl"/>
             </geometry>
-          </collision>
-        </link>
-        <!-- Attach top plate -->
-        <joint name="top_plate_joint" type="fixed">
-          <parent link="base_link" />
-          <child link="top_plate_link"/>
-          <origin xyz="0.0812 0 0.225" rpy="0 0 0"/>
-        </joint>
-        <!-- Top plate front link -->
-        <joint name="top_plate_front_joint" type="fixed">
-          <parent link="top_plate_link" />
-          <child link="top_plate_front_link"/>
-          <origin xyz="0.4125 0 0.00672" rpy="0 0 0"/>
-        </joint>
-        <!-- Top plate rear link-->
-        <joint name="top_plate_rear_joint" type="fixed">
-          <parent link="top_plate_link" />
-          <child link="top_plate_rear_link"/>
-          <origin xyz="-0.4125 0 0.00672" rpy="0 0 0"/>
-        </joint>
-        <link name="top_plate_front_link"/>
-        <link name="top_plate_rear_link"/>
-      </xacro:if>
-      <xacro:if value="${model == 'large'}">
-        <link name="top_plate_link">
-          <visual>
-            <origin xyz="0 0 0" rpy="0 0 0" />
-            <geometry>
-              <mesh filename="package://clearpath_platform_description/meshes/a200/decorations/top_plate.dae" />
-            </geometry>
-          </visual>
-          <collision>
-            <origin xyz="0 0 0" rpy="0 0 0"/>
-            <geometry>
-              <mesh filename="package://clearpath_platform_description/meshes/a200/decorations/top_plate.stl" />
-            </geometry>
-          </collision>
-        </link>
-        <!-- Attach top plate -->
-        <joint name="top_plate_joint" type="fixed">
-          <parent link="base_link" />
-          <child link="top_plate_link"/>
-          <origin xyz="0.0812 0 0.245" rpy="0 0 0"/>
-        </joint>
-        <!-- Top plate front link -->
-        <joint name="top_plate_front_joint" type="fixed">
-          <parent link="top_plate_link" />
-          <child link="top_plate_front_link"/>
-          <origin xyz="0.36367 0 0.00639" rpy="0 0 0"/>
-        </joint>
-        <!-- Top plate rear link-->
-        <joint name="top_plate_rear_joint" type="fixed">
-          <parent link="top_plate_link" />
-          <child link="top_plate_rear_link"/>
-          <origin xyz="-0.36633 0 0.00639" rpy="0 0 0"/>
-        </joint>
-        <!-- Spawn user rails -->
-        <link name="user_rail_link">
-          <visual>
-            <geometry>
-              <mesh filename="package://clearpath_platform_description/meshes/a200/decorations/user_rail.dae" />
-            </geometry>
+            <material name="dark_grey" />
           </visual>
         </link>
-        <!-- Attach user rails to base link -->
-        <joint name="user_rail" type="fixed">
-          <origin xyz="0.272 0 0.245" rpy="0 0 0" />
-          <parent link="base_link" />
-          <child link="user_rail_link" />
+        <joint name="ark_enclosure_joint" type="fixed">
+          <parent link="mid_mount" />
+          <child link="ark_enclosure_link" />
         </joint>
-        <link name="top_plate_front_link"/>
-        <link name="top_plate_rear_link"/>
-      </xacro:if>
-      <xacro:if value="${model == 'pacs'}">
-        <link name="top_plate_link">
-          <visual>
-            <material name="dark_grey" />
-            <geometry>
-              <mesh filename="package://clearpath_platform_description/meshes/a200/decorations/pacs_top_plate.stl" />
-            </geometry>
-          </visual>
-          <collision>
-            <material name="dark_grey" />
-            <origin xyz="0 0 0.00317500531673" rpy="0 0 0"/>
-            <geometry>
-              <box size="0.670000076294 0.590000033379 0.00635001063347"/>
-            </geometry>
-          </collision>
-        </link>
-        <!-- Attach PACS top plate -->
-        <joint name="top_plate_joint" type="fixed">
-          <child link="top_plate_link"/>
-          <parent link="base_link"/>
-          <origin xyz="0.048299998045 0 0.227500006557" rpy="0 0 0"/>
-        </joint>
-        <!-- Generate PACS mounts -->
-        <xacro:full_mounts
-          name="top_plate"
-          parent_link="top_plate_link"
-          column="a"
-          row="1"
-          columns="7"
-          rows="2"
-          x="0.28"
-          y="0.24"
-          z="0.00635" />
-        <xacro:full_mounts
-          name="top_plate"
-          parent_link="top_plate_link"
-          column="a"
-          row="3"
-          columns="1"
-          rows="4"
-          x="0.12"
-          y="0.24"
-          z="0.00635" />
-        <xacro:full_mounts
-          name="top_plate"
-          parent_link="top_plate_link"
-          column="g"
-          row="3"
-          columns="1"
-          rows="4"
-          x="0.12"
-          y="-0.24"
-          z="0.00635" />
-        <xacro:full_mounts
-          name="top_plate"
-          parent_link="top_plate_link"
-          column="a"
-          row="7"
-          columns="7"
-          rows="2"
-          x="-0.20"
-          y="0.24"
-          z="0.00635" />
       </xacro:if>
     </xacro:macro>

File: clearpath_platform_description/urdf/j100/j100.urdf.xacro (robot description, xacro)
@@ -114,5 +114,5 @@
         </xacro:if>
         <xacro:unless value="$(arg is_sim)">
-          <plugin>j100_hardware/J100Hardware</plugin>
+          <plugin>clearpath_platform/J100Hardware</plugin>
           <plugin>fake_components/GenericSystem</plugin>
         </xacro:unless>
