Commit message: Moved IMU filter to platform launch Moved localization into a separate launch file Updated decoration urdfs Added structure urdf

File: clearpath_platform_description/urdf/a200/decorations/bumper.urdf.xacro (robot description, xacro)
@@ -1,5 +1,5 @@
 <?xml version="1.0"?>
 <robot xmlns:xacro="http://ros.org/wiki/xacro">
-    <xacro:macro name="bumper" params="name extension:=0">
+    <xacro:macro name="bumper" params="name extension:=0 *origin">
         <xacro:property name="parent_link" value="front_bumper_mount" />
         <xacro:if value="${'rear' in name}" >

File: clearpath_platform_description/urdf/a200/decorations/top_plate.urdf.xacro (robot description, xacro)
@@ -2,5 +2,5 @@
 <robot xmlns:xacro="http://ros.org/wiki/xacro">
     <!-- <xacro:include filename="$(find clearpath_platform_description)/urdf/common.urdf.xacro" /> -->
-    <xacro:macro name="top_plate" params="model:=default">
+    <xacro:macro name="top_plate" params="model:=default *origin">
         <!-- Spawn the top plate -->
       <xacro:if value="${model == 'large'}">
