Commit message: Fixes to control parameters and naming

File: clearpath_platform_description/urdf/w200/attachments/w200_arm_mount.urdf.xacro (robot description, xacro)
@@ -1,5 +1,5 @@
 <?xml version="1.0"?>
 <robot xmlns:xacro="http://ros.org/wiki/xacro">
-  <xacro:macro name="warthog_arm_mount">
+  <xacro:macro name="w200_arm_mount">
     <link name="arm_mount_link">
       <visual>

File: clearpath_platform_description/urdf/w200/attachments/w200_bulkhead.urdf.xacro (robot description, xacro)
@@ -1,10 +1,10 @@
 <?xml version="1.0"?>
 <robot xmlns:xacro="http://www.ros.org/wiki/xacro">
-  <xacro:macro name="warthog_generator">
-    <link name="generator_link">
+  <xacro:macro name="w200_bulkhead">
+    <link name="bulkhead_link">
       <visual>
         <origin xyz="0 0 0" rpy="0 0 0"/>
         <geometry>
-          <mesh filename="package://clearpath_platform_description/meshes/w200/generator.stl" />
+          <mesh filename="package://clearpath_platform_description/meshes/w200/bulkhead.stl" />
         </geometry>
         <material name="black"><color rgba="0.15 0.15 0.15 1.0" /></material>
@@ -13,5 +13,5 @@
         <origin xyz="0 0 0" rpy="0 0 0"/>
         <geometry>
-          <mesh filename="package://clearpath_platform_description/meshes/w200/generator.stl" />
+          <mesh filename="package://clearpath_platform_description/meshes/w200/bulkhead-collision.stl" />
         </geometry>
       </collision>
@@ -22,4 +22,5 @@
       </inertial>
     </link>
+    <link name="bulkhead_front_mount_link"/>
   </xacro:macro>
 </robot>

File: clearpath_platform_description/urdf/w200/attachments/w200_generator.urdf.xacro (robot description, xacro)
@@ -1,10 +1,10 @@
 <?xml version="1.0"?>
 <robot xmlns:xacro="http://www.ros.org/wiki/xacro">
-  <xacro:macro name="warthog_bulkhead">
-    <link name="bulkhead_link">
+  <xacro:macro name="w200_generator">
+    <link name="generator_link">
       <visual>
         <origin xyz="0 0 0" rpy="0 0 0"/>
         <geometry>
-          <mesh filename="package://clearpath_platform_description/meshes/w200/bulkhead.stl" />
+          <mesh filename="package://clearpath_platform_description/meshes/w200/generator.stl" />
         </geometry>
         <material name="black"><color rgba="0.15 0.15 0.15 1.0" /></material>
@@ -13,5 +13,5 @@
         <origin xyz="0 0 0" rpy="0 0 0"/>
         <geometry>
-          <mesh filename="package://clearpath_platform_description/meshes/w200/bulkhead-collision.stl" />
+          <mesh filename="package://clearpath_platform_description/meshes/w200/generator.stl" />
         </geometry>
       </collision>
@@ -22,5 +22,4 @@
       </inertial>
     </link>
-    <link name="bulkhead_front_mount_link"/>
   </xacro:macro>
 </robot>
