Commit message: Added  to materials

File: clearpath_platform_description/urdf/a200/attachments/bumper.urdf.xacro (robot description, xacro)
@@ -28,5 +28,5 @@
                         <cylinder radius="0.0095" length="${extension}" />
                     </geometry>
-                    <material name="dark_grey" />
+                    <material name="clearpath_dark_grey" />
                     <origin xyz="${extension / 2} 0 0" rpy="0 ${M_PI/2} 0" />
                 </visual>
@@ -37,5 +37,5 @@
                         <cylinder radius="0.0095" length="${extension}" />
                     </geometry>
-                    <material name="dark_grey" />
+                    <material name="clearpath_dark_grey" />
                     <origin xyz="${extension / 2} 0 0" rpy="0 ${M_PI/2} 0" />
                 </visual>

File: clearpath_platform_description/urdf/a200/attachments/top_plate.urdf.xacro (robot description, xacro)
@@ -93,5 +93,5 @@
         <link name="top_plate_link">
           <visual>
-            <material name="dark_grey" />
+            <material name="clearpath_dark_grey" />
             <geometry>
               <mesh filename="package://clearpath_platform_description/meshes/a200/attachments/pacs_top_plate.stl" />
@@ -99,5 +99,5 @@
           </visual>
           <collision>
-            <material name="dark_grey" />
+            <material name="clearpath_dark_grey" />
             <origin xyz="0 0 0.00317500531673" rpy="0 0 0"/>
             <geometry>

File: clearpath_platform_description/urdf/j100/attachments/front_fender.urdf.xacro (robot description, xacro)
@@ -13,5 +13,5 @@
           </xacro:if>
         </geometry>
-        <material name="yellow" />
+        <material name="clearpath_yellow" />
       </visual>
     </link>

File: clearpath_platform_description/urdf/j100/attachments/rear_fender.urdf.xacro (robot description, xacro)
@@ -13,5 +13,5 @@
           </xacro:if>
         </geometry>
-        <material name="yellow" />
+        <material name="clearpath_yellow" />
       </visual>
     </link>

File: clearpath_platform_description/urdf/j100/attachments/top_plate.urdf.xacro (robot description, xacro)
@@ -9,5 +9,5 @@
               <mesh filename="package://clearpath_platform_description/meshes/j100/attachments/ark_enclosure.stl"/>
             </geometry>
-            <material name="dark_grey" />
+            <material name="clearpath_dark_grey" />
           </visual>
         </link>

File: clearpath_platform_description/urdf/j100/j100.urdf.xacro (robot description, xacro)
@@ -72,5 +72,5 @@
           <mesh filename="package://clearpath_platform_description/meshes/j100/j100_base.stl"/>
         </geometry>
-        <material name="dark_grey" />
+        <material name="clearpath_dark_grey" />
       </visual>
       <collision>
@@ -118,5 +118,5 @@
         </geometry>
         <origin xyz="0 0 0.008" />
-        <material name="black" />
+        <material name="clearpath_black" />
       </visual>
     </link>

File: clearpath_platform_description/urdf/w200/attachments/w200_arm_mount.urdf.xacro (robot description, xacro)
@@ -8,5 +8,5 @@
           <mesh filename="package://clearpath_platform_description/meshes/w200/arm-mount-plate.stl" />
         </geometry>
-        <material name="light_grey"/>
+        <material name="clearpath_light_grey"/>
       </visual>
       <collision>

File: clearpath_platform_description/urdf/w200/attachments/w200_bulkhead.urdf.xacro (robot description, xacro)
@@ -8,5 +8,5 @@
           <mesh filename="package://clearpath_platform_description/meshes/w200/bulkhead.stl" />
         </geometry>
-        <material name="black"><color rgba="0.15 0.15 0.15 1.0" /></material>
+        <material name="clearpath_black"><color rgba="0.15 0.15 0.15 1.0" /></material>
       </visual>
       <collision>

File: clearpath_platform_description/urdf/w200/attachments/w200_generator.urdf.xacro (robot description, xacro)
@@ -8,5 +8,5 @@
           <mesh filename="package://clearpath_platform_description/meshes/w200/generator.stl" />
         </geometry>
-        <material name="black"><color rgba="0.15 0.15 0.15 1.0" /></material>
+        <material name="clearpath_black"><color rgba="0.15 0.15 0.15 1.0" /></material>
       </visual>
       <collision>

File: clearpath_platform_description/urdf/w200/w200.urdf.xacro (robot description, xacro)
@@ -67,5 +67,5 @@
           <mesh filename="package://clearpath_platform_description/meshes/w200/wheel.stl" />
         </geometry>
-        <material name="dark_grey" />
+        <material name="clearpath_dark_grey" />
       </visual>
       <collision>
@@ -109,5 +109,5 @@
           <mesh filename="package://clearpath_platform_description/meshes/w200/tracks.dae" />
         </geometry>
-        <material name="dark_grey" />
+        <material name="clearpath_dark_grey" />
       </visual>
       <collision>
@@ -191,5 +191,5 @@
           <mesh filename="package://clearpath_platform_description/meshes/w200/rocker.stl" />
         </geometry>
-        <material name="black"><color rgba="0.15 0.15 0.15 1.0" /></material>
+        <material name="clearpath_black"><color rgba="0.15 0.15 0.15 1.0" /></material>
       </visual>
       <visual>
@@ -198,5 +198,5 @@
           <mesh filename="package://clearpath_platform_description/meshes/w200/fenders.stl" />
         </geometry>
-        <material name="${warthog_color}">
+        <material name="clearpath_${warthog_color}">
           <color rgba="${warthog_color_rgba}" />
         </material>
@@ -223,5 +223,5 @@
           <mesh filename="package://clearpath_platform_description/meshes/w200/light.stl" />
         </geometry>
-        <material name="white"><color rgba="0.9 0.9 0.9 1.0" /></material>
+        <material name="clearpath_white"><color rgba="0.9 0.9 0.9 1.0" /></material>
       </visual>
     </link>
@@ -247,5 +247,5 @@
           <mesh filename="package://clearpath_platform_description/meshes/w200/light.stl" />
         </geometry>
-        <material name="red"><color rgba="0.9 0.0 0.0 1.0" /></material>
+        <material name="clearpath_red"><color rgba="0.9 0.0 0.0 1.0" /></material>
       </visual>
     </link>
@@ -298,5 +298,5 @@
           <mesh filename="package://clearpath_platform_description/meshes/w200/chassis.stl" />
         </geometry>
-        <material name="black"><color rgba="0.15 0.15 0.15 1.0" /></material>
+        <material name="clearpath_black"><color rgba="0.15 0.15 0.15 1.0" /></material>
       </visual>
       <visual>
@@ -305,5 +305,5 @@
           <mesh filename="package://clearpath_platform_description/meshes/w200/e-stop.stl" />
         </geometry>
-        <material name="red"><color rgba="0.9 0.0 0.0 1.0" /></material>
+        <material name="clearpath_red"><color rgba="0.9 0.0 0.0 1.0" /></material>
       </visual>
       <collision>
@@ -327,5 +327,5 @@
           <mesh filename="package://clearpath_platform_description/meshes/w200/diff-link.stl" />
         </geometry>
-        <material name="light_grey" />
+        <material name="clearpath_light_grey" />
       </visual>
       <visual>
@@ -334,5 +334,5 @@
           <mesh filename="package://clearpath_platform_description/meshes/w200/susp-link.stl" />
         </geometry>
-        <material name="light_grey" />
+        <material name="clearpath_light_grey" />
       </visual>
       <visual>
@@ -341,5 +341,5 @@
           <mesh filename="package://clearpath_platform_description/meshes/w200/susp-link.stl" />
         </geometry>
-        <material name="light_grey" />
+        <material name="clearpath_light_grey" />
       </visual>
     </link>
