Commit message: Add mount links for the front & rear 2D lidars (front has a permanent mesh, since it's always assumed to be present)

File: clearpath_platform_description/urdf/a200/attachments/observer_backpack.urdf.xacro (robot description, xacro)
@@ -82,9 +82,21 @@
       <origin xyz="0 0 0.355" rpy="0 0 0" />
     </joint>
-    <link name="${name}_lidar_mount" />
-    <joint name="${name}_lidar_mount_joint" type="fixed">
+    <link name="${name}_center_lidar_mount" />
+    <joint name="${name}_center_lidar_mount_joint" type="fixed">
       <parent link="${name}_shell_link" />
-      <child link="${name}_lidar_mount" />
+      <child link="${name}_center_lidar_mount" />
       <origin xyz="0 0 0.257" rpy="0 0 0" />
+    </joint>
+    <link name="${name}_front_lidar_mount" />
+    <joint name="${name}_front_lidar_mount_joint" type="fixed">
+      <parent link="${name}_shell_link" />
+      <child link="${name}_front_lidar_mount" />
+      <origin xyz="0.45 0 0.06" rpy="3.14159 0 0" />
+    </joint>
+    <link name="${name}_rear_lidar_mount" />
+    <joint name="${name}_rear_lidar_mount_joint" type="fixed">
+      <parent link="${name}_shell_link" />
+      <child link="${name}_rear_lidar_mount" />
+      <origin xyz="-0.45 0 0.06" rpy="3.14159 0 3.14159" />
     </joint>
     <link name="${name}_left_antenna_mount" />

Commit message: Add additional links for the realsense cameras

File: clearpath_platform_description/urdf/a200/attachments/observer_backpack.urdf.xacro (robot description, xacro)
@@ -100,4 +100,16 @@
       <origin xyz="-0.45 0 0.06" rpy="3.14159 0 3.14159" />
     </joint>
+    <link name="${name}_front_realsense_mount" />
+    <joint name="${name}_front_realsense_mount_joint" type="fixed">
+      <parent link="${name}_shell_link" />
+      <child link="${name}_front_realsense_mount" />
+      <origin xyz="0.382 0 0.088" rpy="0 0 0" />
+    </joint>
+    <link name="${name}_rear_realsense_mount" />
+    <joint name="${name}_rear_realsense_mount_joint" type="fixed">
+      <parent link="${name}_shell_link" />
+      <child link="${name}_rear_realsense_mount" />
+      <origin xyz="-0.382 0 0.088" rpy="0 0 3.14159" />
+    </joint>
     <link name="${name}_left_antenna_mount" />
     <joint name="${name}_left_antenna_mount_joint" type="fixed">

Commit message: Add the IMU mount to the URDF

File: clearpath_platform_description/urdf/a200/attachments/observer_backpack.urdf.xacro (robot description, xacro)
@@ -124,4 +124,10 @@
       <origin xyz="-0.25 -0.350 0.695" rpy="0 0 0" />
     </joint>
+    <link name="${name}_imu_mount" />
+    <joint name="${name}_imu_mount_joint" type="fixed">
+      <parent link="${name}_shell_link" />
+      <child link="${name}_imu_mount" />
+      <origin xyz="0.00498 0.0 -0.097312" rpy="0.0 0.0 1.5708" />
+    </joint>
   </xacro:macro>
 </robot>
