Commit message: Added w200 tracks

File: clearpath_platform_description/urdf/w200/diff_unit.urdf.xacro (robot description, xacro)
@@ -12,5 +12,5 @@
     <xacro:if value="${side == 'right'}">
         <xacro:property name="flip" value="-1"/>
-    <xacro:if>
+    </xacro:if>
     <link name="${side}_diff_unit_link">
       <inertial>
@@ -25,7 +25,5 @@
           <mesh filename="package://clearpath_platform_description/meshes/w200/fenders.stl" />
         </geometry>
-        <material name="clearpath_diff_unit">
-          <color rgba="${warthog_color}" />
-        </material>
+        <material name="${warthog_color}"/>
       </visual>
       <collision>
@@ -40,5 +38,5 @@
           <mesh filename="package://clearpath_platform_description/meshes/w200/rocker.stl" />
         </geometry>
-        <material name="clearpath_black"><color rgba="0.15 0.15 0.15 1.0" /></material>
+        <material name="clearpath_black"/>
       </visual>
     </link>
@@ -57,5 +55,5 @@
           <mesh filename="package://clearpath_platform_description/meshes/w200/light.stl" />
         </geometry>
-        <material name="clearpath_white"><color rgba="0.9 0.9 0.9 1.0" /></material>
+        <material name="clearpath_white"/>
       </visual>
     </link>
@@ -81,5 +79,5 @@
           <mesh filename="package://clearpath_platform_description/meshes/w200/light.stl" />
         </geometry>
-        <material name="clearpath_red"><color rgba="0.9 0.0 0.0 1.0" /></material>
+        <material name="clearpath_red"/>
       </visual>
     </link>
@@ -103,6 +101,4 @@
       <visual>
         <material>
-          <ambient>${warthog_color}</ambient>
-          <diffuse>${warthog_color}</diffuse>
           <specular>0.1 0.1 0.1 1</specular>
           <emissive>0 0 0 0</emissive>

File: clearpath_platform_description/urdf/w200/track.urdf.xacro (robot description, xacro)
@@ -2,4 +2,5 @@
 <robot xmlns:xacro="http://ros.org/wiki/xacro" name="w200_track">
   <xacro:macro name="w200_track" params="prefix side *joint_pose">
+    <xacro:property name="rotate" value="${(prefix=='rear')*math.pi}"/>
     <link name="${prefix}_${side}_track_link">
       <visual>
@@ -25,4 +26,16 @@
     <!-- This adds wheels that rotate instead of tracks. -->
     <link name="${prefix}_${side}_wheel_link">
+      <inertial>
+        <origin xyz="0 0 0" rpy="0 0 0" />
+        <mass value="${wheel_mass}" />
+        <xacro:wheel_inertia m="${wheel_mass}" r="${wheel_radius}" h="${wheel_width}" />
+      </inertial>
+      <visual>
+        <material name="clearpath_red"/>
+        <origin xyz="0 0 0" rpy="${PI/2} 0 0"/>
+        <geometry>
+          <cylinder radius="${wheel_radius*wheel_to_track_ratio}" length="${wheel_width}"/>
+        </geometry>
+      </visual>
       <collision>
         <origin xyz="0 0 0" rpy="${PI/2} 0 0"/>
@@ -33,19 +46,16 @@
     </link>
     <joint name="${prefix}_${side}_wheel_joint" type="continuous">
-      <parent link="${side}_diff_unit_link"/>
+      <parent link="${prefix}_${side}_track_link"/>
       <child link="${prefix}_${side}_wheel_link"/>
-      <xacro:insert_block name="joint_pose" />
+      <origin xyz="0.12 0. -0.18" rpy="0 0 ${rotate}"/>
       <axis xyz="0 1 0"/>
     </joint>
-    <transmission name="${prefix}_${side}_wheel_trans">
-      <type>transmission_interface/SimpleTransmission</type>
-      <joint name="${prefix}_${side}_wheel_joint">
-        <hardwareInterface>hardware_interface/VelocityJointInterface</hardwareInterface>
-      </joint>
-      <actuator name="${prefix}_${side}_actuator">
-        <hardwareInterface>hardware_interface/VelocityJointInterface</hardwareInterface>
-        <mechanicalReduction>1</mechanicalReduction>
-      </actuator>
-    </transmission>
+    <gazebo reference="${prefix}_${side}_wheel_link">
+      <selfCollide>false</selfCollide>
+      <mu1>0.5</mu1>
+      <mu2>0.5</mu2>
+      <fdir1 value="1 0 0" />
+      <material>Gazebo/DarkGrey</material>
+    </gazebo>
   </xacro:macro>
 </robot>

File: clearpath_platform_description/urdf/w200/w200.urdf.xacro (robot description, xacro)
@@ -4,5 +4,5 @@
   <xacro:arg name="is_sim" default="false" />
   <xacro:arg name="color" default="yellow"/>
-  <xacro:arg name="wheel" default="wheel" /> <!-- tracks -->
+  <xacro:arg name="wheel" default="track" /> <!-- tracks -->
   <xacro:arg name="gazebo_controllers" default="$(find clearpath_control)/config/w200/control.yaml"/>
   <!-- Include URDF/XACRO Files -->
@@ -19,4 +19,5 @@
   <xacro:property name="axle_y_offset" value="0.0" />
   <xacro:property name="axle_z_offset" value="-0.012977" />
+  <xacro:property name="track_z_offset" value="-0.2" />
   <xacro:property name="diff_unit_length" value="1.34" />
   <xacro:property name="diff_unit_width"  value="0.28" />
@@ -33,20 +34,9 @@
   <!-- Colors: yellow, orange, olive, sand -->
   <xacro:property name="color"          value="$(arg color)"/>
-  <xacro:property name="warthog_yellow" value="0.95 0.816 0.082 1.0"/>
-  <xacro:property name="warthog_orange" value="1.0 0.48 0.0 1.0"/>
-  <xacro:property name="warthog_olive"  value="0.333 0.419 0.184 1.0"/>
-  <xacro:property name="warthog_sand"   value="0.86 0.75 0.54 1.0"/>
-  <xacro:if value="${color == 'yellow'}">
-    <xacro:property name="warthog_color" value="warthog_yellow" />
-  </xacro:if>
-  <xacro:if value="${color == 'orange'}">
-    <xacro:property name="warthog_color" value="warthog_orange" />
-  </xacro:if>
-  <xacro:if value="${color == 'olive'}">
-    <xacro:property name="warthog_color" value="warthog_olive" />
-  </xacro:if>
-  <xacro:if value="${color == 'sand'}">
-    <xacro:property name="warthog_color" value="warthog_sand" />
-  </xacro:if>
+  <xacro:property name="warthog_color"  value="${'warthog_'+color}"/>
+  <material name="warthog_yellow"><color rgba="0.95 0.816 0.082 1.0"/></material>
+  <material name="warthog_orange"><color rgba="1.0 0.48 0.0 1.0"/></material>
+  <material name="warthog_olive"><color rgba="0.333 0.419 0.184 1.0"/></material>
+  <material name="warthog_sand"><color rgba="0.86 0.75 0.54 1.0"/></material>
   <xacro:macro name="w200">
     <!-- Chassis -->
@@ -132,17 +122,17 @@
     </xacro:if>
     <!-- Tracks -->
-    <xacro:if value="${wheel == 'tracks'}">
-      <xacro:track prefix="front" side="left">
+    <xacro:if value="${wheel == 'track'}">
+      <xacro:w200_track prefix="front" side="left">
         <origin xyz="${axle_x_offset*1} ${axle_y_offset*1} ${axle_z_offset}" rpy="0 0 0" />
-      </xacro:track>
-      <xacro:track prefix="front" side="right">
+      </xacro:w200_track>
+      <xacro:w200_track prefix="front" side="right">
         <origin xyz="${axle_x_offset*1} ${axle_y_offset*-1} ${axle_z_offset}" rpy="0 0 0" />
-      </xacro:track>
-      <xacro:track prefix="rear" side="left">
+      </xacro:w200_track>
+      <xacro:w200_track prefix="rear" side="left">
         <origin xyz="${axle_x_offset*-1} ${axle_y_offset*1} ${axle_z_offset}" rpy="0 0 ${PI}" />
-      </xacro:track>
-      <xacro:track prefix="rear" side="right">
+      </xacro:w200_track>
+      <xacro:w200_track prefix="rear" side="right">
         <origin xyz="${axle_x_offset*-1} ${axle_y_offset*-1} ${axle_z_offset}" rpy="0 0 ${PI}" />
-      </xacro:track>
+      </xacro:w200_track>
     </xacro:if>
     <!-- Virtual Mounting Point -->
@@ -188,5 +178,5 @@
           <param name="wheel_diameter">0.6</param>
           <param name="max_accel">50.0</param>
-          <param name="max_speed">5.0</param>
+          <param name="max_speed">25.0</param>
           <param name="polling_timeout">0.1</param>
         </xacro:unless>
@@ -194,6 +184,6 @@
       <joint name="front_left_wheel_joint">
         <command_interface name="velocity">
-          <param name="min">-5</param>
-          <param name="max">5</param>
+          <param name="min">-25</param>
+          <param name="max">25</param>
         </command_interface>
         <state_interface name="position"/>
@@ -202,6 +192,6 @@
       <joint name="rear_left_wheel_joint">
         <command_interface name="velocity">
-          <param name="min">-5</param>
-          <param name="max">5</param>
+          <param name="min">-25</param>
+          <param name="max">25</param>
         </command_interface>
         <state_interface name="position"/>
@@ -210,6 +200,6 @@
       <joint name="front_right_wheel_joint">
         <command_interface name="velocity">
-          <param name="min">-5</param>
-          <param name="max">5</param>
+          <param name="min">-25</param>
+          <param name="max">25</param>
         </command_interface>
         <state_interface name="position"/>
@@ -218,6 +208,6 @@
       <joint name="rear_right_wheel_joint">
         <command_interface name="velocity">
-          <param name="min">-5</param>
-          <param name="max">5</param>
+          <param name="min">-25</param>
+          <param name="max">25</param>
         </command_interface>
         <state_interface name="position"/>

File: clearpath_platform_description/urdf/w200/wheel.urdf.xacro (robot description, xacro)
@@ -37,6 +37,4 @@
       <mu1>0.5</mu1>
       <mu2>0.5</mu2>
-      <!-- <kp value="10000000.0" /> -->
-      <!-- <kd value="1.0" /> -->
       <fdir1 value="1 0 0" />
       <material>Gazebo/DarkGrey</material>
