Commit message: First pass

File: clearpath_platform_description/urdf/w200/w200.urdf.xacro (robot description, xacro)
@@ -1,12 +1,18 @@
 <?xml version='1.0'?>
-<robot name="warthog" xmlns:xacro="http://www.ros.org/wiki/xacro">
-  <xacro:arg name="gazebo_controllers" default="$(find clearpath_control)/config/w200/control.yaml" />
+<robot xmlns:xacro="http://www.ros.org/wiki/xacro">
   <xacro:arg name="namespace" default="" />
   <xacro:arg name="is_sim" default="false" />
+  <xacro:arg name="color" default="yellow"/>
+  <xacro:arg name="wheel" default="wheel" /> <!-- tracks -->
   <xacro:arg name="gazebo_controllers" default="$(find clearpath_control)/config/w200/control.yaml"/>
+  <!-- Include URDF/XACRO Files -->
+  <xacro:include filename="$(find clearpath_platform_description)/urdf/w200/diff_unit.urdf.xacro"/>
+  <xacro:include filename="$(find clearpath_platform_description)/urdf/w200/track.urdf.xacro"/>
+  <xacro:include filename="$(find clearpath_platform_description)/urdf/w200/wheel.urdf.xacro"/>
   <xacro:property name="PI" value="3.1415926535897931"/>
+  <xacro:property name="wheel"        value="$(arg wheel)" />
   <xacro:property name="wheel_radius" value="0.3" />
-  <xacro:property name="wheel_width" value="0.25" />
-  <xacro:property name="wheel_mass" value="15" />
+  <xacro:property name="wheel_width"  value="0.25" />
+  <xacro:property name="wheel_mass"   value="15" />
   <xacro:property name="wheel_to_track_ratio" value="0.5962" />
   <xacro:property name="axle_x_offset" value="0.457367" />
@@ -14,271 +20,35 @@
   <xacro:property name="axle_z_offset" value="-0.012977" />
   <xacro:property name="diff_unit_length" value="1.34" />
-  <xacro:property name="diff_unit_width" value="0.28" />
+  <xacro:property name="diff_unit_width"  value="0.28" />
   <xacro:property name="diff_unit_height" value="0.63"/>
-  <xacro:property name="diff_unit_mass" value="50" />
+  <xacro:property name="diff_unit_mass"   value="50" />
   <xacro:property name="diff_unit_offset_x" value="0.00" />
   <xacro:property name="diff_unit_offset_y" value="0.56821" />
   <xacro:property name="diff_unit_offset_z" value="0.0" />
   <xacro:property name="chassis_length" value="1.35" />
-  <xacro:property name="chassis_width" value="0.70" />
+  <xacro:property name="chassis_width"  value="0.70" />
   <xacro:property name="chassis_height" value="0.30" />
-  <xacro:property name="chassis_mass" value="100" />
+  <xacro:property name="chassis_mass"   value="100" />
   <xacro:property name="dummy_inertia" value="1e-09"/>
-  <!--
-    Optional paint colors.
-    Available colors:
-      - yellow (default)
-      - orange
-      - olive
-      - sand
-  -->
-  <xacro:property name="warthog_color" value="$(optenv WARTHOG_COLOR yellow)" />
-  <xacro:if value="${warthog_color == 'yellow'}">
-    <xacro:property name="warthog_color_rgba" value="0.95 0.816 0.082 1.0" />
-  </xacro:if>
-  <xacro:if value="${warthog_color == 'orange'}">
-    <xacro:property name="warthog_color_rgba" value="1.0 0.48 0.0 1.0" />
-  </xacro:if>
-  <xacro:if value="${warthog_color == 'olive'}">
-    <xacro:property name="warthog_color_rgba" value="0.333 0.419 0.184 1.0" />
-  </xacro:if>
-  <xacro:if value="${warthog_color == 'sand'}">
-    <xacro:property name="warthog_color_rgba" value="0.86 0.75 0.54 1.0" />
-  </xacro:if>
-  <xacro:macro name="wheel_inertia" params="m r h">
-    <inertia ixx="${m*(3*r*r+h*h)/12}" ixy="0" ixz="0"
-             iyy="${m*r*r/2}" iyz="0"
-             izz="${m*(3*r*r+h*h)/12}" />
-  </xacro:macro>
-  <xacro:macro name="box_inertia" params="m x y z">
-    <inertia ixx="${m*(y*y+z*z)/12}" ixy="0" ixz="0"
-             iyy="${m*(x*x+z*z)/12}" iyz="0"
-             izz="${m*(x*x+z*z)/12}" />
-  </xacro:macro>
-  <xacro:macro name="wheel" params="prefix side *joint_pose">
-    <link name="${prefix}_${side}_wheel_link">
-      <inertial>
-        <origin xyz="0 0 0" rpy="0 0 0" />
-        <mass value="${wheel_mass}" />
-        <xacro:wheel_inertia m="${wheel_mass}" r="${wheel_radius}" h="${wheel_width}" />
-      </inertial>
-      <visual>
-        <origin xyz="0 0 0" rpy="0 0 ${PI/2}"/>
-        <geometry>
-          <mesh filename="package://clearpath_platform_description/meshes/w200/wheel.stl" />
-        </geometry>
-        <material name="clearpath_dark_grey" />
-      </visual>
-      <collision>
-        <origin xyz="0 0 0" rpy="${PI/2} 0 0"/>
-        <geometry>
-          <cylinder radius="${wheel_radius}" length="${wheel_width}"/>
-        </geometry>
-      </collision>
-    </link>
-    <joint name="${prefix}_${side}_wheel_joint" type="continuous">
-      <parent link="${side}_diff_unit_link"/>
-      <child link="${prefix}_${side}_wheel_link"/>
-      <xacro:insert_block name="joint_pose" />
-      <axis xyz="0 1 0"/>
-    </joint>
-    <gazebo reference="${prefix}_${side}_wheel_link">
-      <selfCollide>false</selfCollide>
-      <mu1>0.5</mu1>
-      <mu2>0.5</mu2>
-      <!-- <kp value="10000000.0" /> -->
-      <!-- <kd value="1.0" /> -->
-      <fdir1 value="1 0 0" />
-      <material>Gazebo/DarkGrey</material>
-    </gazebo>
-    <transmission name="${prefix}_${side}_wheel_trans">
-      <type>transmission_interface/SimpleTransmission</type>
-      <joint name="${prefix}_${side}_wheel_joint">
-        <hardwareInterface>hardware_interface/VelocityJointInterface</hardwareInterface>
-      </joint>
-      <actuator name="${prefix}_${side}_actuator">
-        <hardwareInterface>hardware_interface/VelocityJointInterface</hardwareInterface>
-        <mechanicalReduction>1</mechanicalReduction>
-      </actuator>
-    </transmission>
-  </xacro:macro>
-  <xacro:macro name="track" params="prefix side *joint_pose">
-    <link name="${prefix}_${side}_track_link">
-      <visual>
-        <origin xyz="0 0 0" rpy="0 0 0"/>
-        <geometry>
-          <mesh filename="package://clearpath_platform_description/meshes/w200/tracks.dae" />
-        </geometry>
-        <material name="clearpath_dark_grey" />
-      </visual>
-      <collision>
-        <origin xyz="0 0 0" rpy="0 0 0"/>
-        <geometry>
-          <mesh filename="package://clearpath_platform_description/meshes/w200/tracks_collision.stl" />
-        </geometry>
-      </collision>
-    </link>
-    <joint name="${prefix}_${side}_track_joint" type="fixed">
-      <parent link="${side}_diff_unit_link"/>
-      <child link="${prefix}_${side}_track_link"/>
-      <xacro:insert_block name="joint_pose" />
-      <axis xyz="0 1 0"/>
-    </joint>
-    <!-- This adds wheels that rotate instead of tracks. -->
-    <link name="${prefix}_${side}_wheel_link">
-      <collision>
-        <origin xyz="0 0 0" rpy="${PI/2} 0 0"/>
-        <geometry>
-          <cylinder radius="${wheel_radius*wheel_to_track_ratio}" length="${wheel_width}"/>
-        </geometry>
-      </collision>
-    </link>
-    <joint name="${prefix}_${side}_wheel_joint" type="continuous">
-      <parent link="${side}_diff_unit_link"/>
-      <child link="${prefix}_${side}_wheel_link"/>
-      <xacro:insert_block name="joint_pose" />
-      <axis xyz="0 1 0"/>
-    </joint>
-    <transmission name="${prefix}_${side}_wheel_trans">
-      <type>transmission_interface/SimpleTransmission</type>
-      <joint name="${prefix}_${side}_wheel_joint">
-        <hardwareInterface>hardware_interface/VelocityJointInterface</hardwareInterface>
-      </joint>
-      <actuator name="${prefix}_${side}_actuator">
-        <hardwareInterface>hardware_interface/VelocityJointInterface</hardwareInterface>
-        <mechanicalReduction>1</mechanicalReduction>
-      </actuator>
-    </transmission>
-  </xacro:macro>
-  <xacro:unless value="$(optenv WARTHOG_TRACKS 0)">
-    <xacro:wheel prefix="front" side="left">
-      <origin xyz="${axle_x_offset*1} ${axle_y_offset*1} ${axle_z_offset}" rpy="0 0 0" />
-    </xacro:wheel>
-    <xacro:wheel prefix="front" side="right">
-      <origin xyz="${axle_x_offset*1} ${axle_y_offset*-1} ${axle_z_offset}" rpy="0 0 0" />
-    </xacro:wheel>
-    <xacro:wheel prefix="rear" side="left">
-      <origin xyz="${axle_x_offset*-1} ${axle_y_offset*1} ${axle_z_offset}" rpy="0 0 0" />
-    </xacro:wheel>
-    <xacro:wheel prefix="rear" side="right">
-      <origin xyz="${axle_x_offset*-1} ${axle_y_offset*-1} ${axle_z_offset}" rpy="0 0 0" />
-    </xacro:wheel>
-  </xacro:unless>
-  <xacro:if value="$(optenv WARTHOG_TRACKS 0)">
-    <xacro:track prefix="front" side="left">
-      <origin xyz="${axle_x_offset*1} ${axle_y_offset*1} ${axle_z_offset}" rpy="0 0 0" />
-    </xacro:track>
-    <xacro:track prefix="front" side="right">
-      <origin xyz="${axle_x_offset*1} ${axle_y_offset*-1} ${axle_z_offset}" rpy="0 0 0" />
-    </xacro:track>
-    <xacro:track prefix="rear" side="left">
-      <origin xyz="${axle_x_offset*-1} ${axle_y_offset*1} ${axle_z_offset}" rpy="0 0 ${PI}" />
-    </xacro:track>
-    <xacro:track prefix="rear" side="right">
-      <origin xyz="${axle_x_offset*-1} ${axle_y_offset*-1} ${axle_z_offset}" rpy="0 0 ${PI}" />
-    </xacro:track>
-  </xacro:if>
-  <xacro:macro name="diff_unit" params="prefix side left">
-    <link name="${prefix}_diff_unit_link">
-      <inertial>
-        <origin xyz="0 ${side*-1*0.05} 0.197" rpy="0 0 0"/>
-        <mass value="${diff_unit_mass}"/>
-        <xacro:box_inertia m="${diff_unit_mass}" x="${diff_unit_length}"
-                           y="${diff_unit_width}" z="${diff_unit_height}" />
-      </inertial>
-      <visual>
-        <origin xyz="0 0 0" rpy="0 0 ${side*PI/2}"/>
-        <geometry>
-          <mesh filename="package://clearpath_platform_description/meshes/w200/fenders.stl" />
-        </geometry>
-        <material name="clearpath_${warthog_color}">
-          <color rgba="${warthog_color_rgba}" />
-        </material>
-      </visual>
-      <collision>
-        <origin xyz="0 0 0" rpy="0 0 ${side*PI/2}"/>
-        <geometry>
-          <mesh filename="package://clearpath_platform_description/meshes/w200/fenders.stl" />
-        </geometry>
-      </collision>
-      <visual>
-        <origin xyz="0 0 0" rpy="0 0 ${side*PI/2}"/>
-        <geometry>
-          <mesh filename="package://clearpath_platform_description/meshes/w200/rocker.stl" />
-        </geometry>
-        <material name="clearpath_black"><color rgba="0.15 0.15 0.15 1.0" /></material>
-      </visual>
-    </link>
-    <joint name="${prefix}_diff_unit_joint" type="fixed">
-      <limit upper="0.4" lower="-0.4" effort="100" velocity="1"/>
-      <parent link="chassis_link"/>
-      <child link="${prefix}_diff_unit_link"/>
-      <origin xyz="${diff_unit_offset_x} ${diff_unit_offset_y*side} ${diff_unit_offset_z}" rpy="0 0 0" />
-      <axis xyz="0 1 0"/>
-      <dynamics damping="100" friction="0.5"/>
-    </joint>
-    <link name="${prefix}_diff_unit_headlight_link">
-      <visual>
-        <origin xyz="0 ${side*-0.0244} 0" rpy="0 0 0"/>
-        <geometry>
-          <mesh filename="package://clearpath_platform_description/meshes/w200/light.stl" />
-        </geometry>
-        <material name="clearpath_white"><color rgba="0.9 0.9 0.9 1.0" /></material>
-      </visual>
-    </link>
-    <joint name="${prefix}_diff_unit_headlight_joint" type="fixed">
-      <parent link="${prefix}_diff_unit_link" />
-      <child link="${prefix}_diff_unit_headlight_link" />
-      <origin xyz="0 0 0" rpy="0 0 0"/>
-    </joint>
-    <gazebo reference="${prefix}_diff_unit_headlight_link">
-      <visual>
-        <material>
-          <ambient>0.9 0.9 0.9 1</ambient>
-          <diffuse>0.9 0.9 0.9 1</diffuse>
-          <specular>0.9 0.9 0.9 1</specular>
-          <emissive>0.9 0.9 0.9 1</emissive>
-        </material>
-      </visual>
-    </gazebo>
-    <link name="${prefix}_diff_unit_taillight_link">
-      <visual>
-        <origin xyz="0 ${side*-0.0244} 0" rpy="0 0 ${side*PI}"/>
-        <geometry>
-          <mesh filename="package://clearpath_platform_description/meshes/w200/light.stl" />
-        </geometry>
-        <material name="clearpath_red"><color rgba="0.9 0.0 0.0 1.0" /></material>
-      </visual>
-    </link>
-    <joint name="${prefix}_diff_unit_taillight_joint" type="fixed">
-      <parent link="${prefix}_diff_unit_link" />
-      <child link="${prefix}_diff_unit_taillight_link" />
-      <origin xyz="0 0 0" rpy="0 0 0"/>
-    </joint>
-    <gazebo reference="${prefix}_diff_unit_taillight_link">
-      <visual>
-        <material>
-          <ambient>0.9 0 0 1</ambient>
-          <diffuse>0.9 0 0 1</diffuse>
-          <specular>0.9 0 0 1</specular>
-          <emissive>0.9 0 0 1</emissive>
-        </material>
-      </visual>
-    </gazebo>
-    <gazebo reference="${prefix}_diff_unit_link">
-      <selfCollide>false</selfCollide>
-      <visual>
-        <material>
-          <ambient>${warthog_color_rgba}</ambient>
-          <diffuse>${warthog_color_rgba}</diffuse>
-          <specular>0.1 0.1 0.1 1</specular>
-          <emissive>0 0 0 0</emissive>
-        </material>
-      </visual>
-    </gazebo>
-  </xacro:macro>
+  <!-- Colors: yellow, orange, olive, sand -->
+  <xacro:property name="color"          value="$(arg color)"/>
+  <xacro:property name="warthog_yellow" value="0.95 0.816 0.082 1.0"/>
+  <xacro:property name="warthog_orange" value="1.0 0.48 0.0 1.0"/>
+  <xacro:property name="warthog_olive"  value="0.333 0.419 0.184 1.0"/>
+  <xacro:property name="warthog_sand"   value="0.86 0.75 0.54 1.0"/>
+  <xacro:if value="${color == 'yellow'}">
+    <xacro:property name="warthog_color" value="warthog_yellow" />
+  </xacro:if>
+  <xacro:if value="${color == 'orange'}">
+    <xacro:property name="warthog_color" value="warthog_orange" />
+  </xacro:if>
+  <xacro:if value="${color == 'olive'}">
+    <xacro:property name="warthog_color" value="warthog_olive" />
+  </xacro:if>
+  <xacro:if value="${color == 'sand'}">
+    <xacro:property name="warthog_color" value="warthog_sand" />
+  </xacro:if>
   <xacro:macro name="w200">
-    <xacro:diff_unit prefix="left" side="1" left="true"/>
-    <xacro:diff_unit prefix="right" side="-1" left="false"/>
+    <!-- Chassis -->
     <link name="base_link"></link>
     <joint name="base_link_joint" type="fixed">
@@ -315,4 +85,66 @@
       </collision>
     </link>
+    <!-- Diff. Unit -->
+    <xacro:w200_diff_unit side="left" />
+    <xacro:w200_diff_unit side="right" />
+    <link name="diff_link">
+      <visual>
+        <origin xyz="0 0 0" rpy="0 0 0"/>
+        <geometry>
+          <mesh filename="package://clearpath_platform_description/meshes/w200/diff-link.stl" />
+        </geometry>
+        <material name="clearpath_light_grey" />
+      </visual>
+      <visual>
+        <origin xyz="0 0 0" rpy="0 0 0"/>
+        <geometry>
+          <mesh filename="package://clearpath_platform_description/meshes/w200/susp-link.stl" />
+        </geometry>
+        <material name="clearpath_light_grey" />
+      </visual>
+      <visual>
+        <origin xyz="0 0 0" rpy="0 0 0"/>
+        <geometry>
+          <mesh filename="package://clearpath_platform_description/meshes/w200/susp-link.stl" />
+        </geometry>
+        <material name="clearpath_light_grey" />
+      </visual>
+    </link>
+    <joint name="diff_link_joint" type="fixed">
+      <parent link="chassis_link"/>
+      <child link="diff_link"/>
+      <origin xyz="-0.5826 0 0.24979" rpy="0 0 0" />
+    </joint>
+    <!-- Wheels -->
+    <xacro:if value="${wheel == 'wheel'}">
+      <xacro:w200_wheel prefix="front" side="left">
+        <origin xyz="${axle_x_offset*1} ${axle_y_offset*1} ${axle_z_offset}" rpy="0 0 0" />
+      </xacro:w200_wheel>
+      <xacro:w200_wheel prefix="front" side="right">
+        <origin xyz="${axle_x_offset*1} ${axle_y_offset*-1} ${axle_z_offset}" rpy="0 0 0" />
+      </xacro:w200_wheel>
+      <xacro:w200_wheel prefix="rear" side="left">
+        <origin xyz="${axle_x_offset*-1} ${axle_y_offset*1} ${axle_z_offset}" rpy="0 0 0" />
+      </xacro:w200_wheel>
+      <xacro:w200_wheel prefix="rear" side="right">
+        <origin xyz="${axle_x_offset*-1} ${axle_y_offset*-1} ${axle_z_offset}" rpy="0 0 0" />
+      </xacro:w200_wheel>
+    </xacro:if>
+    <!-- Tracks -->
+    <xacro:if value="${wheel == 'tracks'}">
+      <xacro:track prefix="front" side="left">
+        <origin xyz="${axle_x_offset*1} ${axle_y_offset*1} ${axle_z_offset}" rpy="0 0 0" />
+      </xacro:track>
+      <xacro:track prefix="front" side="right">
+        <origin xyz="${axle_x_offset*1} ${axle_y_offset*-1} ${axle_z_offset}" rpy="0 0 0" />
+      </xacro:track>
+      <xacro:track prefix="rear" side="left">
+        <origin xyz="${axle_x_offset*-1} ${axle_y_offset*1} ${axle_z_offset}" rpy="0 0 ${PI}" />
+      </xacro:track>
+      <xacro:track prefix="rear" side="right">
+        <origin xyz="${axle_x_offset*-1} ${axle_y_offset*-1} ${axle_z_offset}" rpy="0 0 ${PI}" />
+      </xacro:track>
+    </xacro:if>
+    <!-- Virtual Mounting Point -->
     <link name="default_mount"></link>
     <joint name="default_mount_joint" type="fixed">
@@ -321,33 +153,5 @@
       <child link="default_mount" />
     </joint>
-    <!-- This link is purely to complete the visual look -->
-    <link name="diff_link">
-      <visual>
-        <origin xyz="0 0 0" rpy="0 0 0"/>
-        <geometry>
-          <mesh filename="package://clearpath_platform_description/meshes/w200/diff-link.stl" />
-        </geometry>
-        <material name="clearpath_light_grey" />
-      </visual>
-      <visual>
-        <origin xyz="0 0 0" rpy="0 0 0"/>
-        <geometry>
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
Commit message: Color and wheel are now parameters

File: clearpath_platform_description/urdf/w200/w200.urdf.xacro (robot description, xacro)
@@ -3,41 +3,38 @@
   <xacro:arg name="namespace" default="" />
   <xacro:arg name="is_sim" default="false" />
-  <xacro:arg name="color" default="yellow"/>
-  <xacro:arg name="wheel" default="default" /> <!-- tracks -->
   <xacro:arg name="gazebo_controllers" default="$(find clearpath_control)/config/w200/control.yaml"/>
   <!-- Include URDF/XACRO Files -->
+  <xacro:include filename="$(find clearpath_platform_description)/urdf/w200/wheels/track.urdf.xacro"/>
+  <xacro:include filename="$(find clearpath_platform_description)/urdf/w200/wheels/wheel.urdf.xacro"/>
+  <xacro:property name="PI" value="3.1415926535897931"/>
   <xacro:include filename="$(find clearpath_platform_description)/urdf/w200/diff_unit.urdf.xacro"/>
-  <xacro:include filename="$(find clearpath_platform_description)/urdf/w200/track.urdf.xacro"/>
-  <xacro:include filename="$(find clearpath_platform_description)/urdf/w200/wheel.urdf.xacro"/>
-  <xacro:property name="PI" value="3.1415926535897931"/>
-  <xacro:property name="wheel"        value="$(arg wheel)" />
-  <xacro:property name="wheel_radius" value="0.3" />
-  <xacro:property name="wheel_width"  value="0.25" />
-  <xacro:property name="wheel_mass"   value="15" />
-  <xacro:property name="wheel_to_track_ratio" value="0.5962" />
-  <xacro:property name="axle_x_offset" value="0.457367" />
-  <xacro:property name="axle_y_offset" value="0.0" />
-  <xacro:property name="axle_z_offset" value="-0.012977" />
-  <xacro:property name="track_z_offset" value="-0.2" />
-  <xacro:property name="diff_unit_length" value="1.34" />
-  <xacro:property name="diff_unit_width"  value="0.28" />
-  <xacro:property name="diff_unit_height" value="0.63"/>
-  <xacro:property name="diff_unit_mass"   value="50" />
-  <xacro:property name="diff_unit_offset_x" value="0.00" />
-  <xacro:property name="diff_unit_offset_y" value="0.56821" />
-  <xacro:property name="diff_unit_offset_z" value="0.0" />
-  <xacro:property name="chassis_length" value="1.35" />
-  <xacro:property name="chassis_width"  value="0.70" />
-  <xacro:property name="chassis_height" value="0.30" />
-  <xacro:property name="chassis_mass"   value="100" />
-  <xacro:property name="dummy_inertia" value="1e-09"/>
-  <!-- Colors: yellow, orange, olive, sand -->
-  <xacro:property name="color"          value="$(arg color)"/>
-  <xacro:property name="warthog_color"  value="${'warthog_'+color}"/>
-  <material name="warthog_yellow"><color rgba="0.95 0.816 0.082 1.0"/></material>
-  <material name="warthog_orange"><color rgba="1.0 0.48 0.0 1.0"/></material>
-  <material name="warthog_olive"><color rgba="0.333 0.419 0.184 1.0"/></material>
-  <material name="warthog_sand"><color rgba="0.86 0.75 0.54 1.0"/></material>
-  <xacro:macro name="w200">
+  <xacro:macro name="w200" params="wheel:='default' color:='yellow'">
+    <!-- Colors: yellow, orange, olive, sand -->
+    <xacro:property name="warthog_color"  value="${'warthog_'+color}"/>
+    <material name="warthog_yellow"><color rgba="0.95 0.816 0.082 1.0"/></material>
+    <material name="warthog_orange"><color rgba="1.0 0.48 0.0 1.0"/></material>
+    <material name="warthog_olive"><color rgba="0.333 0.419 0.184 1.0"/></material>
+    <material name="warthog_sand"><color rgba="0.86 0.75 0.54 1.0"/></material>
+    <!-- Variables -->
+    <xacro:property name="wheel_radius" value="0.3" />
+    <xacro:property name="wheel_width"  value="0.25" />
+    <xacro:property name="wheel_mass"   value="15" />
+    <xacro:property name="wheel_to_track_ratio" value="0.5962" />
+    <xacro:property name="axle_x_offset" value="0.457367" />
+    <xacro:property name="axle_y_offset" value="0.0" />
+    <xacro:property name="axle_z_offset" value="-0.012977" />
+    <xacro:property name="track_z_offset" value="-0.2" />
+    <xacro:property name="diff_unit_length" value="1.34" />
+    <xacro:property name="diff_unit_width"  value="0.28" />
+    <xacro:property name="diff_unit_height" value="0.63"/>
+    <xacro:property name="diff_unit_mass"   value="50" />
+    <xacro:property name="diff_unit_offset_x" value="0.00" />
+    <xacro:property name="diff_unit_offset_y" value="0.56821" />
+    <xacro:property name="diff_unit_offset_z" value="0.0" />
+    <xacro:property name="chassis_length" value="1.35" />
+    <xacro:property name="chassis_width"  value="0.70" />
+    <xacro:property name="chassis_height" value="0.30" />
+    <xacro:property name="chassis_mass"   value="100" />
+    <xacro:property name="dummy_inertia" value="1e-09"/>
     <!-- Chassis -->
     <link name="base_link"></link>
