Commit message: Removed testing visual for track virtual wheel

File: clearpath_platform_description/urdf/w200/wheels/track.urdf.xacro (robot description, xacro)
@@ -37,11 +37,4 @@
         <xacro:wheel_inertia m="${wheel_mass}" r="${wheel_radius}" h="${wheel_width}" />
       </inertial>
-      <visual>
-        <material name="clearpath_red"/>
-        <origin xyz="0 0 0" rpy="${PI/2} 0 0"/>
-        <geometry>
-          <cylinder radius="${wheel_radius*wheel_to_track_ratio}" length="${wheel_width}"/>
-        </geometry>
-      </visual>
       <collision>
         <origin xyz="0 0 0" rpy="${PI/2} 0 0"/>
