Commit message: Initial commit with platform, decoration and mounts generating

File: clearpath_mounts_description/urdf/fath_pivot.urdf.xacro (robot description, xacro)
@@ -1,6 +1,6 @@
 <?xml version="1.0"?>
 <robot xmlns:xacro="http://wiki.ros.org/xacro">
-  <xacro:macro name="fath_pivot_mount" params="parent_link prefix angle *origin">
-    <link name="${prefix}_base_link">
+  <xacro:macro name="fath_pivot" params="name parent_link mounting_link angle:=0.0 *origin">
+    <link name="${name}_link">
       <visual>
         <geometry>
@@ -22,5 +22,5 @@
       </collision>
     </link>
-    <link name="${prefix}_hinge_link">
+    <link name="${name}_hinge_link">
       <visual>
         <geometry>
@@ -36,18 +36,18 @@
       </collision>
     </link>
-    <link name="${prefix}_mount" />
-    <joint name="${prefix}_base_joint" type="fixed">
+    <link name="${mounting_link}" />
+    <joint name="${name}_joint" type="fixed">
       <parent link="${parent_link}" />
-      <child link="${prefix}_base_link" />
+      <child link="${name}_link" />
       <xacro:insert_block name="origin" />
     </joint>
-    <joint name="${prefix}_hinge_joint" type="fixed">
-      <parent link="${prefix}_base_link" />
-      <child link="${prefix}_hinge_link" />
+    <joint name="${name}_hinge_joint" type="fixed">
+      <parent link="${name}_link" />
+      <child link="${name}_hinge_link" />
       <origin xyz="0 0 0.0225" rpy="0 ${angle} 0" />
     </joint>
-    <joint name="${prefix}_mount_joint" type="fixed">
-      <parent link="${prefix}_hinge_link" />
-      <child link="${prefix}_mount" />
+    <joint name="${name}_mount_joint" type="fixed">
+      <parent link="${name}_hinge_link" />
+      <child link="${mounting_link}" />
       <origin xyz="0 0 0.0225" rpy="0 0 0" />
     </joint>

File: clearpath_platform_description/urdf/a200/a200.urdf.xacro (robot description, xacro)
@@ -1,45 +1,139 @@
 <?xml version="1.0"?>
-<robot xmlns:xacro="http://ros.org/wiki/xacro" name="a200">
-  <!-- robot name parameter -->
-  <!-- <xacro:arg name="name" default="" /> -->
-  <xacro:arg name="prefix" default="" />
-  <xacro:arg name="gazebo_controllers" default="$(find clearpath_control)/config/control.yaml" />
-  <xacro:include filename="$(find clearpath_platform_description)/urdf/a200/a200_macro.urdf.xacro" />
-  <!-- Load a200 description -->
-  <xacro:a200 prefix="$(arg prefix)" />
-  <xacro:if value="$(arg is_sim)">
-    <gazebo>
-      <plugin name="$(arg prefix)gazebo_ros2_control" filename="libgazebo_ros2_control.so">
-        <parameters>$(arg gazebo_controllers)</parameters>
-      </plugin>
-    </gazebo>
-    <gazebo reference="$(arg prefix)imu_link">
-      <sensor name="$(arg prefix)imu_sensor" type="imu">
-      <plugin filename="libgazebo_ros_imu_sensor.so" name="$(arg prefix)imu_plugin">
-          <ros>
-            <namespace>$(arg prefix)</namespace>
-            <remapping>~/out:=imu/data_raw</remapping>
-          </ros>
-          <initial_orientation_as_reference>false</initial_orientation_as_reference>
-        </plugin>
-        <always_on>true</always_on>
-        <update_rate>100</update_rate>
-        <visualize>true</visualize>
-      </sensor>
-    </gazebo>
-    <gazebo reference="$(arg prefix)gps_link">
-      <sensor name="$(arg prefix)gps_sensor" type="gps">
-      <plugin filename="libgazebo_ros_gps_sensor.so" name="$(arg prefix)gps_plugin">
-          <ros>
-            <namespace>$(arg prefix)</namespace>
-            <remapping>~/out:=gps/data</remapping>
-          </ros>
-        </plugin>
-        <always_on>true</always_on>
-        <update_rate>10</update_rate>
-      </sensor>
-    </gazebo>
-  </xacro:if>
-  <!-- Optional custom includes. -->
-  <xacro:include filename="$(arg urdf_extras)" />
+<robot xmlns:xacro="http://ros.org/wiki/xacro">
+  <xacro:arg name="robot_namespace" default="/" />
+  <xacro:arg name="is_sim" default="false" />
+  <!-- Included URDF/XACRO Files -->
+  <xacro:include filename="$(find clearpath_platform_description)/urdf/a200/wheel.urdf.xacro" />
+  <xacro:property name="M_PI" value="3.14159"/>
+  <xacro:macro name="a200">
+    <!-- Base Size -->
+    <xacro:property name="base_x_size" value="0.98740000" />
+    <xacro:property name="base_y_size" value="0.57090000" />
+    <xacro:property name="base_z_size" value="0.24750000" />
+    <!-- Wheel Mounting Positions -->
+    <xacro:property name="wheelbase" value="0.5120" />
+    <xacro:property name="track" value="0.5708" />
+    <xacro:property name="wheel_vertical_offset" value="0.03282" />
+    <!-- Wheel Properties -->
+    <xacro:property name="wheel_length" value="0.1143" />
+    <xacro:property name="wheel_radius" value="0.1651" />
+    <!-- Base link is the center of the robot's bottom plate -->
+    <link name="base_link">
+      <visual>
+        <origin xyz="0 0 0" rpy="0 0 0" />
+        <geometry>
+          <mesh filename="package://clearpath_platform_description/meshes/a200/base_link.dae" />
+        </geometry>
+      </visual>
+      <collision>
+        <origin xyz="0 0 ${base_z_size/4}" rpy="0 0 0" />
+        <geometry>
+          <box size="${base_x_size} ${base_y_size} ${base_z_size/2}"/>
+        </geometry>
+      </collision>
+      <collision>
+        <origin xyz="0 0 ${base_z_size*3/4-0.01}" rpy="0 0 0" />
+        <geometry>
+          <box size="${base_x_size*4/5} ${base_y_size} ${base_z_size/2-0.02}"/>
+        </geometry>
+      </collision>
+    </link>
+    <!-- Base footprint is on the ground under the robot -->
+    <link name="base_footprint"/>
+    <joint name="base_footprint_joint" type="fixed">
+      <origin xyz="0 0 ${wheel_vertical_offset - wheel_radius}" rpy="0 0 0" />
+      <parent link="base_link" />
+      <child link="base_footprint" />
+    </joint>
+    <!-- Spawn A200 chassis -->
+    <link name="top_chassis_link">
+      <visual>
+        <origin xyz="0 0 0" rpy="0 0 0" />
+        <geometry>
+          <mesh filename="package://clearpath_platform_description/meshes/a200/top_chassis.dae" />
+        </geometry>
+      </visual>
+    </link>
+    <!-- Attach chassis to the robot -->
+    <joint name="top_chassis_joint" type="fixed">
+      <parent link="base_link" />
+      <child link="top_chassis_link" />
+    </joint>
+    <!-- Inertial link stores the robot's inertial information -->
+    <link name="inertial_link">
+      <inertial>
+        <mass value="46.034" />
+        <origin xyz="-0.00065 -0.085 0.062" />
+        <inertia ixx="0.6022" ixy="-0.02364" ixz="-0.1197" iyy="1.7386" iyz="-0.001544" izz="2.0296" />
+      </inertial>
+    </link>
+    <joint name="inertial_joint" type="fixed">
+      <origin xyz="0 0 0" rpy="0 0 0" />
+      <parent link="base_link" />
+      <child link="inertial_link" />
+    </joint>
+    <!-- A200 wheel macros -->
+    <xacro:a200_wheel wheel_prefix="front_left">
+      <origin xyz="${wheelbase/2} ${track/2} ${wheel_vertical_offset}" rpy="0 0 0" />
+    </xacro:a200_wheel>
+    <xacro:a200_wheel wheel_prefix="front_right">
+      <origin xyz="${wheelbase/2} ${-track/2} ${wheel_vertical_offset}" rpy="0 0 0" />
+    </xacro:a200_wheel>
+    <xacro:a200_wheel wheel_prefix="rear_left">
+      <origin xyz="${-wheelbase/2} ${track/2} ${wheel_vertical_offset}" rpy="0 0 0" />
+    </xacro:a200_wheel>
+    <xacro:a200_wheel wheel_prefix="rear_right">
+      <origin xyz="${-wheelbase/2} ${-track/2} ${wheel_vertical_offset}" rpy="0 0 0" />
+    </xacro:a200_wheel>
+    <ros2_control name="a200_hardware" type="system">
+      <hardware>
+        <xacro:if value="$(arg is_sim)">
+          <plugin>gazebo_ros2_control/GazeboSystem</plugin>
+        </xacro:if>
+        <xacro:unless value="$(arg is_sim)">
+          <plugin>a200_base/A200Hardware</plugin>
+          <plugin>fake_components/GenericSystem</plugin>
+          <param name="hw_start_duration_sec">2.0</param>
+          <param name="hw_stop_duration_sec">3.0</param>
+          <param name="wheel_diameter">0.3302</param>
+          <param name="max_accel">5.0</param>
+          <param name="max_speed">1.0</param>
+          <param name="polling_timeout">10.0</param>
+          <param name="serial_port">/dev/prolific</param>
+        </xacro:unless>
+      </hardware>
+      <joint name="front_left_wheel_joint">
+        <command_interface name="velocity">
+          <param name="min">-1</param>
+          <param name="max">1</param>
+        </command_interface>
+        <state_interface name="position"/>
+        <state_interface name="velocity"/>
+      </joint>
+      <joint name="rear_left_wheel_joint">
+        <command_interface name="velocity">
+          <param name="min">-1</param>
+          <param name="max">1</param>
+        </command_interface>
+        <state_interface name="position"/>
+        <state_interface name="velocity"/>
+      </joint>
+      <joint name="front_right_wheel_joint">
+        <command_interface name="velocity">
+          <param name="min">-1</param>
+          <param name="max">1</param>
+        </command_interface>
+        <state_interface name="position"/>
+        <state_interface name="velocity"/>
+      </joint>
+      <joint name="rear_right_wheel_joint">
+        <command_interface name="velocity">
+          <param name="min">-1</param>
+          <param name="max">1</param>
+        </command_interface>
+        <state_interface name="position"/>
+        <state_interface name="velocity"/>
+      </joint>
+    </ros2_control>
+  </xacro:macro>
 </robot>

File: clearpath_platform_description/urdf/a200/decorations/decorations.urdf.xacro (robot description, xacro)
@@ -11,18 +11,4 @@
     <xacro:property name="a200_front_bumper_extend" value="$(optenv A200_FRONT_BUMPER_EXTEND 0)" />
     <xacro:property name="a200_rear_bumper_extend" value="$(optenv A200_REAR_BUMPER_EXTEND 0)" />
-    <!-- Spawn A200 chassis -->
-    <link name="top_chassis_link">
-      <visual>
-        <origin xyz="0 0 0" rpy="0 0 0" />
-        <geometry>
-          <mesh filename="package://clearpath_platform_description/meshes/a200/top_chassis.dae" />
-        </geometry>
-      </visual>
-    </link>
-    <!-- Attach chassis to the robot -->
-    <joint name="top_chassis_joint" type="fixed">
-      <parent link="base_link" />
-      <child link="top_chassis_link" />
-    </joint>
     <xacro:if value="$(optenv A200_USER_RAIL_ENABLED true)">
       <!-- Spawn user rails -->
