Commit message: PACS mounts Common PACS Riser Hokuyo and novatel description fixes

File: clearpath_mounts_description/urdf/fath_pivot.urdf.xacro (robot description, xacro)
@@ -1,5 +1,5 @@
 <?xml version="1.0"?>
 <robot xmlns:xacro="http://wiki.ros.org/xacro">
-  <xacro:macro name="fath_pivot" params="name parent_link mounting_link angle:=0.0 *origin">
+  <xacro:macro name="fath_pivot" params="name parent_link angle:=0.0 *origin">
     <link name="${name}_link">
       <visual>
@@ -36,5 +36,5 @@
       </collision>
     </link>
-    <link name="${mounting_link}" />
+    <link name="${name}_mount" />
     <joint name="${name}_joint" type="fixed">
       <parent link="${parent_link}" />
@@ -49,5 +49,5 @@
     <joint name="${name}_mount_joint" type="fixed">
       <parent link="${name}_hinge_link" />
-      <child link="${mounting_link}" />
+      <child link="${name}_mount" />
       <origin xyz="0 0 0.0225" rpy="0 0 0" />
     </joint>

File: clearpath_platform_description/urdf/a200/decorations/front_bumper.urdf.xacro (robot description, xacro)
@@ -6,5 +6,5 @@
             <visual>
                 <geometry>
-                <mesh filename="package://clearpath_platform_description/meshes/a200/bumper.dae" />
+                <mesh filename="package://clearpath_platform_description/meshes/a200/decorations/bumper.dae" />
                 </geometry>
             </visual>
@@ -20,5 +20,5 @@
                 <visual>
                     <geometry>
-                        <mesh filename="package://clearpath_platform_description/meshes/a200/bumper_extension.dae" />
+                        <mesh filename="package://clearpath_platform_description/meshes/a200/decorations/bumper_extension.dae" />
                     </geometry>
                 </visual>

File: clearpath_platform_description/urdf/a200/decorations/rear_bumper.urdf.xacro (robot description, xacro)
@@ -6,5 +6,5 @@
         <visual>
             <geometry>
-            <mesh filename="package://clearpath_platform_description/meshes/a200/bumper.dae" />
+            <mesh filename="package://clearpath_platform_description/meshes/a200/decorations/bumper.dae" />
             </geometry>
         </visual>
@@ -20,5 +20,5 @@
                 <visual>
                     <geometry>
-                        <mesh filename="package://clearpath_platform_description/meshes/a200/bumper_extension.dae" />
+                        <mesh filename="package://clearpath_platform_description/meshes/a200/decorations/bumper_extension.dae" />
                     </geometry>
                 </visual>

File: clearpath_platform_description/urdf/a200/decorations/top_plate.urdf.xacro (robot description, xacro)
@@ -1,12 +1,13 @@
 <?xml version="1.0"?>
 <robot xmlns:xacro="http://ros.org/wiki/xacro">
-    <xacro:macro name="top_plate" params="large:=false">
+    <xacro:include filename="$(find clearpath_mounts_description)/urdf/common.urdf.xacro" />
+    <xacro:macro name="top_plate" params="model:=default">
         <!-- Spawn the top plate -->
-      <xacro:if value="${large}">
+      <xacro:if value="${model == 'default'}">
         <link name="top_plate_link">
           <visual>
             <origin xyz="0 0 0" rpy="0 0 0" />
             <geometry>
-              <mesh filename="package://clearpath_platform_description/meshes/a200/large_top_plate.dae" />
+              <mesh filename="package://clearpath_platform_description/meshes/a200/decorations/large_top_plate.dae" />
             </geometry>
           </visual>
@@ -14,5 +15,5 @@
             <origin xyz="0 0 0" rpy="0 0 0"/>
             <geometry>
-              <mesh filename="package://clearpath_platform_description/meshes/a200/large_top_plate_collision.stl" />
+              <mesh filename="package://clearpath_platform_description/meshes/a200/decorations/large_top_plate_collision.stl" />
             </geometry>
           </collision>
@@ -36,11 +37,13 @@
           <origin xyz="-0.4125 0 0.00672" rpy="0 0 0"/>
         </joint>
+        <link name="top_plate_front_link"/>
+        <link name="top_plate_rear_link"/>
       </xacro:if>
-      <xacro:unless value="${large}">
+      <xacro:if value="${model == 'large'}">
         <link name="top_plate_link">
           <visual>
             <origin xyz="0 0 0" rpy="0 0 0" />
             <geometry>
-              <mesh filename="package://clearpath_platform_description/meshes/a200/top_plate.dae" />
+              <mesh filename="package://clearpath_platform_description/meshes/a200/decorations/top_plate.dae" />
             </geometry>
           </visual>
@@ -48,5 +51,5 @@
             <origin xyz="0 0 0" rpy="0 0 0"/>
             <geometry>
-              <mesh filename="package://clearpath_platform_description/meshes/a200/top_plate.stl" />
+              <mesh filename="package://clearpath_platform_description/meshes/a200/decorations/top_plate.stl" />
             </geometry>
           </collision>
@@ -74,5 +77,5 @@
           <visual>
             <geometry>
-              <mesh filename="package://clearpath_platform_description/meshes/a200/user_rail.dae" />
+              <mesh filename="package://clearpath_platform_description/meshes/a200/decorations/user_rail.dae" />
             </geometry>
           </visual>
@@ -84,7 +87,71 @@
           <child link="user_rail_link" />
         </joint>
-      </xacro:unless>
-      <link name="top_plate_front_link"/>
-      <link name="top_plate_rear_link"/>
+        <link name="top_plate_front_link"/>
+        <link name="top_plate_rear_link"/>
+      </xacro:if>
+      <xacro:if value="${model == 'pacs'}">
+        <link name="top_plate_link">
+          <visual>
+            <material name="dark_grey"><color rgba="0.2 0.2 0.2 1.0" /></material>
+            <geometry>
+              <mesh filename="package://clearpath_platform_description/meshes/a200/decorations/pacs_top_plate.stl" />
+            </geometry>
+          </visual>
+          <collision>
+            <material name="dark_grey"><color rgba="0.2 0.2 0.2 1.0" /></material>
+            <origin xyz="0 0 0.00317500531673" rpy="0 0 0"/>
+            <geometry>
+              <box size="0.670000076294 0.590000033379 0.00635001063347"/>
+            </geometry>
+          </collision>
+        </link>
+        <!-- Attach PACS top plate -->
+        <joint name="top_plate_joint" type="fixed">
+          <child link="top_plate_link"/>
+          <parent link="base_link"/>
+          <origin xyz="0.048299998045 0 0.227500006557" rpy="0 0 0"/>
+        </joint>
+        <!-- Generate PACS mounts -->
+        <xacro:full_mounts
+          name="top_plate"
+          parent_link="top_plate_link"
+          column="a"
+          row="1"
+          columns="7"
+          rows="2"
+          x="0.28"
+          y="0.24"
+          z="0.00635" />
+        <xacro:full_mounts
+          name="top_plate"
+          parent_link="top_plate_link"
+          column="a"
+          row="3"
+          columns="1"
+          rows="4"
+          x="0.12"
+          y="0.24"
+          z="0.00635" />
+        <xacro:full_mounts
+          name="top_plate"
+          parent_link="top_plate_link"
+          column="g"
+          row="3"
+          columns="1"
+          rows="4"
+          x="0.12"
+          y="-0.24"
+          z="0.00635" />
+        <xacro:full_mounts
+          name="top_plate"
+          parent_link="top_plate_link"
+          column="a"
+          row="7"
+          columns="7"
+          rows="2"
+          x="-0.20"
+          y="0.24"
+          z="0.00635" />
+      </xacro:if>
     </xacro:macro>
 </robot>

File: clearpath_sensors_description/urdf/hokuyo_ust10.urdf.xacro (robot description, xacro)
@@ -1,60 +1,6 @@
 <?xml version="1.0"?>
 <robot xmlns:xacro="http://ros.org/wiki/xacro">
-  <xacro:macro name="hokuyo_ust10_mount" params="prefix topic parent_link *origin">
-    <xacro:macro name="hokuyo_ust10" params="frame:=laser topic:=scan sample_size:=720 update_rate:=50
-               min_angle:=-2.35619 max_angle:=2.35619 min_range:=0.1 max_range:=30.0 robot_namespace:=/">
-      <link name="${frame}">
-        <inertial>
-          <mass value="1.1" />
-          <origin xyz="0 0 0" />
-          <inertia ixx="${0.0833333 * 1.1 * (0.102*0.102 + 0.152*0.152)}" ixy="0.0" ixz="0.0"
-            iyy="${0.0833333 * 1.1 * (0.105*0.105 + 0.152*0.152)}" iyz="0.0"
-            izz="${0.0833333 * 1.1 * (0.105*0.105 + 0.102*0.102)}" />
-        </inertial>
-      </link>
-      <gazebo reference="${frame}">
-        <turnGravityOff>true</turnGravityOff>
-        <sensor type="ray" name="${frame}">
-          <pose>0 0 0 0 0 0</pose>
-          <visualize>false</visualize>
-          <update_rate>${update_rate}</update_rate>
-          <ray>
-            <scan>
-              <horizontal>
-                <samples>${sample_size}</samples>
-                <resolution>1</resolution>
-                <min_angle>${min_angle}</min_angle>
-                <max_angle>${max_angle}</max_angle>
-              </horizontal>
-            </scan>
-            <range>
-              <min>${min_range}</min>
-              <max>${max_range}</max>
-              <resolution>0.01</resolution>
-            </range>
-            <noise>
-              <type>gaussian</type>
-              <mean>0.0</mean>
-              <stddev>0.001</stddev>
-            </noise>
-          </ray>
-          <plugin name="gazebo_ros_laser" filename="libgazebo_ros_ray_sensor.so">
-            <ros>
-              <namespace>${robot_namespace}</namespace>
-              <remapping>~/out:=${topic}</remapping>
-            </ros>
-            <output_type>sensor_msgs/LaserScan</output_type>
-            <frame_name>${frame}</frame_name>
-          </plugin>
-        </sensor>
-      </gazebo>
-    </xacro:macro>
-    <xacro:hokuyo_ust10 frame="${prefix}_laser" topic="${topic}"/>
-    <joint name="${prefix}_laser_mount_joint" type="fixed">
-      <xacro:insert_block name="origin" />
-      <parent link="${parent_link}" />
-      <child link="${prefix}_laser_mount" />
-    </joint>
-    <link name="${prefix}_laser_mount">
+  <xacro:macro name="hokuyo_ust10" params="name parent_link *origin">
+    <link name="${name}_link">
       <visual>
         <origin xyz="0 0 0" rpy="0 0 0" />
@@ -66,13 +12,24 @@
       </visual>
     </link>
-    <joint name="${prefix}_laser_joint" type="fixed">
+    <link name="${name}_laser">
+      <inertial>
+        <mass value="1.1" />
+        <origin xyz="0 0 0" />
+        <inertia ixx="${0.0833333 * 1.1 * (0.102*0.102 + 0.152*0.152)}" ixy="0.0" ixz="0.0"
+                  iyy="${0.0833333 * 1.1 * (0.105*0.105 + 0.152*0.152)}" iyz="0.0"
+                  izz="${0.0833333 * 1.1 * (0.105*0.105 + 0.102*0.102)}" />
+      </inertial>
+    </link>
+    <joint name="${name}_joint" type="fixed">
+      <xacro:insert_block name="origin" />
+      <parent link="${parent_link}" />
+      <child link="${name}_link" />
+    </joint>
+    <joint name="${name}_laser_joint" type="fixed">
       <!-- This offset is from the base of the bracket to the LIDAR's focal point. -->
       <origin xyz="0 0 0.0474" rpy="0 0 0" />
-      <parent link="${prefix}_laser_mount" />
-      <child link="${prefix}_laser" />
+      <parent link="${name}_link" />
+      <child link="${name}_laser" />
     </joint>
-    <gazebo reference="${prefix}_laser_mount">
-      <material>Gazebo/DarkGrey</material>
-    </gazebo>
   </xacro:macro>
 </robot>

File: clearpath_sensors_description/urdf/novatel_smart6.urdf.xacro (robot description, xacro)
@@ -1,6 +1,6 @@
 <?xml version="1.0"?>
 <robot xmlns:xacro="http://www.ros.org/wiki/xacro">
-  <xacro:macro name="novatel_smart6" params="prefix">
-  <link name="${prefix}_navsat">
+  <xacro:macro name="novatel_smart6" params="name">
+  <link name="${name}_link">
     <visual>
       <origin xyz="0 0 0" rpy="0 0 0" />

File: clearpath_sensors_description/urdf/novatel_smart7.urdf.xacro (robot description, xacro)
@@ -1,6 +1,6 @@
 <?xml version="1.0"?>
 <robot xmlns:xacro="http://www.ros.org/wiki/xacro">
-  <xacro:macro name="novatel_smart7" params="prefix">
-    <link name="${prefix}_navsat">
+  <xacro:macro name="novatel_smart7" params="name parent_link *origin">
+    <link name="${name}_link">
       <visual>
         <origin xyz="-0.095 0 0" rpy="${pi/2} 0 -${pi/2}" />
@@ -15,29 +15,12 @@
         <origin xyz="-0.095 0 0" rpy="${pi/2} 0 -${pi/2}" />
         <geometry>
-          <mesh filename="package://clearpath_sensors_description/meshes/novatel-smart7.stl"/>
+          <mesh filename="package://clearpath_sensors_description/meshes/novatel_smart7.stl"/>
         </geometry>
       </collision>
     </link>
-  </xacro:macro>
-  <xacro:macro name="novatel_smart7_stand" params="prefix parent height:=14.5 *origin">
-    <link name="${prefix}_navsat_stand">
-      <visual>
-        <origin xyz="0 0 ${height/2}" rpy="0 0 0"/>
-        <geometry>
-          <box size="0.045 0.025 ${height}" />
-        </geometry>
-        <material name="black" />
-      </visual>
-      <collision>
-        <origin xyz="0 0 ${height/2}" rpy="0 0 0"/>
-        <geometry>
-          <box size="0.045 0.025 ${height}" />
-        </geometry>
-      </collision>
-    </link>
-    <joint name="${prefix}_navsat_stand_joint" type="fixed">
+    <joint name="${name}_joint" type="fixed">
       <xacro:insert_block name="origin" />
-      <parent link="${parent}" />
-      <child link="${prefix}_navsat_stand" />
+      <parent link="${parent_link}" />
+      <child link="${name}_link" />
     </joint>
   </xacro:macro>
