Commit message: Update sensor descriptions and plugins for vecow amr simulation on gazebo classic

File: clearpath_mounts_description/urdf/fath_pivot.urdf.xacro (robot description, xacro)
@@ -5,5 +5,5 @@
       <visual>
         <geometry>
-          <mesh filename="package://clearpath_mounts_description/meshes/fath_pivot_mount_base.dae" />
+          <mesh filename="file://$(find clearpath_mounts_description)/meshes/fath_pivot_mount_base.dae" />
         </geometry>
         <origin xyz="0 0 0" rpy="0 0 ${pi/2}" />
@@ -25,5 +25,5 @@
       <visual>
         <geometry>
-          <mesh filename="package://clearpath_mounts_description/meshes/fath_pivot_mount.dae" />
+          <mesh filename="file://$(find clearpath_mounts_description)/meshes/fath_pivot_mount.dae" />
         </geometry>
         <origin xyz="0 0 0" rpy="0 0 ${pi/2}" />

File: clearpath_mounts_description/urdf/pacs/bracket.urdf.xacro (robot description, xacro)
@@ -36,5 +36,5 @@
         <xacro:property name="mesh_z" value="0.010125"/>
         <xacro:property name="mesh_thickness" value="0.010125"/>
-        <xacro:property name="mesh" value="package://clearpath_mounts_description/meshes/pacs/bracket_horizontal.stl"/>
+        <xacro:property name="mesh" value="file://$(find clearpath_mounts_description)/meshes/pacs/bracket_horizontal.stl"/>
     </xacro:if>
     <!-- Horizontal Large -->
@@ -44,5 +44,5 @@
         <xacro:property name="mesh_z" value="0.00635"/>
         <xacro:property name="mesh_thickness" value="0.00635"/>
-        <xacro:property name="mesh" value="package://clearpath_mounts_description/meshes/pacs/bracket_horizontal_large.stl"/>
+        <xacro:property name="mesh" value="file://$(find clearpath_mounts_description)/meshes/pacs/bracket_horizontal_large.stl"/>
     </xacro:if>
     <!-- Vertical -->
@@ -52,5 +52,5 @@
         <xacro:property name="mesh_z" value="0.1419"/>
         <xacro:property name="mesh_thickness" value="0.010125"/>
-        <xacro:property name="mesh" value="package://clearpath_mounts_description/meshes/pacs/bracket_vertical.stl"/>
+        <xacro:property name="mesh" value="file://$(find clearpath_mounts_description)/meshes/pacs/bracket_vertical.stl"/>
         <!-- Vertical Mount -->
         <link name="${name}_vertical_mount"/>

File: clearpath_platform_description/urdf/a200/a200.urdf.xacro (robot description, xacro)
@@ -2,5 +2,5 @@
 <robot xmlns:xacro="http://ros.org/wiki/xacro">
   <xacro:arg name="namespace" default="" />
-  <xacro:arg name="is_sim" default="false" />
+  <xacro:arg name="is_sim" default="true" />
   <xacro:arg name="serial_port" default="/dev/clearpath/prolific" />
   <xacro:arg name="gazebo_controllers" default="$(find clearpath_control)/config/a200/control.yaml"/>
@@ -25,5 +25,5 @@
         <origin xyz="0 0 0" rpy="0 0 0" />
         <geometry>
-          <mesh filename="package://clearpath_platform_description/meshes/a200/base_link.dae" />
+          <mesh filename="file://$(find clearpath_platform_description)/meshes/a200/base_link.dae" />
         </geometry>
       </visual>
@@ -53,5 +53,5 @@
         <origin xyz="0 0 0" rpy="0 0 0" />
         <geometry>
-          <mesh filename="package://clearpath_platform_description/meshes/a200/top_chassis.dae" />
+          <mesh filename="file://$(find clearpath_platform_description)/meshes/a200/top_chassis.dae" />
         </geometry>
       </visual>
@@ -89,26 +89,26 @@
     </xacro:a200_wheel>
     <gazebo>
-      <plugin filename="libignition-gazebo-wheel-slip-system.so" name="ignition::gazebo::systems::WheelSlip">
+      <plugin name="WheelSlip" filename="libgazebo_ros_wheel_slip.so">
         <wheel link_name="front_left_wheel">
-          <slip_compliance_lateral>1.0</slip_compliance_lateral>
-          <slip_compliance_longitudinal>1.0</slip_compliance_longitudinal>
+          <slip_compliance_lateral>0.1</slip_compliance_lateral>
+          <slip_compliance_longitudinal>0.1</slip_compliance_longitudinal>
           <wheel_normal_force>113</wheel_normal_force>
           <wheel_radius>${wheel_radius}</wheel_radius>
         </wheel>
         <wheel link_name="front_right_wheel">
-          <slip_compliance_lateral>1.0</slip_compliance_lateral>
-          <slip_compliance_longitudinal>1.0</slip_compliance_longitudinal>
+          <slip_compliance_lateral>0.1</slip_compliance_lateral>
+          <slip_compliance_longitudinal>0.1</slip_compliance_longitudinal>
           <wheel_normal_force>113</wheel_normal_force>
           <wheel_radius>${wheel_radius}</wheel_radius>
         </wheel>
         <wheel link_name="rear_left_wheel">
-          <slip_compliance_lateral>1.0</slip_compliance_lateral>
-          <slip_compliance_longitudinal>1.0</slip_compliance_longitudinal>
+          <slip_compliance_lateral>0.1</slip_compliance_lateral>
+          <slip_compliance_longitudinal>0.1</slip_compliance_longitudinal>
           <wheel_normal_force>113</wheel_normal_force>
           <wheel_radius>${wheel_radius}</wheel_radius>
         </wheel>
         <wheel link_name="rear_right_wheel">
-          <slip_compliance_lateral>1.0</slip_compliance_lateral>
-          <slip_compliance_longitudinal>1.0</slip_compliance_longitudinal>
+          <slip_compliance_lateral>0.1</slip_compliance_lateral>
+          <slip_compliance_longitudinal>0.1</slip_compliance_longitudinal>
           <wheel_normal_force>113</wheel_normal_force>
           <wheel_radius>${wheel_radius}</wheel_radius>
@@ -143,5 +143,5 @@
       <hardware>
         <xacro:if value="$(arg is_sim)">
-          <plugin>ign_ros2_control/IgnitionSystem</plugin>
+          <plugin>gazebo_ros2_control/GazeboSystem</plugin>
         </xacro:if>
         <xacro:unless value="$(arg is_sim)">

File: clearpath_platform_description/urdf/a200/attachments/bumper.urdf.xacro (robot description, xacro)
@@ -6,5 +6,5 @@
             <visual>
                 <geometry>
-                    <mesh filename="package://clearpath_platform_description/meshes/a200/attachments/bumper.dae" />
+                    <mesh filename="file://$(find clearpath_platform_description)/meshes/a200/attachments/bumper.dae" />
                 </geometry>
             </visual>

File: clearpath_platform_description/urdf/a200/attachments/sensor_arch.urdf.xacro (robot description, xacro)
@@ -8,5 +8,5 @@
           <origin xyz="0 0 0.51" rpy="0 0 0"/>
           <geometry>
-            <mesh filename="package://clearpath_platform_description/meshes/a200/attachments/510_mm_sensor_arch.dae" />
+            <mesh filename="file://$(find clearpath_platform_description)/meshes/a200/attachments/510_mm_sensor_arch.dae" />
           </geometry>
         </visual>
@@ -14,5 +14,5 @@
           <origin xyz="0 0 0.51" rpy="0 0 0"/>
           <geometry>
-            <mesh filename="package://clearpath_platform_description/meshes/a200/attachments/510_mm_sensor_arch.dae" />
+            <mesh filename="file://$(find clearpath_platform_description)/meshes/a200/attachments/510_mm_sensor_arch.dae" />
           </geometry>
         </collision>
@@ -37,5 +37,5 @@
           <origin xyz="0 0 0.3" rpy="0 0 0"/>
           <geometry>
-            <mesh filename="package://clearpath_platform_description/meshes/a200/attachments/300_mm_sensor_arch.dae" />
+            <mesh filename="file://$(find clearpath_platform_description)/meshes/a200/attachments/300_mm_sensor_arch.dae" />
           </geometry>
         </visual>
@@ -43,5 +43,5 @@
           <origin xyz="0 0 0.3" rpy="0 0 0"/>
           <geometry>
-            <mesh filename="package://clearpath_platform_description/meshes/a200/attachments/300_mm_sensor_arch.dae" />
+            <mesh filename="file://$(find clearpath_platform_description)/meshes/a200/attachments/300_mm_sensor_arch.dae" />
           </geometry>
         </collision>

File: clearpath_platform_description/urdf/a200/attachments/top_plate.urdf.xacro (robot description, xacro)
@@ -1,3 +1,3 @@
-<?xml version="1.0"?>
+<?xm version="1.0"?>
 <robot xmlns:xacro="http://ros.org/wiki/xacro">
     <xacro:macro name="top_plate" params="name model:=default parent_link:=default_mount *origin">
@@ -9,5 +9,5 @@
             <origin xyz="0.0812 0 0" rpy="0 0 0" />
             <geometry>
-              <mesh filename="package://clearpath_platform_description/meshes/a200/attachments/large_top_plate.dae" />
+              <mesh filename="file://$(find clearpath_platform_description)/meshes/a200/attachments/large_top_plate.dae" />
             </geometry>
           </visual>
@@ -15,5 +15,5 @@
             <origin xyz="0.0812 0 0" rpy="0 0 0"/>
             <geometry>
-              <mesh filename="package://clearpath_platform_description/meshes/a200/attachments/large_top_plate_collision.stl" />
+              <mesh filename="file://$(find clearpath_platform_description)/meshes/a200/attachments/large_top_plate_collision.stl" />
             </geometry>
           </collision>
@@ -47,5 +47,5 @@
             <origin xyz="0.272 0 0.019"/>
             <geometry>
-              <mesh filename="package://clearpath_platform_description/meshes/a200/attachments/user_rail.dae" />
+              <mesh filename="file://$(find clearpath_platform_description)/meshes/a200/attachments/user_rail.dae" />
             </geometry>
           </visual>
@@ -62,5 +62,5 @@
             <origin xyz="0.0812 0 0" rpy="0 0 0" />
             <geometry>
-              <mesh filename="package://clearpath_platform_description/meshes/a200/attachments/top_plate.dae" />
+              <mesh filename="file://$(find clearpath_platform_description)/meshes/a200/attachments/top_plate.dae" />
             </geometry>
           </visual>
@@ -68,5 +68,5 @@
             <origin xyz="0.0812 0 0" rpy="0 0 0"/>
             <geometry>
-              <mesh filename="package://clearpath_platform_description/meshes/a200/attachments/top_plate.stl" />
+              <mesh filename="file://$(find clearpath_platform_description)/meshes/a200/attachments/top_plate.stl" />
             </geometry>
           </collision>
@@ -101,5 +101,5 @@
             <material name="clearpath_dark_grey" />
             <geometry>
-              <mesh filename="package://clearpath_platform_description/meshes/a200/attachments/pacs_top_plate.stl" />
+              <mesh filename="file://$(find clearpath_platform_description)/meshes/a200/attachments/pacs_top_plate.stl" />
             </geometry>
           </visual>
@@ -160,4 +160,7 @@
           z="0.00635" />
       </xacro:if>
+       <gazebo reference="${name}_link">
+          <material>Gazebo/DarkGrey</material>
+       </gazebo>
     </xacro:macro>
 </robot>

File: clearpath_platform_description/urdf/a200/wheels/wheel.urdf.xacro (robot description, xacro)
@@ -11,5 +11,5 @@
         <origin xyz="0 0 0" rpy="0 0 0" />
         <geometry>
-          <mesh filename="package://clearpath_platform_description/meshes/a200/wheel.dae" />
+          <mesh filename="file://$(find clearpath_platform_description)/meshes/a200/wheel.dae" />
         </geometry>
       </visual>

File: clearpath_platform_description/urdf/generic/gazebo.urdf.xacro (robot description, xacro)
@@ -3,18 +3,10 @@
   <xacro:if value="$(arg is_sim)">
     <gazebo>
-      <plugin filename="libign_ros2_control-system.so" name="ign_ros2_control::IgnitionROS2ControlPlugin">
+      <plugin filename="libgazebo_ros2_control.so" name="gazebo_ros2_control">
         <parameters>$(arg gazebo_controllers)</parameters>
-        <ros>
-          <remapping>~/odom:=platform/odom</remapping>
-          <remapping>~/cmd_vel_unstamped:=platform/cmd_vel_unstamped</remapping>
-          <remapping>/tf:=tf</remapping>
-          <remapping>/tf_static:=tf_static</remapping>
-          <remapping>/diagnostics:=diagnostics</remapping>
-          <remapping>joint_states:=platform/joint_states</remapping>
-          <namespace>$(arg namespace)</namespace>
-        </ros>
       </plugin>
     </gazebo>
-    <gazebo>
+    <!--  commented because we use robot_state_publisher for gazebo classic, and no ignition packages are required -->
+    <!-- <gazebo>
       <plugin filename="libignition-gazebo-pose-publisher-system.so" name="ignition::gazebo::systems::PosePublisher">
         <publish_link_pose>true</publish_link_pose>
@@ -23,5 +15,5 @@
         <update_frequency>50</update_frequency>
       </plugin>
-    </gazebo>
+    </gazebo>-->
   </xacro:if>
 </robot>

File: clearpath_platform_description/urdf/links/box.urdf.xacro (robot description, xacro)
@@ -7,7 +7,10 @@
           <box size="${size}"/>
         </geometry>
-        <material name="clearpath_dark_grey"/>
+        <material name="clearpath_dark_grey"><color rgba="0.2 0.2 0.2 1.0" /></material>
       </visual>
     </link>
+    <gazebo reference="${name}_link">
+    <material>Gazebo/DarkGrey</material>
+    </gazebo>
     <joint name="${name}_joint" type="fixed">
       <parent link="${parent_link}" />

File: clearpath_platform_description/urdf/links/mesh.urdf.xacro (robot description, xacro)
@@ -5,5 +5,5 @@
       <visual>
         <geometry>
-          <mesh filename="${visual}"/>
+          <mesh filename="file://${visual}"/>
         </geometry>
         <material name="clearpath_dark_grey"/>

File: clearpath_sensors_description/urdf/chrobotics_um6.urdf.xacro (robot description, xacro)
@@ -21,11 +21,11 @@
       <child link="${name}_link" />
     </joint>
-    <gazebo reference="${name}_link">
+    <gazebo reference="${name}_base_link">
       <sensor type="imu" name="${name}">
         <always_on>true</always_on>
+        <plugin name="my_imu_plugin" filename="libgazebo_ros_imu_sensor.so"></plugin>
         <update_rate>${update_rate}</update_rate>
         <visualize>true</visualize>
-        <ignition_frame_id>${name}_link</ignition_frame_id>
-      </sensor>
+        </sensor>
     </gazebo>
   </xacro:macro>

File: clearpath_sensors_description/urdf/intel_realsense.urdf.xacro (robot description, xacro)
@@ -48,5 +48,5 @@
             <origin xyz="${d435_zero_depth_to_glass + d435_glass_to_front} ${-d435_cam_depth_py} 0" rpy="${M_PI/2} 0 ${M_PI/2}"/>
             <geometry>
-              <mesh filename="package://realsense2_description/meshes/d435.dae" />
+              <mesh filename="file://$(find realsense2_description)/meshes/d435.dae" />
             </geometry>
           </xacro:if>
@@ -136,22 +136,29 @@
       <xacro:insert_block name="origin" />
     </xacro:sensor_d435>
-    <gazebo reference="${name}_link">
-      <sensor name="${name}" type="rgbd_camera">
-        <camera>
-          <horizontal_fov>1.25</horizontal_fov>
+  <gazebo reference="${name}_link">
+      <sensor name="${name}" type="depth">
+      <pose> 0 0 0 0 0 0 </pose>
+      <plugin name="camera_${name}_controller" filename="libgazebo_ros_camera.so">
+          <min_depth>0.015</min_depth>
+          <max_depth>10.0</max_depth>
+          <hack_baseline>0.07</hack_baseline>
+          <frame_name>camera_depth_link</frame_name>
+          <distortion_k1>0.00000001</distortion_k1>
+          <distortion_k2>0.00000001</distortion_k2>
+          <distortion_k3>0.00000001</distortion_k3>
+          <distortion_t1>0.00000001</distortion_t1>
+          <distortion_t2>0.00000001</distortion_t2>
+        </plugin>
+        <camera >
+          <horizontal_fov>1.50098</horizontal_fov>
           <image>
-            <width>${image_width}</width>
-            <height>${image_height}</height>
+            <width>640</width>
+            <height>480</height>
+            <format>R8G8B8</format>
           </image>
-          <clip>
-            <near>0.3</near>
-            <far>100</far>
-          </clip>
-          <optical_frame_id>${name}_color_optical_frame</optical_frame_id>
         </camera>
-        <always_on>1</always_on>
-        <update_rate>${update_rate}</update_rate>
         <visualize>true</visualize>
-        <ignition_frame_id>${name}_link</ignition_frame_id>
+        <always_on>true</always_on>
+        <update_rate>30.0</update_rate>
       </sensor>
     </gazebo>

File: clearpath_sensors_description/urdf/novatel_smart6.urdf.xacro (robot description, xacro)
@@ -6,5 +6,5 @@
         <origin xyz="0 0 0" rpy="0 0 0" />
         <geometry>
-          <mesh filename="package://clearpath_sensors_description/meshes/novatel_smart6.stl"/>
+          <mesh filename="file://$(find clearpath_sensors_description)/meshes/novatel_smart6.stl"/>
         </geometry>
         <material name="clearpath_novatel_white">
@@ -18,11 +18,12 @@
       <xacro:insert_block name="origin"/>
     </joint>
-    <gazebo reference="${name}_link">
-      <sensor name="${name}" type="navsat">
-        <always_on>1</always_on>
-        <update_rate>1</update_rate>
-        <ignition_frame_id>${name}_link</ignition_frame_id>
-      </sensor>
-    </gazebo>
+<gazebo reference="${name}_link">
+    <sensor name="${name}" type="gps">
+      <update_rate>30</update_rate>
+      <plugin name="${name}_gps_controller" filename="libgazebo_ros_gps_sensor.so"></plugin>
+      <visualize>true</visualize>
+      <always_on>true</always_on>
+    </sensor>
+</gazebo>
   </xacro:macro>
 </robot>

File: clearpath_sensors_description/urdf/velodyne_lidar.urdf.xacro (robot description, xacro)
@@ -19,10 +19,10 @@
       <visual>
         <geometry>
-          <mesh filename="package://velodyne_description/meshes/VLP16_base_1.dae"/>
+          <mesh filename="file://$(find velodyne_description)/meshes/VLP16_base_1.dae"/>
         </geometry>
       </visual>
       <visual>
         <geometry>
-          <mesh filename="package://velodyne_description/meshes/VLP16_base_2.dae"/>
+          <mesh filename="file://$(find velodyne_description)/meshes/VLP16_base_2.dae"/>
         </geometry>
       </visual>
@@ -33,5 +33,5 @@
         </geometry>
       </collision>
-    </link>
+  </link>
     <joint name="${name}_joint" type="fixed">
       <xacro:insert_block name="origin"/>
@@ -48,5 +48,5 @@
         <origin xyz="0 0 -0.0377"/>
         <geometry>
-          <mesh filename="package://velodyne_description/meshes/VLP16_scan.dae"/>
+          <mesh filename="file://$(find velodyne_description)/meshes/VLP16_scan.dae"/>
         </geometry>
       </visual>
@@ -60,30 +60,40 @@
     <xacro:property name="samples_v" value="${round((max_ang_v - min_ang_v) * 180 / (ang_res_v * pi))}"/>
     <gazebo reference="${name}_laser">
-      <sensor name="${name}" type="gpu_lidar">
+      <sensor name="${name}" type="gpu_ray">
+          <pose>0 0 0 0 0 0</pose>
+          <plugin name="gazebo_ros_gpu_laser" filename="libgazebo_ros_velodyne_laser.so">
+            <ros>
+            <remapping>/gazebo_ros_gpu_laser/out:=vecow/LidarPointCloud</remapping>
+            </ros>
+            <frameName>laser_link</frameName>
+            <min_range>${min_range}</min_range>
+            <max_range>${max_range}</max_range>
+            <gaussianNoise>0.008</gaussianNoise>
+            <updateRate>${update_rate}</updateRate>
+          </plugin>
+          <ray>
+            <scan>
+              <horizontal>
+                <samples>${samples_h}</samples>
+                <resolution>${ang_res_h}</resolution>
+                <min_angle>${min_ang_h}</min_angle>
+                <max_angle>${max_ang_h}</max_angle>
+              </horizontal>
+              <vertical>
+                <samples>${samples_v}</samples>
+                <resolution>${ang_res_v}</resolution>
+                <min_angle>${min_ang_v}</min_angle>
+                <max_angle>${max_ang_v}</max_angle>
+              </vertical>
+            </scan>
+            <range>
+              <min>${min_range}</min>
+              <max>${max_range}</max>
+              <resolution>0.004</resolution>
+            </range>
+        </ray>
         <update_rate>${update_rate}</update_rate>
-        <visualize>true</visualize>
+        <visualize>false</visualize>
         <always_on>true</always_on>
-        <ignition_frame_id>${name}_laser</ignition_frame_id>
-        <lidar>
-          <scan>
-            <horizontal>
-              <samples>${samples_h}</samples>
-              <resolution>1</resolution>
-              <min_angle>${min_ang_h}</min_angle>
-              <max_angle>${max_ang_h}</max_angle>
-            </horizontal>
-            <vertical>
-              <samples>${samples_v}</samples>
-              <resolution>1</resolution>
-              <min_angle>${min_ang_v}</min_angle>
-              <max_angle>${max_ang_v}</max_angle>
-            </vertical>
-          </scan>
-          <range>
-            <min>${min_range}</min>
-            <max>${max_range}</max>
-            <resolution>0.01</resolution>
-          </range>
-        </lidar>
       </sensor>
     </gazebo>
