Commit message: Fixed URDF issues

File: clearpath_customization/project_description/urdf/donut.urdf.xacro (robot description, xacro)
@@ -10,5 +10,5 @@
         <origin xyz="0.0 0.0 0.0" rpy="0.0 0.0 0.0"/>
         <!-- set color of the link -->
-        <material name="donut_color">
+        <material name="${name}_color">
           <color rgba="0 1.0 1.0 1.0"/>
         </material>
@@ -23,5 +23,5 @@
         <origin xyz="0.0 0.0 0.0" rpy="0.0 0.0 0.01"/>
         <!-- set color of the bounding box -->
-        <material name="donut_color">
+        <material name="${name}_color">
           <color rgba="0 1.0 1.0 1.0"/>
         </material>
@@ -33,5 +33,5 @@
     </link>
     <!-- Connect to the rest of the robot using the parameters -->
-    <joint name="${name}_joint"/>
+    <joint name="${name}_joint" type="fixed">
       <child link="${name}_link"/>
       <parent link="${parent}"/>

File: clearpath_customization/project_description/urdf/project_description.urdf.xacro (robot description, xacro)
@@ -8,5 +8,5 @@
   </xacro:sensor_d435>
   <!-- Include macro from this package -->
-  <xacro:include filename="$(find project_bringup)/urdf/donut.stl"/>
+  <xacro:include filename="$(find project_description)/urdf/donut.urdf.xacro"/>
   <!-- Call macro to add mesh to robot -->
   <xacro:donut name="donut" parent="default_mount">
