Commit message: Added all joints to the Kinova gripper SRDF

File: clearpath_manipulators_description/srdf/gripper/kinova_2f_lite.srdf.xacro (robot description, xacro)
@@ -4,4 +4,7 @@
     <group name="${name}">
         <joint name="${name}_right_finger_bottom_joint"/>
+        <joint name="${name}_right_finger_tip_joint"/>
+        <joint name="${name}_left_finger_bottom_joint"/>
+        <joint name="${name}_left_finger_tip_joint"/>
     </group>
     <group_state name="open" group="${name}">
