Commit message: Add padding parameter to define finger joint limits

File: clearpath_manipulators_description/srdf/gripper/robotiq_2f_140.srdf.xacro (robot description, xacro)
@@ -6,5 +6,11 @@
     </group_state>
   </xacro:macro>
-  <xacro:macro name="robotiq_2f_140" params="name">
+  <xacro:macro name="robotiq_2f_140" params="name padding:=true">
+    <xacro:if value="${padding}">
+      <xacro:property name="upper_finger_joint_limit" value="0.7"/>
+    </xacro:if>
+    <xacro:unless value="${padding}">
+      <xacro:property name="upper_finger_joint_limit" value="1.0"/>
+    </xacro:unless>
     <group name="${name}">
         <joint name="${name}_finger_joint"/>
@@ -23,5 +29,5 @@
       name="${name}"
       group_state="close"
-      joint_positions="${[0.7]}"
+      joint_positions="${[upper_finger_joint_limit]}"
     />
     <disable_collisions link1="${name}_left_inner_knuckle" link2="${name}_left_inner_finger" reason="User"/>
@@ -29,4 +35,7 @@
     <disable_collisions link1="${name}_left_outer_knuckle" link2="${name}_left_inner_knuckle" reason="User"/>
     <disable_collisions link1="${name}_right_outer_knuckle" link2="${name}_right_inner_knuckle" reason="User"/>
+    <xacro:if value="${padding}">
+      <disable_collisions link1="${name}_right_inner_finger_pad" link2="${name}_left_inner_finger_pad" reason="User"/>
+    </xacro:if>
   </xacro:macro>
 </robot>

File: clearpath_manipulators_description/urdf/gripper/robotiq_2f_140.urdf.xacro (robot description, xacro)
@@ -16,8 +16,15 @@
     isaac_joint_commands:=/isaac_joint_commands
     isaac_joint_states:=/isaac_joint_states
-    com_port:=/dev/ttyUSB0">
+    com_port:=/dev/ttyUSB0
+    padding:=true">
     <!-- Variables Mappings -->
     <xacro:property name="prefix" value="${name}_"/>
     <xacro:property name="stroke" value="140"/>
+    <xacro:if value="${padding}">
+      <xacro:property name="upper_finger_joint_limit" value="0.7"/>
+    </xacro:if>
+    <xacro:unless value="${padding}">
+      <xacro:property name="upper_finger_joint_limit" value="1.0"/>
+    </xacro:unless>
     <!-- this is a temporary link to rotate the 2f-140 gripper to match the 2f-85 -->
     <link name="${prefix}robotiq_base_link"/>
@@ -204,5 +211,5 @@
         <child link="${prefix}left_outer_knuckle" />
         <axis xyz="-1 0 0" />
-        <limit lower="0" upper="0.7" velocity="2.0" effort="1000" />
+        <limit lower="0" upper="${upper_finger_joint_limit}" velocity="2.0" effort="1000" />
       </joint>
       <xacro:finger_joints prefix="${prefix}" fingerprefix="left" reflect="1.0"/>
@@ -259,5 +266,7 @@
       <xacro:inner_knuckle_joint prefix="${prefix}" fingerprefix="${fingerprefix}" reflect="${reflect}"/>
       <xacro:inner_finger_joint prefix="${prefix}" fingerprefix="${fingerprefix}"/>
-      <xacro:inner_finger_pad_joint prefix="${prefix}" fingerprefix="${fingerprefix}"/>
+      <xacro:if value="${padding}">
+        <xacro:inner_finger_pad_joint prefix="${prefix}" fingerprefix="${fingerprefix}"/>
+      </xacro:if>
     </xacro:macro>
     <xacro:macro name="finger_links" params="prefix fingerprefix stroke">
@@ -265,5 +274,7 @@
       <xacro:outer_finger prefix="${prefix}" fingerprefix="${fingerprefix}" stroke="${stroke}"/>
       <xacro:inner_finger prefix="${prefix}" fingerprefix="${fingerprefix}" stroke="${stroke}"/>
-      <xacro:inner_finger_pad prefix="${prefix}" fingerprefix="${fingerprefix}"/>
+      <xacro:if value="${padding}">
+        <xacro:inner_finger_pad prefix="${prefix}" fingerprefix="${fingerprefix}"/>
+      </xacro:if>
       <xacro:inner_knuckle prefix="${prefix}" fingerprefix="${fingerprefix}" stroke="${stroke}"/>
     </xacro:macro>

Commit message: Tune down to 0.767

File: clearpath_manipulators_description/srdf/gripper/robotiq_2f_140.srdf.xacro (robot description, xacro)
@@ -11,5 +11,5 @@
     </xacro:if>
     <xacro:unless value="${padding}">
-      <xacro:property name="upper_finger_joint_limit" value="1.0"/>
+      <xacro:property name="upper_finger_joint_limit" value="0.767"/>
     </xacro:unless>
     <group name="${name}">

File: clearpath_manipulators_description/urdf/gripper/robotiq_2f_140.urdf.xacro (robot description, xacro)
@@ -25,5 +25,5 @@
     </xacro:if>
     <xacro:unless value="${padding}">
-      <xacro:property name="upper_finger_joint_limit" value="1.0"/>
+      <xacro:property name="upper_finger_joint_limit" value="0.767"/>
     </xacro:unless>
     <!-- this is a temporary link to rotate the 2f-140 gripper to match the 2f-85 -->
@@ -221,5 +221,5 @@
         <child link="${prefix}right_outer_knuckle" />
         <axis xyz="1 0 0" />
-        <limit lower="-0.725" upper="0.725" velocity="2.0" effort="1000" />
+        <limit lower="-0.775" upper="0.775" velocity="2.0" effort="1000" />
         <mimic joint="${prefix}finger_joint" multiplier="-1" offset="0" />
       </joint>
