Commit message: Standard mesh names and height parameter for tower shoulder

File: clearpath_platform_description/urdf/r100/attachments/hams.urdf.xacro (robot description, xacro)
@@ -27,5 +27,5 @@
         <origin xyz="${top_mesh_x} ${top_mesh_y} ${table_height + top_mesh_z}"/>
         <geometry>
-          <mesh filename="package://clearpath_platform_description/meshes/r100/attachments/hams-table-top.stl" />
+          <mesh filename="package://clearpath_platform_description/meshes/r100/attachments/hams_top.stl" />
         </geometry>
         <material name="clearpath_black"/>
@@ -34,5 +34,5 @@
         <origin xyz="${top_mesh_x} ${top_mesh_y} ${table_height + top_mesh_z}"/>
         <geometry>
-          <mesh filename="package://clearpath_platform_description/meshes/r100/attachments/hams-table-top.stl" />
+          <mesh filename="package://clearpath_platform_description/meshes/r100/attachments/hams_top.stl" />
         </geometry>
         <material name="clearpath_black"/>
@@ -53,5 +53,5 @@
       <visual>
         <geometry>
-          <mesh filename="package://clearpath_platform_description/meshes/r100/attachments/hams-arm-mount.stl" />
+          <mesh filename="package://clearpath_platform_description/meshes/r100/attachments/hams_mount.stl" />
         </geometry>
         <material name="clearpath_black" />
@@ -60,5 +60,5 @@
         <origin xyz="0 0 0" rpy="0 0 0"/>
         <geometry>
-          <mesh filename="package://clearpath_platform_description/meshes/r100/attachments/hams-arm-mount.stl" />
+          <mesh filename="package://clearpath_platform_description/meshes/r100/attachments/hams_mount.stl" />
         </geometry>
       </collision>

File: clearpath_platform_description/urdf/r100/attachments/legs.urdf.xacro (robot description, xacro)
@@ -9,5 +9,5 @@
       <origin xyz="${pos_x} ${pos_y} 0" rpy="0 0 0"/>
       <geometry>
-        <mesh filename="package://clearpath_platform_description/meshes/r100/attachments/table-leg.stl"
+        <mesh filename="package://clearpath_platform_description/meshes/r100/attachments/leg.stl"
           scale="1.0 1.0 ${table_height/leg_size_z}"/>
       </geometry>
@@ -23,5 +23,5 @@
       <origin xyz="${pos_x} ${-pos_y} 0" rpy="0 0 0"/>
       <geometry>
-        <mesh filename="package://clearpath_platform_description/meshes/r100/attachments/table-leg.stl"
+        <mesh filename="package://clearpath_platform_description/meshes/r100/attachments/leg.stl"
           scale="1.0 1.0 ${table_height/leg_size_z}"/>
       </geometry>
