Commit message: Add RGBA values for the "black" material, rename it to avoid conflicting with any other material definitions

File: clearpath_sensors_description/urdf/axis/axis_q62.urdf.xacro (robot description, xacro)
@@ -95,5 +95,7 @@
         </geometry>
         <origin xyz="-0.01 0 0.05" rpy="0 0 0" />
-        <material name="black" />
+        <material name="axis_black">
+          <color rgba="0 0 0 1" />
+        </material>
       </visual>
       <visual>
@@ -102,5 +104,7 @@
         </geometry>
         <origin xyz="-0.01 0.20 0.05" rpy="0 0 0" />
-        <material name="black" />
+        <material name="axis_black">
+          <color rgba="0 0 0 1" />
+        </material>
       </visual>
     </link>
