Commit message: Copy and modify franka description

File: clearpath_manipulators_description/srdf/arm/franka.srdf.xacro (robot description, xacro)
@@ -3,22 +3,22 @@
   <xacro:macro name="franka_group_state" params="name group_state joint_positions">
     <group_state name="${group_state}" group="${name}">
-      <joint name="${name}_fr3_joint1" value="${joint_positions[0]}"/>
-      <joint name="${name}_fr3_joint2" value="${joint_positions[1]}"/>
-      <joint name="${name}_fr3_joint3" value="${joint_positions[2]}"/>
-      <joint name="${name}_fr3_joint4" value="${joint_positions[3]}"/>
-      <joint name="${name}_fr3_joint5" value="${joint_positions[4]}"/>
-      <joint name="${name}_fr3_joint6" value="${joint_positions[5]}"/>
-      <joint name="${name}_fr3_joint7" value="${joint_positions[6]}"/>
+      <joint name="${name}_joint1" value="${joint_positions[0]}"/>
+      <joint name="${name}_joint2" value="${joint_positions[1]}"/>
+      <joint name="${name}_joint3" value="${joint_positions[2]}"/>
+      <joint name="${name}_joint4" value="${joint_positions[3]}"/>
+      <joint name="${name}_joint5" value="${joint_positions[4]}"/>
+      <joint name="${name}_joint6" value="${joint_positions[5]}"/>
+      <joint name="${name}_joint7" value="${joint_positions[6]}"/>
     </group_state>
   </xacro:macro>
   <xacro:macro name="franka" params="name">
     <group name="${name}">
-      <joint name="${name}_fr3_joint1"/>
-      <joint name="${name}_fr3_joint2"/>
-      <joint name="${name}_fr3_joint3"/>
-      <joint name="${name}_fr3_joint4"/>
-      <joint name="${name}_fr3_joint5"/>
-      <joint name="${name}_fr3_joint6"/>
-      <joint name="${name}_fr3_joint7"/>
+      <joint name="${name}_joint1"/>
+      <joint name="${name}_joint2"/>
+      <joint name="${name}_joint3"/>
+      <joint name="${name}_joint4"/>
+      <joint name="${name}_joint5"/>
+      <joint name="${name}_joint6"/>
+      <joint name="${name}_joint7"/>
     </group>
     <xacro:franka_group_state

File: clearpath_manipulators_description/urdf/arm/franka.urdf.xacro (robot description, xacro)
@@ -4,4 +4,126 @@
   <xacro:arg name="use_fake_hardware" default="false"/>
   <xacro:arg name="use_manipulation_controllers" default="false"/>
+  <!-- Franka Arm Xacro (without the comments) -->
+  <xacro:macro name="franka_arm" params="arm_id arm_prefix:='' no_prefix:=false description_pkg:='franka_description' connected_to:='base' xyz:='0 0 0' rpy:='0 0 0' gazebo:='false' safety_distance:=0 joint_limits inertials kinematics dynamics with_sc:=false" >
+    <!-- Define a property that defaults to 'arm_prefix_arm_id' concatenated with an underscore if 'no_prefix' is not set -->
+    <xacro:property name="prefix" value="${'' if no_prefix else arm_prefix + arm_id + '_'}" />
+    <xacro:if value="${gazebo}">
+      <xacro:property name="connected_to" value="" />
+    </xacro:if>
+    <xacro:unless value="${not connected_to}">
+      <link name="${connected_to}">
+      </link>
+      <joint name="${prefix}${connected_to}_joint" type="fixed">
+        <parent link="${connected_to}"/>
+        <child link="${prefix}link0"/>
+        <origin rpy="${rpy}" xyz="${xyz}"/>
+      </joint>
+    </xacro:unless>
+    <xacro:link_with_sc no_prefix="${no_prefix}" name="link0" gazebo="${gazebo}" with_sc="${with_sc}">
+      <self_collision_geometries>
+        <xacro:collision_capsule xyz="-0.075 0 0.06" direction="x" radius="${0.06+safety_distance}" length="0.03" />
+      </self_collision_geometries>
+    </xacro:link_with_sc>
+    <xacro:link_with_sc no_prefix="${no_prefix}" name="link1" gazebo="${gazebo}" with_sc="${with_sc}">
+      <self_collision_geometries>
+        <xacro:collision_capsule xyz="0 0 -191.5e-3" radius="${0.06+safety_distance}" length="0.283" />
+      </self_collision_geometries>
+    </xacro:link_with_sc>
+    <joint name="${prefix}joint1" type="revolute">
+      <xacro:franka-kinematics name="joint1" config="${kinematics}" />
+      <parent link="${prefix}link0" />
+      <child link="${prefix}link1" />
+      <axis xyz="0 0 1" />
+      <xacro:franka-limits name="joint1" config="${joint_limits}" />
+      <xacro:franka-dynamics name="joint1" config="${dynamics}" />
+    </joint>
+    <xacro:link_with_sc no_prefix="${no_prefix}" name="link2" gazebo="${gazebo}" with_sc="${with_sc}">
+      <self_collision_geometries>
+        <xacro:collision_capsule xyz="0 0 0" radius="${0.06+safety_distance}" length="0.12" />
+      </self_collision_geometries>
+    </xacro:link_with_sc>
+    <joint name="${prefix}joint2" type="revolute">
+      <xacro:franka-kinematics name="joint2" config="${kinematics}" />
+      <parent link="${prefix}link1" />
+      <child link="${prefix}link2" />
+      <axis xyz="0 0 1" />
+      <xacro:franka-limits name="joint2" config="${joint_limits}" />
+      <xacro:franka-dynamics name="joint2" config="${dynamics}" />
+    </joint>
+    <xacro:link_with_sc no_prefix="${no_prefix}" name="link3" gazebo="${gazebo}" with_sc="${with_sc}">
+      <self_collision_geometries>
+        <xacro:collision_capsule xyz="0 0 -0.145" radius="${0.06+safety_distance}" length="0.15" />
+      </self_collision_geometries>
+    </xacro:link_with_sc>
+    <joint name="${prefix}joint3" type="revolute">
+      <xacro:franka-kinematics name="joint3" config="${kinematics}" />
+      <parent link="${prefix}link2" />
+      <child link="${prefix}link3" />
+      <axis xyz="0 0 1" />
+      <xacro:franka-limits name="joint3" config="${joint_limits}" />
+      <xacro:franka-dynamics name="joint3" config="${dynamics}" />
+    </joint>
+    <xacro:link_with_sc no_prefix="${no_prefix}" name="link4" gazebo="${gazebo}" with_sc="${with_sc}">
+      <self_collision_geometries>
+        <xacro:collision_capsule xyz="0 0 0" radius="${0.06+safety_distance}" length="0.12" />
+     </self_collision_geometries>
+    </xacro:link_with_sc>
+    <joint name="${prefix}joint4" type="revolute">
+      <xacro:franka-kinematics name="joint4" config="${kinematics}" />
+      <parent link="${prefix}link3" />
+      <child link="${prefix}link4" />
+      <axis xyz="0 0 1" />
+      <xacro:franka-limits name="joint4" config="${joint_limits}" />
+      <xacro:franka-dynamics name="joint4" config="${dynamics}" />
+    </joint>
+    <xacro:link_with_sc no_prefix="${no_prefix}" name="link5" gazebo="${gazebo}" with_sc="${with_sc}">
+      <self_collision_geometries>
+        <xacro:collision_capsule xyz="0 0 -0.26"    radius="${0.060+safety_distance}" length="0.10" />
+        <xacro:collision_capsule xyz="0 0.08 -0.13" radius="${0.025+safety_distance}" length="0.14" />
+      </self_collision_geometries>
+    </xacro:link_with_sc>
+    <joint name="${prefix}joint5" type="revolute">
+      <xacro:franka-kinematics name="joint5" config="${kinematics}" />
+      <parent link="${prefix}link4" />
+      <child link="${prefix}link5" />
+      <axis xyz="0 0 1" />
+      <xacro:franka-limits name="joint5" config="${joint_limits}" />
+      <xacro:franka-dynamics name="joint5" config="${dynamics}" />
+    </joint>
+    <xacro:link_with_sc no_prefix="${no_prefix}" name="link6" gazebo="${gazebo}" with_sc="${with_sc}">
+      <self_collision_geometries>
+        <xacro:collision_capsule xyz="0 0 -0.03" radius="${0.05+safety_distance}" length="0.08" />
+      </self_collision_geometries>
+    </xacro:link_with_sc>
+    <joint name="${prefix}joint6" type="revolute">
+      <xacro:franka-kinematics name="joint6" config="${kinematics}" />
+      <parent link="${prefix}link5" />
+      <child link="${prefix}link6" />
+      <axis xyz="0 0 1" />
+      <xacro:franka-limits name="joint6" config="${joint_limits}" />
+      <xacro:franka-dynamics name="joint6" config="${dynamics}" />
+    </joint>
+    <xacro:link_with_sc no_prefix="${no_prefix}" name="link7" gazebo="${gazebo}" rpy="0 0 ${pi/4}" with_sc="${with_sc}">
+      <self_collision_geometries>
+        <xacro:collision_capsule xyz="0 0 0.01" direction="z" radius="${0.04+safety_distance}" length="0.14" />
+        <xacro:collision_capsule xyz="0.06 0 0.082" direction="x" radius="${0.03+safety_distance}"  length="0.01" />
+      </self_collision_geometries>
+    </xacro:link_with_sc>
+    <joint name="${prefix}joint7" type="revolute">
+      <xacro:franka-kinematics name="joint7" config="${kinematics}" />
+      <parent link="${prefix}link6"/>
+      <child link="${prefix}link7"/>
+      <axis xyz="0 0 1"/>
+      <xacro:franka-limits name="joint7" config="${joint_limits}" />
+      <xacro:franka-dynamics name="joint7" config="${dynamics}" />
+    </joint>
+    <link name="${prefix}link8"/>
+    <joint name="${prefix}joint8" type="fixed">
+      <xacro:franka-kinematics name="joint8" config="${kinematics}" />
+      <parent link="${prefix}link7" />
+      <child link="${prefix}link8" />
+    </joint>
+  </xacro:macro>
+  <!-- Franka ROS2 Control -->
   <xacro:macro name="franka_arm_ros2_control"
          params="arm_id
@@ -40,8 +162,4 @@
       <xacro:macro name="configure_joint" params="joint_name initial_position">
         <joint name="${joint_name}">
-          <!--
-            deactivated for gazebo velocity and position interface due to a bug
-            https://github.com/ros-controls/gz_ros2_control/issues/343
-            Command Interfaces -->
           <xacro:unless value="${gazebo and gazebo_effort}">
             <command_interface name="position"/>
@@ -51,5 +169,4 @@
             <command_interface name="effort"/>
           </xacro:if>
-          <!-- State Interfaces -->
           <state_interface name="position">
             <param name="initial_value">${initial_position}</param>
@@ -69,4 +186,5 @@
     </ros2_control>
   </xacro:macro>
+  <!-- Franka Parameters -->
   <xacro:macro name="franka_robot"
               params="arm_id
@@ -92,5 +210,4 @@
                       multi_arm:=false">
     <xacro:include filename="$(find franka_description)/robots/common/utils.xacro" />
-    <xacro:include filename="$(find franka_description)/robots/common/franka_arm.xacro" />
     <xacro:property name="arm_prefix_modified" value="${'' if arm_prefix == '' else arm_prefix + '_'}" />
     <xacro:franka_arm
@@ -238,5 +355,5 @@
     </xacro:if>
     <!-- Fixed Parameters -->
-    <xacro:property name="_hand" value="true" lazy_eval="false"/>
+    <xacro:property name="_hand" value="false" lazy_eval="false"/>
     <xacro:property name="_ee_id" value="franka_hand" lazy_eval="false"/>
     <xacro:property name="_multi_arm" value="false" lazy_eval="false"/>
@@ -253,8 +370,8 @@
     <xacro:franka_robot
       arm_id="${_arm_id}"
-      joint_limits="${xacro.load_yaml('$(find franka_description)/robots/' + arm_id + '/joint_limits.yaml')}"
-      inertials="${xacro.load_yaml('$(find franka_description)/robots/' + arm_id + '/inertials.yaml')}"
-      kinematics="${xacro.load_yaml('$(find franka_description)/robots/' + arm_id + '/kinematics.yaml')}"
-      dynamics="${xacro.load_yaml('$(find franka_description)/robots/' + arm_id + '/dynamics.yaml')}"
+      joint_limits="${_joint_limits}"
+      inertials="${_inertials}"
+      kinematics="${_kinematics}"
+      dynamics="${_dynamics}"
       gazebo="${_gazebo}"
       hand="${_hand}"
