Commit message: Add `rgba` parameter to links so additional shapes aren't always dark grey

File: clearpath_platform_description/urdf/links/box.urdf.xacro (robot description, xacro)
@@ -1,5 +1,5 @@
 <?xml version="1.0"?>
 <robot xmlns:xacro="http://ros.org/wiki/xacro">
-  <xacro:macro name="box" params="name parent_link size *origin">
+  <xacro:macro name="box" params="name parent_link size rgba *origin">
     <link name="${name}_link">
       <visual>
@@ -7,5 +7,7 @@
           <box size="${size}"/>
         </geometry>
-        <material name="clearpath_dark_grey"/>
+        <material name="${name}_rgba">
+          <color rgba="${rgba}" />
+        </material>
       </visual>
       <collision>
@@ -13,5 +15,4 @@
           <box size="${size}"/>
         </geometry>
-        <material name="clearpath_dark_grey"/>
       </collision>
     </link>

File: clearpath_platform_description/urdf/links/cylinder.urdf.xacro (robot description, xacro)
@@ -1,5 +1,5 @@
 <?xml version="1.0"?>
 <robot xmlns:xacro="http://ros.org/wiki/xacro">
-  <xacro:macro name="cylinder" params="name parent_link radius length *origin">
+  <xacro:macro name="cylinder" params="name parent_link radius length rgba *origin">
     <link name="${name}_link">
       <visual>
@@ -7,5 +7,7 @@
           <cylinder radius="${radius}" length="${length}"/>
         </geometry>
-        <material name="clearpath_dark_grey"/>
+        <material name="${name}_rgba">
+          <color rgba="${rgba}" />
+        </material>
       </visual>
       <collision>
@@ -13,5 +15,4 @@
           <cylinder radius="${radius}" length="${length}"/>
         </geometry>
-        <material name="clearpath_dark_grey"/>
       </collision>
     </link>

File: clearpath_platform_description/urdf/links/mesh.urdf.xacro (robot description, xacro)
@@ -1,5 +1,5 @@
 <?xml version="1.0"?>
 <robot xmlns:xacro="http://ros.org/wiki/xacro">
-  <xacro:macro name="mesh" params="name parent_link visual *origin">
+  <xacro:macro name="mesh" params="name parent_link visual rgba *origin">
     <link name="${name}_link">
       <visual>
@@ -7,5 +7,7 @@
           <mesh filename="${visual}"/>
         </geometry>
-        <material name="clearpath_dark_grey"/>
+        <material name="${name}_rgba">
+          <color rgba="${rgba}" />
+        </material>
       </visual>
       <collision>
@@ -13,5 +15,4 @@
           <mesh filename="${visual}"/>
         </geometry>
-        <material name="clearpath_dark_grey"/>
       </collision>
     </link>

File: clearpath_platform_description/urdf/links/sphere.urdf.xacro (robot description, xacro)
@@ -1,5 +1,5 @@
 <?xml version="1.0"?>
 <robot xmlns:xacro="http://ros.org/wiki/xacro">
-  <xacro:macro name="sphere" params="name parent_link radius *origin">
+  <xacro:macro name="sphere" params="name parent_link radius rgba *origin">
     <link name="${name}_link">
       <visual>
@@ -7,5 +7,7 @@
           <sphere radius="${radius}"/>
         </geometry>
-        <material name="clearpath_dark_grey"/>
+        <material name="${name}_rgba">
+          <color rgba="${rgba}" />
+        </material>
       </visual>
       <collision>
@@ -13,5 +15,4 @@
           <sphere radius="${radius}"/>
         </geometry>
-        <material name="clearpath_dark_grey"/>
       </collision>
     </link>

Commit message: Add collision attribute to optionally disable collision geometry for links

File: clearpath_platform_description/urdf/links/box.urdf.xacro (robot description, xacro)
@@ -1,5 +1,5 @@
 <?xml version="1.0"?>
 <robot xmlns:xacro="http://ros.org/wiki/xacro">
-  <xacro:macro name="box" params="name parent_link size rgba *origin">
+  <xacro:macro name="box" params="name parent_link size rgba collision *origin">
     <link name="${name}_link">
       <visual>
@@ -11,9 +11,11 @@
         </material>
       </visual>
-      <collision>
-        <geometry>
-          <box size="${size}"/>
-        </geometry>
-      </collision>
+      <xacro:if value="${collision}">
+        <collision>
+          <geometry>
+            <box size="${size}"/>
+          </geometry>
+        </collision>
+      </xacro:if>
     </link>
     <joint name="${name}_joint" type="fixed">

File: clearpath_platform_description/urdf/links/cylinder.urdf.xacro (robot description, xacro)
@@ -1,5 +1,5 @@
 <?xml version="1.0"?>
 <robot xmlns:xacro="http://ros.org/wiki/xacro">
-  <xacro:macro name="cylinder" params="name parent_link radius length rgba *origin">
+  <xacro:macro name="cylinder" params="name parent_link radius length rgba collision *origin">
     <link name="${name}_link">
       <visual>
@@ -11,9 +11,11 @@
         </material>
       </visual>
-      <collision>
-        <geometry>
-          <cylinder radius="${radius}" length="${length}"/>
-        </geometry>
-      </collision>
+      <xacro:if value="${collision}">
+        <collision>
+          <geometry>
+            <cylinder radius="${radius}" length="${length}"/>
+          </geometry>
+        </collision>
+      </xacro:if>
     </link>
     <joint name="${name}_joint" type="fixed">

File: clearpath_platform_description/urdf/links/mesh.urdf.xacro (robot description, xacro)
@@ -1,5 +1,5 @@
 <?xml version="1.0"?>
 <robot xmlns:xacro="http://ros.org/wiki/xacro">
-  <xacro:macro name="mesh" params="name parent_link visual rgba *origin">
+  <xacro:macro name="mesh" params="name parent_link visual rgba collision *origin">
     <link name="${name}_link">
       <visual>
@@ -11,9 +11,11 @@
         </material>
       </visual>
-      <collision>
-        <geometry>
-          <mesh filename="${visual}"/>
-        </geometry>
-      </collision>
+      <xacro:if value="${collision}">
+        <collision>
+          <geometry>
+            <mesh filename="${visual}"/>
+          </geometry>
+        </collision>
+      </xacro:if>
     </link>
     <joint name="${name}_joint" type="fixed">

File: clearpath_platform_description/urdf/links/sphere.urdf.xacro (robot description, xacro)
@@ -1,5 +1,5 @@
 <?xml version="1.0"?>
 <robot xmlns:xacro="http://ros.org/wiki/xacro">
-  <xacro:macro name="sphere" params="name parent_link radius rgba *origin">
+  <xacro:macro name="sphere" params="name parent_link radius rgba collision *origin">
     <link name="${name}_link">
       <visual>
@@ -11,9 +11,11 @@
         </material>
       </visual>
-      <collision>
-        <geometry>
-          <sphere radius="${radius}"/>
-        </geometry>
-      </collision>
+      <xacro:if value="${collision}">
+        <collision>
+          <geometry>
+            <sphere radius="${radius}"/>
+          </geometry>
+        </collision>
+      </xacro:if>
     </link>
     <joint name="${name}_joint" type="fixed">
