Commit message: Add new URDFs from Rhys, add cellular & wifi antennas to the observer arch. Add new wireless charger attachment

File: clearpath_platform_description/urdf/a300/attachments/observer_arch.urdf.xacro (robot description, xacro)
@@ -2,4 +2,7 @@
 <robot xmlns:xacro="http://wiki.ros.org.xacro">
   <xacro:macro name="observer_arch" params="name parent_link:=default_mount model:=observer_arch *origin">
+    <!--
+      Main sensor arch
+    -->
     <link name="${name}_link">
       <visual>
@@ -26,5 +29,50 @@
     </joint>
     <!--
-        Sensor mounting points
+      Standard antennas & accessories
+    -->
+    <link name="${name}_cellular_antenna">
+      <visual>
+        <geometry>
+          <mesh filename="package://clearpath_platform_description/meshes/a300/attachments/observer_cellular_antenna.stl" scale="0.001 0.001 0.001" />
+        </geometry>
+        <material name="clearpath_black" />
+        <origin xyz="0 0 0" rpy="0 0 0" />
+      </visual>
+      <collision>
+        <geometry>
+          <!-- TODO: replace with box -->
+          <mesh filename="package://clearpath_platform_description/meshes/a300/attachments/observer_cellular_antenna.stl" scale="0.001 0.001 0.001" />
+        </geometry>
+        <origin xyz="0 0 0" rpy="0 0 0" />
+      </collision>
+    </link>
+    <joint name="${name}_cellular_antenna_joint" type="fixed">
+      <parent link="${name}_link" />
+      <child link="${name}_cellular_antenna" />
+      <origin xyz="0 0 0" rpy="0 0 0" />
+    </joint>
+    <link name="${name}_wifi_antennas">
+      <visual>
+        <geometry>
+          <mesh filename="package://clearpath_platform_description/meshes/a300/attachments/observer_wifi_antennas.stl" scale="0.001 0.001 0.001" />
+        </geometry>
+        <material name="clearpath_black" />
+        <origin xyz="0 0 0" rpy="0 0 0" />
+      </visual>
+      <collision>
+        <geometry>
+          <!-- TODO: replace with dual cylinders -->
+          <mesh filename="package://clearpath_platform_description/meshes/a300/attachments/observer_wifi_antennas.stl" scale="0.001 0.001 0.001" />
+        </geometry>
+        <origin xyz="0 0 0" rpy="0 0 0" />
+      </collision>
+    </link>
+    <joint name="${name}_wifi_antennas_joint" type="fixed">
+      <parent link="${name}_link" />
+      <child link="${name}_wifi_antennas" />
+      <origin xyz="0 0 0" rpy="0 0 0" />
+    </joint>
+    <!--
+      Sensor mounting points
     -->
     <link name="${name}_left_antenna_mount" />

Commit message: Merge all arch antennas into a single frame, put an oversized box collider around all of it

File: clearpath_platform_description/urdf/a300/attachments/observer_arch.urdf.xacro (robot description, xacro)
@@ -31,5 +31,5 @@
       Standard antennas & accessories
     -->
-    <link name="${name}_cellular_antenna">
+    <link name="${name}_antennas">
       <visual>
         <geometry>
@@ -39,18 +39,4 @@
         <origin xyz="0 0 0" rpy="0 0 0" />
       </visual>
-      <collision>
-        <geometry>
-          <!-- TODO: replace with box -->
-          <mesh filename="package://clearpath_platform_description/meshes/a300/attachments/observer_cellular_antenna.stl" scale="0.001 0.001 0.001" />
-        </geometry>
-        <origin xyz="0 0 0" rpy="0 0 0" />
-      </collision>
-    </link>
-    <joint name="${name}_cellular_antenna_joint" type="fixed">
-      <parent link="${name}_link" />
-      <child link="${name}_cellular_antenna" />
-      <origin xyz="0 0 0" rpy="0 0 0" />
-    </joint>
-    <link name="${name}_wifi_antennas">
       <visual>
         <geometry>
@@ -62,13 +48,13 @@
       <collision>
         <geometry>
-          <!-- TODO: replace with dual cylinders -->
-          <mesh filename="package://clearpath_platform_description/meshes/a300/attachments/observer_wifi_antennas.stl" scale="0.001 0.001 0.001" />
+          <box size="0.170 0.350 0.12" />
         </geometry>
-        <origin xyz="0 0 0" rpy="0 0 0" />
+        <material name="clearpath_black" />
+        <origin xyz="0 0 0.490" rpy="0 0 0" />
       </collision>
     </link>
-    <joint name="${name}_wifi_antennas_joint" type="fixed">
+    <joint name="${name}_antennas_joint" type="fixed">
       <parent link="${name}_link" />
-      <child link="${name}_wifi_antennas" />
+      <child link="${name}_antennas" />
       <origin xyz="0 0 0" rpy="0 0 0" />
     </joint>
