Commit message: Remove the old AMP arch; AMP & Observer use the same arch. Observer -> AMP for attachment names. Remove the lights STL as it wasn't being used

File: clearpath_platform_description/urdf/a300/attachments/amp_enclosure.urdf.xacro (robot description, xacro)
@@ -1,5 +1,5 @@
 <?xml version="1.0" ?>
 <robot xmlns:xacro="http://wiki.ros.org.xacro">
-  <xacro:macro name="observer_backpack" params="name parent_link:=base_link model:=observer_backpack *origin">
+  <xacro:macro name="amp_enclosure" params="name parent_link:=base_link model:=amp_enclosure *origin">
     <link name="${name}_enclosure_link">
       <visual>

File: clearpath_platform_description/urdf/a300/attachments/amp_sensor_arch.urdf.xacro (robot description, xacro)
@@ -1,5 +1,5 @@
 <?xml version="1.0" ?>
 <robot xmlns:xacro="http://wiki.ros.org.xacro">
-  <xacro:macro name="observer_arch" params="name parent_link:=default_mount model:=observer_arch *origin">
+  <xacro:macro name="amp_sensor_arch" params="name parent_link:=default_mount model:=amp_sensor_arch *origin">
     <!--
       Main sensor arch
