Commit message: Add a link to the face of the charger, as this may be useful for docking

File: clearpath_platform_description/urdf/a300/attachments/wireless_charger.urdf.xacro (robot description, xacro)
@@ -23,4 +23,10 @@
             <xacro:insert_block name="origin" />
         </joint>
+        <link name="${name}_face" />
+        <joint name="${name}_face_joint" type="fixed">
+            <parent link="${name}_link" />
+            <child link="${name}_face" />
+            <origin xyz="0 -0.34 0.15" rpy="0 0 0" />
+        </joint>
     </xacro:macro>
 </robot>

Commit message: Rotate the charger face link so the X axis points outward

File: clearpath_platform_description/urdf/a300/attachments/wireless_charger.urdf.xacro (robot description, xacro)
@@ -27,5 +27,5 @@
             <parent link="${name}_link" />
             <child link="${name}_face" />
-            <origin xyz="0 -0.34 0.15" rpy="0 0 0" />
+            <origin xyz="0 -0.34 0.15" rpy="0 0 -${pi / 2}" />
         </joint>
     </xacro:macro>

Commit message: Use a box collider for the wireless charger

File: clearpath_platform_description/urdf/a300/attachments/wireless_charger.urdf.xacro (robot description, xacro)
@@ -12,8 +12,7 @@
         <collision>
             <geometry>
-                <!-- TODO: replace with box -->
-                <mesh filename="package://clearpath_platform_description/meshes/a300/attachments/wireless_charger.stl" scale="0.001 0.001 0.001" />
+                 <box size="0.170 0.145 0.195" />
             </geometry>
-            <origin xyz="0 0 0" rpy="0 0 0" />
+            <origin xyz="0 -0.265 0.18" rpy="0 0 0" />
         </collision>
         </link>
