Commit message: Add the third antenna (bluetooth) to the top of the AMP frame

File: clearpath_platform_description/urdf/a300/attachments/amp_sensor_arch.urdf.xacro (robot description, xacro)
@@ -32,4 +32,11 @@
     -->
     <link name="${name}_antennas">
+      <visual>
+        <geometry>
+          <mesh filename="package://clearpath_platform_description/meshes/a300/attachments/observer_bluetooth_antenna.stl" scale="0.001 0.001 0.001" />
+        </geometry>
+        <material name="clearpath_black" />
+        <origin xyz="0 0 0" rpy="0 0 0" />
+      </visual>
       <visual>
         <geometry>
