Commit message: Dingo-D

File: clearpath_platform_description/urdf/dd100/drivetrain/wheels/indoor.urdf.xacro (robot description, xacro)
@@ -1,10 +1,13 @@
 <?xml version="1.0"?>
-<robot xmlns:xacro="http://ros.org/wiki/xacro" name="dd100_wheel">
-  <xacro:macro name="dd100_wheel" params="prefix *joint_pose">
+<robot xmlns:xacro="http://ros.org/wiki/xacro" name="dd100_indoor_wheel">
+  <xacro:property name="dd100_indoor_wheel_radius" value="0.049" />
+  <xacro:property name="dd100_indoor_wheel_mass" value="0.111" />
+  <xacro:property name="dd100_indoor_wheel_width" value="0.02032" />
+  <xacro:macro name="dd100_indoor_wheel" params="prefix *joint_pose">
     <link name="${prefix}_wheel_link">
       <visual>
         <origin xyz="0 0 0" rpy="0 0 0"/>
         <geometry>
-          <mesh filename="package://clearpath_platform_description/meshes/dd100/wheel.stl"/>
+          <mesh filename="package://clearpath_platform_description/meshes/dd100/wheels/indoor.stl"/>
         </geometry>
         <material name="clearpath_black" />
@@ -13,10 +16,10 @@
         <origin xyz="0 0 0" rpy="${PI/2} 0 0"/>
         <geometry>
-          <cylinder radius="${wheel_radius}" length="${wheel_width}"/>
+          <cylinder radius="${dd100_indoor_wheel_radius}" length="${dd100_indoor_wheel_width}"/>
         </geometry>
       </collision>
       <inertial>
         <origin xyz="0 0 0" rpy="0 0 0"/>
-        <mass value="${wheel_mass}"/>
+        <mass value="${dd100_indoor_wheel_mass}"/>
         <inertia
           ixx="0.0003234" ixy="0" ixz="0"

File: clearpath_platform_description/urdf/do100/drivetrain/wheels.urdf.xacro (robot description, xacro)
@@ -15,5 +15,5 @@
     </xacro:if>
     <xacro:unless value="${front_wheels == 'mecanum'}">
-      <xacro:error message="Invalid DO100 front wheels ${front_wheels}"/>
+      <xacro:error message="Invalid Dingo-O front wheels ${front_wheels}"/>
     </xacro:unless>
     <!-- Rear Wheels -->
@@ -29,5 +29,5 @@
     </xacro:if>
     <xacro:unless value="${rear_wheels == 'mecanum'}">
-      <xacro:error message="Invalid DO100 rear wheels ${rear_wheels}"/>
+      <xacro:error message="Invalid Dingo-O rear wheels ${rear_wheels}"/>
     </xacro:unless>
   </xacro:macro>

Commit message: R100

File: clearpath_platform_description/urdf/dd100/drivetrain/wheels/indoor.urdf.xacro (robot description, xacro)
@@ -28,4 +28,14 @@
       </inertial>
     </link>
+    <gazebo>
+      <plugin filename="libgz-sim-wheel-slip-system.so" name="gz::sim::systems::WheelSlip">
+        <wheel link_name="${prefix}_wheel_link">
+          <slip_compliance_lateral>1.0</slip_compliance_lateral>
+          <slip_compliance_longitudinal>1.0</slip_compliance_longitudinal>
+          <wheel_normal_force>39.2</wheel_normal_force>
+          <wheel_radius>${dd100_indoor_wheel_radius}</wheel_radius>
+        </wheel>
+      </plugin>
+    </gazebo>
     <gazebo reference="${prefix}_wheel_link">
       <material>Gazebo/DarkGrey</material>

File: clearpath_platform_description/urdf/do100/drivetrain/wheels/mecanum.urdf.xacro (robot description, xacro)
@@ -33,5 +33,5 @@
           <slip_compliance_longitudinal>1.0</slip_compliance_longitudinal>
           <wheel_normal_force>20</wheel_normal_force>
-          <do100_mecanum_wheel_radius>${do100_mecanum_wheel_radius}</do100_mecanum_wheel_radius>
+          <wheel_radius>${do100_mecanum_wheel_radius}</wheel_radius>
         </wheel>
       </plugin>

File: clearpath_platform_description/urdf/r100/r100.urdf.xacro (robot description, xacro)
@@ -3,14 +3,8 @@
   <xacro:arg name="namespace" default="" />
   <xacro:arg name="is_sim" default="false" />
-  <xacro:arg name="gazebo_controllers" default="$(find clearpath_control)/config/r100/control.yaml"/>
-  <!-- Includes -->
-  <xacro:include filename="$(find clearpath_platform_description)/urdf/r100/wheels/wheel.urdf.xacro"/>
-  <xacro:include filename="$(find clearpath_platform_description)/urdf/r100/rocker.urdf.xacro"/>
+  <xacro:arg name="gazebo_controllers" default="$(find clearpath_control)/config/r100/control/omni_4wd.yaml"/>
   <!-- R100 Platform Macro -->
-  <xacro:macro name="r100" params="wheel:='defaut'">
+  <xacro:macro name="r100" params="control:='omni_4wd' front_wheels:='mecanum' rear_wheels:='mecanum'">
     <!-- Variables -->
-    <xacro:property name="wheel_radius" value="0.0759" />
-    <xacro:property name="wheel_width" value="0.0790" />
-    <xacro:property name="wheel_mass" value="2.5" />
     <xacro:property name="chassis_length" value="0.960" />
     <xacro:property name="chassis_width" value="0.793" />
@@ -199,39 +193,26 @@
       </collision>
     </link>
-    <!-- Rocker -->
-    <xacro:r100_rocker prefix="front" joint_type="fixed" location="1" >
-      <limit lower="-0.08726" upper="0.08726" effort="0" velocity="0" />
-    </xacro:r100_rocker>
-    <xacro:r100_rocker prefix="rear" joint_type="fixed" location="-1" >
-      <limit effort="0" velocity="0" />
-    </xacro:r100_rocker>
-    <gazebo>
-      <plugin filename="libgz-sim-wheel-slip-system.so" name="gz::sim::systems::WheelSlip">
-        <wheel link_name="front_left_wheel_link">
-          <slip_compliance_lateral>1.0</slip_compliance_lateral>
-          <slip_compliance_longitudinal>1.0</slip_compliance_longitudinal>
-          <wheel_normal_force>200</wheel_normal_force>
-          <wheel_radius>${wheel_radius}</wheel_radius>
-        </wheel>
-        <wheel link_name="front_right_wheel_link">
-          <slip_compliance_lateral>1.0</slip_compliance_lateral>
-          <slip_compliance_longitudinal>1.0</slip_compliance_longitudinal>
-          <wheel_normal_force>200</wheel_normal_force>
-          <wheel_radius>${wheel_radius}</wheel_radius>
-        </wheel>
-        <wheel link_name="rear_left_wheel_link">
-          <slip_compliance_lateral>1.0</slip_compliance_lateral>
-          <slip_compliance_longitudinal>1.0</slip_compliance_longitudinal>
-          <wheel_normal_force>200</wheel_normal_force>
-          <wheel_radius>${wheel_radius}</wheel_radius>
-        </wheel>
-        <wheel link_name="rear_right_wheel_link">
-          <slip_compliance_lateral>1.0</slip_compliance_lateral>
-          <slip_compliance_longitudinal>1.0</slip_compliance_longitudinal>
-          <wheel_normal_force>200</wheel_normal_force>
-          <wheel_radius>${wheel_radius}</wheel_radius>
-        </wheel>
-      </plugin>
-    </gazebo>
+    <!-- Add wheels -->
+    <xacro:include filename="$(find clearpath_platform_description)/urdf/r100/drivetrain/wheels.urdf.xacro"/>
+    <xacro:r100_drivetrain_wheels front_wheels="${front_wheels}" rear_wheels="${rear_wheels}"/>
+    <!-- Add drivetrain -->
+    <xacro:include filename="$(find clearpath_platform_description)/urdf/generic/drivetrain/drivetrain.urdf.xacro"/>
+    <!-- Hardware  -->
+    <xacro:if value="$(arg is_sim)">
+      <xacro:property name="hardware_plugin" value="gz_ros2_control/GazeboSimSystem"/>
+    </xacro:if>
+    <xacro:unless value="$(arg is_sim)">
+      <xacro:property name="hardware_plugin" value="clearpath_hardware_interfaces/PumaHardware"/>
+    </xacro:unless>
+    <xacro:unless value="${control == 'omni_4wd' or control == 'diff_4wd'}">
+      <xacro:error message="Invalid drivetrain control ${control}"/>
+    </xacro:unless>
+    <xacro:generic_drivetrain
+      name="r100"
+      control="${control}"
+      front_wheels="${front_wheels}"
+      rear_wheels="${rear_wheels}"
+      hardware_plugin="${hardware_plugin}"
+    />
     <!-- Internal IMU -->
     <link name="imu_0_link">
@@ -262,37 +243,4 @@
       <origin xyz="0 0 ${riser_height + deck_thickness}" rpy="0 0 0"/>
     </joint>
-    <!-- Gazebo Controller -->
-    <xacro:include filename="$(find clearpath_platform_description)/urdf/generic/gazebo.urdf.xacro"/>
-    <!-- ROS2 controls -->
-    <ros2_control name="r100_hardware" type="system">
-      <hardware>
-        <xacro:if value="$(arg is_sim)">
-          <plugin>gz_ros2_control/GazeboSimSystem</plugin>
-        </xacro:if>
-        <xacro:unless value="$(arg is_sim)">
-          <plugin>clearpath_hardware_interfaces/PumaHardware</plugin>
-        </xacro:unless>
-      </hardware>
-      <joint name="front_left_wheel_joint">
-        <command_interface name="velocity"/>
-        <state_interface name="position"/>
-        <state_interface name="velocity"/>
-      </joint>
-      <joint name="front_right_wheel_joint">
-        <command_interface name="velocity"/>
-        <state_interface name="position"/>
-        <state_interface name="velocity"/>
-      </joint>
-      <joint name="rear_left_wheel_joint">
-        <command_interface name="velocity"/>
-        <state_interface name="position"/>
-        <state_interface name="velocity"/>
-      </joint>
-      <joint name="rear_right_wheel_joint">
-        <command_interface name="velocity"/>
-        <state_interface name="position"/>
-        <state_interface name="velocity"/>
-      </joint>
-    </ros2_control>
   </xacro:macro>
 </robot>
