Commit message: Separated caster wheel into swivel and wheel links

File: clearpath_platform_description/urdf/a300/drivetrain/wheels/caster.urdf.xacro (robot description, xacro)
@@ -5,12 +5,44 @@
   <xacro:property name="a300_caster_wheel_width" value="0.05" />
   <xacro:macro name="a300_caster_wheel" params="prefix side">
-    <xacro:property name="mesh"
-      value="${'primary' if ((prefix == 'front' and side == 'right') or (prefix == 'rear' and side == 'left')) else 'secondary'}"/>
     <xacro:property name="rotation_yaw" value="${math.pi if prefix == 'rear' else 0}"/>
-    <link name="${prefix}_${side}_wheel_mount"/>
-    <joint name="${prefix}_${side}_wheel_mount_joint" type="fixed">
+    <link name="${prefix}_${side}_bracket_plate_link">
+      <visual>
+        <origin xyz="0 0 0" rpy="${math.pi / 2} 0 ${-math.pi / 2}"/>
+        <material name="clearpath_dark_grey"/>
+        <geometry>
+          <mesh filename="package://clearpath_platform_description/meshes/a300/drivetrain/caster_bracket_plate.stl" />
+        </geometry>
+      </visual>
+    </link>
+    <joint name="${prefix}_${side}_bracket_plate_joint" type="fixed">
       <parent link="${prefix}_${side}_flange_mount"/>
-      <child link="${prefix}_${side}_wheel_mount"/>
+      <child link="${prefix}_${side}_bracket_plate_link"/>
     </joint>
+    <link name="${prefix}_${side}_bracket_swivel_link">
+      <inertial>
+        <mass value="0.5" />
+        <origin xyz="0 0 0" />
+        <inertia
+          ixx="0.01" ixy="0" ixz="0"
+          iyy="0.01" iyz="0"
+          izz="0.01" />
+      </inertial>
+      <visual>
+        <origin xyz="0 0 0" rpy="${math.pi / 2} 0 ${-math.pi / 2}"/>
+        <material name="clearpath_dark_grey"/>
+        <geometry>
+          <mesh filename="package://clearpath_platform_description/meshes/a300/drivetrain/caster_bracket_swivel.stl" />
+        </geometry>
+      </visual>
+    </link>
+    <joint name="${prefix}_${side}_bracket_swivel_joint" type="fixed">
+      <parent link="${prefix}_${side}_bracket_plate_link"/>
+      <child link="${prefix}_${side}_bracket_swivel_link"/>
+      <origin xyz="0 0 -0.006237119"/>
+      <axis xyz="0 0 1"/>
+    </joint>
+    <gazebo reference="${prefix}_${side}_bracket_swivel_joint">
+      <springStiffness>0.5</springStiffness>
+    </gazebo>
     <link name="${prefix}_${side}_wheel_link">
       <inertial>
@@ -36,4 +68,15 @@
       </collision>
     </link>
+    <gazebo reference="${prefix}_${side}_wheel_link">
+      <turnGravityOff>false</turnGravityOff>
+      <kp>1000000.0</kp>
+      <kd>100.0</kd>
+      <mu1>0.05</mu1>
+      <mu2>0.05</mu2>
+      <fdir1>1 0 0</fdir1>
+      <minDepth>0.00</minDepth>
+      <implicitSpringDamper>1</implicitSpringDamper>
+    </gazebo>
+<!--
     <gazebo>
       <plugin filename="libgz-sim-wheel-slip-system.so" name="gz::sim::systems::WheelSlip">
@@ -41,14 +84,14 @@
           <slip_compliance_lateral>1.0</slip_compliance_lateral>
           <slip_compliance_longitudinal>1.0</slip_compliance_longitudinal>
-          <wheel_normal_force>113</wheel_normal_force>
+          <wheel_normal_force>0</wheel_normal_force>
           <wheel_radius>${a300_caster_wheel_radius}</wheel_radius>
         </wheel>
       </plugin>
-    </gazebo>
+    </gazebo> -->
     <joint name="${prefix}_${side}_wheel_joint" type="continuous">
-      <parent link="${prefix}_${side}_wheel_mount"/>
+      <parent link="${prefix}_${side}_bracket_swivel_link"/>
       <child link="${prefix}_${side}_wheel_link"/>
-      <origin xyz="-0.054 0 -0.115" rpy="0 0 0"/>
-      <axis xyz="1 1 0" rpy="0 0 0" />
+      <origin xyz="-0.054 0 -0.108762881" rpy="0 0 0"/>
+      <axis xyz="0 1 0"/>
     </joint>
   </xacro:macro>

File: clearpath_platform_description/urdf/a300/drivetrain/wheels/mecanum.urdf.xacro (robot description, xacro)
@@ -1,4 +1,4 @@
 <?xml version="1.0"?>
-<robot xmlns:xacro="http://ros.org/wiki/xacro" name="a300_mecanum_wheel">
+<robot xmlns:xacro="http://ros.org/wiki/xacro" name="a300_mecanum_wheel" xmlns:gz="http://gazebosim.org/schema">
   <xacro:property name="a300_mecanum_wheel_radius" value="0.1524" />
   <xacro:property name="a300_mecanum_wheel_mass" value="2.5" />
@@ -7,4 +7,5 @@
     <xacro:property name="mesh"
       value="${'primary' if ((prefix == 'front' and side == 'left') or (prefix == 'rear' and side == 'right')) else 'secondary'}"/>
+    <xacro:property name="fdir_side" value="${1 if side == 'left' else -1}"/>
     <link name="${prefix}_${side}_wheel_link">
       <inertial>
@@ -40,4 +41,17 @@
       </plugin>
     </gazebo>
+    <gazebo reference="${prefix}_wheel_link">
+      <collision>
+        <surface>
+          <friction>
+            <ode>
+              <mu>1.0</mu>
+              <mu2>0.0</mu2>
+              <fdir1 gz:expressed_in="base_link">1 ${fdir_side} 0</fdir1>
+            </ode>
+          </friction>
+        </surface>
+      </collision>
+    </gazebo>
     <joint name="${prefix}_${side}_wheel_joint" type="continuous">
       <parent link="${prefix}_${side}_motor_mount"/>

File: clearpath_platform_description/urdf/a300/drivetrain/wheels/outdoor.urdf.xacro (robot description, xacro)
@@ -31,6 +31,6 @@
       <plugin filename="libgz-sim-wheel-slip-system.so" name="gz::sim::systems::WheelSlip">
         <wheel link_name="${prefix}_${side}_wheel_link">
-          <slip_compliance_lateral>1.0</slip_compliance_lateral>
-          <slip_compliance_longitudinal>1.0</slip_compliance_longitudinal>
+          <slip_compliance_lateral>0.75</slip_compliance_lateral>
+          <slip_compliance_longitudinal>0.75</slip_compliance_longitudinal>
           <wheel_normal_force>113</wheel_normal_force>
           <wheel_radius>${a300_outdoor_wheel_radius}</wheel_radius>
