Commit message: Fix: Made the A300 caster joint fixed.

File: clearpath_platform_description/urdf/a300/drivetrain/wheels/caster.urdf.xacro (robot description, xacro)
@@ -89,9 +89,8 @@
       </plugin>
     </gazebo> -->
-    <joint name="${prefix}_${side}_wheel_joint" type="continuous">
+    <joint name="${prefix}_${side}_wheel_joint" type="fixed">
       <parent link="${prefix}_${side}_bracket_swivel_link"/>
       <child link="${prefix}_${side}_wheel_link"/>
       <origin xyz="-0.054 0 -0.108762881" rpy="0 0 0"/>
-      <axis xyz="0 1 0"/>
     </joint>
   </xacro:macro>
