Commit message: W200 drivetrain urdf

File: clearpath_platform_description/urdf/w200/drivetrain/wheels/tracks.urdf.xacro (robot description, xacro)
@@ -1,5 +1,8 @@
 <?xml version="1.0"?>
-<robot xmlns:xacro="http://ros.org/wiki/xacro" name="w200_track">
-  <xacro:macro name="w200_track" params="prefix side *joint_pose">
+<robot xmlns:xacro="http://ros.org/wiki/xacro" name="w200_tracks">
+  <xacro:property name="w200_tracks_radius" value="0.3" />
+  <xacro:property name="w200_tracks_mass" value="15.0" />
+  <xacro:property name="w200_tracks_width" value="0.25" />
+  <xacro:macro name="w200_tracks" params="prefix side *joint_pose">
     <xacro:property name="rotate" value="${(prefix=='rear')*math.pi}"/>
     <link name="${prefix}_${side}_track_link">
@@ -7,5 +10,5 @@
         <origin xyz="0 0 0" rpy="0 0 0"/>
         <geometry>
-          <mesh filename="package://clearpath_platform_description/meshes/w200/tracks.dae" />
+          <mesh filename="package://clearpath_platform_description/meshes/w200/wheels/tracks.dae" />
         </geometry>
         <material name="clearpath_dark_grey" />
@@ -34,11 +37,11 @@
       <inertial>
         <origin xyz="0 0 0" rpy="0 0 0" />
-        <mass value="${wheel_mass}" />
-        <xacro:wheel_inertia m="${wheel_mass}" r="${wheel_radius}" h="${wheel_width}" />
+        <mass value="${w200_tracks_mass}" />
+        <xacro:wheel_inertia m="${w200_tracks_mass}" r="${w200_tracks_radius}" h="${w200_tracks_width}" />
       </inertial>
       <collision>
         <origin xyz="0 0 0" rpy="${PI/2} 0 0"/>
         <geometry>
-          <cylinder radius="${wheel_radius*wheel_to_track_ratio}" length="${wheel_width}"/>
+          <cylinder radius="${w200_tracks_radius*wheel_to_track_ratio}" length="${w200_tracks_width}"/>
         </geometry>
       </collision>
@@ -50,4 +53,14 @@
       <axis xyz="0 1 0"/>
     </joint>
+    <gazebo>
+      <plugin filename="libgz-sim-wheel-slip-system.so" name="gz::sim::systems::WheelSlip">
+        <wheel link_name="${prefix}_${side}_wheel_link">
+          <slip_compliance_lateral>1.0</slip_compliance_lateral>
+          <slip_compliance_longitudinal>1.0</slip_compliance_longitudinal>
+          <wheel_normal_force>686</wheel_normal_force>
+          <wheel_radius>${w200_tracks_radius}</wheel_radius>
+        </wheel>
+      </plugin>
+    </gazebo>
     <gazebo reference="${prefix}_${side}_wheel_link">
       <selfCollide>false</selfCollide>
