Commit message: A300 urdf

File: clearpath_platform_description/urdf/a300/a300.urdf.xacro (robot description, xacro)
@@ -5,15 +5,31 @@
   <xacro:arg name="gazebo_controllers" default="$(find clearpath_control)/config/a300/control.yaml"/>
   <xacro:arg name="use_platform_controllers" default="true"/>
-  <!-- Included URDF/XACRO Files -->
-  <xacro:include filename="$(find clearpath_platform_description)/urdf/a300/mobility/diff_drive.urdf.xacro" />
   <!-- Global Variables -->
   <xacro:property name="M_PI" value="${math.pi}"/>
-  <xacro:macro name="a300" params="wheel:='default'">
-    <!-- Base Size -->
-    <xacro:property name="base_mass" value="70"/>
-    <xacro:property name="base_x_size" value="0.860"/>
-    <xacro:property name="base_y_size" value="0.378"/>
-    <xacro:property name="base_z_size" value="0.229559"/>
-    <xacro:property name="base_z_narrow" value="0.0568"/>
+  <xacro:macro name="a300" params="control:='diff_4wd' front_wheels:='outdoor' rear_wheels:='outdoor'">
+    <!-- Chassis Size -->
+    <xacro:property name="chassis_mass" value="70"/>
+    <xacro:property name="chassis_x_size" value="0.860"/>
+    <xacro:property name="chassis_y_size" value="0.378"/>
+    <xacro:property name="chassis_z_size" value="0.229559"/>
+    <!-- Wheel base and track  -->
+    <xacro:property name="wheel_base" value="0.512"/>
+    <xacro:property name="wheel_track" value="0.562"/>
+    <!-- Chassis Positions relative to center of rotation -->
+    <xacro:if value="${control == 'diff_4wd' or control == 'omni_4wd'}">
+      <xacro:property name="chassis_x" value="0"/>
+      <xacro:property name="chassis_y" value="0"/>
+      <xacro:property name="chassis_z" value="0"/>
+    </xacro:if>
+    <xacro:if value="${control == 'diff_fwd'}">
+      <xacro:property name="chassis_x" value="${-wheel_base / 2}"/>
+      <xacro:property name="chassis_y" value="0"/>
+      <xacro:property name="chassis_z" value="0"/>
+    </xacro:if>
+    <xacro:if value="${control == 'diff_rwd'}">
+      <xacro:property name="chassis_x" value="${wheel_base / 2}"/>
+      <xacro:property name="chassis_y" value="0"/>
+      <xacro:property name="chassis_z" value="0"/>
+    </xacro:if>
     <!-- Bumper Mounting Positions -->
     <xacro:property name="bumper_x" value="0.368500"/>
@@ -23,7 +39,9 @@
     <xacro:property name="top_x" value="0.0"/>
     <xacro:property name="top_y" value="0.0"/>
-    <xacro:property name="top_z" value="${base_z_size}"/>
-    <!-- Base Link: center of the bottom of the robot -->
-    <link name="base_link">
+    <xacro:property name="top_z" value="${chassis_z_size}"/>
+    <!-- Base Link: center of rotation at the bottom of the robot -->
+    <link name="base_link"/>
+    <!-- Chassis Link: center of the bottom of the robot chassis -->
+    <link name="chassis_link">
       <visual>
         <geometry>
@@ -48,13 +66,18 @@
       </collision>
       <inertial>
-        <mass value="${base_mass}"/>
-        <origin xyz="0 0 ${base_z_size/2}" rpy="0 0 0"/>
+        <mass value="${chassis_mass}"/>
+        <origin xyz="0 0 ${chassis_z_size/2}" rpy="0 0 0"/>
         <inertia
-          ixx="${ base_mass/12 * (base_y_size**2 + base_z_size**2) }" ixy="0" ixz="0"
-          iyy="${ base_mass/12 * (base_x_size**2 + base_z_size**2) }" iyz="0"
-          izz="${ base_mass/12 * (base_x_size**2 + base_y_size**2) }"
+          ixx="${ chassis_mass/12 * (chassis_y_size**2 + chassis_z_size**2) }" ixy="0" ixz="0"
+          iyy="${ chassis_mass/12 * (chassis_x_size**2 + chassis_z_size**2) }" iyz="0"
+          izz="${ chassis_mass/12 * (chassis_x_size**2 + chassis_y_size**2) }"
         />
       </inertial>
     </link>
+    <joint name="chassis_joint" type="fixed">
+      <child link="chassis_link"/>
+      <parent link="base_link"/>
+      <origin xyz="${chassis_x} ${chassis_y} ${chassis_z}" rpy="0 0 0"/>
+    </joint>
     <!-- Bumper Mounts -->
     <link name="front_bumper_mount"/>
@@ -62,10 +85,10 @@
     <joint name="front_bumper_mount_joint" type="fixed">
       <child link="front_bumper_mount"/>
-      <parent link="base_link"/>
+      <parent link="chassis_link"/>
       <origin xyz="${bumper_x} ${bumper_y} ${bumper_z}" rpy="0 0 0"/>
     </joint>
     <joint name="rear_bumper_mount_joint" type="fixed">
       <child link="rear_bumper_mount"/>
-      <parent link="base_link"/>
+      <parent link="chassis_link"/>
       <origin xyz="${-bumper_x} ${bumper_y} ${bumper_z}" rpy="0 0 ${math.pi}"/>
     </joint>
@@ -74,11 +97,79 @@
     <joint name="default_mount_joint" type="fixed">
       <child link="default_mount"/>
-      <parent link="base_link"/>
+      <parent link="chassis_link"/>
       <origin xyz="${top_x} ${top_y} ${top_z}"/>
     </joint>
-    <!-- Gazebo Controller -->
-    <xacro:include filename="$(find clearpath_platform_description)/urdf/generic/gazebo.urdf.xacro"/>
-    <!-- Mobility Kit -->
-    <xacro:mobility_diff_drive wheel='${wheel}'/>
+    <!-- Suspension beams -->
+    <link name="left_suspension_beam_link">
+      <visual>
+        <material name="clearpath_dark_grey"/>
+        <geometry>
+          <mesh filename="package://clearpath_platform_description/meshes/a300/mobility/suspension_beam.dae" />
+        </geometry>
+      </visual>
+      <collision>
+        <geometry>
+          <mesh filename="package://clearpath_platform_description/meshes/a300/mobility/diff_drive_collision.stl" />
+        </geometry>
+      </collision>
+    </link>
+    <joint name="left_suspension_beam_joint" type="fixed">
+      <parent link="chassis_link"/>
+      <child link="left_suspension_beam_link"/>
+      <origin xyz="0 0 0" rpy="0 0 ${math.pi}" />
+    </joint>
+    <link name="right_suspension_beam_link">
+      <visual>
+        <material name="clearpath_dark_grey"/>
+        <geometry>
+          <mesh filename="package://clearpath_platform_description/meshes/a300/mobility/suspension_beam.dae" />
+        </geometry>
+      </visual>
+      <collision>
+        <geometry>
+          <mesh filename="package://clearpath_platform_description/meshes/a300/mobility/diff_drive_collision.stl" />
+        </geometry>
+      </collision>
+    </link>
+    <joint name="right_suspension_beam_joint" type="fixed">
+      <parent link="chassis_link"/>
+      <child link="right_suspension_beam_link"/>
+      <origin xyz="0 0 0" rpy="0 0 0" />
+    </joint>
+    <!-- Add wheels -->
+    <xacro:include filename="$(find clearpath_platform_description)/urdf/a300/drivetrain/wheels.urdf.xacro"/>
+    <xacro:a300_drivetrain_wheels front_wheels="${front_wheels}" rear_wheels="${rear_wheels}"/>
+    <!-- Add drivetrain -->
+    <xacro:include filename="$(find clearpath_platform_description)/urdf/generic/drivetrain/drivetrain.urdf.xacro"/>
+    <!-- Hardware  -->
+    <xacro:if value="$(arg is_sim)">
+      <xacro:property name="hardware_plugin" value="gz_ros2_control/GazeboSimSystem"/>
+    </xacro:if>
+    <xacro:unless value="$(arg is_sim)">
+      <xacro:property name="hardware_plugin" value="clearpath_hardware_interfaces/LynxHardware"/>
+    </xacro:unless>
+    <xacro:generic_drivetrain
+      name="a300"
+      control="${control}"
+      front_wheels="${front_wheels}"
+      rear_wheels="${rear_wheels}"
+      hardware_plugin="${hardware_plugin}"
+    />
+    <!-- Base Footprint: on the ground below the robot -->
+    <link name="base_footprint"/>
+    <xacro:if value="${control == 'diff_4wd' or control == 'omni_4wd' or control == 'diff_fwd'}">
+      <joint name="base_footprint_joint" type="fixed">
+        <origin xyz="0 0 ${front_wheel_radius}" rpy="0 0 0" />
+        <parent link="chassis_link" />
+        <child link="base_footprint" />
+      </joint>
+    </xacro:if>
+    <xacro:if value="${control == 'diff_rwd'}">
+      <joint name="base_footprint_joint" type="fixed">
+        <origin xyz="0 0 ${rear_wheel_radius}" rpy="0 0 0" />
+        <parent link="chassis_link" />
+        <child link="base_footprint" />
+      </joint>
+    </xacro:if>
   </xacro:macro>
 </robot>

Commit message: Updated A300 meshes Mecanum and caster support

File: clearpath_platform_description/urdf/a300/a300.urdf.xacro (robot description, xacro)
@@ -32,4 +32,8 @@
       <xacro:property name="chassis_z" value="0"/>
     </xacro:if>
+    <!-- Suspension Beam Mounting Positions -->
+    <xacro:property name="chassis_suspension_mount_x" value="0.0"/>
+    <xacro:property name="chassis_suspension_mount_y" value="0.192"/>
+    <xacro:property name="chassis_suspension_mount_z" value="0.03763"/>
     <!-- Bumper Mounting Positions -->
     <xacro:property name="bumper_x" value="0.368500"/>
@@ -80,4 +84,16 @@
       <origin xyz="${chassis_x} ${chassis_y} ${chassis_z}" rpy="0 0 0"/>
     </joint>
+    <link name="chassis_left_suspension_mount"/>
+    <link name="chassis_right_suspension_mount"/>
+    <joint name="chassis_left_suspension_mount_joint" type="fixed">
+      <child link="chassis_left_suspension_mount"/>
+      <parent link="chassis_link"/>
+      <origin xyz="${chassis_suspension_mount_x} ${chassis_suspension_mount_y} ${chassis_suspension_mount_z}" rpy="0 0 0"/>
+    </joint>
+    <joint name="chassis_right_suspension_mount_joint" type="fixed">
+      <child link="chassis_right_suspension_mount"/>
+      <parent link="chassis_link"/>
+      <origin xyz="${chassis_suspension_mount_x} ${-chassis_suspension_mount_y} ${chassis_suspension_mount_z}" rpy="0 0 0"/>
+    </joint>
     <!-- Bumper Mounts -->
     <link name="front_bumper_mount"/>
@@ -101,40 +117,7 @@
     </joint>
     <!-- Suspension beams -->
-    <link name="left_suspension_beam_link">
-      <visual>
-        <material name="clearpath_dark_grey"/>
-        <geometry>
-          <mesh filename="package://clearpath_platform_description/meshes/a300/mobility/suspension_beam.dae" />
-        </geometry>
-      </visual>
-      <collision>
-        <geometry>
-          <mesh filename="package://clearpath_platform_description/meshes/a300/mobility/diff_drive_collision.stl" />
-        </geometry>
-      </collision>
-    </link>
-    <joint name="left_suspension_beam_joint" type="fixed">
-      <parent link="chassis_link"/>
-      <child link="left_suspension_beam_link"/>
-      <origin xyz="0 0 0" rpy="0 0 ${math.pi}" />
-    </joint>
-    <link name="right_suspension_beam_link">
-      <visual>
-        <material name="clearpath_dark_grey"/>
-        <geometry>
-          <mesh filename="package://clearpath_platform_description/meshes/a300/mobility/suspension_beam.dae" />
-        </geometry>
-      </visual>
-      <collision>
-        <geometry>
-          <mesh filename="package://clearpath_platform_description/meshes/a300/mobility/diff_drive_collision.stl" />
-        </geometry>
-      </collision>
-    </link>
-    <joint name="right_suspension_beam_joint" type="fixed">
-      <parent link="chassis_link"/>
-      <child link="right_suspension_beam_link"/>
-      <origin xyz="0 0 0" rpy="0 0 0" />
-    </joint>
+    <xacro:include filename="$(find clearpath_platform_description)/urdf/a300/drivetrain/suspension_beam.urdf.xacro"/>
+    <xacro:a300_suspension_beam side="left"/>
+    <xacro:a300_suspension_beam side="right"/>
     <!-- Add wheels -->
     <xacro:include filename="$(find clearpath_platform_description)/urdf/a300/drivetrain/wheels.urdf.xacro"/>

File: clearpath_platform_description/urdf/a300/drivetrain/motor.urdf.xacro (robot description, xacro)
@@ -1,23 +1,32 @@
 <?xml version="1.0"?>
 <robot xmlns:xacro="http://ros.org/wiki/xacro" name="a300_motor">
-  <xacro:macro name="a300_motor" params="prefix *joint_pose">
-    <link name="${prefix}_motor_link">
-        <visual>
-          <material name="clearpath_dark_grey"/>
-          <geometry>
-            <mesh filename="package://clearpath_platform_description/meshes/a300/mobility/motor.dae" />
-          </geometry>
-        </visual>
-        <collision>
-          <geometry>
-            <mesh filename="package://clearpath_platform_description/meshes/a300/mobility/motor.dae" />
-          </geometry>
-        </collision>
-      </link>
-      <joint name="${prefix}_motor_joint" type="fixed">
-        <parent link="chassis_link"/>
-        <child link="${prefix}_motor_link"/>
-        <xacro:insert_block name="joint_pose"/>
-      </joint>
+  <xacro:macro name="a300_motor" params="prefix side">
+    <xacro:property name="rotation_yaw" value="${math.pi if side == 'left' else 0}"/>
+    <xacro:property name="translation_y" value="${0.0655 if side == 'left' else -0.0655}"/>
+    <link name="${prefix}_${side}_motor_link">
+      <visual>
+        <material name="clearpath_dark_grey"/>
+        <geometry>
+          <mesh filename="package://clearpath_platform_description/meshes/a300/drivetrain/motor.stl"/>
+        </geometry>
+        <origin rpy="0 0 ${rotation_yaw}"/>
+      </visual>
+      <collision>
+        <geometry>
+          <mesh filename="package://clearpath_platform_description/meshes/a300/drivetrain/motor.stl"/>
+        </geometry>
+      </collision>
+    </link>
+    <joint name="${prefix}_${side}_motor_joint" type="fixed">
+      <parent link="${side}_suspension_beam_${prefix}_mount"/>
+      <child link="${prefix}_${side}_motor_link"/>
+      <origin rpy="0 0 0"/>
+    </joint>
+    <link name="${prefix}_${side}_motor_mount"/>
+    <joint name="${prefix}_${side}_motor_mount_joint" type="fixed">
+      <parent link="${prefix}_${side}_motor_link"/>
+      <child link="${prefix}_${side}_motor_mount"/>
+      <origin xyz="0 ${translation_y} 0"/>
+    </joint>
   </xacro:macro>
 </robot>

File: clearpath_platform_description/urdf/a300/drivetrain/wheels.urdf.xacro (robot description, xacro)
@@ -3,53 +3,70 @@
   <xacro:macro name="a300_drivetrain_wheels" params="front_wheels rear_wheels">
     <xacro:include filename="$(find clearpath_platform_description)/urdf/a300/drivetrain/wheels/outdoor.urdf.xacro" />
+    <xacro:include filename="$(find clearpath_platform_description)/urdf/a300/drivetrain/wheels/mecanum.urdf.xacro" />
+    <xacro:include filename="$(find clearpath_platform_description)/urdf/a300/drivetrain/wheels/caster.urdf.xacro" />
     <xacro:include filename="$(find clearpath_platform_description)/urdf/a300/drivetrain/motor.urdf.xacro" />
+    <xacro:include filename="$(find clearpath_platform_description)/urdf/a300/drivetrain/caster_flange.urdf.xacro" />
     <!-- Front Wheels -->
     <xacro:if value="${front_wheels == 'outdoor'}">
       <xacro:property name="front_wheel_radius" value="${a300_outdoor_wheel_radius}" scope="parent"/>
       <xacro:property name="front_wheel_width" value="${a300_outdoor_wheel_width}" scope="parent"/>
-      <!-- Wheel -->
-      <xacro:a300_outdoor_wheel prefix="front_left">
-        <origin xyz="${wheel_base/2} ${wheel_track/2} 0" rpy="0 0 0"/>
-      </xacro:a300_outdoor_wheel>
-      <!-- Motor -->
-      <xacro:a300_motor prefix="front_left">
-        <origin xyz="0 0 0" rpy="0 0 ${math.pi}"/>
-      </xacro:a300_motor>
-      <!-- Wheel -->
-      <xacro:a300_outdoor_wheel prefix="front_right">
-        <origin xyz="${wheel_base/2} ${-wheel_track/2} 0" rpy="0 0 0"/>
-      </xacro:a300_outdoor_wheel>
-      <!-- Motor -->
-      <xacro:a300_motor prefix="front_right">
-        <origin xyz="0 0 0" rpy="${math.pi} 0 ${math.pi}"/>
-      </xacro:a300_motor>
+      <!-- Motors -->
+      <xacro:a300_motor prefix="front" side="left"/>
+      <xacro:a300_motor prefix="front" side="right"/>
+      <!-- Wheels -->
+      <xacro:a300_outdoor_wheel prefix="front" side="left"/>
+      <xacro:a300_outdoor_wheel prefix="front" side="right"/>
     </xacro:if>
-    <xacro:unless value="${front_wheels == 'outdoor'}">
-      <xacro:error message="Invalid A300 front wheels ${front_wheels}"/>
-    </xacro:unless>
+    <xacro:if value="${front_wheels == 'mecanum'}">
+      <xacro:property name="front_wheel_radius" value="${a300_mecanum_wheel_radius}" scope="parent"/>
+      <xacro:property name="front_wheel_width" value="${a300_mecanum_wheel_width}" scope="parent"/>
+      <!-- Motors -->
+      <xacro:a300_motor prefix="front" side="left"/>
+      <xacro:a300_motor prefix="front" side="right"/>
+      <!-- Wheels -->
+      <xacro:a300_mecanum_wheel prefix="front" side="left"/>
+      <xacro:a300_mecanum_wheel prefix="front" side="right"/>
+    </xacro:if>
+    <xacro:if value="${front_wheels == 'caster'}">
+      <xacro:property name="front_wheel_radius" value="${a300_caster_wheel_radius}" scope="parent"/>
+      <xacro:property name="front_wheel_width" value="${a300_caster_wheel_width}" scope="parent"/>
+      <!-- Flanges -->
+      <xacro:a300_caster_flange prefix="front" side="left"/>
+      <xacro:a300_caster_flange prefix="front" side="right"/>
+      <!-- Wheels -->
+      <xacro:a300_caster_wheel prefix="front" side="left"/>
+      <xacro:a300_caster_wheel prefix="front" side="right"/>
+    </xacro:if>
     <!-- Rear Wheels -->
     <xacro:if value="${rear_wheels == 'outdoor'}">
       <xacro:property name="rear_wheel_radius" value="${a300_outdoor_wheel_radius}" scope="parent"/>
       <xacro:property name="rear_wheel_width" value="${a300_outdoor_wheel_width}" scope="parent"/>
-      <!-- Wheel -->
-      <xacro:a300_outdoor_wheel prefix="rear_left">
-        <origin xyz="${-wheel_base/2} ${wheel_track/2} 0" rpy="0 0 0"/>
-      </xacro:a300_outdoor_wheel>
-      <!-- Motor -->
-      <xacro:a300_motor prefix="rear_left">
-        <origin xyz="0 0 0" rpy="${math.pi} 0 0"/>
-      </xacro:a300_motor>
-      <!-- Wheel -->
-      <xacro:a300_outdoor_wheel prefix="rear_right">
-        <origin xyz="${-wheel_base/2} ${-wheel_track/2} 0" rpy="0 0 0"/>
-      </xacro:a300_outdoor_wheel>
-      <!-- Motor -->
-      <xacro:a300_motor prefix="rear_right">
-        <origin xyz="0 0 0" rpy="0 0 0"/>
-      </xacro:a300_motor>
+      <!-- Motors -->
+      <xacro:a300_motor prefix="rear" side="left"/>
+      <xacro:a300_motor prefix="rear" side="right"/>
+      <!-- Wheels -->
+      <xacro:a300_outdoor_wheel prefix="rear" side="left"/>
+      <xacro:a300_outdoor_wheel prefix="rear" side="right"/>
     </xacro:if>
-    <xacro:unless value="${rear_wheels == 'outdoor'}">
-      <xacro:error message="Invalid A300 rear wheels ${rear_wheels}"/>
-    </xacro:unless>
+    <xacro:if value="${rear_wheels == 'mecanum'}">
+      <xacro:property name="rear_wheel_radius" value="${a300_mecanum_wheel_radius}" scope="parent"/>
+      <xacro:property name="rear_wheel_width" value="${a300_mecanum_wheel_width}" scope="parent"/>
+      <!-- Motors -->
+      <xacro:a300_motor prefix="rear" side="left"/>
+      <xacro:a300_motor prefix="rear" side="right"/>
+      <!-- Wheels -->
+      <xacro:a300_mecanum_wheel prefix="rear" side="left"/>
+      <xacro:a300_mecanum_wheel prefix="rear" side="right"/>
+    </xacro:if>
+    <xacro:if value="${rear_wheels == 'caster'}">
+      <xacro:property name="rear_wheel_radius" value="${a300_caster_wheel_radius}" scope="parent"/>
+      <xacro:property name="rear_wheel_width" value="${a300_caster_wheel_width}" scope="parent"/>
+      <!-- Flanges -->
+      <xacro:a300_caster_flange prefix="rear" side="left"/>
+      <xacro:a300_caster_flange prefix="rear" side="right"/>
+      <!-- Wheels -->
+      <xacro:a300_caster_wheel prefix="rear" side="left"/>
+      <xacro:a300_caster_wheel prefix="rear" side="right"/>
+    </xacro:if>
   </xacro:macro>
 </robot>

File: clearpath_platform_description/urdf/a300/drivetrain/wheels/outdoor.urdf.xacro (robot description, xacro)
@@ -4,6 +4,6 @@
   <xacro:property name="a300_outdoor_wheel_mass" value="2.5" />
   <xacro:property name="a300_outdoor_wheel_width" value="0.1143" />
-  <xacro:macro name="a300_outdoor_wheel" params="prefix *joint_pose">
-    <link name="${prefix}_wheel_link">
+  <xacro:macro name="a300_outdoor_wheel" params="prefix side">
+    <link name="${prefix}_${side}_wheel_link">
       <inertial>
         <mass value="${a300_outdoor_wheel_mass}" />
@@ -15,8 +15,8 @@
       </inertial>
       <visual>
-        <origin xyz="0 0 0" rpy="0 0 ${math.pi}"/>
+        <origin xyz="0 0 0" rpy="0 0 ${math.pi if side == 'right' else 0}"/>
         <material name="clearpath_dark_grey"/>
         <geometry>
-          <mesh filename="package://clearpath_platform_description/meshes/a300/wheels/outdoor.dae" />
+          <mesh filename="package://clearpath_platform_description/meshes/a300/drivetrain/wheels/outdoor_${side}.stl" />
         </geometry>
       </visual>
@@ -30,5 +30,5 @@
     <gazebo>
       <plugin filename="libgz-sim-wheel-slip-system.so" name="gz::sim::systems::WheelSlip">
-        <wheel link_name="${prefix}_wheel_link">
+        <wheel link_name="${prefix}_${side}_wheel_link">
           <slip_compliance_lateral>1.0</slip_compliance_lateral>
           <slip_compliance_longitudinal>1.0</slip_compliance_longitudinal>
@@ -38,8 +38,7 @@
       </plugin>
     </gazebo>
-    <joint name="${prefix}_wheel_joint" type="continuous">
-      <parent link="chassis_link"/>
-      <child link="${prefix}_wheel_link"/>
-      <xacro:insert_block name="joint_pose"/>
+    <joint name="${prefix}_${side}_wheel_joint" type="continuous">
+      <parent link="${prefix}_${side}_motor_mount"/>
+      <child link="${prefix}_${side}_wheel_link"/>
       <axis xyz="0 1 0" rpy="0 0 0" />
     </joint>
