Commit message: switch urdfs to glb mesh refs

File: clearpath_platform_description/urdf/a300/a300.urdf.xacro (robot description, xacro)
@@ -50,15 +50,5 @@
       <visual>
         <geometry>
-          <mesh filename="package://clearpath_platform_description/meshes/a300/chassis.dae" />
-        </geometry>
-      </visual>
-      <visual>
-        <geometry>
-          <mesh filename="package://clearpath_platform_description/meshes/a300/livery.dae" />
-        </geometry>
-      </visual>
-      <visual>
-        <geometry>
-          <mesh filename="package://clearpath_platform_description/meshes/a300/status_lights.dae" />
+          <mesh filename="package://clearpath_platform_description/meshes/a300/a300_chassis.glb" />
         </geometry>
       </visual>

File: clearpath_platform_description/urdf/a300/drivetrain/motor.urdf.xacro (robot description, xacro)
@@ -8,5 +8,5 @@
         <material name="clearpath_dark_grey"/>
         <geometry>
-          <mesh filename="package://clearpath_platform_description/meshes/a300/drivetrain/motor.stl"/>
+          <mesh filename="package://clearpath_platform_description/meshes/a300/drivetrain/motor.glb"/>
         </geometry>
         <origin rpy="0 0 ${rotation_yaw}"/>
@@ -14,5 +14,5 @@
       <collision>
         <geometry>
-          <mesh filename="package://clearpath_platform_description/meshes/a300/drivetrain/motor.stl"/>
+          <mesh filename="package://clearpath_platform_description/meshes/a300/drivetrain/motor.glb"/>
         </geometry>
       </collision>

File: clearpath_platform_description/urdf/a300/drivetrain/suspension_beam.urdf.xacro (robot description, xacro)
@@ -9,5 +9,5 @@
         <material name="clearpath_dark_grey"/>
         <geometry>
-          <mesh filename="package://clearpath_platform_description/meshes/a300/drivetrain/suspension_spacer.stl"/>
+          <mesh filename="package://clearpath_platform_description/meshes/a300/drivetrain/suspension_spacer.glb"/>
         </geometry>
         <origin rpy="0 0 ${rotation_yaw}"/>
@@ -15,5 +15,5 @@
       <collision>
         <geometry>
-          <mesh filename="package://clearpath_platform_description/meshes/a300/drivetrain/suspension_spacer.stl"/>
+          <mesh filename="package://clearpath_platform_description/meshes/a300/drivetrain/suspension_spacer.glb"/>
         </geometry>
       </collision>
@@ -28,5 +28,5 @@
         <material name="clearpath_dark_grey"/>
         <geometry>
-          <mesh filename="package://clearpath_platform_description/meshes/a300/drivetrain/suspension_beam.stl"/>
+          <mesh filename="package://clearpath_platform_description/meshes/a300/drivetrain/suspension_beam.glb"/>
         </geometry>
         <origin rpy="0 0 ${rotation_yaw}"/>
@@ -34,5 +34,5 @@
       <collision>
         <geometry>
-          <mesh filename="package://clearpath_platform_description/meshes/a300/drivetrain/suspension_beam.stl"/>
+          <mesh filename="package://clearpath_platform_description/meshes/a300/drivetrain/suspension_beam.glb"/>
         </geometry>
       </collision>

File: clearpath_platform_description/urdf/a300/drivetrain/wheels/outdoor.urdf.xacro (robot description, xacro)
@@ -18,5 +18,5 @@
         <material name="clearpath_dark_grey"/>
         <geometry>
-          <mesh filename="package://clearpath_platform_description/meshes/a300/drivetrain/wheels/outdoor_${side}.stl" />
+          <mesh filename="package://clearpath_platform_description/meshes/a300/drivetrain/wheels/outdoor_${side}.glb" />
         </geometry>
       </visual>

File: clearpath_platform_description/urdf/do100/do100.urdf.xacro (robot description, xacro)
@@ -23,5 +23,5 @@
         <origin xyz="0 0 0" rpy="0 0 0"/>
         <geometry>
-          <mesh filename="package://clearpath_platform_description/meshes/do100/omni_chassis.dae"/>
+          <mesh filename="package://clearpath_platform_description/meshes/do100/do100_chassis.glb"/>
         </geometry>
       </visual>
@@ -34,5 +34,5 @@
       <inertial>
         <!-- Center of mass -->
-        <origin xyz="0 0 0" rpy="0 0 0"/>
+        <origin xyz="0 0 ${wheel_vertical_offset}" rpy="0 0 0"/>
         <mass value="14"/>
         <!-- Moments of inertia: ( chassis without wheels ) -->

File: clearpath_platform_description/urdf/j100/drivetrain/wheels/outdoor.urdf.xacro (robot description, xacro)
@@ -9,5 +9,5 @@
         <origin xyz="0 0 0" rpy="${PI/2} 0 0"/>
         <geometry>
-          <mesh filename="package://clearpath_platform_description/meshes/j100/wheels/outdoor.stl"/>
+          <mesh filename="package://clearpath_platform_description/meshes/j100/wheels/outdoor.glb"/>
         </geometry>
         <material name="clearpath_black" />

File: clearpath_platform_description/urdf/j100/j100.urdf.xacro (robot description, xacro)
@@ -28,5 +28,5 @@
         <origin xyz="0 0 ${footprint_vertical_offset}" rpy="${PI/2} 0 ${PI/2}"/>
         <geometry>
-          <mesh filename="package://clearpath_platform_description/meshes/j100/j100_base.stl"/>
+          <mesh filename="package://clearpath_platform_description/meshes/j100/j100_chassis.glb"/>
         </geometry>
         <material name="clearpath_dark_grey" />
