Commit message: Initial add do100

File: clearpath_platform_description/urdf/do100/do100.urdf.xacro (robot description, xacro)
@@ -3,17 +3,17 @@
   <xacro:arg name="namespace" default="" />
   <xacro:arg name="is_sim" default="false" />
-  <xacro:arg name="gazebo_controllers" default="$(find clearpath_control)/config/dd100/control.yaml"/>
-  <!-- Included URDF/XACRO Files -->
-  <xacro:include filename="$(find clearpath_platform_description)/urdf/dd100/wheels/wheel.urdf.xacro"/>
+  <xacro:arg name="gazebo_controllers" default="$(find clearpath_control)/config/do100/control.yaml"/>
+  <!-- Included URDF/Xacro Files -->
+  <xacro:include filename="$(find clearpath_platform_description)/urdf/do100/wheels/wheel.urdf.xacro"/>
   <xacro:property name="PI" value="${math.pi}" />
-  <!-- DD100 Platform Macro -->
-  <xacro:macro name="dd100" params="wheel:='default'">
+  <!-- D0100 Platform Macro -->
+  <xacro:macro name="do100" params="wheel:='defaut'">
     <!-- Variables -->
-    <xacro:property name="wheel_radius" value="0.049" />
-    <xacro:property name="wheel_mass" value="0.111" />
-    <xacro:property name="wheel_width" value="0.02032" />
-    <xacro:property name="wheel_x_offset" value="0.0989838" />
-    <xacro:property name="wheel_z_offset" value="0.0345" />
-    <xacro:property name="wheelbase" value="0.2160016" />
+    <xacro:property name="wheelbase" value="0.570" />
+    <xacro:property name="track" value="0.3708" />
+    <xacro:property name="wheel_vertical_offset" value="0.035145" />
+    <xacro:property name="wheel_radius" value="0.050" />
+    <xacro:property name="wheel_mass" value="0.4" />
+    <xacro:property name="wheel_width" value="0.050" />
     <xacro:property name="dummy_inertia" value="1e-09"/>
     <!-- Chassis -->
@@ -28,29 +28,38 @@
         <origin xyz="0 0 0" rpy="0 0 0"/>
         <geometry>
-          <mesh filename="package://clearpath_platform_description/meshes/dd100/chassis.dae"/>
+          <mesh filename="package://clearpath_platform_description/meshes/do100/omni_chassis.dae"/>
         </geometry>
+        <material name="clearpath_dark_grey" />
       </visual>
       <collision>
         <origin xyz="0 0 0"/>
         <geometry>
-          <mesh filename="package://clearpath_platform_description/meshes/dd100/chassis_collision.stl"/>
+          <mesh filename="package://clearpath_platform_description/meshes/do100/omni_chassis_collision.stl"/>
         </geometry>
       </collision>
       <inertial>
+        <!-- Center of mass -->
         <origin xyz="0 0 0" rpy="0 0 0"/>
-        <mass value="10.0"/>
+        <mass value="14"/>
+        <!-- Moments of inertia: ( chassis without wheels ) -->
         <inertia
-          ixx="0.2216" ixy="0" ixz="0"
-          iyy="0.2458" iyz="0"
-          izz="0.4474"/>
+          ixx="0.35498" ixy="0" ixz="0"
+          iyy="0.7266" iyz="0"
+          izz="1.0553"/>
         </inertial>
     </link>
     <!-- Wheels -->
-    <xacro:dd100_wheel prefix="front_left">
-      <origin xyz="${wheel_x_offset} ${wheelbase+wheel_width/2} ${wheel_z_offset}" rpy="0 0 0" />
-    </xacro:dd100_wheel>
-    <xacro:dd100_wheel prefix="front_right">
-      <origin xyz="${wheel_x_offset} ${-wheelbase-wheel_width/2} ${wheel_z_offset}" rpy="0 0 0" />
-    </xacro:dd100_wheel>
+    <xacro:do100_wheel prefix="front_left">
+      <origin xyz="${wheelbase/2} ${track/2+wheel_width/2} ${wheel_vertical_offset}" rpy="0 0 0" />
+    </xacro:do100_wheel>
+    <xacro:do100_wheel prefix="front_right">
+      <origin xyz="${wheelbase/2} ${-track/2-wheel_width/2} ${wheel_vertical_offset}" rpy="0 0 0" />
+    </xacro:do100_wheel>
+    <xacro:do100_wheel prefix="rear_left">
+      <origin xyz="${-wheelbase/2} ${track/2+wheel_width/2} ${wheel_vertical_offset}" rpy="0 0 0" />
+    </xacro:do100_wheel>
+    <xacro:do100_wheel prefix="rear_right">
+      <origin xyz="${-wheelbase/2} ${-track/2-wheel_width/2} ${wheel_vertical_offset}" rpy="0 0 0" />
+    </xacro:do100_wheel>
     <gazebo>
       <plugin filename="libignition-gazebo-wheel-slip-system.so" name="ignition::gazebo::systems::WheelSlip">
@@ -58,5 +67,5 @@
           <slip_compliance_lateral>1.0</slip_compliance_lateral>
           <slip_compliance_longitudinal>1.0</slip_compliance_longitudinal>
-          <wheel_normal_force>39.2</wheel_normal_force>
+          <wheel_normal_force>20</wheel_normal_force>
           <wheel_radius>${wheel_radius}</wheel_radius>
         </wheel>
@@ -64,56 +73,22 @@
           <slip_compliance_lateral>1.0</slip_compliance_lateral>
           <slip_compliance_longitudinal>1.0</slip_compliance_longitudinal>
-          <wheel_normal_force>39.2</wheel_normal_force>
+          <wheel_normal_force>20</wheel_normal_force>
           <wheel_radius>${wheel_radius}</wheel_radius>
         </wheel>
       </plugin>
-    </gazebo>
-    <!-- Caster -->
-    <link name="rear_caster">
-      <visual>
-        <origin rpy="0 0 0" xyz="0 0 0"/>
-        <geometry>
-          <sphere radius="0.01"/>
-        </geometry>
-        <material name="clearpath_black"/>
-      </visual>
-      <collision>
-        <geometry>
-          <sphere radius="0.01"/>
-        </geometry>
-        <origin rpy="0 0 0" xyz="0 0 0"/>
-        <surface>
-          <friction>
-            <ode>
-              <mu>0.0</mu>
-              <mu2>0.0</mu2>
-              <slip1>1.0</slip1>
-              <slip2>1.0</slip2>
-            </ode>
-          </friction>
-        </surface>
-      </collision>
-      <inertial>
-        <mass value="0.1" />
-        <origin xyz="0 0 0" />
-        <inertia ixx="0.001" ixy="0.0" ixz="0.0"
-                iyy="0.001" iyz="0.0"
-                izz="0.001" />
-      </inertial>
-    </link>
-    <joint name="rear_caster_joint" type="fixed">
-      <parent link="chassis_link"/>
-      <child link="rear_caster"/>
-      <origin xyz="-0.244 0 -0.00674" rpy="0 0 0"/>
-    </joint>
-    <gazebo reference="rear_caster">
-      <turnGravityOff>false</turnGravityOff>
-      <kp>1000000.0</kp>
-      <kd>100.0</kd>
-      <mu1>0.2</mu1>
-      <mu2>0.2</mu2>
-      <fdir1>1 0 0</fdir1>
-      <minDepth>0.00</minDepth>
-      <implicitSpringDamper>1</implicitSpringDamper>
+      <plugin filename="libignition-gazebo-wheel-slip-system.so" name="ignition::gazebo::systems::WheelSlip">
+        <wheel link_name="rear_left_wheel_link">
+          <slip_compliance_lateral>1.0</slip_compliance_lateral>
+          <slip_compliance_longitudinal>1.0</slip_compliance_longitudinal>
+          <wheel_normal_force>20</wheel_normal_force>
+          <wheel_radius>${wheel_radius}</wheel_radius>
+        </wheel>
+        <wheel link_name="rear_right_wheel_link">
+          <slip_compliance_lateral>1.0</slip_compliance_lateral>
+          <slip_compliance_longitudinal>1.0</slip_compliance_longitudinal>
+          <wheel_normal_force>20</wheel_normal_force>
+          <wheel_radius>${wheel_radius}</wheel_radius>
+        </wheel>
+      </plugin>
     </gazebo>
     <!-- Internal IMU -->
@@ -146,11 +121,11 @@
     <link name="rear_0_mount"/>
     <joint name="default_mount_joint" type="fixed">
-      <origin xyz="0 0 0" rpy="0 0 0"/>
-      <parent link="front_0_mount"/>
-      <child link="default_mount"/>
+      <origin xyz="0 0 0.069023" rpy="0 0 0" />
+      <parent link="chassis_link"/>
+      <child link="default_mount" />
     </joint>
     <joint name="front_0_mount_joint" type="fixed">
-      <origin xyz="0.040 0 0.064263" rpy="0 0 0" />
-      <parent link="chassis_link"/>
+      <origin xyz="0.080 0 0" rpy="0 0 0" />
+      <parent link="default_mount"/>
       <child link="front_0_mount" />
     </joint>
@@ -166,6 +141,6 @@
     </joint>
     <joint name="rear_0_mount_joint" type="fixed">
-      <origin xyz="-0.040 0 0.064263" rpy="0 0 0" />
-      <parent link="chassis_link"/>
+      <origin xyz="-0.080 0 0" rpy="0 0 0" />
+      <parent link="default_mount"/>
       <child link="rear_0_mount" />
     </joint>
@@ -175,5 +150,5 @@
       <child link="rear_1_mount" />
     </joint>
-    <joint name="rear_2_moint_joint" type="fixed">
+    <joint name="rear_2_mount_joint" type="fixed">
       <origin xyz="-0.080 0 0" rpy="0 0 0" />
       <parent link="rear_1_mount"/>
@@ -184,10 +159,10 @@
     <link name="rear_bumper_mount"/>
     <joint name="front_bumper_mount_joint" type="fixed">
-      <origin xyz="0.274 0 0.0345125" rpy="0 0 0" />
+      <origin xyz="0.34159 0 0.0345115" rpy="0 0 0" />
       <parent link="chassis_link"/>
       <child link="front_bumper_mount" />
     </joint>
     <joint name="rear_bumper_mount_joint" type="fixed">
-      <origin xyz="-0.274 0 0.0345125" rpy="0 0 ${PI}" />
+      <origin xyz="-0.34159 0 0.0345115" rpy="0 0 0" />
       <parent link="chassis_link"/>
       <child link="rear_bumper_mount" />
@@ -196,5 +171,5 @@
     <xacro:include filename="$(find clearpath_platform_description)/urdf/generic/gazebo.urdf.xacro"/>
     <!-- ROS2 controls -->
-    <ros2_control name="dd100_hardware" type="system">
+    <ros2_control name="do100_hardware" type="system">
       <hardware>
         <xacro:if value="$(arg is_sim)">
@@ -202,5 +177,5 @@
         </xacro:if>
         <xacro:unless value="$(arg is_sim)">
-          <plugin>clearpath_platform/DD100Hardware</plugin>
+          <plugin>clearpath_platform/DO100Hardware</plugin>
           <plugin>fake_components/GenericSystem</plugin>
         </xacro:unless>
@@ -216,4 +191,14 @@
         <state_interface name="velocity"/>
       </joint>
+      <joint name="rear_left_wheel_joint">
+        <command_interface name="velocity"/>
+        <state_interface name="position"/>
+        <state_interface name="velocity"/>
+      </joint>
+      <joint name="rear_right_wheel_joint">
+        <command_interface name="velocity"/>
+        <state_interface name="position"/>
+        <state_interface name="velocity"/>
+      </joint>
     </ros2_control>
   </xacro:macro>

Commit message: Only load mecanum wheels in simulation

File: clearpath_platform_description/urdf/do100/do100.urdf.xacro (robot description, xacro)
@@ -51,16 +51,32 @@
     </link>
     <!-- Wheels -->
-    <xacro:do100_mecanum_wheel prefix="front_left" side="-1">
-      <origin xyz="${wheelbase/2} ${track/2+wheel_width/2} ${wheel_vertical_offset}" rpy="0 0 0" />
-    </xacro:do100_mecanum_wheel>
-    <xacro:do100_mecanum_wheel prefix="front_right" side="1">
-      <origin xyz="${wheelbase/2} ${-track/2-wheel_width/2} ${wheel_vertical_offset}" rpy="0 0 0" />
-    </xacro:do100_mecanum_wheel>
-    <xacro:do100_mecanum_wheel prefix="rear_left" side="1">
-      <origin xyz="${-wheelbase/2} ${track/2+wheel_width/2} ${wheel_vertical_offset}" rpy="0 0 0" />
-    </xacro:do100_mecanum_wheel>
-    <xacro:do100_mecanum_wheel prefix="rear_right" side="-1">
-      <origin xyz="${-wheelbase/2} ${-track/2-wheel_width/2} ${wheel_vertical_offset}" rpy="0 0 0" />
-    </xacro:do100_mecanum_wheel>
+    <xacro:if value="$(arg is_sim)">
+      <xacro:do100_mecanum_wheel prefix="front_left" side="-1">
+        <origin xyz="${wheelbase/2} ${track/2+wheel_width/2} ${wheel_vertical_offset}" rpy="0 0 0" />
+      </xacro:do100_mecanum_wheel>
+      <xacro:do100_mecanum_wheel prefix="front_right" side="1">
+        <origin xyz="${wheelbase/2} ${-track/2-wheel_width/2} ${wheel_vertical_offset}" rpy="0 0 0" />
+      </xacro:do100_mecanum_wheel>
+      <xacro:do100_mecanum_wheel prefix="rear_left" side="1">
+        <origin xyz="${-wheelbase/2} ${track/2+wheel_width/2} ${wheel_vertical_offset}" rpy="0 0 0" />
+      </xacro:do100_mecanum_wheel>
+      <xacro:do100_mecanum_wheel prefix="rear_right" side="-1">
+        <origin xyz="${-wheelbase/2} ${-track/2-wheel_width/2} ${wheel_vertical_offset}" rpy="0 0 0" />
+      </xacro:do100_mecanum_wheel>
+    </xacro:if>
+    <xacro:unless value="$(arg is_sim)">
+      <xacro:do100_wheel prefix="front_left">
+        <origin xyz="${wheelbase/2} ${track/2+wheel_width/2} ${wheel_vertical_offset}" rpy="0 0 0" />
+      </xacro:do100_wheel>
+      <xacro:do100_wheel prefix="front_right">
+        <origin xyz="${wheelbase/2} ${-track/2-wheel_width/2} ${wheel_vertical_offset}" rpy="0 0 0" />
+      </xacro:do100_wheel>
+      <xacro:do100_wheel prefix="rear_left">
+        <origin xyz="${-wheelbase/2} ${track/2+wheel_width/2} ${wheel_vertical_offset}" rpy="0 0 0" />
+      </xacro:do100_wheel>
+      <xacro:do100_wheel prefix="rear_right">
+        <origin xyz="${-wheelbase/2} ${-track/2-wheel_width/2} ${wheel_vertical_offset}" rpy="0 0 0" />
+      </xacro:do100_wheel>
+    </xacro:unless>
     <gazebo>
       <plugin filename="libignition-gazebo-wheel-slip-system.so" name="ignition::gazebo::systems::WheelSlip">
