Commit message: URDF Mecanum Updates

File: clearpath_platform_description/urdf/do100/do100.urdf.xacro (robot description, xacro)
@@ -6,5 +6,4 @@
   <!-- Included URDF/Xacro Files -->
   <xacro:include filename="$(find clearpath_platform_description)/urdf/do100/wheels/wheel.urdf.xacro"/>
-  <xacro:include filename="$(find clearpath_platform_description)/urdf/do100/wheels/mecanum_wheel.urdf.xacro"/>
   <xacro:property name="PI" value="${math.pi}" />
   <!-- D0100 Platform Macro -->
@@ -31,5 +30,4 @@
           <mesh filename="package://clearpath_platform_description/meshes/do100/omni_chassis.dae"/>
         </geometry>
-        <material name="clearpath_dark_grey" />
       </visual>
       <collision>
@@ -51,33 +49,17 @@
     </link>
     <!-- Wheels -->
-    <xacro:if value="$(arg is_sim)">
-      <xacro:do100_mecanum_wheel prefix="front_left" side="-1">
-        <origin xyz="${wheelbase/2} ${track/2+wheel_width/2} ${wheel_vertical_offset}" rpy="0 0 0" />
-      </xacro:do100_mecanum_wheel>
-      <xacro:do100_mecanum_wheel prefix="front_right" side="1">
-        <origin xyz="${wheelbase/2} ${-track/2-wheel_width/2} ${wheel_vertical_offset}" rpy="0 0 0" />
-      </xacro:do100_mecanum_wheel>
-      <xacro:do100_mecanum_wheel prefix="rear_left" side="1">
-        <origin xyz="${-wheelbase/2} ${track/2+wheel_width/2} ${wheel_vertical_offset}" rpy="0 0 0" />
-      </xacro:do100_mecanum_wheel>
-      <xacro:do100_mecanum_wheel prefix="rear_right" side="-1">
-        <origin xyz="${-wheelbase/2} ${-track/2-wheel_width/2} ${wheel_vertical_offset}" rpy="0 0 0" />
-      </xacro:do100_mecanum_wheel>
-    </xacro:if>
-    <xacro:unless value="$(arg is_sim)">
-      <xacro:do100_wheel prefix="front_left">
-        <origin xyz="${wheelbase/2} ${track/2+wheel_width/2} ${wheel_vertical_offset}" rpy="0 0 0" />
-      </xacro:do100_wheel>
-      <xacro:do100_wheel prefix="front_right">
-        <origin xyz="${wheelbase/2} ${-track/2-wheel_width/2} ${wheel_vertical_offset}" rpy="0 0 0" />
-      </xacro:do100_wheel>
-      <xacro:do100_wheel prefix="rear_left">
-        <origin xyz="${-wheelbase/2} ${track/2+wheel_width/2} ${wheel_vertical_offset}" rpy="0 0 0" />
-      </xacro:do100_wheel>
-      <xacro:do100_wheel prefix="rear_right">
-        <origin xyz="${-wheelbase/2} ${-track/2-wheel_width/2} ${wheel_vertical_offset}" rpy="0 0 0" />
-      </xacro:do100_wheel>
-    </xacro:unless>
-    <gazebo>
+    <xacro:do100_wheel prefix="front_left" side="-1">
+      <origin xyz="${wheelbase/2} ${track/2+wheel_width/2} ${wheel_vertical_offset}" rpy="0 0 0" />
+    </xacro:do100_wheel>
+    <xacro:do100_wheel prefix="front_right" side="1">
+      <origin xyz="${wheelbase/2} ${-track/2-wheel_width/2} ${wheel_vertical_offset}" rpy="0 0 0" />
+    </xacro:do100_wheel>
+    <xacro:do100_wheel prefix="rear_left" side="1">
+      <origin xyz="${-wheelbase/2} ${track/2+wheel_width/2} ${wheel_vertical_offset}" rpy="0 0 0" />
+    </xacro:do100_wheel>
+    <xacro:do100_wheel prefix="rear_right" side="-1">
+      <origin xyz="${-wheelbase/2} ${-track/2-wheel_width/2} ${wheel_vertical_offset}" rpy="0 0 0" />
+    </xacro:do100_wheel>
+    <!-- <gazebo>
       <plugin filename="libignition-gazebo-wheel-slip-system.so" name="ignition::gazebo::systems::WheelSlip">
         <wheel link_name="front_left_wheel_link">
@@ -106,5 +88,5 @@
         </wheel>
       </plugin>
-    </gazebo>
+    </gazebo> -->
     <!-- Internal IMU -->
     <link name="imu_0_link">

File: clearpath_platform_description/urdf/do100/wheels/wheel.urdf.xacro (robot description, xacro)
@@ -1,12 +1,11 @@
 <?xml version="1.0"?>
-<robot xmlns:xacro="http://ros.org/wiki/xacro" name="do100_wheel">
-  <xacro:macro name="do100_wheel" params="prefix *joint_pose">
+<robot xmlns:xacro="http://ros.org/wiki/xacro" xmlns:ignition="http://gazebosim.org/schema" name="do100_wheel">
+  <xacro:macro name="do100_wheel" params="prefix side *joint_pose">
     <link name="${prefix}_wheel_link">
       <visual>
-        <origin xyz="0 0 0" rpy="${PI/2} 0 0"/>
+        <origin xyz="0 ${side * 0.027} 0" rpy="0 0 ${PI/2}"/>
         <geometry>
-          <cylinder radius="${wheel_radius}" length="${wheel_width}"/>
+          <mesh filename="package://clearpath_platform_description/meshes/do100/mecanum_wheel.dae" scale="${side} 1 1" />
         </geometry>
-        <material name="clearpath_black" />
       </visual>
       <collision>
@@ -20,15 +19,21 @@
         <mass value="${wheel_mass}"/>
         <inertia
-          ixx="0.0003234" ixy="0" ixz="0"
-          iyy="0.0003234" iyz="0"
-          izz="0.0004901"/>
+          ixx="${wheel_mass/12 * (3 * wheel_radius * wheel_radius + wheel_width * wheel_width)}" ixy="0" ixz="0"
+          iyy="${(wheel_radius * wheel_radius * wheel_mass)/2}" iyz="0"
+          izz="${wheel_mass/12 * (3 * wheel_radius * wheel_radius + wheel_width * wheel_width)}"/>
       </inertial>
     </link>
     <gazebo reference="${prefix}_wheel_link">
-      <material>Gazebo/DarkGrey</material>
-      <selfCollide>false</selfCollide>
-      <mu1 value="0.5"/>
-      <mu2 value="0.5"/>
-      <!-- <fdir1 value="1 0 0"/> -->
+      <collision>
+        <surface>
+          <friction>
+            <ode>
+              <mu>1.0</mu>
+              <mu2>0.0</mu2>
+              <fdir1 ignition:expressed_in="base_link">1 ${side} 0</fdir1>
+            </ode>
+          </friction>
+        </surface>
+      </collision>
     </gazebo>
     <joint name="${prefix}_wheel_joint" type="continuous">

File: clearpath_platform_description/urdf/generic/gazebo.urdf.xacro (robot description, xacro)
@@ -12,4 +12,6 @@
           <remapping>/diagnostics:=diagnostics</remapping>
           <remapping>joint_states:=platform/joint_states</remapping>
+          <remapping>~/reference:=platform/cmd_vel</remapping>
+          <remapping>~/odometry:=platform/odom</remapping>
           <namespace>$(arg namespace)</namespace>
         </ros>

File: clearpath_platform_description/urdf/r100/r100.urdf.xacro (robot description, xacro)
@@ -12,5 +12,5 @@
     <xacro:property name="wheel_radius" value="0.0759" />
     <xacro:property name="wheel_width" value="0.0790" />
-    <xacro:property name="wheel_mass" value="0.8" />
+    <xacro:property name="wheel_mass" value="2.5" />
     <xacro:property name="chassis_length" value="0.960" />
     <xacro:property name="chassis_width" value="0.793" />
@@ -211,5 +211,5 @@
           <slip_compliance_lateral>1.0</slip_compliance_lateral>
           <slip_compliance_longitudinal>1.0</slip_compliance_longitudinal>
-          <wheel_normal_force>20</wheel_normal_force>
+          <wheel_normal_force>200</wheel_normal_force>
           <wheel_radius>${wheel_radius}</wheel_radius>
         </wheel>
@@ -217,5 +217,5 @@
           <slip_compliance_lateral>1.0</slip_compliance_lateral>
           <slip_compliance_longitudinal>1.0</slip_compliance_longitudinal>
-          <wheel_normal_force>20</wheel_normal_force>
+          <wheel_normal_force>200</wheel_normal_force>
           <wheel_radius>${wheel_radius}</wheel_radius>
         </wheel>
@@ -223,5 +223,5 @@
           <slip_compliance_lateral>1.0</slip_compliance_lateral>
           <slip_compliance_longitudinal>1.0</slip_compliance_longitudinal>
-          <wheel_normal_force>20</wheel_normal_force>
+          <wheel_normal_force>200</wheel_normal_force>
           <wheel_radius>${wheel_radius}</wheel_radius>
         </wheel>
@@ -229,5 +229,5 @@
           <slip_compliance_lateral>1.0</slip_compliance_lateral>
           <slip_compliance_longitudinal>1.0</slip_compliance_longitudinal>
-          <wheel_normal_force>20</wheel_normal_force>
+          <wheel_normal_force>200</wheel_normal_force>
           <wheel_radius>${wheel_radius}</wheel_radius>
         </wheel>

File: clearpath_platform_description/urdf/r100/rocker.urdf.xacro (robot description, xacro)
@@ -2,5 +2,4 @@
 <robot xmlns:xacro="http://ros.org/wiki/xacro" name="r100_rocker">
   <xacro:include filename="$(find clearpath_platform_description)/urdf/r100/wheels/wheel.urdf.xacro"/>
-  <xacro:include filename="$(find clearpath_platform_description)/urdf/r100/wheels/mecanum_wheel.urdf.xacro"/>
   <xacro:macro name="r100_rocker" params="prefix joint_type location *joint_limits">
     <link name="${prefix}_rocker_link">
@@ -28,20 +27,10 @@
       <xacro:insert_block name="joint_limits" />
     </joint>
-    <xacro:if value="$(arg is_sim)">
-      <xacro:r100_mecanum_wheel parent="${prefix}_rocker_link" prefix="${prefix}_left" side="${-location}">
-          <origin xyz="0 ${rocker_width/2 + wheel_width/2} 0" rpy="0 0 0" />
-        </xacro:r100_mecanum_wheel>
-        <xacro:r100_mecanum_wheel parent="${prefix}_rocker_link" prefix="${prefix}_right" side="${location}">
-          <origin xyz="0 ${-(rocker_width/2 + wheel_width/2)} 0" rpy="0 0 0" />
-        </xacro:r100_mecanum_wheel>
-    </xacro:if>
-    <xacro:unless value="$(arg is_sim)">
-      <xacro:r100_wheel parent="${prefix}_rocker_link" prefix="${prefix}_left">
-        <origin xyz="0 ${rocker_width/2 + wheel_width/2} 0" rpy="0 0 0" />
-      </xacro:r100_wheel>
-      <xacro:r100_wheel parent="${prefix}_rocker_link" prefix="${prefix}_right">
-        <origin xyz="0 ${-(rocker_width/2 + wheel_width/2)} 0" rpy="0 0 0" />
-      </xacro:r100_wheel>
-    </xacro:unless>
+    <xacro:r100_wheel parent="${prefix}_rocker_link" prefix="${prefix}_left" side="${-location}">
+      <origin xyz="0 ${rocker_width/2 + wheel_width/2} 0" rpy="0 0 0" />
+    </xacro:r100_wheel>
+    <xacro:r100_wheel parent="${prefix}_rocker_link" prefix="${prefix}_right" side="${location}">
+      <origin xyz="0 ${-(rocker_width/2 + wheel_width/2)} 0" rpy="0 0 0" />
+    </xacro:r100_wheel>
   </xacro:macro>
 </robot>

File: clearpath_platform_description/urdf/r100/wheels/wheel.urdf.xacro (robot description, xacro)
@@ -1,5 +1,5 @@
 <?xml version="1.0"?>
-<robot xmlns:xacro="http://ros.org/wiki/xacro" name="r100_wheel">
-  <xacro:macro name="r100_wheel" params="parent prefix *joint_pose">
+<robot xmlns:xacro="http://ros.org/wiki/xacro" xmlns:ignition="http://gazebosim.org/schema" name="r100_wheel">
+  <xacro:macro name="r100_wheel" params="parent prefix side *joint_pose">
     <link name="${prefix}_wheel_link">
       <visual>
@@ -18,17 +18,23 @@
       <inertial>
         <origin xyz="0 0 0" rpy="0 0 0"/>
-        <mass value="2.3"/>
+        <mass value="${wheel_mass}"/>
         <inertia
-          ixx="3.3212e-3" ixy="0" ixz="0"
-          iyy="6.6424e-3" iyz="0"
-          izz="3.3212e-3"/>
+          ixx="${wheel_mass/12 * (3 * wheel_radius * wheel_radius + wheel_width * wheel_width)}" ixy="0" ixz="0"
+          iyy="${(wheel_radius * wheel_radius * wheel_mass)/2}" iyz="0"
+          izz="${wheel_mass/12 * (3 * wheel_radius * wheel_radius + wheel_width * wheel_width)}"/>
       </inertial>
     </link>
     <gazebo reference="${prefix}_wheel_link">
-      <material>Gazebo/DarkGrey</material>
-      <selfCollide>false</selfCollide>
-      <mu1 value="0.5"/>
-      <mu2 value="0.5"/>
-      <!-- <fdir1 value="1 0 0"/> -->
+      <collision>
+        <surface>
+          <friction>
+            <ode>
+              <mu>1.0</mu>
+              <mu2>0.0</mu2>
+              <fdir1 ignition:expressed_in="base_link">1 ${side} 0</fdir1>
+            </ode>
+          </friction>
+        </surface>
+      </collision>
     </gazebo>
     <joint name="${prefix}_wheel_joint" type="continuous">

Commit message: Moved meshes to wheels folder Mecanum drivetrain for do100

File: clearpath_platform_description/urdf/do100/do100.urdf.xacro (robot description, xacro)
@@ -5,15 +5,12 @@
   <xacro:arg name="gazebo_controllers" default="$(find clearpath_control)/config/do100/control.yaml"/>
   <!-- Included URDF/Xacro Files -->
-  <xacro:include filename="$(find clearpath_platform_description)/urdf/do100/wheels/wheel.urdf.xacro"/>
+  <!-- <xacro:include filename="$(find clearpath_platform_description)/urdf/do100/wheels/wheel.urdf.xacro"/> -->
   <xacro:property name="PI" value="${math.pi}" />
   <!-- D0100 Platform Macro -->
-  <xacro:macro name="do100" params="wheel:='defaut'">
+  <xacro:macro name="do100" params="drivetrain:='omni_4wd' wheels:='mecanum'">
     <!-- Variables -->
     <xacro:property name="wheelbase" value="0.570" />
     <xacro:property name="track" value="0.3708" />
     <xacro:property name="wheel_vertical_offset" value="0.035145" />
-    <xacro:property name="wheel_radius" value="0.050" />
-    <xacro:property name="wheel_mass" value="0.4" />
-    <xacro:property name="wheel_width" value="0.050" />
     <xacro:property name="dummy_inertia" value="1e-09"/>
     <!-- Chassis -->
@@ -48,45 +45,9 @@
         </inertial>
     </link>
-    <!-- Wheels -->
-    <xacro:do100_wheel prefix="front_left" side="-1">
-      <origin xyz="${wheelbase/2} ${track/2+wheel_width/2} ${wheel_vertical_offset}" rpy="0 0 0" />
-    </xacro:do100_wheel>
-    <xacro:do100_wheel prefix="front_right" side="1">
-      <origin xyz="${wheelbase/2} ${-track/2-wheel_width/2} ${wheel_vertical_offset}" rpy="0 0 0" />
-    </xacro:do100_wheel>
-    <xacro:do100_wheel prefix="rear_left" side="1">
-      <origin xyz="${-wheelbase/2} ${track/2+wheel_width/2} ${wheel_vertical_offset}" rpy="0 0 0" />
-    </xacro:do100_wheel>
-    <xacro:do100_wheel prefix="rear_right" side="-1">
-      <origin xyz="${-wheelbase/2} ${-track/2-wheel_width/2} ${wheel_vertical_offset}" rpy="0 0 0" />
-    </xacro:do100_wheel>
-    <gazebo>
-      <plugin filename="libgz-sim-wheel-slip-system.so" name="gz::sim::systems::WheelSlip">
-        <wheel link_name="front_left_wheel_link">
-          <slip_compliance_lateral>1.0</slip_compliance_lateral>
-          <slip_compliance_longitudinal>1.0</slip_compliance_longitudinal>
-          <wheel_normal_force>20</wheel_normal_force>
-          <wheel_radius>${wheel_radius}</wheel_radius>
-        </wheel>
-        <wheel link_name="front_right_wheel_link">
-          <slip_compliance_lateral>1.0</slip_compliance_lateral>
-          <slip_compliance_longitudinal>1.0</slip_compliance_longitudinal>
-          <wheel_normal_force>20</wheel_normal_force>
-          <wheel_radius>${wheel_radius}</wheel_radius>
-        </wheel>
-        <wheel link_name="rear_left_wheel_link">
-          <slip_compliance_lateral>1.0</slip_compliance_lateral>
-          <slip_compliance_longitudinal>1.0</slip_compliance_longitudinal>
-          <wheel_normal_force>20</wheel_normal_force>
-          <wheel_radius>${wheel_radius}</wheel_radius>
-        </wheel>
-        <wheel link_name="rear_right_wheel_link">
-          <slip_compliance_lateral>1.0</slip_compliance_lateral>
-          <slip_compliance_longitudinal>1.0</slip_compliance_longitudinal>
-          <wheel_normal_force>20</wheel_normal_force>
-          <wheel_radius>${wheel_radius}</wheel_radius>
-        </wheel>
-      </plugin>
-    </gazebo>
+    <!-- Add drivetrain -->
+    <xacro:if value="${drivetrain == 'omni_4wd'}">
+      <xacro:include filename="$(find clearpath_platform_description)/urdf/do100/drivetrain/type/omni_4wd.urdf.xacro"/>
+      <xacro:do100_drivetrain_type_omni wheels="${wheels}"/>
+    </xacro:if>
     <!-- Internal IMU -->
     <link name="imu_0_link">
@@ -165,37 +126,4 @@
       <child link="rear_bumper_mount" />
     </joint>
-    <!-- Gazebo Controller -->
-    <xacro:include filename="$(find clearpath_platform_description)/urdf/generic/gazebo.urdf.xacro"/>
-    <!-- ROS2 controls -->
-    <ros2_control name="do100_hardware" type="system">
-      <hardware>
-        <xacro:if value="$(arg is_sim)">
-          <plugin>gz_ros2_control/GazeboSimSystem</plugin>
-        </xacro:if>
-        <xacro:unless value="$(arg is_sim)">
-          <plugin>clearpath_hardware_interfaces/PumaHardware</plugin>
-        </xacro:unless>
-      </hardware>
-      <joint name="front_left_wheel_joint">
-        <command_interface name="velocity"/>
-        <state_interface name="position"/>
-        <state_interface name="velocity"/>
-      </joint>
-      <joint name="front_right_wheel_joint">
-        <command_interface name="velocity"/>
-        <state_interface name="position"/>
-        <state_interface name="velocity"/>
-      </joint>
-      <joint name="rear_left_wheel_joint">
-        <command_interface name="velocity"/>
-        <state_interface name="position"/>
-        <state_interface name="velocity"/>
-      </joint>
-      <joint name="rear_right_wheel_joint">
-        <command_interface name="velocity"/>
-        <state_interface name="position"/>
-        <state_interface name="velocity"/>
-      </joint>
-    </ros2_control>
   </xacro:macro>
   <!-- Joint State Publisher -->

File: clearpath_platform_description/urdf/do100/drivetrain/wheels/mecanum.urdf.xacro (robot description, xacro)
@@ -1,10 +1,13 @@
 <?xml version="1.0"?>
 <robot xmlns:xacro="http://ros.org/wiki/xacro" xmlns:ignition="http://gazebosim.org/schema" name="do100_wheel">
-  <xacro:macro name="do100_wheel" params="prefix side *joint_pose">
+  <xacro:property name="wheel_radius" value="0.050" />
+  <xacro:property name="wheel_mass" value="0.4" />
+  <xacro:property name="wheel_width" value="0.050" />
+  <xacro:macro name="do100_mecanum_wheel" params="prefix side *joint_pose">
     <link name="${prefix}_wheel_link">
       <visual>
         <origin xyz="0 ${side * 0.027} 0" rpy="0 0 ${PI/2}"/>
         <geometry>
-          <mesh filename="package://clearpath_platform_description/meshes/do100/mecanum_wheel.dae" scale="${side} 1 1" />
+          <mesh filename="package://clearpath_platform_description/meshes/do100/wheels/mecanum.dae" scale="${side} 1 1" />
         </geometry>
       </visual>

Commit message: Generic drivetrain URDFs

File: clearpath_platform_description/urdf/do100/do100.urdf.xacro (robot description, xacro)
@@ -4,9 +4,7 @@
   <xacro:arg name="is_sim" default="false" />
   <xacro:arg name="gazebo_controllers" default="$(find clearpath_control)/config/do100/control.yaml"/>
-  <!-- Included URDF/Xacro Files -->
-  <!-- <xacro:include filename="$(find clearpath_platform_description)/urdf/do100/wheels/wheel.urdf.xacro"/> -->
   <xacro:property name="PI" value="${math.pi}" />
   <!-- D0100 Platform Macro -->
-  <xacro:macro name="do100" params="drivetrain:='omni_4wd' wheels:='mecanum'">
+  <xacro:macro name="do100" params="control:='omni_4wd' front_wheels:='mecanum' rear_wheels:='mecanum'">
     <!-- Variables -->
     <xacro:property name="wheelbase" value="0.570" />
@@ -45,9 +43,21 @@
         </inertial>
     </link>
+    <!-- Add wheels -->
+    <xacro:include filename="$(find clearpath_platform_description)/urdf/do100/drivetrain/wheels.urdf.xacro"/>
+    <xacro:do100_drivetrain_wheels front_wheels="${front_wheels}" rear_wheels="${rear_wheels}"/>
     <!-- Add drivetrain -->
-    <xacro:if value="${drivetrain == 'omni_4wd'}">
-      <xacro:include filename="$(find clearpath_platform_description)/urdf/do100/drivetrain/type/omni_4wd.urdf.xacro"/>
-      <xacro:do100_drivetrain_type_omni wheels="${wheels}"/>
-    </xacro:if>
+    <xacro:include filename="$(find clearpath_platform_description)/urdf/generic/drivetrain/drivetrain.urdf.xacro"/>
+    <!-- Hardware  -->
+    <xacro:property name="hardware">
+      <xacro:if value="$(arg is_sim)">
+        <hardware plugin="gz_ros2_control/GazeboSimSystem"/>
+      </xacro:if>
+      <xacro:unless value="$(arg is_sim)">
+        <hardware plugin="clearpath_hardware_interfaces/PumaHardware"/>
+      </xacro:unless>
+    </xacro:property>
+    <xacro:generic_drivetrain name="do100" control="${control}" front_wheels="${front_wheels}" rear_wheels="${rear_wheels}">
+      <xacro:insert_block name="hardware"/>
+    </xacro:generic_drivetrain>
     <!-- Internal IMU -->
     <link name="imu_0_link">

File: clearpath_platform_description/urdf/do100/drivetrain/wheels/mecanum.urdf.xacro (robot description, xacro)
@@ -1,7 +1,7 @@
 <?xml version="1.0"?>
-<robot xmlns:xacro="http://ros.org/wiki/xacro" xmlns:ignition="http://gazebosim.org/schema" name="do100_wheel">
-  <xacro:property name="wheel_radius" value="0.050" />
-  <xacro:property name="wheel_mass" value="0.4" />
-  <xacro:property name="wheel_width" value="0.050" />
+<robot xmlns:xacro="http://ros.org/wiki/xacro" xmlns:ignition="http://gazebosim.org/schema" name="do100_mecanum_wheel">
+  <xacro:property name="do100_mecanum_wheel_radius" value="0.050" />
+  <xacro:property name="do100_mecanum_wheel_mass" value="0.4" />
+  <xacro:property name="do100_mecanum_wheel_width" value="0.050" />
   <xacro:macro name="do100_mecanum_wheel" params="prefix side *joint_pose">
     <link name="${prefix}_wheel_link">
@@ -15,16 +15,26 @@
         <origin xyz="0 0 0" rpy="${PI/2} 0 0"/>
         <geometry>
-          <cylinder radius="${wheel_radius}" length="${wheel_width}"/>
+          <cylinder radius="${do100_mecanum_wheel_radius}" length="${do100_mecanum_wheel_width}"/>
         </geometry>
       </collision>
       <inertial>
         <origin xyz="0 0 0" rpy="0 0 0"/>
-        <mass value="${wheel_mass}"/>
+        <mass value="${do100_mecanum_wheel_mass}"/>
         <inertia
-          ixx="${wheel_mass/12 * (3 * wheel_radius * wheel_radius + wheel_width * wheel_width)}" ixy="0" ixz="0"
-          iyy="${(wheel_radius * wheel_radius * wheel_mass)/2}" iyz="0"
-          izz="${wheel_mass/12 * (3 * wheel_radius * wheel_radius + wheel_width * wheel_width)}"/>
+          ixx="${do100_mecanum_wheel_mass/12 * (3 * do100_mecanum_wheel_radius * do100_mecanum_wheel_radius + do100_mecanum_wheel_width * do100_mecanum_wheel_width)}" ixy="0" ixz="0"
+          iyy="${(do100_mecanum_wheel_radius * do100_mecanum_wheel_radius * do100_mecanum_wheel_mass)/2}" iyz="0"
+          izz="${do100_mecanum_wheel_mass/12 * (3 * do100_mecanum_wheel_radius * do100_mecanum_wheel_radius + do100_mecanum_wheel_width * do100_mecanum_wheel_width)}"/>
       </inertial>
     </link>
+    <gazebo>
+      <plugin filename="libgz-sim-wheel-slip-system.so" name="gz::sim::systems::WheelSlip">
+        <wheel link_name="${prefix}_wheel_link">
+          <slip_compliance_lateral>1.0</slip_compliance_lateral>
+          <slip_compliance_longitudinal>1.0</slip_compliance_longitudinal>
+          <wheel_normal_force>20</wheel_normal_force>
+          <do100_mecanum_wheel_radius>${do100_mecanum_wheel_radius}</do100_mecanum_wheel_radius>
+        </wheel>
+      </plugin>
+    </gazebo>
     <gazebo reference="${prefix}_wheel_link">
       <collision>
