Commit message: Pass hardware plugin string rather than block

File: clearpath_platform_description/urdf/do100/do100.urdf.xacro (robot description, xacro)
@@ -49,15 +49,17 @@
     <xacro:include filename="$(find clearpath_platform_description)/urdf/generic/drivetrain/drivetrain.urdf.xacro"/>
     <!-- Hardware  -->
-    <xacro:property name="hardware">
-      <xacro:if value="$(arg is_sim)">
-        <hardware plugin="gz_ros2_control/GazeboSimSystem"/>
-      </xacro:if>
-      <xacro:unless value="$(arg is_sim)">
-        <hardware plugin="clearpath_hardware_interfaces/PumaHardware"/>
-      </xacro:unless>
-    </xacro:property>
-    <xacro:generic_drivetrain name="do100" control="${control}" front_wheels="${front_wheels}" rear_wheels="${rear_wheels}">
-      <xacro:insert_block name="hardware"/>
-    </xacro:generic_drivetrain>
+    <xacro:if value="$(arg is_sim)">
+      <xacro:property name="hardware_plugin" value="gz_ros2_control/GazeboSimSystem"/>
+    </xacro:if>
+    <xacro:unless value="$(arg is_sim)">
+      <xacro:property name="hardware_plugin" value="clearpath_hardware_interfaces/PumaHardware"/>
+    </xacro:unless>
+    <xacro:generic_drivetrain
+      name="do100"
+      control="${control}"
+      front_wheels="${front_wheels}"
+      rear_wheels="${rear_wheels}"
+      hardware_plugin="${hardware_plugin}"
+    />
     <!-- Internal IMU -->
     <link name="imu_0_link">

File: clearpath_platform_description/urdf/generic/drivetrain/control/diff_4wd.urdf.xacro (robot description, xacro)
@@ -1,8 +1,8 @@
 <?xml version="1.0"?>
 <robot xmlns:xacro="http://ros.org/wiki/xacro" xmlns:ignition="http://gazebosim.org/schema" name="generic_drivetrain_control_diff_4wd">
-  <xacro:macro name="generic_drivetrain_control_diff_4wd" params="name *hardware">
+  <xacro:macro name="generic_drivetrain_control_diff_4wd" params="name hardware_plugin">
     <!-- This is the same as omni_4wd -->
     <xacro:include filename="$(find clearpath_platform_description)/urdf/generic/drivetrain/control/omni_4wd.urdf.xacro"/>
-    <xacro:generic_drivetrain_control_omni_4wd name="${name}" hardware="${hardware}"/>
+    <xacro:generic_drivetrain_control_omni_4wd name="${name}" hardware_plugin="${hardware_plugin}"/>
   </xacro:macro>
 </robot>

File: clearpath_platform_description/urdf/generic/drivetrain/control/diff_fwd.urdf.xacro (robot description, xacro)
@@ -1,10 +1,12 @@
 <?xml version="1.0"?>
 <robot xmlns:xacro="http://ros.org/wiki/xacro" xmlns:ignition="http://gazebosim.org/schema" name="generic_drivetrain_control_diff_fwd">
-  <xacro:macro name="generic_drivetrain_control_diff_fwd" params="name *hardware">
+  <xacro:macro name="generic_drivetrain_control_diff_fwd" params="name hardware_plugin">
     <!-- Gazebo Controller -->
     <xacro:include filename="$(find clearpath_platform_description)/urdf/generic/gazebo.urdf.xacro"/>
     <!-- ROS2 controls -->
     <ros2_control name="${name}_hardware" type="system">
-      <xacro:insert_block name="hardware"/>
+      <hardware>
+        <plugin>${hardware_plugin}</plugin>
+      </hardware>
       <joint name="front_left_wheel_joint">
         <command_interface name="velocity"/>

File: clearpath_platform_description/urdf/generic/drivetrain/control/diff_rwd.urdf.xacro (robot description, xacro)
@@ -1,10 +1,12 @@
 <?xml version="1.0"?>
 <robot xmlns:xacro="http://ros.org/wiki/xacro" xmlns:ignition="http://gazebosim.org/schema" name="generic_drivetrain_control_diff_rwd">
-  <xacro:macro name="generic_drivetrain_control_diff_rwd" params="name *hardware">
+  <xacro:macro name="generic_drivetrain_control_diff_rwd" params="name hardware_plugin">
     <!-- Gazebo Controller -->
     <xacro:include filename="$(find clearpath_platform_description)/urdf/generic/gazebo.urdf.xacro"/>
     <!-- ROS2 controls -->
     <ros2_control name="${name}_hardware" type="system">
-      <xacro:insert_block name="hardware"/>
+      <hardware>
+        <plugin>${hardware_plugin}</plugin>
+      </hardware>
       <joint name="rear_left_wheel_joint">
         <command_interface name="velocity"/>

File: clearpath_platform_description/urdf/generic/drivetrain/control/omni_4wd.urdf.xacro (robot description, xacro)
@@ -1,10 +1,12 @@
 <?xml version="1.0"?>
 <robot xmlns:xacro="http://ros.org/wiki/xacro" xmlns:ignition="http://gazebosim.org/schema" name="generic_drivetrain_control_omni_4wd">
-  <xacro:macro name="generic_drivetrain_control_omni_4wd" params="name *hardware">
+  <xacro:macro name="generic_drivetrain_control_omni_4wd" params="name hardware_plugin">
     <!-- Gazebo Controller -->
     <xacro:include filename="$(find clearpath_platform_description)/urdf/generic/gazebo.urdf.xacro"/>
     <!-- ROS2 controls -->
     <ros2_control name="${name}_hardware" type="system">
-      <xacro:insert_block name="hardware"/>
+      <hardware>
+        <plugin>${hardware_plugin}</plugin>
+      </hardware>
       <joint name="front_left_wheel_joint">
         <command_interface name="velocity"/>

File: clearpath_platform_description/urdf/generic/drivetrain/drivetrain.urdf.xacro (robot description, xacro)
@@ -1,32 +1,27 @@
 <?xml version="1.0"?>
 <robot xmlns:xacro="http://ros.org/wiki/xacro" xmlns:ignition="http://gazebosim.org/schema" name="generic_drivetrain">
-  <xacro:macro name="generic_drivetrain" params="name control front_wheels rear_wheels *hardware">
+  <xacro:macro name="generic_drivetrain" params="name control front_wheels rear_wheels hardware_plugin">
+    <xacro:property name="hardware">
+      <hardware plugin="${hardware_plugin}"/>
+    </xacro:property>
     <!-- Omni drivetrain -->
     <xacro:if value="${control == 'omni_4wd'}">
       <xacro:include filename="$(find clearpath_platform_description)/urdf/generic/drivetrain/control/omni_4wd.urdf.xacro"/>
-      <xacro:generic_drivetrain_control_omni_4wd name="${name}">
-        <xacro:insert_block name="hardware"/>
-      </xacro:generic_drivetrain_control_omni_4wd>
+      <xacro:generic_drivetrain_control_omni_4wd name="${name}" hardware_plugin="${hardware_plugin}"/>
     </xacro:if>
     <!-- Diff 4WD drivetrain -->
     <xacro:if value="${control == 'diff_4wd'}">
       <xacro:include filename="$(find clearpath_platform_description)/urdf/generic/drivetrain/control/diff_4wd.urdf.xacro"/>
-      <xacro:generic_drivetrain_control_diff_4wd name="${name}">
-        <xacro:insert_block name="hardware"/>
-      </xacro:generic_drivetrain_control_diff_4wd>
+      <xacro:generic_drivetrain_control_diff_4wd name="${name}" hardware_plugin="${hardware_plugin}"/>
     </xacro:if>
     <!-- Diff FWD drivetrain -->
     <xacro:if value="${control == 'diff_fwd'}">
       <xacro:include filename="$(find clearpath_platform_description)/urdf/generic/drivetrain/control/diff_fwd.urdf.xacro"/>
-      <xacro:generic_drivetrain_control_diff_fwd name="${name}">
-        <xacro:insert_block name="hardware"/>
-      </xacro:generic_drivetrain_control_diff_fwd>
+      <xacro:generic_drivetrain_control_diff_fwd name="${name}" hardware_plugin="${hardware_plugin}"/>
     </xacro:if>
     <!-- Diff RWD drivetrain -->
     <xacro:if value="${control == 'diff_rwd'}">
       <xacro:include filename="$(find clearpath_platform_description)/urdf/generic/drivetrain/control/diff_rwd.urdf.xacro"/>
-      <xacro:generic_drivetrain_control_diff_rwd name="${name}">
-        <xacro:insert_block name="hardware"/>
-      </xacro:generic_drivetrain_control_diff_rwd>
+      <xacro:generic_drivetrain_control_diff_rwd name="${name}" hardware_plugin="${hardware_plugin}"/>
     </xacro:if>
   </xacro:macro>

Commit message: Removed 2WD for Dingo-O

File: clearpath_platform_description/urdf/do100/do100.urdf.xacro (robot description, xacro)
@@ -54,4 +54,7 @@
     <xacro:unless value="$(arg is_sim)">
       <xacro:property name="hardware_plugin" value="clearpath_hardware_interfaces/PumaHardware"/>
+    </xacro:unless>
+    <xacro:unless value="${control == 'omni_4wd' or control == 'diff_4wd'}">
+      <xacro:error message="Invalid drivetrain control ${control}"/>
     </xacro:unless>
     <xacro:generic_drivetrain

File: clearpath_platform_description/urdf/generic/drivetrain/drivetrain.urdf.xacro (robot description, xacro)
@@ -2,7 +2,4 @@
 <robot xmlns:xacro="http://ros.org/wiki/xacro" xmlns:ignition="http://gazebosim.org/schema" name="generic_drivetrain">
   <xacro:macro name="generic_drivetrain" params="name control front_wheels rear_wheels hardware_plugin">
-    <xacro:property name="hardware">
-      <hardware plugin="${hardware_plugin}"/>
-    </xacro:property>
     <!-- Omni drivetrain -->
     <xacro:if value="${control == 'omni_4wd'}">

Commit message: DO150

File: clearpath_platform_description/urdf/do100/do100.urdf.xacro (robot description, xacro)
@@ -3,5 +3,5 @@
   <xacro:arg name="namespace" default="" />
   <xacro:arg name="is_sim" default="false" />
-  <xacro:arg name="gazebo_controllers" default="$(find clearpath_control)/config/do100/control.yaml"/>
+  <xacro:arg name="gazebo_controllers" default="$(find clearpath_control)/config/do100/control/omni_4wd.yaml"/>
   <xacro:property name="PI" value="${math.pi}" />
   <!-- D0100 Platform Macro -->

File: clearpath_platform_description/urdf/do150/do150.urdf.xacro (robot description, xacro)
@@ -3,17 +3,147 @@
   <xacro:arg name="namespace" default="" />
   <xacro:arg name="is_sim" default="false" />
-  <xacro:arg name="gazebo_controllers" default="$(find clearpath_control)/config/do150/control.yaml"/>
-  <!-- Included URDF/Xacro Files -->
-  <xacro:include filename="$(find clearpath_platform_description)/urdf/do100/do100.urdf.xacro"/>
-  <!-- D0100 Platform Macro -->
-  <xacro:macro name="do150" params="wheel:='defaut'">
-    <xacro:do100 wheel="${wheel}"/>
+  <xacro:arg name="gazebo_controllers" default="$(find clearpath_control)/config/do150/control/omni_4wd.yaml"/>
+  <xacro:property name="PI" value="${math.pi}" />
+  <!-- D0150 Platform Macro -->
+  <xacro:macro name="do150" params="control:='omni_4wd' front_wheels:='mecanum' rear_wheels:='mecanum'">
+    <!-- Variables -->
+    <xacro:property name="wheelbase" value="0.570" />
+    <xacro:property name="track" value="0.3708" />
+    <xacro:property name="wheel_vertical_offset" value="0.035145" />
+    <xacro:property name="dummy_inertia" value="1e-09"/>
+    <!-- Chassis -->
+    <link name="base_link"></link>
+    <joint name="base_link_joint" type="fixed">
+      <origin xyz="0 0 0" rpy="0 0 0" />
+      <parent link="base_link"/>
+      <child link="chassis_link" />
+    </joint>
+    <link name="chassis_link">
+      <visual>
+        <origin xyz="0 0 0" rpy="0 0 0"/>
+        <geometry>
+          <mesh filename="package://clearpath_platform_description/meshes/do100/omni_chassis.dae"/>
+        </geometry>
+      </visual>
+      <collision>
+        <origin xyz="0 0 0"/>
+        <geometry>
+          <mesh filename="package://clearpath_platform_description/meshes/do100/omni_chassis_collision.stl"/>
+        </geometry>
+      </collision>
+      <inertial>
+        <!-- Center of mass -->
+        <origin xyz="0 0 0" rpy="0 0 0"/>
+        <mass value="14"/>
+        <!-- Moments of inertia: ( chassis without wheels ) -->
+        <inertia
+          ixx="0.35498" ixy="0" ixz="0"
+          iyy="0.7266" iyz="0"
+          izz="1.0553"/>
+        </inertial>
+    </link>
+    <!-- Add wheels (Same as DO100) -->
+    <xacro:include filename="$(find clearpath_platform_description)/urdf/do100/drivetrain/wheels.urdf.xacro"/>
+    <xacro:do100_drivetrain_wheels front_wheels="${front_wheels}" rear_wheels="${rear_wheels}"/>
+    <!-- Add drivetrain -->
+    <xacro:include filename="$(find clearpath_platform_description)/urdf/generic/drivetrain/drivetrain.urdf.xacro"/>
+    <!-- Hardware  -->
+    <xacro:if value="$(arg is_sim)">
+      <xacro:property name="hardware_plugin" value="gz_ros2_control/GazeboSimSystem"/>
+    </xacro:if>
+    <xacro:unless value="$(arg is_sim)">
+      <xacro:property name="hardware_plugin" value="clearpath_hardware_interfaces/PumaHardware"/>
+    </xacro:unless>
+    <xacro:unless value="${control == 'omni_4wd' or control == 'diff_4wd'}">
+      <xacro:error message="Invalid drivetrain control ${control}"/>
+    </xacro:unless>
+    <xacro:generic_drivetrain
+      name="do150"
+      control="${control}"
+      front_wheels="${front_wheels}"
+      rear_wheels="${rear_wheels}"
+      hardware_plugin="${hardware_plugin}"
+    />
+    <!-- Internal IMU -->
+    <link name="imu_0_link">
+      <inertial>
+        <mass value="0.001"/>
+        <origin xyz="0 0 0" rpy="0 0 0"/>
+        <inertia ixx="${dummy_inertia}" ixy="0.0" ixz="0.0" iyy="${dummy_inertia}" iyz="0.0" izz="${dummy_inertia}"/>
+      </inertial>
+    </link>
+    <joint name="imu_joint" type="fixed">
+      <parent link="chassis_link" />
+      <child link="imu_0_link" />
+    </joint>
+    <gazebo reference="imu_0_link">
+      <sensor type="imu" name="imu_0">
+        <always_on>true</always_on>
+        <update_rate>50</update_rate>
+        <visualize>true</visualize>
+        <gz_frame_id>imu_0_link</gz_frame_id>
+      </sensor>
+    </gazebo>
+    <!-- Mounting Hard Points -->
+    <link name="default_mount"/>
+    <link name="front_2_mount"/>
+    <link name="front_1_mount"/>
+    <link name="front_0_mount"/>
+    <link name="rear_2_mount"/>
+    <link name="rear_1_mount"/>
+    <link name="rear_0_mount"/>
+    <joint name="default_mount_joint" type="fixed">
+      <origin xyz="0 0 0.069023" rpy="0 0 0" />
+      <parent link="chassis_link"/>
+      <child link="default_mount" />
+    </joint>
+    <joint name="front_0_mount_joint" type="fixed">
+      <origin xyz="0.080 0 0" rpy="0 0 0" />
+      <parent link="default_mount"/>
+      <child link="front_0_mount" />
+    </joint>
+    <joint name="front_1_mount_joint" type="fixed">
+      <origin xyz="0.080 0 0" rpy="0 0 0" />
+      <parent link="front_0_mount"/>
+      <child link="front_1_mount" />
+    </joint>
+    <joint name="front_2_mount_joint" type="fixed">
+      <origin xyz="0.080 0 0" rpy="0 0 0" />
+      <parent link="front_1_mount"/>
+      <child link="front_2_mount" />
+    </joint>
+    <joint name="rear_0_mount_joint" type="fixed">
+      <origin xyz="-0.080 0 0" rpy="0 0 0" />
+      <parent link="default_mount"/>
+      <child link="rear_0_mount" />
+    </joint>
+    <joint name="rear_1_mount_joint" type="fixed">
+      <origin xyz="-0.080 0 0" rpy="0 0 0" />
+      <parent link="rear_0_mount"/>
+      <child link="rear_1_mount" />
+    </joint>
+    <joint name="rear_2_mount_joint" type="fixed">
+      <origin xyz="-0.080 0 0" rpy="0 0 0" />
+      <parent link="rear_1_mount"/>
+      <child link="rear_2_mount" />
+    </joint>
+    <!-- Bumper Mounts -->
+    <link name="front_bumper_mount"/>
+    <link name="rear_bumper_mount"/>
+    <joint name="front_bumper_mount_joint" type="fixed">
+      <origin xyz="0.34159 0 0.0345115" rpy="0 0 0" />
+      <parent link="chassis_link"/>
+      <child link="front_bumper_mount" />
+    </joint>
+    <joint name="rear_bumper_mount_joint" type="fixed">
+      <origin xyz="-0.34159 0 0.0345115" rpy="0 0 0" />
+      <parent link="chassis_link"/>
+      <child link="rear_bumper_mount" />
+    </joint>
   </xacro:macro>
   <!-- Joint State Publisher -->
-  <gazebo>
-    <plugin
-      filename="ignition-gazebo-joint-state-publisher-system"
-      name="ignition::gazebo::systems::JointStatePublisher"
-    />
-  </gazebo>
+  <plugin
+    filename="gz-sim-joint-state-publisher-system"
+    name="gz::sim::systems::JointStatePublisher"
+  />
 </robot>

Commit message: Drivetrains (#237)
* Moved meshes to wheels folder
Mecanum drivetrain for do100

* Generic drivetrain URDFs

* Pass hardware plugin string rather than block

* Added drivetrain control parameters

* Removed 2WD for Dingo-O

* DO150

* Dingo-D

* R100

* A300 urdf

* Fixed xacro generate print

* Generic teleop configs per controller
Platform specific teleop only defines velocity limits

* A200 drivetrain changes

* W200 drivetrain urdf

* Updated A300 meshes
Mecanum and caster support

* Separated caster wheel into swivel and wheel links

* Fixed joystick axis mapping

* Updated wheel_separation_multiplier for fwd and rwd on A300

* URDF structure changes for J100
Updated A200 and W200 to be 4WD

* Linting

File: clearpath_platform_description/urdf/do100/do100.urdf.xacro (robot description, xacro)
@@ -3,17 +3,12 @@
   <xacro:arg name="namespace" default="" />
   <xacro:arg name="is_sim" default="false" />
-  <xacro:arg name="gazebo_controllers" default="$(find clearpath_control)/config/do100/control.yaml"/>
-  <!-- Included URDF/Xacro Files -->
-  <xacro:include filename="$(find clearpath_platform_description)/urdf/do100/wheels/wheel.urdf.xacro"/>
+  <xacro:arg name="gazebo_controllers" default="$(find clearpath_control)/config/do100/control/omni_4wd.yaml"/>
   <xacro:property name="PI" value="${math.pi}" />
   <!-- D0100 Platform Macro -->
-  <xacro:macro name="do100" params="wheel:='defaut'">
+  <xacro:macro name="do100" params="control:='omni_4wd' front_wheels:='mecanum' rear_wheels:='mecanum'">
     <!-- Variables -->
     <xacro:property name="wheelbase" value="0.570" />
     <xacro:property name="track" value="0.3708" />
     <xacro:property name="wheel_vertical_offset" value="0.035145" />
-    <xacro:property name="wheel_radius" value="0.050" />
-    <xacro:property name="wheel_mass" value="0.4" />
-    <xacro:property name="wheel_width" value="0.050" />
     <xacro:property name="dummy_inertia" value="1e-09"/>
     <!-- Chassis -->
@@ -48,45 +43,26 @@
         </inertial>
     </link>
-    <!-- Wheels -->
-    <xacro:do100_wheel prefix="front_left" side="-1">
-      <origin xyz="${wheelbase/2} ${track/2+wheel_width/2} ${wheel_vertical_offset}" rpy="0 0 0" />
-    </xacro:do100_wheel>
-    <xacro:do100_wheel prefix="front_right" side="1">
-      <origin xyz="${wheelbase/2} ${-track/2-wheel_width/2} ${wheel_vertical_offset}" rpy="0 0 0" />
-    </xacro:do100_wheel>
-    <xacro:do100_wheel prefix="rear_left" side="1">
-      <origin xyz="${-wheelbase/2} ${track/2+wheel_width/2} ${wheel_vertical_offset}" rpy="0 0 0" />
-    </xacro:do100_wheel>
-    <xacro:do100_wheel prefix="rear_right" side="-1">
-      <origin xyz="${-wheelbase/2} ${-track/2-wheel_width/2} ${wheel_vertical_offset}" rpy="0 0 0" />
-    </xacro:do100_wheel>
-    <gazebo>
-      <plugin filename="libgz-sim-wheel-slip-system.so" name="gz::sim::systems::WheelSlip">
-        <wheel link_name="front_left_wheel_link">
-          <slip_compliance_lateral>1.0</slip_compliance_lateral>
-          <slip_compliance_longitudinal>1.0</slip_compliance_longitudinal>
-          <wheel_normal_force>20</wheel_normal_force>
-          <wheel_radius>${wheel_radius}</wheel_radius>
-        </wheel>
-        <wheel link_name="front_right_wheel_link">
-          <slip_compliance_lateral>1.0</slip_compliance_lateral>
-          <slip_compliance_longitudinal>1.0</slip_compliance_longitudinal>
-          <wheel_normal_force>20</wheel_normal_force>
-          <wheel_radius>${wheel_radius}</wheel_radius>
-        </wheel>
-        <wheel link_name="rear_left_wheel_link">
-          <slip_compliance_lateral>1.0</slip_compliance_lateral>
-          <slip_compliance_longitudinal>1.0</slip_compliance_longitudinal>
-          <wheel_normal_force>20</wheel_normal_force>
-          <wheel_radius>${wheel_radius}</wheel_radius>
-        </wheel>
-        <wheel link_name="rear_right_wheel_link">
-          <slip_compliance_lateral>1.0</slip_compliance_lateral>
-          <slip_compliance_longitudinal>1.0</slip_compliance_longitudinal>
-          <wheel_normal_force>20</wheel_normal_force>
-          <wheel_radius>${wheel_radius}</wheel_radius>
-        </wheel>
-      </plugin>
-    </gazebo>
+    <!-- Add wheels -->
+    <xacro:include filename="$(find clearpath_platform_description)/urdf/do100/drivetrain/wheels.urdf.xacro"/>
+    <xacro:do100_drivetrain_wheels front_wheels="${front_wheels}" rear_wheels="${rear_wheels}"/>
+    <!-- Add drivetrain -->
+    <xacro:include filename="$(find clearpath_platform_description)/urdf/generic/drivetrain/drivetrain.urdf.xacro"/>
+    <!-- Hardware  -->
+    <xacro:if value="$(arg is_sim)">
+      <xacro:property name="hardware_plugin" value="gz_ros2_control/GazeboSimSystem"/>
+    </xacro:if>
+    <xacro:unless value="$(arg is_sim)">
+      <xacro:property name="hardware_plugin" value="clearpath_hardware_interfaces/PumaHardware"/>
+    </xacro:unless>
+    <xacro:unless value="${control == 'omni_4wd' or control == 'diff_4wd'}">
+      <xacro:error message="Invalid drivetrain control ${control}"/>
+    </xacro:unless>
+    <xacro:generic_drivetrain
+      name="do100"
+      control="${control}"
+      front_wheels="${front_wheels}"
+      rear_wheels="${rear_wheels}"
+      hardware_plugin="${hardware_plugin}"
+    />
     <!-- Internal IMU -->
     <link name="imu_0_link">
@@ -165,37 +141,4 @@
       <child link="rear_bumper_mount" />
     </joint>
-    <!-- Gazebo Controller -->
-    <xacro:include filename="$(find clearpath_platform_description)/urdf/generic/gazebo.urdf.xacro"/>
-    <!-- ROS2 controls -->
-    <ros2_control name="do100_hardware" type="system">
-      <hardware>
-        <xacro:if value="$(arg is_sim)">
-          <plugin>gz_ros2_control/GazeboSimSystem</plugin>
-        </xacro:if>
-        <xacro:unless value="$(arg is_sim)">
-          <plugin>clearpath_hardware_interfaces/PumaHardware</plugin>
-        </xacro:unless>
-      </hardware>
-      <joint name="front_left_wheel_joint">
-        <command_interface name="velocity"/>
-        <state_interface name="position"/>
-        <state_interface name="velocity"/>
-      </joint>
-      <joint name="front_right_wheel_joint">
-        <command_interface name="velocity"/>
-        <state_interface name="position"/>
-        <state_interface name="velocity"/>
-      </joint>
-      <joint name="rear_left_wheel_joint">
-        <command_interface name="velocity"/>
-        <state_interface name="position"/>
-        <state_interface name="velocity"/>
-      </joint>
-      <joint name="rear_right_wheel_joint">
-        <command_interface name="velocity"/>
-        <state_interface name="position"/>
-        <state_interface name="velocity"/>
-      </joint>
-    </ros2_control>
   </xacro:macro>
   <!-- Joint State Publisher -->
