Commit message: Added argument to toggle manipulator controllers

File: clearpath_manipulators_description/urdf/arm/kinova_gen3_lite.urdf.xacro (robot description, xacro)
@@ -3,4 +3,5 @@
   <xacro:arg name="is_sim" default="false"/>
   <xacro:arg name="use_fake_hardware" default="false"/>
+  <xacro:arg name="use_manipulation_controllers" default="false"/>
   <xacro:macro name="kinova_gen3_lite" params="
     name
@@ -22,4 +23,5 @@
     gripper_max_force:=100.0
     use_fake_hardware:=$(arg use_fake_hardware)
+    use_controllers:=$(arg use_manipulation_controllers)
     fake_sensor_commands:=false
     sim_gazebo:=false
@@ -234,114 +236,116 @@
     </joint>
     <!-- ROS2 Controls -->
-    <ros2_control name="${name}_hardware" type="system">
-      <hardware>
-        <xacro:if value="${sim_gazebo}">
-          <plugin>gazebo_ros2_control/GazeboSystem</plugin>
-        </xacro:if>
-        <xacro:if value="${sim_ignition}">
-          <plugin>ign_ros2_control/IgnitionSystem</plugin>
-        </xacro:if>
-        <xacro:if value="${sim_isaac}">
-          <plugin>topic_based_ros2_control/TopicBasedSystem</plugin>
-          <param name="joint_commands_topic">${isaac_joint_commands}</param>
-          <param name="joint_states_topic">${isaac_joint_states}</param>
-        </xacro:if>
-        <xacro:if value="${use_fake_hardware}">
-          <plugin>mock_components/GenericSystem</plugin>
-          <param name="fake_sensor_commands">${fake_sensor_commands}</param>
-          <param name="state_following_offset">0.0</param>
-        </xacro:if>
+    <xacro:if value="${use_controllers}">
+      <ros2_control name="${name}_hardware" type="system">
+        <hardware>
+          <xacro:if value="${sim_gazebo}">
+            <plugin>gazebo_ros2_control/GazeboSystem</plugin>
+          </xacro:if>
+          <xacro:if value="${sim_ignition}">
+            <plugin>ign_ros2_control/IgnitionSystem</plugin>
+          </xacro:if>
+          <xacro:if value="${sim_isaac}">
+            <plugin>topic_based_ros2_control/TopicBasedSystem</plugin>
+            <param name="joint_commands_topic">${isaac_joint_commands}</param>
+            <param name="joint_states_topic">${isaac_joint_states}</param>
+          </xacro:if>
+          <xacro:if value="${use_fake_hardware}">
+            <plugin>mock_components/GenericSystem</plugin>
+            <param name="fake_sensor_commands">${fake_sensor_commands}</param>
+            <param name="state_following_offset">0.0</param>
+          </xacro:if>
+          <xacro:unless value="${use_fake_hardware or sim_gazebo or sim_ignition or sim_isaac}">
+            <plugin>kortex_driver/KortexMultiInterfaceHardware</plugin>
+            <param name="robot_ip">${robot_ip}</param>
+            <param name="username">${username}</param>
+            <param name="password">${password}</param>
+            <param name="port">${port}</param>
+            <param name="port_realtime">${port_realtime}</param>
+            <param name="session_inactivity_timeout_ms">${session_inactivity_timeout_ms}</param>
+            <param name="connection_inactivity_timeout_ms">${connection_inactivity_timeout_ms}</param>
+            <param name="tf_prefix">"${tf_prefix}"</param>
+            <param name="use_internal_bus_gripper_comm">${use_internal_bus_gripper_comm}</param>
+            <param name="gripper_joint_name">${gripper_joint_name}</param>
+            <param name="gripper_max_velocity">${gripper_max_velocity}</param>
+            <param name="gripper_max_force">${gripper_max_force}</param>
+          </xacro:unless>
+        </hardware>
+        <joint name="${name}_joint_1">
+          <command_interface name="position">
+            <param name="min">-2.69</param>
+            <param name="max">2.69</param>
+          </command_interface>
+          <state_interface name="position">
+            <param name="initial_value">${initial_positions['joint_1']}</param>
+          </state_interface>
+          <state_interface name="velocity"/>
+          <state_interface name="effort"/>
+        </joint>
+        <joint name="${name}_joint_2">
+          <command_interface name="position">
+            <param name="min">-2.69</param>
+            <param name="max">2.36</param>
+          </command_interface>
+          <state_interface name="position">
+            <param name="initial_value">${initial_positions['joint_2']}</param>
+          </state_interface>
+          <state_interface name="velocity"/>
+          <state_interface name="effort"/>
+        </joint>
+        <joint name="${name}_joint_3">
+          <command_interface name="position">
+            <param name="min">-2.69</param>
+            <param name="max">2.69</param>
+          </command_interface>
+          <state_interface name="position">
+            <param name="initial_value">${initial_positions['joint_3']}</param>
+          </state_interface>
+          <state_interface name="velocity"/>
+          <state_interface name="effort"/>
+        </joint>
+        <joint name="${name}_joint_4">
+          <command_interface name="position">
+            <param name="min">-2.59</param>
+            <param name="max">2.59</param>
+          </command_interface>
+          <state_interface name="position">
+            <param name="initial_value">${initial_positions['joint_4']}</param>
+          </state_interface>
+          <state_interface name="velocity"/>
+          <state_interface name="effort"/>
+        </joint>
+        <joint name="${name}_joint_5">
+          <command_interface name="position">
+            <param name="min">-2.57</param>
+            <param name="max">2.57</param>
+          </command_interface>
+          <state_interface name="position">
+            <param name="initial_value">${initial_positions['joint_5']}</param>
+          </state_interface>
+          <state_interface name="velocity"/>
+          <state_interface name="effort"/>
+        </joint>
+        <joint name="${name}_joint_6">
+          <command_interface name="position">
+            <param name="min">-2.59</param>
+            <param name="max">2.59</param>
+          </command_interface>
+          <state_interface name="position">
+            <param name="initial_value">${initial_positions['joint_6']}</param>
+          </state_interface>
+          <state_interface name="velocity"/>
+          <state_interface name="effort"/>
+        </joint>
         <xacro:unless value="${use_fake_hardware or sim_gazebo or sim_ignition or sim_isaac}">
-          <plugin>kortex_driver/KortexMultiInterfaceHardware</plugin>
-          <param name="robot_ip">${robot_ip}</param>
-          <param name="username">${username}</param>
-          <param name="password">${password}</param>
-          <param name="port">${port}</param>
-          <param name="port_realtime">${port_realtime}</param>
-          <param name="session_inactivity_timeout_ms">${session_inactivity_timeout_ms}</param>
-          <param name="connection_inactivity_timeout_ms">${connection_inactivity_timeout_ms}</param>
-          <param name="tf_prefix">"${tf_prefix}"</param>
-          <param name="use_internal_bus_gripper_comm">${use_internal_bus_gripper_comm}</param>
-          <param name="gripper_joint_name">${gripper_joint_name}</param>
-          <param name="gripper_max_velocity">${gripper_max_velocity}</param>
-          <param name="gripper_max_force">${gripper_max_force}</param>
+          <xacro:if value="${use_internal_bus_gripper_comm}">
+            <joint name="gripper_0_right_finger_bottom_joint">
+              <command_interface name="position"/>
+              <state_interface name="position"/>
+              <state_interface name="velocity"/>
+            </joint>
+          </xacro:if>
         </xacro:unless>
-      </hardware>
-      <joint name="${name}_joint_1">
-        <command_interface name="position">
-          <param name="min">-2.69</param>
-          <param name="max">2.69</param>
-        </command_interface>
-        <state_interface name="position">
-          <param name="initial_value">${initial_positions['joint_1']}</param>
-        </state_interface>
-        <state_interface name="velocity"/>
-        <state_interface name="effort"/>
-      </joint>
-      <joint name="${name}_joint_2">
-        <command_interface name="position">
-          <param name="min">-2.69</param>
-          <param name="max">2.36</param>
-        </command_interface>
-        <state_interface name="position">
-          <param name="initial_value">${initial_positions['joint_2']}</param>
-        </state_interface>
-        <state_interface name="velocity"/>
-        <state_interface name="effort"/>
-      </joint>
-      <joint name="${name}_joint_3">
-        <command_interface name="position">
-          <param name="min">-2.69</param>
-          <param name="max">2.69</param>
-        </command_interface>
-        <state_interface name="position">
-          <param name="initial_value">${initial_positions['joint_3']}</param>
-        </state_interface>
-        <state_interface name="velocity"/>
-        <state_interface name="effort"/>
-      </joint>
-      <joint name="${name}_joint_4">
-        <command_interface name="position">
-          <param name="min">-2.59</param>
-          <param name="max">2.59</param>
-        </command_interface>
-        <state_interface name="position">
-          <param name="initial_value">${initial_positions['joint_4']}</param>
-        </state_interface>
-        <state_interface name="velocity"/>
-        <state_interface name="effort"/>
-      </joint>
-      <joint name="${name}_joint_5">
-        <command_interface name="position">
-          <param name="min">-2.57</param>
-          <param name="max">2.57</param>
-        </command_interface>
-        <state_interface name="position">
-          <param name="initial_value">${initial_positions['joint_5']}</param>
-        </state_interface>
-        <state_interface name="velocity"/>
-        <state_interface name="effort"/>
-      </joint>
-      <joint name="${name}_joint_6">
-        <command_interface name="position">
-          <param name="min">-2.59</param>
-          <param name="max">2.59</param>
-        </command_interface>
-        <state_interface name="position">
-          <param name="initial_value">${initial_positions['joint_6']}</param>
-        </state_interface>
-        <state_interface name="velocity"/>
-        <state_interface name="effort"/>
-      </joint>
-      <xacro:unless value="${use_fake_hardware or sim_gazebo or sim_ignition or sim_isaac}">
-        <xacro:if value="${use_internal_bus_gripper_comm}">
-          <joint name="gripper_0_right_finger_bottom_joint">
-            <command_interface name="position"/>
-            <state_interface name="position"/>
-            <state_interface name="velocity"/>
-          </joint>
-        </xacro:if>
-      </xacro:unless>
-    </ros2_control>
+      </ros2_control>
+    </xacro:if>
   </xacro:macro>
 </robot>

File: clearpath_manipulators_description/urdf/gripper/kinova_2f_lite.urdf.xacro (robot description, xacro)
@@ -3,4 +3,5 @@
   <xacro:arg name="is_sim" default="false"/>
   <xacro:arg name="use_fake_hardware" default="false"/>
+  <xacro:arg name="use_manipulation_controllers" default="false"/>
   <xacro:macro name="kinova_2f_lite" params="
     name
@@ -8,4 +9,5 @@
     *origin
     use_fake_hardware:=$(arg use_fake_hardware)
+    use_controllers:=$(arg use_manipulation_controllers)
     fake_sensor_commands:=false
     sim_ignition:=$(arg is_sim)
@@ -182,5 +184,5 @@
       <mimic joint="${name}_right_finger_bottom_joint" multiplier="-0.676" offset="0.149" />
     </joint>
-    <xacro:if value="${use_fake_hardware or sim_gazebo or sim_ignition or sim_isaac}">
+    <xacro:if value="${use_controllers and (use_fake_hardware or sim_gazebo or sim_ignition or sim_isaac)}">
       <ros2_control name="${name}_hardware" type="system">
           <hardware>

Commit message: Remove prefix from Kinova gripper joint

File: clearpath_manipulators_description/urdf/arm/kinova_gen3_6dof.urdf.xacro (robot description, xacro)
@@ -482,5 +482,5 @@
         <xacro:unless value="${use_fake_hardware or sim_gazebo or sim_ignition or sim_isaac}">
           <xacro:if value="${use_internal_bus_gripper_comm}">
-            <joint name="${name}_${gripper_joint_name}">
+            <joint name="${gripper_joint_name}">
               <command_interface name="position" />
               <state_interface name="position"/>

File: clearpath_manipulators_description/urdf/arm/kinova_gen3_7dof.urdf.xacro (robot description, xacro)
@@ -612,5 +612,5 @@
         <xacro:unless value="${use_fake_hardware or sim_gazebo or sim_ignition or sim_isaac}">
           <xacro:if value="${use_internal_bus_gripper_comm}">
-            <joint name="${name}_${gripper_joint_name}">
+            <joint name="${gripper_joint_name}">
               <command_interface name="position" />
               <state_interface name="position"/>
