Commit message: Added all descriptions for kinova manipulators

File: clearpath_manipulators_description/urdf/arm/kinova_gen3_7dof.urdf.xacro (robot description, xacro)
@@ -1,13 +1,12 @@
 <?xml version="1.0"?>
 <robot xmlns:xacro="http://ros.org/wiki/xacro">
-  <!-- Propagate last link name information because it is the gripper's parent link -->
-  <xacro:property name="last_arm_link" value="end_effector_link"/>
-  <xacro:property name="PI" value="3.1415926535897931"/>
-  <xacro:macro name="kinova_gen3_6dof" params="
+  <xacro:arg name="is_sim" default="false"/>
+  <xacro:arg name="use_fake_hardware" default="false"/>
+  <xacro:macro name="kinova_gen3_7dof" params="
     name
     parent_link
     *origin
     tf_prefix:=''
-    dof:=6
+    dof:=7
     vision:=false
     robot_ip:=192.168.131.40
@@ -22,5 +21,5 @@
     gripper_max_velocity:=100.0
     gripper_max_force:=100.0
-    use_fake_hardware:=false
+    use_fake_hardware:=$(arg use_fake_hardware)
     fake_sensor_commands:=false
     sim_gazebo:=false
@@ -28,5 +27,6 @@
     sim_isaac:=false
     use_external_cable:=false
-    initial_positions:=${dict(joint_1=0.0,joint_2=0.0,joint_3=0.0,joint_4=0.0,joint_5=0.0,joint_6=0.0)}" >
+    initial_positions:=${dict(joint_1=0.0,joint_2=0.0,joint_3=0.0,joint_4=0.0,joint_5=0.0,joint_6=0.0,joint_7=0.0)}" >
+    <!-- Instantiate the Arm -->
     <joint name="${name}_base_joint" type="fixed">
       <xacro:insert_block name="origin" />
@@ -59,5 +59,5 @@
       <inertial>
         <origin xyz="-2.3E-05 -0.010364 -0.07336" rpy="0 0 0" />
-        <mass value="1.377" />
+        <mass value="1.3773" />
         <inertia ixx="0.00457" ixy="1E-06" ixz="2E-06" iyy="0.004831" iyz="0.000448" izz="0.001409" />
       </inertial>
@@ -80,12 +80,13 @@
     <xacro:if value="${use_external_cable}">
       <joint
-        name="${name}_joint_1"
-        type="revolute">
-        <origin
-          xyz="0 0 0.15643"
-          rpy="-3.1416 0.0 0.0" />
-        <parent link="${name}_base_link" />
-        <child link="${name}_shoulder_link" />
-        <axis xyz="0 0 1" />
+      name="${name}_joint_1"
+      type="revolute">
+        <origin xyz="0 0 0.15643" rpy="3.1416 2.7629E-18 -4.9305E-36" />
+        <parent
+          link="${name}_base_link" />
+        <child
+          link="${name}_shoulder_link" />
+        <axis
+          xyz="0 0 1" />
         <limit
           lower="${-2*PI}"
@@ -99,10 +100,11 @@
         name="${name}_joint_1"
         type="continuous">
-        <origin
-          xyz="0 0 0.15643"
-          rpy="-3.1416 0.0 0.0" />
-        <parent link="${name}_base_link" />
-        <child link="${name}_shoulder_link" />
-        <axis xyz="0 0 1" />
+        <origin xyz="0 0 0.15643" rpy="3.1416 2.7629E-18 -4.9305E-36" />
+        <parent
+          link="${name}_base_link" />
+        <child
+          link="${name}_shoulder_link" />
+        <axis
+          xyz="0 0 1" />
         <limit
           effort="39"
@@ -110,24 +112,14 @@
       </joint>
     </xacro:unless>
-    <link name="${name}_bicep_link">
+    <link name="${name}_half_arm_1_link">
       <inertial>
-        <origin
-          xyz="3.5E-05 -0.208207 -0.01889"
-          rpy="0 0 0" />
-        <mass value="1.262" />
-        <inertia
-          ixx="0.046752"
-          ixy="-9E-06"
-          ixz="0"
-          iyy="0.00085"
-          iyz="-9.8E-05"
-          izz="0.047188" />
+        <origin xyz="-4.4E-05 -0.09958 -0.013278" rpy="0 0 0" />
+        <mass value="1.1636" />
+        <inertia ixx="0.011088" ixy="5E-06" ixz="0" iyy="0.001072" iyz="-0.000691" izz="0.011255" />
       </inertial>
       <visual>
-        <origin
-          xyz="0 0 0"
-          rpy="0 0 0" />
-        <geometry>
-          <mesh filename="file://$(find kortex_description)/arms/gen3/${dof}dof/meshes/bicep_link.STL" />
+        <origin xyz="0 0 0" rpy="0 0 0" />
+        <geometry>
+          <mesh filename="file://$(find kortex_description)/arms/gen3/${dof}dof/meshes/half_arm_1_link.STL" />
         </geometry>
         <material name="">
@@ -136,29 +128,32 @@
       </visual>
       <collision>
-        <origin
-          xyz="0 0 0"
-          rpy="0 0 0" />
-        <geometry>
-          <mesh filename="file://$(find kortex_description)/arms/gen3/${dof}dof/meshes/bicep_link.STL" />
+        <origin xyz="0 0 0" rpy="0 0 0" />
+        <geometry>
+          <mesh filename="file://$(find kortex_description)/arms/gen3/${dof}dof/meshes/half_arm_1_link.STL" />
         </geometry>
       </collision>
     </link>
-    <joint name="${name}_joint_2" type="revolute">
-      <origin xyz="0 0.005375 -0.12838" rpy="1.5708 0.0 0.0" />
-      <parent link="${name}_shoulder_link" />
-      <child link="${name}_bicep_link" />
-      <axis xyz="0 0 1" />
+    <joint
+      name="${name}_joint_2"
+      type="revolute">
+      <origin xyz="0 0.005375 -0.12838" rpy="1.5708 2.1343E-17 -1.1102E-16" />
+      <parent
+        link="${name}_shoulder_link" />
+      <child
+        link="${name}_half_arm_1_link" />
+      <axis
+        xyz="0 0 1" />
       <limit lower="-2.41" upper="2.41" effort="39" velocity="1.3963" />
     </joint>
-    <link name="${name}_forearm_link">
+    <link name="${name}_half_arm_2_link">
       <inertial>
-        <origin xyz="1.8E-05 0.076168 -0.01397" rpy="0 0 0" />
-        <mass value="0.93" />
-        <inertia ixx="0.008292" ixy="-1E-06" ixz="0" iyy="0.000628" iyz="0.000432" izz="0.008464" />
+        <origin xyz="-4.4E-05 -0.006641 -0.117892" rpy="0 0 0" />
+        <mass value="1.1636" />
+        <inertia ixx="0.010932" ixy="0" ixz="-7E-06" iyy="0.011127" iyz="0.000606" izz="0.001043" />
       </inertial>
       <visual>
         <origin xyz="0 0 0" rpy="0 0 0" />
         <geometry>
-          <mesh filename="file://$(find kortex_description)/arms/gen3/${dof}dof/meshes/forearm_link.STL" />
+          <mesh filename="file://$(find kortex_description)/arms/gen3/${dof}dof/meshes/half_arm_2_link.STL" />
         </geometry>
         <material name="">
@@ -169,25 +164,52 @@
         <origin xyz="0 0 0" rpy="0 0 0" />
         <geometry>
-          <mesh filename="file://$(find kortex_description)/arms/gen3/${dof}dof/meshes/forearm_link.STL" />
+          <mesh filename="file://$(find kortex_description)/arms/gen3/${dof}dof/meshes/half_arm_2_link.STL" />
         </geometry>
       </collision>
     </link>
-    <joint name="${name}_joint_3" type="revolute">
-      <origin xyz="0 -0.41 0" rpy="3.1416 0 0" />
-      <parent link="${name}_bicep_link" />
-      <child link="${name}_forearm_link" />
-      <axis xyz="0 0 1" />
-      <limit lower="-2.66" upper="2.66" effort="39" velocity="1.3963" />
-    </joint>
-    <link name="${name}_spherical_wrist_1_link">
+    <xacro:if value="${use_external_cable}">
+      <joint
+        name="${name}_joint_3"
+        type="revolute">
+        <origin xyz="0 -0.21038 -0.006375" rpy="-1.5708 1.2326E-32 -2.9122E-16" />
+        <parent
+          link="${name}_half_arm_1_link" />
+        <child
+          link="${name}_half_arm_2_link" />
+        <axis
+          xyz="0 0 1" />
+        <limit
+          lower="${-2*PI}"
+          upper="${2*PI}"
+          effort="39"
+          velocity="1.3963" />
+      </joint>
+    </xacro:if>
+    <xacro:unless value="${use_external_cable}">
+      <joint
+        name="${name}_joint_3"
+        type="continuous">
+        <origin xyz="0 -0.21038 -0.006375" rpy="-1.5708 1.2326E-32 -2.9122E-16" />
+        <parent
+          link="${name}_half_arm_1_link" />
+        <child
+          link="${name}_half_arm_2_link" />
+        <axis
+          xyz="0 0 1" />
+        <limit
+          effort="39"
+          velocity="1.3963" />
+      </joint>
+    </xacro:unless>
+    <link name="${name}_forearm_link">
       <inertial>
-        <origin xyz="-1E-06 0.008486 -0.062937" rpy="0 0 0" />
-        <mass value="0.6781" />
-        <inertia ixx="0.001645" ixy="0" ixz="0" iyy="0.001666" iyz="-0.000234" izz="0.000389" />
+        <origin xyz="-1.8E-05 -0.075478 -0.015006" rpy="0 0 0" />
+        <mass value="0.9302" />
+        <inertia ixx="0.008147" ixy="-1E-06" ixz="0" iyy="0.000631" iyz="-0.0005" izz="0.008316" />
       </inertial>
       <visual>
         <origin xyz="0 0 0" rpy="0 0 0" />
         <geometry>
-          <mesh filename="file://$(find kortex_description)/arms/gen3/${dof}dof/meshes/spherical_wrist_1_link.STL" />
+          <mesh filename="file://$(find kortex_description)/arms/gen3/${dof}dof/meshes/forearm_link.STL" />
         </geometry>
         <material name="">
@@ -198,36 +220,30 @@
         <origin xyz="0 0 0" rpy="0 0 0" />
         <geometry>
-          <mesh filename="file://$(find kortex_description)/arms/gen3/${dof}dof/meshes/spherical_wrist_1_link.STL" />
+          <mesh filename="file://$(find kortex_description)/arms/gen3/${dof}dof/meshes/forearm_link.STL" />
         </geometry>
       </collision>
     </link>
-    <xacro:if value="${use_external_cable}">
-      <joint name="${name}_joint_4" type="revolute">
-        <origin xyz="0 0.20843 -0.006375" rpy="1.5708 0.0 0.0" />
-        <parent link="${name}_forearm_link" />
-        <child link="${name}_spherical_wrist_1_link" />
-        <axis xyz="0 0 1" />
-        <limit lower="${-2*PI}" upper="${2*PI}" effort="9" velocity="1.2218" />
-      </joint>
-    </xacro:if>
-    <xacro:unless value="${use_external_cable}">
-      <joint name="${name}_joint_4" type="continuous">
-        <origin xyz="0 0.20843 -0.006375" rpy="1.5708 0.0 0.0" />
-        <parent link="${name}_forearm_link" />
-        <child link="${name}_spherical_wrist_1_link" />
-        <axis xyz="0 0 1" />
-        <limit effort="9" velocity="1.2218" />
-      </joint>
-    </xacro:unless>
-    <link name="${name}_spherical_wrist_2_link">
+    <joint
+      name="${name}_joint_4"
+      type="revolute">
+      <origin xyz="0 0.006375 -0.21038" rpy="1.5708 -6.6954E-17 -1.6653E-16" />
+      <parent
+        link="${name}_half_arm_2_link" />
+      <child
+        link="${name}_forearm_link" />
+      <axis
+        xyz="0 0 1" />
+      <limit lower="-2.66" upper="2.66" effort="39" velocity="1.3963" />
+    </joint>
+    <link name="${name}_spherical_wrist_1_link">
       <inertial>
-        <origin xyz="-1E-06 0.046429 -0.008704" rpy="0 0 0" />
-        <mass value="0.678" />
-        <inertia ixx="0.001685" ixy="0" ixz="0" iyy="0.0004" iyz="0.000255" izz="0.001696" />
+        <origin xyz="1E-06 -0.009432 -0.063883" rpy="0 0 0" />
+        <mass value="0.6781" />
+        <inertia ixx="0.001596" ixy="0" ixz="0" iyy="0.001607" iyz="0.000256" izz="0.000399" />
       </inertial>
       <visual>
         <origin xyz="0 0 0" rpy="0 0 0" />
         <geometry>
-          <mesh filename="file://$(find kortex_description)/arms/gen3/${dof}dof/meshes/spherical_wrist_2_link.STL" />
+          <mesh filename="file://$(find kortex_description)/arms/gen3/${dof}dof/meshes/spherical_wrist_1_link.STL" />
         </geometry>
         <material name="">
@@ -238,26 +254,52 @@
         <origin xyz="0 0 0" rpy="0 0 0" />
         <geometry>
-          <mesh filename="file://$(find kortex_description)/arms/gen3/${dof}dof/meshes/spherical_wrist_2_link.STL" />
+          <mesh filename="file://$(find kortex_description)/arms/gen3/${dof}dof/meshes/spherical_wrist_1_link.STL" />
         </geometry>
       </collision>
     </link>
-    <joint name="${name}_joint_5" type="revolute">
-      <origin xyz="0 -0.00017505 -0.10593" rpy="-1.5708 0.0 0.0" />
-      <parent link="${name}_spherical_wrist_1_link" />
-      <child link="${name}_spherical_wrist_2_link" />
-      <axis xyz="0 0 1" />
-      <limit lower="-2.23" upper="2.23" effort="9" velocity="1.2218" />
-    </joint>
-    <xacro:if value="${vision}">
-    <link name="${name}_bracelet_link">
+    <xacro:if value="${use_external_cable}">
+      <joint
+        name="${name}_joint_5"
+        type="revolute">
+        <origin xyz="0 -0.20843 -0.006375" rpy="-1.5708 2.2204E-16 -6.373E-17" />
+        <parent
+          link="${name}_forearm_link" />
+        <child
+          link="${name}_spherical_wrist_1_link" />
+        <axis
+          xyz="0 0 1" />
+        <limit
+          lower="${-2*PI}"
+          upper="${2*PI}"
+          effort="9"
+          velocity="1.2218" />
+      </joint>
+    </xacro:if>
+    <xacro:unless value="${use_external_cable}">
+      <joint
+        name="${name}_joint_5"
+        type="continuous">
+        <origin xyz="0 -0.20843 -0.006375" rpy="-1.5708 2.2204E-16 -6.373E-17" />
+        <parent
+          link="${name}_forearm_link" />
+        <child
+          link="${name}_spherical_wrist_1_link" />
+        <axis
+          xyz="0 0 1" />
+        <limit
+          effort="9"
+          velocity="1.2218" />
+      </joint>
+    </xacro:unless>
+    <link name="${name}_spherical_wrist_2_link">
       <inertial>
-        <origin xyz="0.000281 0.011402 -0.029798" rpy="0 0 0" />
-        <mass value="0.5" />
-        <inertia ixx="0.000587" ixy="3E-06" ixz="3E-06" iyy="0.000369" iyz="-0.000118" izz="0.000609" />
+        <origin xyz="1E-06 -0.045483 -0.00965" rpy="0 0 0" />
+        <mass value="0.6781" />
+        <inertia ixx="0.001641" ixy="0" ixz="0" iyy="0.00041" iyz="-0.000278" izz="0.001641" />
       </inertial>
       <visual>
         <origin xyz="0 0 0" rpy="0 0 0" />
         <geometry>
-          <mesh filename="file://$(find kortex_description)/arms/gen3/${dof}dof/meshes/bracelet_with_vision_link.STL" />
+          <mesh filename="file://$(find kortex_description)/arms/gen3/${dof}dof/meshes/spherical_wrist_2_link.STL" />
         </geometry>
         <material name="">
@@ -268,49 +310,103 @@
         <origin xyz="0 0 0" rpy="0 0 0" />
         <geometry>
-          <mesh filename="file://$(find kortex_description)/arms/gen3/${dof}dof/meshes/bracelet_with_vision_link.STL" />
+          <mesh filename="file://$(find kortex_description)/arms/gen3/${dof}dof/meshes/spherical_wrist_2_link.STL" />
         </geometry>
       </collision>
     </link>
+    <joint
+      name="${name}_joint_6"
+      type="revolute">
+      <origin xyz="0 0.00017505 -0.10593" rpy="1.5708 9.2076E-28 -8.2157E-15" />
+      <parent
+        link="${name}_spherical_wrist_1_link" />
+      <child
+        link="${name}_spherical_wrist_2_link" />
+      <axis
+        xyz="0 0 1" />
+      <limit lower="-2.23" upper="2.23" effort="9" velocity="1.2218" />
+    </joint>
+    <!-- Bracelet with Vision -->
+    <xacro:if value="${vision}">
+      <link name="${name}_bracelet_link">
+        <inertial>
+          <origin xyz="0.000281 0.011402 -0.029798" rpy="0 0 0" />
+          <mass value="0.5" />
+          <inertia ixx="0.000587" ixy="3E-06" ixz="3E-06" iyy="0.000369" iyz="-0.000118" izz="0.000609" />
+        </inertial>
+        <visual>
+          <origin xyz="0 0 0" rpy="0 0 0" />
+          <geometry>
+            <mesh filename="file://$(find kortex_description)/arms/gen3/${dof}dof/meshes/bracelet_with_vision_link.STL" />
+          </geometry>
+          <material name="">
+            <color rgba="0.75294 0.75294 0.75294 1" />
+          </material>
+        </visual>
+        <collision>
+          <origin xyz="0 0 0" rpy="0 0 0" />
+          <geometry>
+            <mesh filename="file://$(find kortex_description)/arms/gen3/${dof}dof/meshes/bracelet_with_vision_link.STL" />
+          </geometry>
+        </collision>
+      </link>
     </xacro:if>
+    <!-- Bracelet without Vision -->
     <xacro:unless value="${vision}">
-    <link name="${name}_bracelet_link">
-      <inertial>
-        <origin xyz="-9.3E-05 0.000132 -0.022905" rpy="0 0 0" />
-        <mass value="0.364" />
-        <inertia ixx="0.000214" ixy="0" ixz="1E-06" iyy="0.000223" iyz="-2E-06" izz="0.00024" />
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
Commit message: Gripper joint set through arm URD

File: clearpath_manipulators_description/urdf/arm/kinova_gen3_7dof.urdf.xacro (robot description, xacro)
@@ -470,5 +470,5 @@
     </xacro:if>
     <!-- ROS2 Controls -->
-    <xacro:if value="${use_controllers}"/>
+    <xacro:if value="${use_controllers}">
       <ros2_control name="${name}_hardware" type="system">
         <hardware>

File: clearpath_manipulators_description/urdf/arm/kinova_gen3_lite.urdf.xacro (robot description, xacro)
@@ -18,6 +18,6 @@
     session_inactivity_timeout_ms:=6000
     connection_inactivity_timeout_ms:=2000
-    use_internal_bus_gripper_comm:=true
-    gripper_joint_name:=gripper_0_right_finger_bottom_joint
+    use_internal_bus_gripper_comm:=false
+    gripper_joint_name:=finger_joint
     gripper_max_velocity:=100.0
     gripper_max_force:=100.0
@@ -339,5 +339,5 @@
         <xacro:unless value="${use_fake_hardware or sim_gazebo or sim_ignition or sim_isaac}">
           <xacro:if value="${use_internal_bus_gripper_comm}">
-            <joint name="gripper_0_right_finger_bottom_joint">
+            <joint name="${gripper_joint_name}">
               <command_interface name="position"/>
               <state_interface name="position"/>
