Commit message: Replace 'PI' property with 'math.pi'

File: clearpath_manipulators_description/urdf/arm/kinova_gen3_7dof.urdf.xacro (robot description, xacro)
@@ -92,6 +92,6 @@
           xyz="0 0 1" />
         <limit
-          lower="${-2*PI}"
-          upper="${2*PI}"
+          lower="${-2*math.pi}"
+          upper="${2*math.pi}"
           effort="39"
           velocity="1.3963" />
@@ -182,6 +182,6 @@
           xyz="0 0 1" />
         <limit
-          lower="${-2*PI}"
-          upper="${2*PI}"
+          lower="${-2*math.pi}"
+          upper="${2*math.pi}"
           effort="39"
           velocity="1.3963" />
@@ -272,6 +272,6 @@
           xyz="0 0 1" />
         <limit
-          lower="${-2*PI}"
-          upper="${2*PI}"
+          lower="${-2*math.pi}"
+          upper="${2*math.pi}"
           effort="9"
           velocity="1.2218" />
@@ -391,6 +391,6 @@
           xyz="0 0 1" />
         <limit
-          lower="${-2*PI}"
-          upper="${2*PI}"
+          lower="${-2*math.pi}"
+          upper="${2*math.pi}"
           effort="9"
           velocity="1.2218" />
@@ -431,5 +431,5 @@
         <link name="${name}_camera_link" />
         <joint name="${name}_camera_module" type="fixed">
-          <origin xyz="0 0.05639 0.01305" rpy="0 ${-PI/2} ${-PI/2}" />
+          <origin xyz="0 0.05639 0.01305" rpy="0 ${-math.pi/2} ${-math.pi/2}" />
           <parent link="${name}_end_effector_link" />
           <child  link="${name}_camera_link" />
@@ -437,5 +437,5 @@
         <link name="${name}_camera_depth_frame" />
         <joint name="${name}_depth_module" type="fixed">
-          <origin xyz="0.0275 0.066 0.01305" rpy="0 ${-PI/2} ${-PI/2}" />
+          <origin xyz="0.0275 0.066 0.01305" rpy="0 ${-math.pi/2} ${-math.pi/2}" />
           <parent link="${name}_end_effector_link" />
           <child  link="${name}_camera_depth_frame" />
@@ -443,5 +443,5 @@
         <link name="${name}_camera_color_frame" />
         <joint name="${name}_color_module" type="fixed">
-          <origin xyz="0 0.05639 0.01305" rpy="0 ${-PI/2} ${-PI/2}" />
+          <origin xyz="0 0.05639 0.01305" rpy="0 ${-math.pi/2} ${-math.pi/2}" />
           <parent link="${name}_end_effector_link" />
           <child  link="${name}_camera_color_frame" />
@@ -451,5 +451,5 @@
         <link name="${name}_camera_link" />
         <joint name="${name}_camera_module" type="fixed">
-          <origin xyz="0 0.05639 -0.00305" rpy="${PI} ${PI} 0" />
+          <origin xyz="0 0.05639 -0.00305" rpy="${math.pi} ${math.pi} 0" />
           <parent link="${name}_end_effector_link" />
           <child  link="${name}_camera_link" />
@@ -457,5 +457,5 @@
         <link name="${name}_camera_depth_frame" />
         <joint name="${name}_depth_module" type="fixed">
-          <origin xyz="0.0275 0.066 -0.00305" rpy="${PI} ${PI} 0" />
+          <origin xyz="0.0275 0.066 -0.00305" rpy="${math.pi} ${math.pi} 0" />
           <parent link="${name}_end_effector_link" />
           <child  link="${name}_camera_depth_frame" />
@@ -463,5 +463,5 @@
         <link name="${name}_camera_color_frame" />
         <joint name="${name}_color_module" type="fixed">
-          <origin xyz="0 0.05639 -0.00305" rpy="${PI} ${PI} 0" />
+          <origin xyz="0 0.05639 -0.00305" rpy="${math.pi} ${math.pi} 0" />
           <parent link="${name}_end_effector_link" />
           <child  link="${name}_camera_color_frame" />
