Commit message: Create joint instead of using connected_to parameter

File: clearpath_manipulators_description/urdf/arm/franka.urdf.xacro (robot description, xacro)
@@ -48,9 +48,8 @@
     <xacro:property name="_no_prefix" value="false" lazy_eval="false"/>
     <xacro:property name="_arm_prefix" value="${name}" lazy_eval="false"/>
-    <xacro:property name="_connected_to" value="${name}_${arm_id}_base_link" lazy_eval="false"/>
+    <xacro:property name="_connected_to" value="" lazy_eval="false"/>
     <xacro:property name="_multi_arm" value="false" lazy_eval="false"/>
-    <link name="${name}_${arm_id}_base_link"/>
-    <joint name="${name}_${arm_id}_base_joint" type="fixed">
-      <child link="${name}_${arm_id}_base_link"/>
+    <joint name="${name}_${arm_id}_joint0" type="fixed">
+      <child link="${name}_${arm_id}_link0"/>
       <parent link="${parent_link}"/>
       <xacro:insert_block name="origin"/>
@@ -58,9 +57,9 @@
     <xacro:include filename="$(find franka_description)/robots/common/franka_robot.xacro"/>
     <xacro:franka_robot
-      arm_id="fr3"
-      joint_limits="${xacro.load_yaml('$(find franka_description)/robots/fr3/joint_limits.yaml')}"
-      inertials="${xacro.load_yaml('$(find franka_description)/robots/fr3/inertials.yaml')}"
-      kinematics="${xacro.load_yaml('$(find franka_description)/robots/fr3/kinematics.yaml')}"
-      dynamics="${xacro.load_yaml('$(find franka_description)/robots/fr3/dynamics.yaml')}"
+      arm_id="${_arm_id}"
+      joint_limits="${xacro.load_yaml('$(find franka_description)/robots/' + arm_id + '/joint_limits.yaml')}"
+      inertials="${xacro.load_yaml('$(find franka_description)/robots/' + arm_id + '/inertials.yaml')}"
+      kinematics="${xacro.load_yaml('$(find franka_description)/robots/' + arm_id + '/kinematics.yaml')}"
+      dynamics="${xacro.load_yaml('$(find franka_description)/robots/' + arm_id + '/dynamics.yaml')}"
       gazebo="${_gazebo}"
       hand="${_hand}"

Commit message: Modify entire Franka arm xacro

File: clearpath_manipulators_description/urdf/arm/franka.urdf.xacro (robot description, xacro)
@@ -4,9 +4,157 @@
   <xacro:arg name="use_fake_hardware" default="false"/>
   <xacro:arg name="use_manipulation_controllers" default="false"/>
+  <xacro:macro name="franka_arm_ros2_control"
+         params="arm_id
+             robot_ip
+             use_fake_hardware:=^|false
+             fake_sensor_commands:=^|false
+             gazebo:=^|false
+             hand:=^|false
+             gazebo_effort:=^|false
+             arm_prefix:=''
+             multi_arm:=false">
+    <xacro:property name="arm_prefix_modified" value="${'' if arm_prefix == '' else arm_prefix + '_'}" />
+    <ros2_control name="${arm_prefix_modified}FrankaHardwareInterface" type="system">
+        <hardware>
+          <param name="arm_id">${arm_id}</param>
+          <param name="prefix">${arm_prefix}</param>
+          <xacro:if value="${use_fake_hardware}">
+            <plugin>fake_components/GenericSystem</plugin>
+            <param name="fake_sensor_commands">${fake_sensor_commands}</param>
+            <param name="state_following_offset">0.0</param>
+          </xacro:if>
+          <xacro:if value="${gazebo}">
+            <plugin>ign_ros2_control/IgnitionSystem</plugin>
+          </xacro:if>
+          <xacro:if value="${use_fake_hardware == 0 and gazebo == 0 and multi_arm == 0}">
+            <plugin>franka_hardware/FrankaHardwareInterface</plugin>
+            <param name="robot_ip">${robot_ip}</param>
+            <param name="arm_prefix">${arm_prefix}</param>
+          </xacro:if>
+          <xacro:if value="${use_fake_hardware == 0 and gazebo == 0 and multi_arm == 1}">
+            <plugin>franka_hardware/MultiFrankaHardwareInterface</plugin>
+            <param name="robot_ip">${robot_ip}</param>
+            <param name="arm_prefix">${arm_prefix}</param>
+          </xacro:if>
+        </hardware>
+      <xacro:macro name="configure_joint" params="joint_name initial_position">
+        <joint name="${joint_name}">
+          <!--
+            deactivated for gazebo velocity and position interface due to a bug
+            https://github.com/ros-controls/gz_ros2_control/issues/343
+            Command Interfaces -->
+          <xacro:unless value="${gazebo and gazebo_effort}">
+            <command_interface name="position"/>
+            <command_interface name="velocity"/>
+          </xacro:unless>
+          <xacro:if value="${gazebo_effort}">
+            <command_interface name="effort"/>
+          </xacro:if>
+          <!-- State Interfaces -->
+          <state_interface name="position">
+            <param name="initial_value">${initial_position}</param>
+          </state_interface>
+          <state_interface name="velocity"/>
+            <param name="initial_value">0.0</param>
+          <state_interface name="effort"/>
+        </joint>
+      </xacro:macro>
+      <xacro:configure_joint joint_name="${arm_prefix_modified}${arm_id}_joint1" initial_position="0.0"/>
+      <xacro:configure_joint joint_name="${arm_prefix_modified}${arm_id}_joint2" initial_position="${-pi/4}"/>
+      <xacro:configure_joint joint_name="${arm_prefix_modified}${arm_id}_joint3" initial_position="0.0"/>
+      <xacro:configure_joint joint_name="${arm_prefix_modified}${arm_id}_joint4" initial_position="${-3*pi/4}"/>
+      <xacro:configure_joint joint_name="${arm_prefix_modified}${arm_id}_joint5" initial_position="0.0"/>
+      <xacro:configure_joint joint_name="${arm_prefix_modified}${arm_id}_joint6" initial_position="${pi/2}"/>
+      <xacro:configure_joint joint_name="${arm_prefix_modified}${arm_id}_joint7" initial_position="${pi/4}"/>
+    </ros2_control>
+  </xacro:macro>
+  <xacro:macro name="franka_robot"
+              params="arm_id
+                      joint_limits
+                      kinematics
+                      inertials
+                      dynamics
+                      parent:='world'
+                      xyz:='0 0 0'
+                      rpy:='0 0 0'
+                      hand:='true'
+                      ee_id:=none
+                      gazebo:='false'
+                      with_sc:='false'
+                      ros2_control:=false
+                      robot_ip:=''
+                      use_fake_hardware:=false
+                      fake_sensor_commands:=false
+                      gazebo_effort:=false
+                      no_prefix:='false'
+                      arm_prefix:=''
+                      connected_to:='base'
+                      multi_arm:=false">
+    <xacro:include filename="$(find franka_description)/robots/common/utils.xacro" />
+    <xacro:include filename="$(find franka_description)/robots/common/franka_arm.xacro" />
+    <xacro:property name="arm_prefix_modified" value="${'' if arm_prefix == '' else arm_prefix + '_'}" />
+    <xacro:franka_arm
+      arm_id="${arm_id}"
+      arm_prefix="${arm_prefix_modified}"
+      no_prefix="${no_prefix}"
+      xyz="${xyz}"
+      rpy="${rpy}"
+      safety_distance="0.03"
+      gazebo="${gazebo}"
+      joint_limits="${joint_limits}"
+      kinematics="${kinematics}"
+      inertials="${inertials}"
+      dynamics="${dynamics}"
+      with_sc="${with_sc}"
+      connected_to="${connected_to}"
+    />
+    <!-- Definition of additional Gazebo tags -->
+    <xacro:if value="${gazebo}">
+      <xacro:gazebo-joint joint="${arm_prefix_modified}${arm_id}_joint1" transmission="hardware_interface/PositionJointInterface" />
+      <xacro:gazebo-joint joint="${arm_prefix_modified}${arm_id}_joint2" transmission="hardware_interface/PositionJointInterface" />
+      <xacro:gazebo-joint joint="${arm_prefix_modified}${arm_id}_joint3" transmission="hardware_interface/PositionJointInterface" />
+      <xacro:gazebo-joint joint="${arm_prefix_modified}${arm_id}_joint4" transmission="hardware_interface/PositionJointInterface" />
+      <xacro:gazebo-joint joint="${arm_prefix_modified}${arm_id}_joint5" transmission="hardware_interface/PositionJointInterface" />
+      <xacro:gazebo-joint joint="${arm_prefix_modified}${arm_id}_joint6" transmission="hardware_interface/PositionJointInterface" />
+      <xacro:gazebo-joint joint="${arm_prefix_modified}${arm_id}_joint7" transmission="hardware_interface/PositionJointInterface" />
+      <xacro:gazebo-joint joint="${arm_prefix_modified}${arm_id}_joint1" transmission="hardware_interface/VelocityJointInterface" />
+      <xacro:gazebo-joint joint="${arm_prefix_modified}${arm_id}_joint2" transmission="hardware_interface/VelocityJointInterface" />
+      <xacro:gazebo-joint joint="${arm_prefix_modified}${arm_id}_joint3" transmission="hardware_interface/VelocityJointInterface" />
+      <xacro:gazebo-joint joint="${arm_prefix_modified}${arm_id}_joint4" transmission="hardware_interface/VelocityJointInterface" />
+      <xacro:gazebo-joint joint="${arm_prefix_modified}${arm_id}_joint5" transmission="hardware_interface/VelocityJointInterface" />
+      <xacro:gazebo-joint joint="${arm_prefix_modified}${arm_id}_joint6" transmission="hardware_interface/VelocityJointInterface" />
+      <xacro:gazebo-joint joint="${arm_prefix_modified}${arm_id}_joint7" transmission="hardware_interface/VelocityJointInterface" />
+      <xacro:gazebo-joint joint="${arm_prefix_modified}${arm_id}_joint1" transmission="hardware_interface/EffortJointInterface" />
+      <xacro:gazebo-joint joint="${arm_prefix_modified}${arm_id}_joint2" transmission="hardware_interface/EffortJointInterface" />
+      <xacro:gazebo-joint joint="${arm_prefix_modified}${arm_id}_joint3" transmission="hardware_interface/EffortJointInterface" />
+      <xacro:gazebo-joint joint="${arm_prefix_modified}${arm_id}_joint4" transmission="hardware_interface/EffortJointInterface" />
+      <xacro:gazebo-joint joint="${arm_prefix_modified}${arm_id}_joint5" transmission="hardware_interface/EffortJointInterface" />
+      <xacro:gazebo-joint joint="${arm_prefix_modified}${arm_id}_joint6" transmission="hardware_interface/EffortJointInterface" />
+      <xacro:gazebo-joint joint="${arm_prefix_modified}${arm_id}_joint7" transmission="hardware_interface/EffortJointInterface" />
+      <xacro:transmission-franka-state arm_id="${arm_id}" />
+      <xacro:transmission-franka-model arm_id="${arm_id}"
+         root="${arm_prefix_modified}${arm_id}_joint1"
+         tip="${arm_prefix_modified}${arm_id}_joint8"
+       />
+    </xacro:if>
+    <xacro:if value="${ros2_control}">
+      <xacro:franka_arm_ros2_control
+          arm_id="${arm_id}"
+          robot_ip="${robot_ip}"
+          use_fake_hardware="${use_fake_hardware}"
+          fake_sensor_commands="${fake_sensor_commands}"
+          gazebo="${gazebo}"
+          hand="${hand}"
+          gazebo_effort="${gazebo_effort}"
+          arm_prefix="${arm_prefix}"
+          multi_arm="${multi_arm}"
+      />
+    </xacro:if>
+  </xacro:macro>
   <xacro:macro name="franka" params="
     name
     parent_link
     *origin
-    arm_id:=fr3
+    arm_id:=''
     joint_limits:=''
     joint_limits_parameters_file:=''
@@ -17,37 +165,85 @@
     dynamics:=''
     dynamics_parameters_file:=''
-    gazebo:=''
-    hand:=''
-    ee_id:=''
-    with_sc:=''
     ros2_control:=''
     robot_ip:=''
     use_fake_hardware:=''
     fake_sensor_commands:=''
+    gazebo:=''
     gazebo_effort:=''
-    no_prefix:=''
-    arm_prefix:=''
-    connected_to:=''
   ">
-    <xacro:property name="_arm_id" value="${arm_id}" lazy_eval="false"/>
-    <xacro:property name="_joint_limits" value="" lazy_eval="false"/>
-    <xacro:property name="_inertials" value="" lazy_eval="false"/>
-    <xacro:property name="_kinematics" value="" lazy_eval="false"/>
-    <xacro:property name="_dynamics" value="" lazy_eval="false"/>
-    <!-- End Effector -->
+    <!-- Franka Type -->
+    <xacro:property name="_arm_id" value="fr3" lazy_eval="false"/>
+    <xacro:if value="${arm_id != ''}">
+      <xacro:property name="_arm_id" value="${arm_id}" lazy_eval="false"/>
+    </xacro:if>
+    <!-- Description Parameter Files -->
+    <xacro:property name="_joint_limits_parameters_file" value="$(find franka_description)/robots/${_arm_id}/joint_limits.yaml" lazy_eval="false"/>
+    <xacro:property name="_inertials_parameters_file" value="$(find franka_description)/robots/${_arm_id}/inertials.yaml" lazy_eval="false"/>
+    <xacro:property name="_kinematics_parameters_file" value="$(find franka_description)/robots/${_arm_id}/kinematics.yaml" lazy_eval="false"/>
+    <xacro:property name="_dynamics_parameters_file" value="$(find franka_description)/robots/${_arm_id}/dynamics.yaml" lazy_eval="false"/>
+    <xacro:if value="${joint_limits_parameters_file != ''}">
+      <xacro:property name="_joint_limits_parameters_file" value="${joint_limits_parameters_file}" lazy_eval="false"/>
+    </xacro:if>
+    <xacro:if value="${inertials_parameters_file != ''}">
+      <xacro:property name="_inertials_parameters_file" value="${inertials_parameters_file}" lazy_eval="false"/>
+    </xacro:if>
+    <xacro:if value="${kinematics_parameters_file != ''}">
+      <xacro:property name="_kinematics_parameters_file" value="${kinematics_parameters_file}" lazy_eval="false"/>
+    </xacro:if>
+    <xacro:if value="${dynamics_parameters_file != ''}">
+      <xacro:property name="_dynamics_parameters_file" value="${dynamics_parameters_file}" lazy_eval="false"/>
+    </xacro:if>
+    <!-- Loaded Parameters -->
+    <xacro:property name="_joint_limits" value="${xacro.load_yaml(_joint_limits_parameters_file)}" lazy_eval="false"/>
+    <xacro:property name="_inertials" value="${xacro.load_yaml(_inertials_parameters_file)}" lazy_eval="false"/>
+    <xacro:property name="_kinematics" value="${xacro.load_yaml(_kinematics_parameters_file)}" lazy_eval="false"/>
+    <xacro:property name="_dynamics" value="${xacro.load_yaml(_dynamics_parameters_file)}" lazy_eval="false"/>
+    <xacro:if value="${joint_limits != ''}">
+      <xacro:property name="_joint_limits" value="${joint_limits}" lazy_eval="false"/>
+    </xacro:if>
+    <xacro:if value="${inertials != ''}">
+      <xacro:property name="_inertials" value="${inertials}" lazy_eval="false"/>
+    </xacro:if>
+    <xacro:if value="${kinematics != ''}">
+      <xacro:property name="_kinematics" value="${kinematics}" lazy_eval="false"/>
+    </xacro:if>
+    <xacro:if value="${dynamics != ''}">
+      <xacro:property name="_dynamics" value="${dynamics}" lazy_eval="false"/>
+    </xacro:if>
+    <!-- Control Parameters -->
+    <xacro:property name="_ros2_control" value="$(arg use_manipulation_controllers)" lazy_eval="false"/>
+    <xacro:property name="_robot_ip" value="192.168.131.40" lazy_eval="false"/>
+    <xacro:if value="${ros2_control != ''}">
+      <xacro:property name="_ros2_control" value="${ros2_control}" lazy_eval="false"/>
+    </xacro:if>
+    <xacro:if value="${robot_ip != ''}">
+      <xacro:property name="_robot_ip" value="${robot_ip}" lazy_eval="false"/>
+    </xacro:if>
+    <!-- Simulation -->
+    <xacro:property name="_gazebo" value="$(arg is_sim)" lazy_eval="false"/>
+    <xacro:property name="_gazebo_effort" value="false" lazy_eval="false"/>
+    <xacro:property name="_use_fake_hardware" value="false" lazy_eval="false"/>
+    <xacro:property name="_fake_sensor_commands" value="false" lazy_eval="false"/>
+    <xacro:if value="${gazebo != ''}">
+      <xacro:property name="_gazebo" value="${gazebo}" lazy_eval="false"/>
+    </xacro:if>
+    <xacro:if value="${gazebo_effort != ''}">
+      <xacro:property name="_gazebo_effort" value="${gazebo_effort}" lazy_eval="false"/>
+    </xacro:if>
+    <xacro:if value="${use_fake_hardware != ''}">
+      <xacro:property name="_use_fake_hardware" value="${use_fake_hardware}" lazy_eval="false"/>
+    </xacro:if>
+    <xacro:if value="${fake_sensor_commands != ''}">
+      <xacro:property name="_fake_sensor_commands" value="${fake_sensor_commands}" lazy_eval="false"/>
+    </xacro:if>
+    <!-- Fixed Parameters -->
     <xacro:property name="_hand" value="true" lazy_eval="false"/>
     <xacro:property name="_ee_id" value="franka_hand" lazy_eval="false"/>
-    <!-- Simulation -->
-    <xacro:property name="_gazebo" value="$(arg is_sim)" lazy_eval="false"/>
+    <xacro:property name="_multi_arm" value="false" lazy_eval="false"/>
+    <xacro:property name="_connected_to" value="" lazy_eval="false"/>
     <xacro:property name="_with_sc" value="false" lazy_eval="false"/>
-    <xacro:property name="_ros2_control" value="$(arg use_manipulation_controllers)" lazy_eval="false"/>
-    <xacro:property name="_robot_ip" value="192.168.131.40" lazy_eval="false"/>
-    <xacro:property name="_use_fake_hardware" value="false" lazy_eval="false"/>
-    <xacro:property name="_fake_sensor_commands" value="false" lazy_eval="false"/>
-    <xacro:property name="_gazebo_effort" value="false" lazy_eval="false"/>
     <xacro:property name="_no_prefix" value="false" lazy_eval="false"/>
     <xacro:property name="_arm_prefix" value="${name}" lazy_eval="false"/>
-    <xacro:property name="_connected_to" value="" lazy_eval="false"/>
-    <xacro:property name="_multi_arm" value="false" lazy_eval="false"/>
+    <!-- Parent Joint -->
     <joint name="${name}_${arm_id}_joint0" type="fixed">
       <child link="${name}_${arm_id}_link0"/>
@@ -55,5 +251,4 @@
       <xacro:insert_block name="origin"/>
     </joint>
-    <xacro:include filename="$(find franka_description)/robots/common/franka_robot.xacro"/>
     <xacro:franka_robot
       arm_id="${_arm_id}"
