Commit message: Initial rework to match new franka URDF

File: clearpath_manipulators_description/urdf/arm/franka.urdf.xacro (robot description, xacro)
@@ -4,149 +4,140 @@
   <xacro:arg name="use_fake_hardware" default="false"/>
   <xacro:arg name="use_manipulation_controllers" default="false"/>
-  <!-- Franka ROS2 Control -->
-  <xacro:macro name="franka_arm_ros2_control"
-         params="arm_id
-             robot_ip
-             use_fake_hardware:=^|false
-             fake_sensor_commands:=^|false
-             gazebo:=^|false
-             hand:=^|false
-             gazebo_effort:=^|false
-             arm_prefix:=''
-             multi_arm:=false">
-    <xacro:property name="arm_prefix_modified" value="${'' if arm_prefix == '' else arm_prefix + '_'}" />
-    <ros2_control name="${arm_prefix_modified}FrankaHardwareInterface" type="system">
-        <hardware>
-          <param name="version">0.1.0</param>
-          <param name="arm_id">${arm_id}</param>
-          <param name="prefix">${arm_prefix}</param>
-          <xacro:if value="${use_fake_hardware}">
-            <plugin>fake_components/GenericSystem</plugin>
-            <param name="fake_sensor_commands">${fake_sensor_commands}</param>
-            <param name="state_following_offset">0.0</param>
-          </xacro:if>
-          <xacro:if value="${gazebo}">
-            <plugin>gz_ros2_control/GazeboSimSystem</plugin>
-          </xacro:if>
-          <xacro:if value="${use_fake_hardware == 0 and gazebo == 0 and multi_arm == 0}">
-            <plugin>franka_hardware/FrankaHardwareInterface</plugin>
-            <param name="robot_ip">${robot_ip}</param>
-            <param name="arm_prefix">${arm_prefix}</param>
-          </xacro:if>
-          <xacro:if value="${use_fake_hardware == 0 and gazebo == 0 and multi_arm == 1}">
-            <plugin>franka_hardware/MultiFrankaHardwareInterface</plugin>
-            <param name="robot_ip">${robot_ip}</param>
-            <param name="arm_prefix">${arm_prefix}</param>
-          </xacro:if>
-        </hardware>
-      <xacro:macro name="configure_joint" params="joint_name initial_position">
-        <joint name="${joint_name}">
-          <command_interface name="position"/>
-          <command_interface name="velocity"/>
-          <xacro:if value="${gazebo == 0 or gazebo_effort == 1}">
-            <command_interface name="effort"/>
-          </xacro:if>
-          <state_interface name="position">
-            <param name="initial_value">${initial_position}</param>
-          </state_interface>
-          <state_interface name="velocity"/>
-            <param name="initial_value">0.0</param>
-          <state_interface name="effort"/>
-        </joint>
-      </xacro:macro>
-      <xacro:configure_joint joint_name="${arm_prefix_modified}${arm_id}_joint1" initial_position="0.0"/>
-      <xacro:configure_joint joint_name="${arm_prefix_modified}${arm_id}_joint2" initial_position="${-pi/4}"/>
-      <xacro:configure_joint joint_name="${arm_prefix_modified}${arm_id}_joint3" initial_position="0.0"/>
-      <xacro:configure_joint joint_name="${arm_prefix_modified}${arm_id}_joint4" initial_position="${-3*pi/4}"/>
-      <xacro:configure_joint joint_name="${arm_prefix_modified}${arm_id}_joint5" initial_position="0.0"/>
-      <xacro:configure_joint joint_name="${arm_prefix_modified}${arm_id}_joint6" initial_position="${pi/2}"/>
-      <xacro:configure_joint joint_name="${arm_prefix_modified}${arm_id}_joint7" initial_position="${pi/4}"/>
-    </ros2_control>
-  </xacro:macro>
-  <!-- Franka Parameters -->
-  <xacro:macro name="franka_robot"
-              params="arm_id
-                      joint_limits
-                      kinematics
-                      accelerometer_config:=none
-                      inertials
-                      dynamics
-                      parent:='world'
-                      xyz:='0 0 0'
-                      rpy:='0 0 0'
-                      hand:='true'
-                      ee_id:=none
-                      gazebo:='false'
-                      with_sc:='false'
-                      ros2_control:=false
-                      robot_ip:=''
-                      use_fake_hardware:=false
-                      fake_sensor_commands:=false
-                      gazebo_effort:=false
-                      no_prefix:='false'
-                      arm_prefix:=''
-                      connected_to:='base'
-                      multi_arm:=false">
-    <xacro:include filename="$(find franka_description)/robots/common/utils.xacro" />
-    <xacro:include filename="$(find franka_description)/robots/common/franka_arm.xacro" />
-    <xacro:property name="arm_prefix_modified" value="${'' if arm_prefix == '' else arm_prefix + '_'}" />
-    <xacro:franka_arm
-      arm_id="${arm_id}"
-      arm_prefix="${arm_prefix_modified}"
-      no_prefix="${no_prefix}"
-      xyz="${xyz}"
-      rpy="${rpy}"
-      safety_distance="0.03"
-      gazebo="${gazebo}"
-      joint_limits="${joint_limits}"
-      kinematics="${kinematics}"
-      accelerometer_config="${accelerometer_config}"
-      inertials="${inertials}"
-      dynamics="${dynamics}"
-      with_sc="${with_sc}"
-      connected_to="${connected_to}"
-    />
-    <!-- Definition of additional Gazebo tags -->
-    <xacro:if value="${gazebo}">
-      <xacro:gazebo-joint joint="${arm_prefix_modified}${arm_id}_joint1" transmission="hardware_interface/PositionJointInterface" />
-      <xacro:gazebo-joint joint="${arm_prefix_modified}${arm_id}_joint2" transmission="hardware_interface/PositionJointInterface" />
-      <xacro:gazebo-joint joint="${arm_prefix_modified}${arm_id}_joint3" transmission="hardware_interface/PositionJointInterface" />
-      <xacro:gazebo-joint joint="${arm_prefix_modified}${arm_id}_joint4" transmission="hardware_interface/PositionJointInterface" />
-      <xacro:gazebo-joint joint="${arm_prefix_modified}${arm_id}_joint5" transmission="hardware_interface/PositionJointInterface" />
-      <xacro:gazebo-joint joint="${arm_prefix_modified}${arm_id}_joint6" transmission="hardware_interface/PositionJointInterface" />
-      <xacro:gazebo-joint joint="${arm_prefix_modified}${arm_id}_joint7" transmission="hardware_interface/PositionJointInterface" />
-      <xacro:gazebo-joint joint="${arm_prefix_modified}${arm_id}_joint1" transmission="hardware_interface/VelocityJointInterface" />
-      <xacro:gazebo-joint joint="${arm_prefix_modified}${arm_id}_joint2" transmission="hardware_interface/VelocityJointInterface" />
-      <xacro:gazebo-joint joint="${arm_prefix_modified}${arm_id}_joint3" transmission="hardware_interface/VelocityJointInterface" />
-      <xacro:gazebo-joint joint="${arm_prefix_modified}${arm_id}_joint4" transmission="hardware_interface/VelocityJointInterface" />
-      <xacro:gazebo-joint joint="${arm_prefix_modified}${arm_id}_joint5" transmission="hardware_interface/VelocityJointInterface" />
-      <xacro:gazebo-joint joint="${arm_prefix_modified}${arm_id}_joint6" transmission="hardware_interface/VelocityJointInterface" />
-      <xacro:gazebo-joint joint="${arm_prefix_modified}${arm_id}_joint7" transmission="hardware_interface/VelocityJointInterface" />
-      <xacro:gazebo-joint joint="${arm_prefix_modified}${arm_id}_joint1" transmission="hardware_interface/EffortJointInterface" />
-      <xacro:gazebo-joint joint="${arm_prefix_modified}${arm_id}_joint2" transmission="hardware_interface/EffortJointInterface" />
-      <xacro:gazebo-joint joint="${arm_prefix_modified}${arm_id}_joint3" transmission="hardware_interface/EffortJointInterface" />
-      <xacro:gazebo-joint joint="${arm_prefix_modified}${arm_id}_joint4" transmission="hardware_interface/EffortJointInterface" />
-      <xacro:gazebo-joint joint="${arm_prefix_modified}${arm_id}_joint5" transmission="hardware_interface/EffortJointInterface" />
-      <xacro:gazebo-joint joint="${arm_prefix_modified}${arm_id}_joint6" transmission="hardware_interface/EffortJointInterface" />
-      <xacro:gazebo-joint joint="${arm_prefix_modified}${arm_id}_joint7" transmission="hardware_interface/EffortJointInterface" />
-      <xacro:transmission-franka-state arm_id="${arm_id}" />
-      <xacro:transmission-franka-model arm_id="${arm_id}"
-         root="${arm_prefix_modified}${arm_id}_joint1"
-         tip="${arm_prefix_modified}${arm_id}_joint8"
-       />
-    </xacro:if>
-    <xacro:if value="${ros2_control}">
-      <xacro:franka_arm_ros2_control
-          arm_id="${arm_id}"
-          robot_ip="${robot_ip}"
-          use_fake_hardware="${use_fake_hardware}"
-          fake_sensor_commands="${fake_sensor_commands}"
-          gazebo="${gazebo}"
-          hand="${hand}"
-          gazebo_effort="${gazebo_effort}"
-          arm_prefix="${arm_prefix}"
-          multi_arm="${multi_arm}"
-      />
-    </xacro:if>
+  <!-- Includes -->
+  <xacro:include filename="$(find franka_description)/robots/common/utils.xacro" />
+  <xacro:include filename="$(find franka_hardware)/ros2_control/franka_arm.ros2_control.xacro"/>
+  <!-- safety_distance: Minimum safety distance in [m] by which the collision volumes are expanded and which is enforced during robot motions -->
+  <!-- robot_type: the franka robot arm type -->
+  <!-- joint_limits: description of the joint limits that comes from a YAML file. Example definition: ${xacro.load_yaml('$(find franka_description)/robots/fr3/joint_limits.yaml')} -->
+  <!-- kinematics: description of the kinematics that comes from a YAML file. Example definition: ${xacro.load_yaml('$(find franka_description)/robots/fr3/kinematics.yaml')} -->
+  <!-- inertials: description of the inertials that comes from a YAML file. Example definition: ${xacro.load_yaml('$(find franka_description)/robots/fr3/inertials.yaml')} -->
+  <!-- dynamics: description of the dynamics that comes from a YAML file. Example definition: ${xacro.load_yaml('$(find franka_description)/robots/fr3/dynamics.yaml')} -->
+  <!-- Re-definiton of `franka_arm` to adhere to Clearpath descriptions -->
+  <xacro:macro name="franka_arm" params="
+    robot_type
+    parent_link
+    *origin
+    joint_limits
+    inertials
+    kinematics
+    accelerometer_config
+    dynamics
+    arm_prefix:=''
+    no_prefix:=false'
+    gazebo:='false'
+    safety_distance:=0
+    with_sc:=false">
+    <!-- Define a property that defaults to 'arm_prefix_robot_type' concatenated with an underscore if 'no_prefix' is not set -->
+    <xacro:property name="prefix" value="${'' if no_prefix else arm_prefix + robot_type + '_'}" />
+    <xacro:property name="with_accelerometers" value="${'false' if accelerometer_config == 'none' else 'true'}" />
+    <joint name="${prefix}joint0" type="fixed">
+      <parent link="${parent_link}"/>
+      <child link="${prefix}link0"/>
+      <xacro:insert_block name="origin" />
+    </joint>
+    <xacro:link_with_sc no_prefix="${no_prefix}" name="link0" gazebo="${gazebo}" with_sc="${with_sc}" with_accelerometers="${with_accelerometers}">
+      <self_collision_geometries>
+        <xacro:collision_capsule xyz="-0.075 0 0.06" direction="x" radius="${0.06+safety_distance}" length="0.03" />
+      </self_collision_geometries>
+    </xacro:link_with_sc>
+    <xacro:link_with_sc no_prefix="${no_prefix}" name="link1" gazebo="${gazebo}" with_sc="${with_sc}" with_accelerometers="${with_accelerometers}">
+      <self_collision_geometries>
+        <xacro:collision_capsule xyz="0 0 -191.5e-3" radius="${0.06+safety_distance}" length="0.283" />
+      </self_collision_geometries>
+    </xacro:link_with_sc>
+    <joint name="${prefix}joint1" type="revolute">
+      <xacro:franka-kinematics name="joint1" config="${kinematics}" />
+      <parent link="${prefix}link0" />
+      <child link="${prefix}link1" />
+      <axis xyz="0 0 1" />
+      <xacro:franka-limits name="joint1" config="${joint_limits}" />
+      <xacro:franka-dynamics name="joint1" config="${dynamics}" />
+    </joint>
+    <xacro:link_with_sc no_prefix="${no_prefix}" name="link2" gazebo="${gazebo}" with_sc="${with_sc}" with_accelerometers="${with_accelerometers}">
+      <self_collision_geometries>
+        <xacro:collision_capsule xyz="0 0 0" radius="${0.06+safety_distance}" length="0.12" />
+      </self_collision_geometries>
+    </xacro:link_with_sc>
+    <joint name="${prefix}joint2" type="revolute">
+      <xacro:franka-kinematics name="joint2" config="${kinematics}" />
+      <parent link="${prefix}link1" />
+      <child link="${prefix}link2" />
+      <axis xyz="0 0 1" />
+      <xacro:franka-limits name="joint2" config="${joint_limits}" />
+      <xacro:franka-dynamics name="joint2" config="${dynamics}" />
+    </joint>
+    <xacro:link_with_sc no_prefix="${no_prefix}" name="link3" gazebo="${gazebo}" with_sc="${with_sc}" with_accelerometers="${with_accelerometers}">
+      <self_collision_geometries>
+        <xacro:collision_capsule xyz="0 0 -0.145" radius="${0.06+safety_distance}" length="0.15" />
+      </self_collision_geometries>
+    </xacro:link_with_sc>
+    <joint name="${prefix}joint3" type="revolute">
+      <xacro:franka-kinematics name="joint3" config="${kinematics}" />
+      <parent link="${prefix}link2" />
+      <child link="${prefix}link3" />
+      <axis xyz="0 0 1" />
+      <xacro:franka-limits name="joint3" config="${joint_limits}" />
+      <xacro:franka-dynamics name="joint3" config="${dynamics}" />
+    </joint>
+    <xacro:link_with_sc no_prefix="${no_prefix}" name="link4" gazebo="${gazebo}" with_sc="${with_sc}" with_accelerometers="${with_accelerometers}">
+      <self_collision_geometries>
+        <xacro:collision_capsule xyz="0 0 0" radius="${0.06+safety_distance}" length="0.12" />
+     </self_collision_geometries>
+    </xacro:link_with_sc>
+    <joint name="${prefix}joint4" type="revolute">
+      <xacro:franka-kinematics name="joint4" config="${kinematics}" />
+      <parent link="${prefix}link3" />
+      <child link="${prefix}link4" />
+      <axis xyz="0 0 1" />
+      <xacro:franka-limits name="joint4" config="${joint_limits}" />
+      <xacro:franka-dynamics name="joint4" config="${dynamics}" />
+    </joint>
+    <xacro:link_with_sc no_prefix="${no_prefix}" name="link5" gazebo="${gazebo}" with_sc="${with_sc}" with_accelerometers="${with_accelerometers}">
+      <self_collision_geometries>
+        <xacro:collision_capsule xyz="0 0 -0.26"    radius="${0.060+safety_distance}" length="0.10" />
+        <xacro:collision_capsule xyz="0 0.08 -0.13" radius="${0.025+safety_distance}" length="0.14" />
+      </self_collision_geometries>
+    </xacro:link_with_sc>
+    <joint name="${prefix}joint5" type="revolute">
+      <xacro:franka-kinematics name="joint5" config="${kinematics}" />
+      <parent link="${prefix}link4" />
+      <child link="${prefix}link5" />
+      <axis xyz="0 0 1" />
+      <xacro:franka-limits name="joint5" config="${joint_limits}" />
+      <xacro:franka-dynamics name="joint5" config="${dynamics}" />
+    </joint>
+    <xacro:link_with_sc no_prefix="${no_prefix}" name="link6" gazebo="${gazebo}" with_sc="${with_sc}" with_accelerometers="false">
+      <self_collision_geometries>
+        <xacro:collision_capsule xyz="0 0 -0.03" radius="${0.05+safety_distance}" length="0.08" />
+      </self_collision_geometries>
+    </xacro:link_with_sc>
+    <joint name="${prefix}joint6" type="revolute">
+      <xacro:franka-kinematics name="joint6" config="${kinematics}" />
+      <parent link="${prefix}link5" />
+      <child link="${prefix}link6" />
+      <axis xyz="0 0 1" />
+      <xacro:franka-limits name="joint6" config="${joint_limits}" />
+      <xacro:franka-dynamics name="joint6" config="${dynamics}" />
+    </joint>
+    <xacro:link_with_sc no_prefix="${no_prefix}" name="link7" gazebo="${gazebo}" rpy="0 0 ${pi/4}" with_sc="${with_sc}" with_accelerometers="false">
+      <self_collision_geometries>
+        <xacro:collision_capsule xyz="0 0 0.01" direction="z" radius="${0.04+safety_distance}" length="0.14" />
+        <xacro:collision_capsule xyz="0.06 0 0.082" direction="x" radius="${0.03+safety_distance}"  length="0.01" />
+      </self_collision_geometries>
+    </xacro:link_with_sc>
+    <joint name="${prefix}joint7" type="revolute">
+      <xacro:franka-kinematics name="joint7" config="${kinematics}" />
+      <parent link="${prefix}link6"/>
+      <child link="${prefix}link7"/>
+      <axis xyz="0 0 1"/>
+      <xacro:franka-limits name="joint7" config="${joint_limits}" />
+      <xacro:franka-dynamics name="joint7" config="${dynamics}" />
+    </joint>
+    <link name="${prefix}link8"/>
+    <joint name="${prefix}joint8" type="fixed">
+      <xacro:franka-kinematics name="joint8" config="${kinematics}" />
+      <parent link="${prefix}link7" />
+      <child link="${prefix}link8" />
+    </joint>
   </xacro:macro>
   <xacro:macro name="franka" params="
@@ -154,5 +145,5 @@
     parent_link
     *origin
-    arm_id:=''
+    robot_type:=''
     joint_limits:=''
     joint_limits_parameters_file:=''
@@ -170,15 +161,19 @@
     gazebo:=''
     gazebo_effort:=''
+    safety_distance:=''
+    with_sc:=''
+    is_async:=''
+    thread_priority:=''
   ">
     <!-- Franka Type -->
-    <xacro:property name="_arm_id" value="fr3" lazy_eval="false"/>
-    <xacro:if value="${arm_id != ''}">
-      <xacro:property name="_arm_id" value="${arm_id}" lazy_eval="false"/>
+    <xacro:property name="_robot_type" value="fr3" lazy_eval="false"/>
+    <xacro:if value="${robot_type != ''}">
+      <xacro:property name="_robot_type" value="${robot_type}" lazy_eval="false"/>
     </xacro:if>
     <!-- Description Parameter Files -->
-    <xacro:property name="_joint_limits_parameters_file" value="$(find franka_description)/robots/${_arm_id}/joint_limits.yaml" lazy_eval="false"/>
-    <xacro:property name="_inertials_parameters_file" value="$(find franka_description)/robots/${_arm_id}/inertials.yaml" lazy_eval="false"/>
-    <xacro:property name="_kinematics_parameters_file" value="$(find franka_description)/robots/${_arm_id}/kinematics.yaml" lazy_eval="false"/>
-    <xacro:property name="_dynamics_parameters_file" value="$(find franka_description)/robots/${_arm_id}/dynamics.yaml" lazy_eval="false"/>
+    <xacro:property name="_joint_limits_parameters_file" value="$(find franka_description)/robots/${_robot_type}/joint_limits.yaml" lazy_eval="false"/>
+    <xacro:property name="_inertials_parameters_file" value="$(find franka_description)/robots/${_robot_type}/inertials.yaml" lazy_eval="false"/>
+    <xacro:property name="_kinematics_parameters_file" value="$(find franka_description)/robots/${_robot_type}/kinematics.yaml" lazy_eval="false"/>
+    <xacro:property name="_dynamics_parameters_file" value="$(find franka_description)/robots/${_robot_type}/dynamics.yaml" lazy_eval="false"/>
     <xacro:if value="${joint_limits_parameters_file != ''}">
       <xacro:property name="_joint_limits_parameters_file" value="${joint_limits_parameters_file}" lazy_eval="false"/>
@@ -213,4 +208,6 @@
     <xacro:property name="_ros2_control" value="$(arg use_manipulation_controllers)" lazy_eval="false"/>
     <xacro:property name="_robot_ip" value="192.168.131.40" lazy_eval="false"/>
+    <xacro:property name="_is_async" value="false" lazy_eval="false"/>
+    <xacro:property name="_thread_priority" value="50" lazy_eval="false"/>
     <xacro:if value="${ros2_control != ''}">
       <xacro:property name="_ros2_control" value="${ros2_control}" lazy_eval="false"/>
@@ -218,4 +215,10 @@
     <xacro:if value="${robot_ip != ''}">
       <xacro:property name="_robot_ip" value="${robot_ip}" lazy_eval="false"/>
+    </xacro:if>
+    <xacro:if value="${is_async != ''}">
+      <xacro:property name="_is_async" value="${is_async}" lazy_eval="false"/>
+    </xacro:if>
+    <xacro:if value="${thread_priority != ''}">
+      <xacro:property name="_thread_priority" value="${thread_priority}" lazy_eval="false"/>
     </xacro:if>
     <!-- Simulation -->
@@ -236,4 +239,13 @@
       <xacro:property name="_fake_sensor_commands" value="${fake_sensor_commands}" lazy_eval="false"/>
     </xacro:if>
+    <!-- Collision Parameter -->
+    <xacro:property name="_safety_distance" value="0.03" lazy_eval="false"/>
+    <xacro:property name="_with_sc" value="false" lazy_eval="false"/>
+    <xacro:if value="${safety_distance != ''}">
+      <xacro:property name="_safety_distance" value="${safety_distance}" lazy_eval="false"/>
+    </xacro:if>
+    <xacro:if value="${with_sc != ''}">
+      <xacro:property name="_with_sc" value="${with_sc}" lazy_eval="false"/>
+    </xacro:if>
     <!-- Fixed Parameters -->
     <xacro:property name="_hand" value="false" lazy_eval="false"/>
@@ -241,35 +253,85 @@
     <xacro:property name="_multi_arm" value="false" lazy_eval="false"/>
     <xacro:property name="_connected_to" value="" lazy_eval="false"/>
-    <xacro:property name="_with_sc" value="false" lazy_eval="false"/>
     <xacro:property name="_no_prefix" value="false" lazy_eval="false"/>
     <xacro:property name="_arm_prefix" value="${name}" lazy_eval="false"/>
     <xacro:property name="_accelerometer_config" value="none" lazy_eval="false"/>
-    <!-- Parent Joint -->
-    <joint name="${name}_${arm_id}_joint0" type="fixed">
-      <child link="${name}_${arm_id}_link0"/>
-      <parent link="${parent_link}"/>
-      <xacro:insert_block name="origin"/>
-    </joint>
-    <xacro:franka_robot
-      arm_id="${_arm_id}"
+    <!-- Instantiate Clearpath version of franka_arm xacro-->
+     <xacro:franka_arm
+      robot_type="${_robot_type}"
+      parent_link="${parent_link}"
       joint_limits="${_joint_limits}"
       inertials="${_inertials}"
       kinematics="${_kinematics}"
+      dynamics="${_dynamics}"
       accelerometer_config="${_accelerometer_config}"
-      dynamics="${_dynamics}"
-      gazebo="${_gazebo}"
-      hand="${_hand}"
-      ee_id="none"
-      with_sc="${_with_sc}"
-      ros2_control="${_ros2_control}"
+      arm_prefix:="${_arm_prefix}"
+      no_prefix:="${_no_prefix}"
+      gazebo:="${_gazebo}"
+      safety_distance:="${_safety_distance}"
+      with_sc:="${_with_sc}">
+      <xacro:insert_block name="origin" />
+    </xacro:franka_arm>
+    <!-- Definition of additional Gazebo tags -->
+    <xacro:if value="${_gazebo}">
+      <xacro:gazebo-joint joint="${arm_prefix}${robot_type}_joint1"
+        transmission="hardware_interface/PositionJointInterface"/>
+      <xacro:gazebo-joint joint="${arm_prefix}${robot_type}_joint2"
+        transmission="hardware_interface/PositionJointInterface"/>
+      <xacro:gazebo-joint joint="${arm_prefix}${robot_type}_joint3"
+        transmission="hardware_interface/PositionJointInterface"/>
+      <xacro:gazebo-joint joint="${arm_prefix}${robot_type}_joint4"
+        transmission="hardware_interface/PositionJointInterface"/>
+      <xacro:gazebo-joint joint="${arm_prefix}${robot_type}_joint5"
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