Commit message: R100 mecanum

File: clearpath_platform_description/urdf/r100/r100.urdf.xacro (robot description, xacro)
@@ -12,4 +12,5 @@
     <xacro:property name="wheel_radius" value="0.0759" />
     <xacro:property name="wheel_width" value="0.0790" />
+    <xacro:property name="wheel_mass" value="0.8" />
     <xacro:property name="chassis_length" value="0.960" />
     <xacro:property name="chassis_width" value="0.793" />
@@ -219,6 +220,4 @@
           <wheel_radius>${wheel_radius}</wheel_radius>
         </wheel>
-      </plugin>
-      <plugin filename="libignition-gazebo-wheel-slip-system.so" name="ignition::gazebo::systems::WheelSlip">
         <wheel link_name="rear_left_wheel_link">
           <slip_compliance_lateral>1.0</slip_compliance_lateral>

File: clearpath_platform_description/urdf/r100/rocker.urdf.xacro (robot description, xacro)
@@ -2,4 +2,5 @@
 <robot xmlns:xacro="http://ros.org/wiki/xacro" name="r100_rocker">
   <xacro:include filename="$(find clearpath_platform_description)/urdf/r100/wheels/wheel.urdf.xacro"/>
+  <xacro:include filename="$(find clearpath_platform_description)/urdf/r100/wheels/mecanum_wheel.urdf.xacro"/>
   <xacro:macro name="r100_rocker" params="prefix joint_type location *joint_limits">
     <link name="${prefix}_rocker_link">
@@ -27,10 +28,20 @@
       <xacro:insert_block name="joint_limits" />
     </joint>
-    <xacro:r100_wheel prefix="${prefix}" side="left">
-      <origin xyz="0 ${rocker_width/2 + wheel_width/2} 0" rpy="0 0 0" />
-    </xacro:r100_wheel>
-    <xacro:r100_wheel prefix="${prefix}" side="right">
-      <origin xyz="0 ${-(rocker_width/2 + wheel_width/2)} 0" rpy="0 0 0" />
-    </xacro:r100_wheel>
+    <xacro:if value="$(arg is_sim)">
+      <xacro:r100_mecanum_wheel parent="${prefix}_rocker_link" prefix="${prefix}_left" side="${-location}">
+          <origin xyz="0 ${rocker_width/2 + wheel_width/2} 0" rpy="0 0 0" />
+        </xacro:r100_mecanum_wheel>
+        <xacro:r100_mecanum_wheel parent="${prefix}_rocker_link" prefix="${prefix}_right" side="${location}">
+          <origin xyz="0 ${-(rocker_width/2 + wheel_width/2)} 0" rpy="0 0 0" />
+        </xacro:r100_mecanum_wheel>
+    </xacro:if>
+    <xacro:unless value="$(arg is_sim)">
+      <xacro:r100_wheel parent="${prefix}_rocker_link" prefix="${prefix}_left">
+        <origin xyz="0 ${rocker_width/2 + wheel_width/2} 0" rpy="0 0 0" />
+      </xacro:r100_wheel>
+      <xacro:r100_wheel parent="${prefix}_rocker_link" prefix="${prefix}_right">
+        <origin xyz="0 ${-(rocker_width/2 + wheel_width/2)} 0" rpy="0 0 0" />
+      </xacro:r100_wheel>
+    </xacro:unless>
   </xacro:macro>
 </robot>

File: clearpath_platform_description/urdf/r100/wheels/wheel.urdf.xacro (robot description, xacro)
@@ -1,6 +1,6 @@
 <?xml version="1.0"?>
 <robot xmlns:xacro="http://ros.org/wiki/xacro" name="r100_wheel">
-  <xacro:macro name="r100_wheel" params="prefix side *joint_pose">
-    <link name="${prefix}_${side}_wheel_link">
+  <xacro:macro name="r100_wheel" params="parent prefix *joint_pose">
+    <link name="${prefix}_wheel_link">
       <visual>
         <origin xyz="0 0 0" rpy="${math.pi/2} 0 0"/>
@@ -32,7 +32,7 @@
       <!-- <fdir1 value="1 0 0"/> -->
     </gazebo>
-    <joint name="${prefix}_${side}_wheel_joint" type="continuous">
-      <parent link="${prefix}_rocker_link"/>
-      <child link="${prefix}_${side}_wheel_link" />
+    <joint name="${prefix}_wheel_joint" type="continuous">
+      <parent link="${parent}"/>
+      <child link="${prefix}_wheel_link" />
       <xacro:insert_block name="joint_pose" />
       <axis xyz="0 1 0" />

Commit message: Added use_platform_controllers for R100. (#313)
(cherry picked from commit 932f706f04788b9bbaeae62ebd798b0c98e47a16)

# Conflicts:
#	clearpath_platform_description/urdf/r100/r100.urdf.xacro

File: clearpath_platform_description/urdf/r100/r100.urdf.xacro (robot description, xacro)
@@ -3,4 +3,5 @@
   <xacro:arg name="namespace" default="" />
   <xacro:arg name="is_sim" default="false" />
+<<<<<<< HEAD
   <xacro:arg name="gazebo_controllers" default="$(find clearpath_control)/config/r100/control.yaml"/>
   <xacro:arg name="use_platform_controllers" default="true"/>
@@ -8,4 +9,8 @@
   <xacro:include filename="$(find clearpath_platform_description)/urdf/r100/wheels/wheel.urdf.xacro"/>
   <xacro:include filename="$(find clearpath_platform_description)/urdf/r100/rocker.urdf.xacro"/>
+=======
+  <xacro:arg name="gazebo_controllers" default="$(find clearpath_control)/config/r100/control/omni_4wd.yaml"/>
+  <xacro:arg name="use_platform_controllers" default="true"/>
+>>>>>>> 932f706 (Added use_platform_controllers for R100. (#313))
   <!-- R100 Platform Macro -->
   <xacro:macro name="r100" params="wheel:='defaut'">
@@ -207,4 +212,5 @@
       <limit effort="0" velocity="0" />
     </xacro:r100_rocker>
+<<<<<<< HEAD
     <gazebo>
       <plugin filename="libignition-gazebo-wheel-slip-system.so" name="ignition::gazebo::systems::WheelSlip">
@@ -235,4 +241,25 @@
       </plugin>
     </gazebo>
+=======
+    <!-- Hardware  -->
+    <xacro:if value="$(arg is_sim)">
+      <xacro:property name="hardware_plugin" value="gz_ros2_control/GazeboSimSystem"/>
+    </xacro:if>
+    <xacro:unless value="$(arg is_sim)">
+      <xacro:property name="hardware_plugin" value="clearpath_hardware_interfaces/PumaHardware"/>
+    </xacro:unless>
+    <xacro:unless value="${control == 'omni_4wd' or control == 'diff_4wd'}">
+      <xacro:error message="Invalid drivetrain control ${control}"/>
+    </xacro:unless>
+    <xacro:if value="$(arg use_platform_controllers)">
+      <xacro:generic_drivetrain
+        name="r100"
+        control="${control}"
+        front_wheels="${front_wheels}"
+        rear_wheels="${rear_wheels}"
+        hardware_plugin="${hardware_plugin}"
+      />
+    </xacro:if>
+>>>>>>> 932f706 (Added use_platform_controllers for R100. (#313))
     <!-- Internal IMU -->
     <link name="imu_0_link">

Commit message: Changes to support mobile manipulation
- Add meshes to some links missing collision geometry
- Support different hardware plugins, including mock hardware

File: clearpath_platform_description/urdf/r100/r100.urdf.xacro (robot description, xacro)
@@ -6,5 +6,5 @@
   <xacro:arg name="use_platform_controllers" default="true"/>
   <!-- R100 Platform Macro -->
-  <xacro:macro name="r100" params="control:='omni_4wd' front_wheels:='mecanum' rear_wheels:='mecanum'">
+  <xacro:macro name="r100" params="control:='omni_4wd' front_wheels:='mecanum' rear_wheels:='mecanum' hardware_plugin_name='mock_components/GenericSystem'">
     <!-- Variables -->
     <xacro:property name="chassis_length" value="0.960" />
@@ -70,4 +70,10 @@
         <material name="clearpath_yellow" />
       </visual>
+      <collision>
+        <origin xyz="0 0 0" rpy="0 0 ${math.pi}" />
+        <geometry>
+          <mesh filename="package://clearpath_platform_description/meshes/r100/side-cover.stl"/>
+        </geometry>
+      </collision>
     </link>
     <link name="right_side_cover_link">
@@ -79,4 +85,10 @@
         <material name="clearpath_yellow" />
       </visual>
+      <collision>
+        <origin xyz="0 0 0" rpy="0 0 0" />
+        <geometry>
+          <mesh filename="package://clearpath_platform_description/meshes/r100/side-cover.stl"/>
+        </geometry>
+      </collision>
     </link>
     <joint name="front_cover_link_joint" type="fixed">
@@ -93,4 +105,10 @@
         <material name="clearpath_black" />
       </visual>
+      <collision>
+        <origin xyz="0 0 0" rpy="0 0 0" />
+        <geometry>
+          <mesh filename="package://clearpath_platform_description/meshes/r100/end-cover.stl" />
+        </geometry>
+      </collision>
     </link>
     <joint name="rear_cover_link_joint" type="fixed">
@@ -107,4 +125,10 @@
         <material name="clearpath_black" />
       </visual>
+      <collision>
+        <origin xyz="0 0 0" rpy="0 0 ${math.pi}" />
+        <geometry>
+          <mesh filename="package://clearpath_platform_description/meshes/r100/end-cover.stl" />
+        </geometry>
+      </collision>
     </link>
     <!-- Ligths -->
@@ -127,4 +151,10 @@
         <material name="clearpath_white" />
       </visual>
+      <collision>
+        <origin xyz="0 0 0" rpy="0 0 0" />
+        <geometry>
+          <mesh filename="package://clearpath_platform_description/meshes/r100/lights.stl" />
+        </geometry>
+      </collision>
     </link>
     <link name="rear_lights_link">
@@ -136,4 +166,10 @@
         <material name="clearpath_red" />
       </visual>
+      <collision>
+        <origin xyz="0 0 0" rpy="0 0 ${math.pi}" />
+        <geometry>
+          <mesh filename="package://clearpath_platform_description/meshes/r100/lights.stl" />
+        </geometry>
+      </collision>
     </link>
     <!-- Axle -->
@@ -151,4 +187,10 @@
         <material name="clearpath_black" />
       </visual>
+      <collision>
+        <origin xyz="0 0 0" rpy="0 ${math.pi/2} 0" />
+        <geometry>
+          <mesh filename="package://clearpath_platform_description/meshes/r100/axle.stl" />
+        </geometry>
+      </collision>
     </link>
     <!-- Riser -->
@@ -200,10 +242,5 @@
     <xacro:include filename="$(find clearpath_platform_description)/urdf/generic/drivetrain/drivetrain.urdf.xacro"/>
     <!-- Hardware  -->
-    <xacro:if value="$(arg is_sim)">
-      <xacro:property name="hardware_plugin" value="gz_ros2_control/GazeboSimSystem"/>
-    </xacro:if>
-    <xacro:unless value="$(arg is_sim)">
-      <xacro:property name="hardware_plugin" value="clearpath_hardware_interfaces/PumaHardware"/>
-    </xacro:unless>
+    <xacro:property name="hardware_plugin" value="${hardware_plugin_name}"/>
     <xacro:unless value="${control == 'omni_4wd' or control == 'diff_4wd'}">
       <xacro:error message="Invalid drivetrain control ${control}"/>

File: clearpath_platform_description/urdf/r100/rocker.urdf.xacro (robot description, xacro)
@@ -10,4 +10,11 @@
         <material name="clearpath_black" />
       </visual>
+      <collision>
+        <origin xyz="0 0 0" rpy="${math.pi/2} 0 ${math.pi/2}" />
+        <geometry>
+          <mesh filename="package://clearpath_platform_description/meshes/r100/rocker.stl"/>
+        </geometry>
+        <material name="clearpath_black" />
+      </collision>
       <inertial>
         <origin xyz="0 0 0" rpy="${math.pi/2} 0 ${math.pi/2}"/>

File: clearpath_sensors_description/urdf/hokuyo_ust.urdf.xacro (robot description, xacro)
@@ -13,4 +13,11 @@
         <material name="clearpath_dark_grey" />
       </visual>
+      <collision>
+        <origin xyz="0 0 0" rpy="0 0 0" />
+        <geometry>
+          <mesh filename="package://clearpath_sensors_description/meshes/hokuyo_ust.stl" />
+        </geometry>
+        <material name="clearpath_dark_grey" />
+      </collision>
     </link>
     <link name="${name}_laser">
