Commit message: rework do100 mecanum wheel model

File: clearpath_platform_description/urdf/do100/drivetrain/wheels/mecanum.urdf.xacro (robot description, xacro)
@@ -4,18 +4,84 @@
   <xacro:property name="do100_mecanum_wheel_mass" value="0.4" />
   <xacro:property name="do100_mecanum_wheel_width" value="0.050" />
+  <!-- Mecanum wheel = driven hub + ring of 9 passive barrel rollers. Meshes are
+       baked into the wheel_link frame (axle = +Y); the rollers touch the ground. -->
+  <xacro:property name="do100_roller_count"  value="9" />
+  <xacro:property name="do100_roller_delta"  value="0.6981317" />  <!-- 2*pi/9 -->
+  <xacro:property name="do100_roller_ring_r" value="0.04043" />
+  <xacro:property name="do100_roller_len"    value="0.0470" />
+  <xacro:property name="do100_roller_rad"    value="0.00977" />
+  <xacro:property name="do100_roller_mass"   value="0.02" />
+  <!-- Roller spin axis, ~45 deg to the +Y axle (side = +1). -->
+  <xacro:property name="do100_roller_ax" value="0.00321" />
+  <xacro:property name="do100_roller_ay" value="0.70342" />
+  <xacro:property name="do100_roller_az" value="0.71077" />
+    <!-- Roller barrel = 5 spheres along the spin axis: one on the centre (widest)
+      plus two mirrored pairs tapering to the ends, so contact stays a point. -->
+  <xacro:property name="do100_roller_half"       value="${do100_roller_len / 2.0}" />
+  <xacro:property name="do100_roller_off_inner"  value="${0.27 * do100_roller_half}" />
+  <xacro:property name="do100_roller_off_mid"    value="${0.52 * do100_roller_half}" />
+  <xacro:property name="do100_roller_rad_center" value="${do100_roller_rad}" />
+  <xacro:property name="do100_roller_rad_inner"  value="${0.96 * do100_roller_rad}" />
+  <xacro:property name="do100_roller_rad_mid"    value="${0.88 * do100_roller_rad}" />
+  <!-- One collision sphere at signed offset 'off' along the spin axis. -->
+  <xacro:macro name="do100_roller_sphere" params="side off rad">
+    <collision>
+      <origin xyz="${off * side * do100_roller_ax} ${off * do100_roller_ay} ${off * do100_roller_az}" rpy="0 0 0"/>
+      <geometry>
+        <sphere radius="${rad}"/>
+      </geometry>
+    </collision>
+  </xacro:macro>
+  <!-- One passive roller (instance 'index'), free-spinning on the hub ring. -->
+  <xacro:macro name="do100_mecanum_roller" params="prefix side count index">
+    <link name="${prefix}_roller_${index}_link">
+      <visual>
+        <origin xyz="0 0 0" rpy="0 0 0"/>
+        <geometry>
+          <mesh filename="package://clearpath_platform_description/meshes/do100/wheels/mecanum_roller.glb"
+                scale="${side} 1 1"/>
+        </geometry>
+        <material name="dingo_black"><color rgba="0.15 0.15 0.15 1.0"/></material>
+      </visual>
+      <!-- Crowned barrel: 5 spheres, peak sphere on the centre. -->
+      <xacro:do100_roller_sphere side="${side}" off="0"                          rad="${do100_roller_rad_center}"/>
+      <xacro:do100_roller_sphere side="${side}" off=" ${do100_roller_off_inner}"  rad="${do100_roller_rad_inner}"/>
+      <xacro:do100_roller_sphere side="${side}" off="${-do100_roller_off_inner}"  rad="${do100_roller_rad_inner}"/>
+      <xacro:do100_roller_sphere side="${side}" off=" ${do100_roller_off_mid}"    rad="${do100_roller_rad_mid}"/>
+      <xacro:do100_roller_sphere side="${side}" off="${-do100_roller_off_mid}"    rad="${do100_roller_rad_mid}"/>
+      <inertial>
+        <origin xyz="0 0 0" rpy="0 0 0"/>
+        <mass value="${do100_roller_mass}"/>
+        <inertia ixx="2.0e-6" ixy="0" ixz="0" iyy="2.0e-6" iyz="0" izz="2.0e-6"/>
+      </inertial>
+    </link>
+    <joint name="${prefix}_roller_${index}_joint" type="continuous">
+      <parent link="${prefix}_wheel_link"/>
+      <child  link="${prefix}_roller_${index}_link"/>
+      <origin xyz="${side * do100_roller_ring_r * cos(side * index * do100_roller_delta)} 0 ${-side * do100_roller_ring_r * sin(side * index * do100_roller_delta)}"
+              rpy="0 ${side * index * do100_roller_delta} 0"/>
+      <axis   xyz="${side * do100_roller_ax} ${do100_roller_ay} ${do100_roller_az}"/>
+      <!-- Light bearing drag so a free-spun roller settles instead of windmilling. -->
+      <dynamics damping="0.002" friction="0.0"/>
+    </joint>
+  </xacro:macro>
+  <!-- Recursively instantiate the full roller ring. -->
+  <xacro:macro name="do100_mecanum_roller_ring" params="prefix side count index:=0">
+    <xacro:if value="${index &lt; count}">
+      <xacro:do100_mecanum_roller prefix="${prefix}" side="${side}" count="${count}" index="${index}"/>
+      <xacro:do100_mecanum_roller_ring prefix="${prefix}" side="${side}" count="${count}" index="${index + 1}"/>
+    </xacro:if>
+  </xacro:macro>
   <xacro:macro name="do100_mecanum_wheel" params="prefix side *joint_pose">
+    <!-- Driven hub, visual only - the rollers carry all ground contact. -->
     <link name="${prefix}_wheel_link">
       <visual>
-        <origin xyz="0 ${side * 0.027} 0" rpy="0 0 ${PI/2}"/>
+        <origin xyz="0 0 0" rpy="0 0 0"/>
         <geometry>
-          <mesh filename="package://clearpath_platform_description/meshes/do100/wheels/mecanum.dae" scale="${side} 1 1" />
+          <mesh filename="package://clearpath_platform_description/meshes/do100/wheels/mecanum_hub.glb"
+                scale="${side} 1 1"/>
         </geometry>
+        <material name="dingo_black"><color rgba="0.15 0.15 0.15 1.0"/></material>
       </visual>
-      <collision>
-        <origin xyz="0 0 0" rpy="${PI/2} 0 0"/>
-        <geometry>
-          <cylinder radius="${do100_mecanum_wheel_radius}" length="${do100_mecanum_wheel_width}"/>
-        </geometry>
-      </collision>
       <inertial>
         <origin xyz="0 0 0" rpy="0 0 0"/>
@@ -27,27 +93,4 @@
       </inertial>
     </link>
-    <gazebo>
-      <plugin filename="libgz-sim-wheel-slip-system.so" name="gz::sim::systems::WheelSlip">
-        <wheel link_name="${prefix}_wheel_link">
-          <slip_compliance_lateral>1.0</slip_compliance_lateral>
-          <slip_compliance_longitudinal>1.0</slip_compliance_longitudinal>
-          <wheel_normal_force>20</wheel_normal_force>
-          <wheel_radius>${do100_mecanum_wheel_radius}</wheel_radius>
-        </wheel>
-      </plugin>
-    </gazebo>
-    <gazebo reference="${prefix}_wheel_link">
-      <collision>
-        <surface>
-          <friction>
-            <ode>
-              <mu>1.0</mu>
-              <mu2>0.0</mu2>
-              <fdir1 gz:expressed_in="base_link">1 ${side} 0</fdir1>
-            </ode>
-          </friction>
-        </surface>
-      </collision>
-    </gazebo>
     <joint name="${prefix}_wheel_joint" type="continuous">
       <parent link="chassis_link"/>
@@ -56,4 +99,5 @@
       <axis xyz="0 1 0" />
     </joint>
+    <xacro:do100_mecanum_roller_ring prefix="${prefix}" side="${side}" count="${do100_roller_count}"/>
   </xacro:macro>
 </robot>
