Commit message: Add corrected D435 mesh with fixed normals

File: clearpath_sensors_description/urdf/intel/d435.urdf.xacro (robot description, xacro)
@@ -46,5 +46,5 @@
           <origin xyz="${d435_zero_depth_to_glass + d435_glass_to_front} ${-d435_cam_depth_py} 0" rpy="${M_PI/2} 0 ${M_PI/2}"/>
           <geometry>
-            <mesh filename="file://$(find realsense2_description)/meshes/d435.dae" />
+            <mesh filename="file://$(find clearpath_sensors_description)/meshes/d435.dae" />
           </geometry>
         </xacro:if>
